File: Hardware/GeneralPurposeAlarmDevicePCB/GeneralPurposeAlarmDevicePCB/GeneralPurposeAlarmDevicePCB.sch (KiCad schematic (older format))
At the start: 23 parts

Commit message: Annote reference designators.
Parts:
- gave numbers to parts that had none: 23
Changed lines of the file:
@@
 $EndDescr
 $Comp
-L dk_Crystals:NX3225GD-8MHZ-STD-CRA-3 XTAL?
+L dk_Crystals:NX3225GD-8MHZ-STD-CRA-3 XTAL101
 U 1 1 62B3A927
 P 2600 4050
-F 0 "XTAL?" H 2600 4290 50  0000 C CNN
+F 0 "XTAL101" H 2600 4290 50  0000 C CNN
 F 1 "16MHZ 20PF HC-49S/SMD" H 2700 4200 50  0000 C CNN
 F 2 "" H 2800 4250 60  0001 L CNN
@@
 $EndComp
 $Comp
-L Device:C C?
+L Device:C C104
 U 1 1 62B45335
 P 2100 4400
-F 0 "C?" H 2215 4446 50  0000 L CNN
+F 0 "C104" H 2215 4446 50  0000 L CNN
 F 1 "39pF" H 2215 4355 50  0000 L CNN
 F 2 "Capacitor_SMD:C_0603_1608Metric" H 2138 4250 50  0001 C CNN
@@
 $EndComp
 $Comp
-L Device:C C?
+L Device:C C106
 U 1 1 62B46140
 P 2950 4400
-F 0 "C?" H 3065 4446 50  0000 L CNN
+F 0 "C106" H 3065 4446 50  0000 L CNN
 F 1 "39pF" H 3065 4355 50  0000 L CNN
 F 2 "Capacitor_SMD:C_0603_1608Metric_Pad1.08x0.95mm_HandSolder" H 2988 4250 50  0001 C CNN
@@
 Note: Check pad sized for 0603 and 0603HandSolder
 $Comp
-L Device:D_Schottky D?
+L Device:D_Schottky D101
 U 1 1 62B4A83F
 P 1600 1000
-F 0 "D?" H 1600 783 50  0000 C CNN
+F 0 "D101" H 1600 783 50  0000 C CNN
 F 1 "Schottky 2A" H 1600 874 50  0000 C CNN
 F 2 "Diode_SMD:D_SMB" H 1600 1000 50  0001 C CNN
@@
 $EndComp
 $Comp
-L dk_LED-Indication-Discrete:LTST-C171KRKT D?
+L dk_LED-Indication-Discrete:LTST-C171KRKT D102
 U 1 1 62B52665
 P 5300 4550
-F 0 "D?" H 5250 4887 60  0000 C CNN
+F 0 "D102" H 5250 4887 60  0000 C CNN
 F 1 "RED 0603" H 5250 4781 60  0000 C CNN
 F 2 "LED_SMD:LED_0603_1608Metric" H 5500 4750 60  0001 L CNN
@@
 $EndComp
 $Comp
-L Device:CP C?
+L Device:CP C102
 U 1 1 62B5ACAD
 P 1850 1300
-F 0 "C?" H 1968 1346 50  0000 L CNN
+F 0 "C102" H 1968 1346 50  0000 L CNN
 F 1 "47uF 16V" H 1968 1255 50  0000 L CNN
 F 2 "Capacitor_SMD:CP_Elec_5x5.4" H 1888 1150 50  0001 C CNN
@@
 $EndComp
 $Comp
-L Device:CP C?
+L Device:CP C108
 U 1 1 62B5B741
 P 3750 1200
-F 0 "C?" H 3868 1246 50  0000 L CNN
+F 0 "C108" H 3868 1246 50  0000 L CNN
 F 1 "47uF 16V" H 3868 1155 50  0000 L CNN
 F 2 "Capacitor_SMD:CP_Elec_5x5.4" H 3788 1050 50  0001 C CNN
@@
 $EndComp
 $Comp
-L dk_PMIC-Voltage-Regulators-Linear:NCP1117ST50T3G U?
+L dk_PMIC-Voltage-Regulators-Linear:NCP1117ST50T3G U101
 U 1 1 62B5C195
 P 2500 1000
-F 0 "U?" H 2550 1287 60  0000 C CNN
+F 0 "U101" H 2550 1287 60  0000 C CNN
 F 1 "NCP1117ST50T3G" H 2550 1181 60  0000 C CNN
 F 2 "digikey-footprints:SOT-223" H 2700 1200 60  0001 L CNN
@@
 $EndComp
 $Comp
-L Device:C C?
+L Device:C C107
 U 1 1 62B5D253
 P 3200 1200
-F 0 "C?" H 3315 1246 50  0000 L CNN
+F 0 "C107" H 3315 1246 50  0000 L CNN
 F 1 "100nF" H 3315 1155 50  0000 L CNN
 F 2 "Capacitor_SMD:C_0603_1608Metric_Pad1.08x0.95mm_HandSolder" H 3238 1050 50  0001 C CNN
@@
 $EndComp
 $Comp
-L Device:R R?
+L Device:R R103
 U 1 1 62B42216
 P 5200 4100
-F 0 "R?" V 5000 4050 50  0000 C CNN
+F 0 "R103" V 5000 4050 50  0000 C CNN
 F 1 "330R" V 5100 4100 50  0000 C CNN
 F 2 "Resistor_SMD:R_0603_1608Metric" V 5130 4100 50  0001 C CNN
@@
 $EndComp
 $Comp
-L power:+5V #PWR?
+L power:+5V #PWR0113
 U 1 1 62B6F384
 P 3900 900
-F 0 "#PWR?" H 3900 750 50  0001 C CNN
+F 0 "#PWR0113" H 3900 750 50  0001 C CNN
 F 1 "+5V" H 3915 1073 50  0000 C CNN
 F 2 "" H 3900 900 50  0001 C CNN
@@
 $EndComp
 $Comp
-L GPAD_SCH_LIB:Barrel_Jack_Switch_SMT J?
+L GPAD_SCH_LIB:Barrel_Jack_Switch_SMT J101
 U 1 1 62BBF172
 P 850 1100
-F 0 "J?" H 907 1491 50  0000 C CNN
+F 0 "J101" H 907 1491 50  0000 C CNN
 F 1 "Barrel_Jack_Switch_SMT" H 907 1400 50  0000 C CNN
 F 2 "Connector_BarrelJack:BarrelJack_CLIFF_FC681465S_SMT_Horizontal" H 900 1060 50  0001 C CNN
@@
 $EndComp
 $Comp
-L GPAD_SCH_LIB:PI_ATMEGA328P-AU-InOrder U?
+L GPAD_SCH_LIB:PI_ATMEGA328P-AU-InOrder U102
 U 1 1 62B3A84B
 P 4250 3350
-F 0 "U?" H 3250 4250 60  0000 L CNN
+F 0 "U102" H 3250 4250 60  0000 L CNN
 F 1 "PI_ATMEGA328P-AU-InOrder" H 3600 2900 60  0000 L CNN
 F 2 "digikey-footprints:TQFP-32_7x7mm" H 3400 3400 60  0001 L CNN
@@
 $EndComp
 $Comp
-L power:GND #PWR?
+L power:GND #PWR0112
 U 1 1 62B4EB2C
 P 2550 3500
-F 0 "#PWR?" H 2550 3250 50  0001 C CNN
+F 0 "#PWR0112" H 2550 3250 50  0001 C CNN
 F 1 "GND" H 2555 3327 50  0000 C CNN
 F 2 "" H 2550 3500 50  0001 C CNN
@@
 $EndComp
 $Comp
-L power:GND #PWR?
+L power:GND #PWR0110
 U 1 1 62B4EB26
 P 2000 3550
-F 0 "#PWR?" H 2000 3300 50  0001 C CNN
+F 0 "#PWR0110" H 2000 3300 50  0001 C CNN
 F 1 "GND" H 2005 3377 50  0000 C CNN
 F 2 "" H 2000 3550 50  0001 C CNN
@@
 $EndComp
 $Comp
-L Device:C C?
+L Device:C C103
 U 1 1 62B4EB20
 P 2000 3300
-F 0 "C?" H 2115 3346 50  0000 L CNN
+F 0 "C103" H 2115 3346 50  0000 L CNN
 F 1 "100nF" H 2115 3255 50  0000 L CNN
 F 2 "Capacitor_SMD:C_0603_1608Metric_Pad1.08x0.95mm_HandSolder" H 2038 3150 50  0001 C CNN
@@
 $EndComp
 $Comp
-L Device:CP C?
+L Device:CP C105
 U 1 1 62B4EB15
 P 2550 3300
-F 0 "C?" H 2668 3346 50  0000 L CNN
+F 0 "C105" H 2668 3346 50  0000 L CNN
 F 1 "47uF 16V" H 2668 3255 50  0000 L CNN
 F 2 "Capacitor_SMD:CP_Elec_5x5.4" H 2588 3150 50  0001 C CNN
@@
 $EndComp
 $Comp
-L power:GND #PWR?
+L power:GND #PWR0115
 U 1 1 62B56993
 P 5500 3300
-F 0 "#PWR?" H 5500 3050 50  0001 C CNN
+F 0 "#PWR0115" H 5500 3050 50  0001 C CNN
 F 1 "GND" H 5505 3127 50  0000 C CNN
 F 2 "" H 5500 3300 50  0001 C CNN
@@
 $EndComp
 $Comp
-L Device:CP C?
+L Device:CP C111
 U 1 1 62B56FAA
 P 5950 3750
-F 0 "C?" H 6068 3796 50  0000 L CNN
+F 0 "C111" H 6068 3796 50  0000 L CNN
 F 1 "47uF 16V" H 6068 3705 50  0000 L CNN
 F 2 "Capacitor_SMD:CP_Elec_5x5.4" H 5988 3600 50  0001 C CNN
@@
 $EndComp
 $Comp
-L Device:C C?
+L Device:C C110
 U 1 1 62B57F1E
 P 5500 3750
-F 0 "C?" H 5615 3796 50  0000 L CNN
+F 0 "C110" H 5615 3796 50  0000 L CNN
 F 1 "100nF" H 5615 3705 50  0000 L CNN
 F 2 "Capacitor_SMD:C_0603_1608Metric_Pad1.08x0.95mm_HandSolder" H 5538 3600 50  0001 C CNN
@@
 Notes:\nArduino Pin to ATmega328\nA0 PC0\nA1 PC1\nA2 PC2\nA3 PC3\nA4 PC4\nA5 PC5\nD0 PD0\nD1 PD1\nD2 PD2\n'D3 PD3\nD4 PD4\n`D5 PD5\n`D6 PD6\nD7 PD7\nD8 PB0\n`D9 PB1\n`D10 PB2\n`D11 PB3\nD12 PB4\nD13 PB5
 $Comp
-L power:GND #PWR?
+L power:GND #PWR0116
 U 1 1 62BAF22E
 P 5500 4000
-F 0 "#PWR?" H 5500 3750 50  0001 C CNN
+F 0 "#PWR0116" H 5500 3750 50  0001 C CNN
 F 1 "GND" H 5505 3827 50  0000 C CNN
 F 2 "" H 5500 4000 50  0001 C CNN
@@
 $EndSheet
 $Comp
-L GPAD_SCH_LIB:SWITCH_TACTILE_SPST-NO_0.05A_24V S?
+L GPAD_SCH_LIB:SWITCH_TACTILE_SPST-NO_0.05A_24V S101
 U 1 1 62BA946B
 P 5550 2200
-F 0 "S?" H 5550 2547 60  0000 C CNN
+F 0 "S101" H 5550 2547 60  0000 C CNN
 F 1 "SWITCH_TACTILE_SPST-NO_0.05A_24V" H 5550 2441 60  0000 C CNN
 F 2 "digikey-footprints:Switch_Tactile_THT_6x6mm" H 5750 2400 60  0001 L CNN
@@
 $EndComp
 $Comp
-L power:GND #PWR?
+L power:GND #PWR0117
 U 1 1 62BAA497
 P 6050 2100
-F 0 "#PWR?" H 6050 1850 50  0001 C CNN
+F 0 "#PWR0117" H 6050 1850 50  0001 C CNN
 F 1 "GND" H 6055 1927 50  0000 C CNN
 F 2 "" H 6050 2100 50  0001 C CNN
@@
 $EndComp
 $Comp
-L Device:C C?
+L Device:C C109
 U 1 1 62BAB737
 P 5050 2300
-F 0 "C?" H 5165 2346 50  0000 L CNN
+F 0 "C109" H 5165 2346 50  0000 L CNN
 F 1 "100nF" H 5165 2255 50  0000 L CNN
 F 2 "Capacitor_SMD:C_0603_1608Metric_Pad1.08x0.95mm_HandSolder" H 5088 2150 50  0001 C CNN
@@
 $EndComp
 $Comp
-L power:GND #PWR?
+L power:GND #PWR0114
 U 1 1 62BAC0E9
 P 5050 2550
-F 0 "#PWR?" H 5050 2300 50  0001 C CNN
+F 0 "#PWR0114" H 5050 2300 50  0001 C CNN
 F 1 "GND" H 5055 2377 50  0000 C CNN
 F 2 "" H 5050 2550 50  0001 C CNN
@@
 $EndComp
 $Comp
-L Device:R R?
+L Device:R R102
 U 1 1 62BAC86D
 P 4500 2100
-F 0 "R?" V 4300 2050 50  0000 C CNN
+F 0 "R102" V 4300 2050 50  0000 C CNN
 F 1 "10K" V 4400 2100 50  0000 C CNN
 F 2 "Resistor_SMD:R_0603_1608Metric" V 4430 2100 50  0001 C CNN
@@
 	4750 2100 5050 2100
 $Comp
-L Device:R R?
+L Device:R R101
 U 1 1 62BF3016
 P 2600 2950
-AR Path="/62BF3016" Ref="R?"  Part="1"
+AR Path="/62BF3016" Ref="R101"  Part="1"
 AR Path="/62B871EE/62BF3016" Ref="R?"  Part="1"
-F 0 "R?" V 2400 2900 50  0000 C CNN
+F 0 "R101" V 2400 2900 50  0000 C CNN
 F 1 "1R0" V 2500 2950 50  0000 C CNN
 F 2 "Resistor_SMD:R_0603_1608Metric" V 2530 2950 50  0001 C CNN
@@
 $EndComp
 $Comp
-L power:+5V #PWR?
+L power:+5V #PWR0105
 U 1 1 62BF301C
 P 1850 2950
-AR Path="/62BF301C" Ref="#PWR?"  Part="1"
+AR Path="/62BF301C" Ref="#PWR0105"  Part="1"
 AR Path="/62B871EE/62BF301C" Ref="#PWR?"  Part="1"
-F 0 "#PWR?" H 1850 2800 50  0001 C CNN
+F 0 "#PWR0105" H 1850 2800 50  0001 C CNN
 F 1 "+5V" H 1865 3123 50  0000 C CNN
 F 2 "" H 1850 2950 50  0001 C CNN
@@
 	1300 1000 1250 1000
 $Comp
-L power:GND #PWR?
+L power:GND #PWR0111
 U 1 1 62C08ABB
 P 2500 1500
-F 0 "#PWR?" H 2500 1250 50  0001 C CNN
+F 0 "#PWR0111" H 2500 1250 50  0001 C CNN
 F 1 "GND" H 2505 1327 50  0000 C CNN
 F 2 "" H 2500 1500 50  0001 C CNN
@@
 $EndComp
 $Comp
-L Device:C C?
+L Device:C C101
 U 1 1 62B4BD4B
 P 1300 1450
-F 0 "C?" H 1415 1496 50  0000 L CNN
+F 0 "C101" H 1415 1496 50  0000 L CNN
 F 1 "39pF" H 1415 1405 50  0000 L CNN
 F 2 "Capacitor_SMD:C_0603_1608Metric_Pad1.08x0.95mm_HandSolder" H 1338 1300 50  0001 C CNN
@@
 	2850 7350 2700 7350
 $Comp
-L dk_Rectangular-Connectors-Headers-Male-Pins:22-23-2021 J?
+L dk_Rectangular-Connectors-Headers-Male-Pins:22-23-2021 J102
 U 1 1 62CD8EE4
 P 4650 850
-F 0 "J?" H 4563 812 50  0000 R CNN
+F 0 "J102" H 4563 812 50  0000 R CNN
 F 1 "22-23-2021" H 4563 903 50  0000 R CNN
 F 2 "digikey-footprints:PinHeader_1x2_P2.54mm_Drill1.02mm" H 4850 1050 60  0001 L CNN
@@
 	4750 1000 4750 950
 $Comp
-L dk_Rectangular-Connectors-Headers-Male-Pins:22-23-2021 J?
+L dk_Rectangular-Connectors-Headers-Male-Pins:22-23-2021 J103
 U 1 1 62D1C4B1
 P 5600 1200
-F 0 "J?" H 5513 1162 50  0000 R CNN
+F 0 "J103" H 5513 1162 50  0000 R CNN
 F 1 "22-23-2021" H 5513 1253 50  0000 R CNN
 F 2 "digikey-footprints:PinHeader_1x2_P2.54mm_Drill1.02mm" H 5800 1400 60  0001 L CNN

Commit message: Clear several DRC warnings.
Connections:
- net VccControler: now also C110.1, U102.18 (AVCC), U102.20 (AREF)
- no-connect marks 8 -> 9
Changed lines of the file:
@@
 	5200 3400 5200 3600
 Wire Wire Line
-	5200 3600 4950 3600
-Wire Wire Line
 	5200 3600 5500 3600
-Connection ~ 5200 3600
 Wire Wire Line
 	1150 1100 1250 1100
@@
 	1250 1000 1150 1000
 Wire Wire Line
-	1450 1000 1300 1000
+	1450 1000 1400 1000
 Connection ~ 1250 1000
 Connection ~ 1300 1000
@@
 Connection ~ 1850 1000
 Wire Wire Line
-	1850 1000 2200 1000
+	1850 1000 2050 1000
 Wire Wire Line
 	1850 1450 1850 1550
@@
 Wire Wire Line
 	4200 5150 3350 5150
+$Comp
+L power:PWR_FLAG #FLG0101
+U 1 1 62E136FF
+P 1400 1000
+F 0 "#FLG0101" H 1400 1075 50  0001 C CNN
+F 1 "PWR_FLAG" H 1400 1173 50  0000 C CNN
+F 2 "" H 1400 1000 50  0001 C CNN
+F 3 "~" H 1400 1000 50  0001 C CNN
+	1    1400 1000
+	1    0    0    -1
+$EndComp
+Connection ~ 1400 1000
+Wire Wire Line
+	1400 1000 1300 1000
+$Comp
+L power:PWR_FLAG #FLG0102
+U 1 1 62E14B5B
+P 2050 1000
+F 0 "#FLG0102" H 2050 1075 50  0001 C CNN
+F 1 "PWR_FLAG" H 2050 1173 50  0000 C CNN
+F 2 "" H 2050 1000 50  0001 C CNN
+F 3 "~" H 2050 1000 50  0001 C CNN
+	1    2050 1000
+	1    0    0    -1
+$EndComp
+Connection ~ 2050 1000
+Wire Wire Line
+	2050 1000 2200 1000
+NoConn ~ 4950 3500
+Wire Wire Line
+	4950 3600 5200 3600
+Connection ~ 5200 3600
+Wire Wire Line
+	5500 3600 5950 3600
+Connection ~ 5500 3600
+Connection ~ 5950 3600
 $EndSCHEMATC

Commit message: Clear several more DRC warnings.
Other:
- moved on the sheet: S101
Changed lines of the file:
@@
 L GPAD_SCH_LIB:SWITCH_TACTILE_SPST-NO_0.05A_24V S101
 U 1 1 62BA946B
-P 5550 2200
-F 0 "S101" H 5550 2547 60  0000 C CNN
-F 1 "SWITCH_TACTILE_SPST-NO_0.05A_24V" H 5550 2441 60  0000 C CNN
-F 2 "digikey-footprints:Switch_Tactile_THT_6x6mm" H 5750 2400 60  0001 L CNN
-F 3 "https://www.te.com/commerce/DocumentDelivery/DDEController?Action=srchrtrv&DocNm=1825910&DocType=Customer+Drawing&DocLang=English" H 5750 2500 60  0001 L CNN
-F 4 "JLCPCB" H 5550 2200 50  0001 C CNN "Distributor 1"
-F 5 "C592982" H 5550 2200 50  0001 C CNN "Distributor 1 PN"
-F 6 "Digikey" H 5550 2200 50  0001 C CNN "Distributor 2"
-F 7 "450-1804-ND" H 5750 2600 60  0001 L CNN "Distributor 2 PN"
-F 8 "TE Connectivity ALCOSWITCH Switches" H 5750 3300 60  0001 L CNN "Manufacturer"
-F 9 "1825910-7" H 5750 2700 60  0001 L CNN "MPN"
-F 10 "Switches" H 5750 2800 60  0001 L CNN "Category"
-F 11 "Tactile Switches" H 5750 2900 60  0001 L CNN "Family"
-F 12 "https://www.te.com/commerce/DocumentDelivery/DDEController?Action=srchrtrv&DocNm=1825910&DocType=Customer+Drawing&DocLang=English" H 5750 3000 60  0001 L CNN "DK_Datasheet_Link"
-F 13 "/product-detail/en/te-connectivity-alcoswitch-switches/1825910-7/450-1804-ND/1731414" H 5750 3100 60  0001 L CNN "DK_Detail_Page"
-F 14 "SWITCH TACTILE SPST-NO 0.05A 24V" H 5750 3200 60  0001 L CNN "Description"
-F 15 "Active" H 5750 3400 60  0001 L CNN "Status"
-	1    5550 2200
+P 5800 2200
+F 0 "S101" H 5800 2547 60  0000 C CNN
+F 1 "SWITCH_TACTILE_SPST-NO_0.05A_24V" H 5800 2441 60  0000 C CNN
+F 2 "digikey-footprints:Switch_Tactile_THT_6x6mm" H 6000 2400 60  0001 L CNN
+F 3 "https://www.te.com/commerce/DocumentDelivery/DDEController?Action=srchrtrv&DocNm=1825910&DocType=Customer+Drawing&DocLang=English" H 6000 2500 60  0001 L CNN
+F 4 "JLCPCB" H 5800 2200 50  0001 C CNN "Distributor 1"
+F 5 "C592982" H 5800 2200 50  0001 C CNN "Distributor 1 PN"
+F 6 "Digikey" H 5800 2200 50  0001 C CNN "Distributor 2"
+F 7 "450-1804-ND" H 6000 2600 60  0001 L CNN "Distributor 2 PN"
+F 8 "TE Connectivity ALCOSWITCH Switches" H 6000 3300 60  0001 L CNN "Manufacturer"
+F 9 "1825910-7" H 6000 2700 60  0001 L CNN "MPN"
+F 10 "Switches" H 6000 2800 60  0001 L CNN "Category"
+F 11 "Tactile Switches" H 6000 2900 60  0001 L CNN "Family"
+F 12 "https://www.te.com/commerce/DocumentDelivery/DDEController?Action=srchrtrv&DocNm=1825910&DocType=Customer+Drawing&DocLang=English" H 6000 3000 60  0001 L CNN "DK_Datasheet_Link"
+F 13 "/product-detail/en/te-connectivity-alcoswitch-switches/1825910-7/450-1804-ND/1731414" H 6000 3100 60  0001 L CNN "DK_Detail_Page"
+F 14 "SWITCH TACTILE SPST-NO 0.05A 24V" H 6000 3200 60  0001 L CNN "Description"
+F 15 "Active" H 6000 3400 60  0001 L CNN "Status"
+	1    5800 2200
 	1    0    0    -1
 $EndComp
@@
 L power:GND #PWR0117
 U 1 1 62BAA497
-P 6050 2100
-F 0 "#PWR0117" H 6050 1850 50  0001 C CNN
-F 1 "GND" H 6055 1927 50  0000 C CNN
-F 2 "" H 6050 2100 50  0001 C CNN
-F 3 "" H 6050 2100 50  0001 C CNN
-	1    6050 2100
+P 6300 2100
+F 0 "#PWR0117" H 6300 1850 50  0001 C CNN
+F 1 "GND" H 6305 1927 50  0000 C CNN
+F 2 "" H 6300 2100 50  0001 C CNN
+F 3 "" H 6300 2100 50  0001 C CNN
+	1    6300 2100
 	1    0    0    -1
 $EndComp
@@
 Connection ~ 5050 2100
 Wire Wire Line
-	5050 2100 5250 2100
-Wire Wire Line
 	5050 2450 5050 2550
 Wire Wire Line
-	5350 2300 5250 2300
-Wire Wire Line
-	5250 2300 5250 2100
-Connection ~ 5250 2100
-Wire Wire Line
-	5250 2100 5350 2100
-Wire Wire Line
-	5750 2100 5850 2100
-Wire Wire Line
-	5750 2300 5850 2300
-Wire Wire Line
-	5850 2300 5850 2100
-Connection ~ 5850 2100
-Wire Wire Line
-	5850 2100 6050 2100
+	6000 2100 6100 2100
+Wire Wire Line
+	6000 2300 6100 2300
+Wire Wire Line
+	6100 2300 6100 2100
+Connection ~ 6100 2100
+Wire Wire Line
+	6100 2100 6300 2100
 Wire Wire Line
 	4200 2250 4750 2250
@@
 	3200 1050 3200 1000
 Connection ~ 3200 1000
-Wire Wire Line
-	3200 1000 3750 1000
 Wire Wire Line
 	2900 1100 3000 1100
@@
 Connection ~ 5500 3600
 Connection ~ 5950 3600
+Wire Wire Line
+	5550 2300 5550 2100
+Wire Wire Line
+	5550 2300 5600 2300
+Connection ~ 5550 2100
+Wire Wire Line
+	5550 2100 5600 2100
+Wire Wire Line
+	5050 2100 5550 2100
+Wire Wire Line
+	3200 1000 3750 1000
+Text Label 3450 1000 0    50   ~ 0
++5V
 $EndSCHEMATC

Commit message: Pull parts into PCB Begin rough placement into groups.
Parts:
- added R104: 1R0, Resistor_SMD:R_0603_1608Metric, symbol Device:R
- XTAL101: footprint (none) -> Crystal:Crystal_SMD_HC49-SD
Connections:
- net +5V: now also R104.1; no longer U101.4 (OUT)
- net GND: now also J101.2, J101.3
- new net: R104.2, U101.4 (OUT)
Other:
- note added: "To do: Remove resistor from U101 pin 2 to 4."
Changed lines of the file:
@@
 F 0 "XTAL101" H 2600 4290 50  0000 C CNN
 F 1 "16MHZ 20PF HC-49S/SMD" H 2700 4200 50  0000 C CNN
-F 2 "" H 2800 4250 60  0001 L CNN
+F 2 "Crystal:Crystal_SMD_HC49-SD" H 2800 4250 60  0001 L CNN
 F 3 "1811061718_TAE-Zhejiang-Abel-Elec-TAXM16M2GLFBET2T_C111377.pdf" H 2800 4350 60  0001 L CNN
 F 4 "JLCPCB" H 2600 4050 50  0001 C CNN "Distributor 1"
@@
 	2500 1500 2500 1400
 Wire Wire Line
-	2900 1000 3000 1000
-Wire Wire Line
 	3900 1000 3900 900
 Wire Wire Line
@@
 Connection ~ 3200 1000
 Wire Wire Line
-	2900 1100 3000 1100
-Wire Wire Line
-	3000 1100 3000 1000
-Connection ~ 3000 1000
-Wire Wire Line
-	3000 1000 3200 1000
-Wire Wire Line
 	3200 1350 3200 1450
 Wire Wire Line
@@
 Wire Wire Line
 	1300 1300 1300 1000
-Wire Wire Line
-	1300 1600 1300 1700
 $Comp
 L power:GND #PWR0101
@@
 Connection ~ 4250 2100
 Wire Wire Line
-	4250 2100 2950 2100
+	4250 2100 3050 2100
 Wire Wire Line
 	2950 4550 2950 4650
@@
 Text Label 3450 1000 0    50   ~ 0
 +5V
+$Comp
+L power:PWR_FLAG #FLG0105
+U 1 1 62E7BE21
+P 3050 2100
+F 0 "#FLG0105" H 3050 2175 50  0001 C CNN
+F 1 "PWR_FLAG" H 3050 2273 50  0000 C CNN
+F 2 "" H 3050 2100 50  0001 C CNN
+F 3 "~" H 3050 2100 50  0001 C CNN
+	1    3050 2100
+	1    0    0    -1
+$EndComp
+Connection ~ 3050 2100
+Wire Wire Line
+	3050 2100 2950 2100
+Wire Wire Line
+	1300 1600 1300 1650
+Wire Wire Line
+	2900 1000 3050 1000
+$Comp
+L Device:R R104
+U 1 1 62E95591
+P 3050 1350
+AR Path="/62E95591" Ref="R104"  Part="1"
+AR Path="/62B871EE/62E95591" Ref="R?"  Part="1"
+F 0 "R104" V 2850 1300 50  0000 C CNN
+F 1 "1R0" V 2950 1350 50  0000 C CNN
+F 2 "Resistor_SMD:R_0603_1608Metric" V 2980 1350 50  0001 C CNN
+F 3 "~" H 3050 1350 50  0001 C CNN
+F 4 "JLCPCB" V 3050 1350 50  0001 C CNN "Distributor 1"
+F 5 "C269434" V 3050 1350 50  0001 C CNN "Distributor 1 PN"
+F 6 "TyoHM" V 3050 1350 50  0001 C CNN "Manufacturer"
+F 7 "RMC060315%N" V 3050 1350 50  0001 C CNN "MPN"
+F 8 "0.1W ±5% 1Ω 0603 Chip Resistor - Surface Mount ROHS" H 3050 1350 50  0001 C CNN "Description"
+	1    3050 1350
+	1    0    0    -1
+$EndComp
+Wire Wire Line
+	3050 1200 3050 1000
+Connection ~ 3050 1000
+Wire Wire Line
+	3050 1000 3200 1000
+Wire Wire Line
+	2900 1100 2900 1700
+Wire Wire Line
+	2900 1700 3050 1700
+Wire Wire Line
+	3050 1700 3050 1500
+Text Notes 2300 1450 0    50   ~ 10
+To do: Remove resistor from U101 pin 2 to 4.
+Wire Wire Line
+	1250 1200 1250 1350
+Wire Wire Line
+	1250 1350 1000 1350
+Wire Wire Line
+	1000 1350 1000 1650
+Wire Wire Line
+	1000 1650 1300 1650
+Connection ~ 1250 1200
+Connection ~ 1300 1650
+Wire Wire Line
+	1300 1650 1300 1700
 $EndSCHEMATC
