File: Hardware/GeneralPurposeAlarmDevicePCB/GeneralPurposeAlarmDevicePCB/GeneralPurposeAlarmDevicePCB.sch (KiCad schematic (older format))
At the start: 24 parts, among them J101 Barrel_Jack_Switch_SMT, J102 22-23-2021, J103 22-23-2021, U101 NCP1117ST50T3G, U102 PI_ATMEGA328P-AU-InOrder

Commit message: Add new LED, RJ12 footprints to footprint library. Add STEP model.
Parts:
- removed R104: 1R0, Resistor_SMD:R_0603_1608Metric, symbol Device:R
- removed U101: NCP1117ST50T3G, digikey-footprints:SOT-223, symbol dk_PMIC-Voltage-Regulators-Linear:NCP1117ST50T3G
- added C105: 100nF, Capacitor_SMD:C_0603_1608Metric_Pad1.08x0.95mm_HandSolder, symbol Device:C
- added H101, H102, H103, H104: MountingHole_Pad_3.5mm, GeneralPurposeAlarmDevicePCB:MountingHole_3.5mm_Pad_Via, symbol GPAD_SCH_LIB:MountingHole_Pad_3.5mm
- added U101: NCP1117ST50T3G, digikey-footprints:SOT-223, symbol GPAD_SCH_LIB:NCP1117ST50T3G
- D102: footprint LED_SMD:LED_0603_1608Metric -> digikey-footprints:0805; DK_Datasheet_Link (none) -> http://optoelectronics.liteon.com/upload/download/DS22-2000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; DK_Detail_Page (none) -> /product-detail/en/lite-on-inc/LTST-C171KRKT/160-1427-1-ND/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; Digi-Key_PN (none) -> 160-1427-1-ND; MPN KT-0603R -> LTST-C171KRKT; Manufacturer Hubei KENTO Elec -> Lite-On Inc.
- J101: footprint Connector_BarrelJack:BarrelJack_CLIFF_FC681465S_SMT_Horizontal -> GeneralPurposeAlarmDevicePCB:BarrelJack_CLIFF_FC681465S_SMT_Horizontal
- S101: footprint digikey-footprints:Switch_Tactile_THT_6x6mm -> GeneralPurposeAlarmDevicePCB:Switch_Tactile_THT_6x6mm; Distributor 1 PN C592982 -> C13828; MPN 1825910-7 -> TE Connectivity 1825910-7, Dongguan Guangzhu Industrial C13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
- XTAL101: footprint Crystal:Crystal_SMD_HC49-SD -> digikey-footprints:SMD-2_3.2x2.5mm; DK_Datasheet_Link (none) -> http://www.ndk.com/images/products/catalog/c_NX3225GD-STD-C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; DK_Detail_Page (none) -> /product-detail/en/ndk-america-inc/NX3225GD-8MHZ-STD-CRA-3/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; Description CRYSTAL 16.0000MHZ 20PF HC49SSMD -> CRYSTAL 8.0000MHZ 8PF SMD; Digi-Key_PN (none) -> 644-1178-1-ND; MPN TAXM16M2GLFBET2T -> NX3225GD-8MHZ-STD-CRA-3; Manufacturer TAE -> NDK America, Inc.
- renumbered C105 to C106, C106 to C107, C107 to C108, C108 to C109, C109 to C110, C110 to C111, C111 to C112
Connections:
- net labels added: Switch_Mute
- wire segments 161 -> 173
- no-connect marks 9 -> 8
Other:
- note removed: "To do: Remove resistor from U101 pin 2 to 4."
- moved on the sheet: C102

Commit message: Add JST connector for I2C and more.
Parts:
- removed J102, J103: 22-23-2021, digikey-footprints:PinHeader_1x2_P2.54mm_Drill1.02mm, symbol dk_Rectangular-Connectors-Headers-Male-Pins:22-23-2021
- added C113, C114: 33pF, Capacitor_SMD:C_0603_1608Metric_Pad1.08x0.95mm_HandSolder, symbol Device:C
- added J102, J103: 22-23-2021, Connector_Molex:Molex_KK-254_AE-6410-02A_1x02_P2.54mm_Vertical, symbol GPAD_SCH_LIB:22-23-2021
- added J105: S04B-XASK-1(LF)(SN), Connector_PinHeader_2.54mm:PinHeader_1x04_P2.54mm_Horizontal, symbol GPAD_SCH_LIB:S04B-XASK-1(LF)(SN)
- added R104, R105: 39R, Resistor_SMD:R_0603_1608Metric, symbol Device:R
Connections:
- wire segments 173 -> 191

Commit message: Add more parts including a place holder only for power jack 3D, USB micro is incomplete. Added I2C daisy chain connector.
Parts:
- added D103: 1N5819WS, GeneralPurposeAlarmDevicePCB:D_SOD-323, symbol GPAD_SCH_LIB:1N5819WS
- U102: footprint digikey-footprints:TQFP-32_7x7mm -> Package_QFP:TQFP-32_7x7mm_P0.8mm
Connections:
- wire segments 191 -> 196
Changed lines of the file:
@@
 F 0 "U102" H 3150 4100 60  0000 L CNN
 F 1 "PI_ATMEGA328P-AU-InOrder" H 3600 2900 60  0000 L CNN
-F 2 "digikey-footprints:TQFP-32_7x7mm" H 3400 3400 60  0001 L CNN
+F 2 "Package_QFP:TQFP-32_7x7mm_P0.8mm" H 3400 3400 60  0001 L CNN
 F 3 "http://www.microchip.com/mymicrochip/filehandler.aspx?ddocname=en608326" V 4900 2240 60  0001 L CNN
 F 4 "DigiKey" H 3100 3050 50  0001 C CNN "Distributor 1"
@@
 Connection ~ 4750 2100
 Wire Wire Line
-	4750 2100 5050 2100
+	4750 2100 4900 2100
 $Comp
 L Device:R R101
@@
 Wire Wire Line
 	8500 2600 8950 2600
+Wire Wire Line
+	4900 1650 4900 2100
+Connection ~ 4900 2100
+Wire Wire Line
+	4900 2100 5050 2100
+Wire Wire Line
+	4400 1650 4250 1650
+Wire Wire Line
+	4250 1650 4250 1800
+Connection ~ 4250 1800
+Wire Wire Line
+	4700 1650 4900 1650
+$Comp
+L GPAD_SCH_LIB:1N5819WS D103
+U 1 1 62EB37D5
+P 4500 1650
+F 0 "D103" H 4550 1875 50  0000 C CNN
+F 1 "1N5819WS" H 4550 1784 50  0000 C CNN
+F 2 "GeneralPurposeAlarmDevicePCB:D_SOD-323" H 4700 1850 60  0001 L CNN
+F 3 "https://www.diodes.com/assets/Datasheets/ds30217.pdf" H 4700 1950 60  0001 L CNN
+F 4 "1N5819WS" H 4700 2150 60  0001 L CNN "MPN"
+F 5 "Discrete Semiconductor Products" H 4700 2250 60  0001 L CNN "Category"
+F 6 "Diodes - Rectifiers - Single" H 4700 2350 60  0001 L CNN "Family"
+F 7 "40V 600mV@1A 1A SOD-323  Schottky Barrier Diodes (SBD) ROHS" H 4700 2650 60  0001 L CNN "Description"
+F 8 "Guangdong Hottech" H 4700 2750 60  0001 L CNN "Manufacturer"
+F 9 "Active" H 4700 2850 60  0001 L CNN "Status"
+F 10 "JLCPCB" H 4500 1650 50  0001 C CNN "Distributor 1"
+F 11 "C191023" H 4500 1650 50  0001 C CNN "Distributor 1 PN"
+	1    4500 1650
+	1    0    0    -1
+$EndComp
 $EndSCHEMATC

Commit message: Add current limit to CongtollerVcc, and Barrel Input. Add jumper resistors for headers selecting VBus and ControllerVcc.
Parts:
- added A101: Arduino_UNO_R3, Module:Arduino_UNO_R3, symbol MCU_Module:Arduino_UNO_R3
- added D?: Schottky 2A, Diode_SMD:D_SMB, symbol Device:D_Schottky
- added F?: Polyfuse_Small, symbol Device:Polyfuse_Small
- added R? (x2): DNI, Resistor_SMD:R_0603_1608Metric, symbol Device:R
Connections:
- net labels added: Attenuate
- wire segments 196 -> 224
- no-connect marks 8 -> 7
Other:
- note added: "Notes:\nArduino Pin to ATmega328\nA0 PC0\nA1 PC1\nA2 PC2\nA3 PC3\nA4 PC4\nA5 PC5\nD0 PD0\nD1 PD1\nD2 PD2\n'D3 PD3\nD4 PD4\n`D5 PD5\n`D6 PD6\nD7 PD7\nD8 PB0\n`D9 PB1\n`D10 PB2\n`D11 PB3\nD12 PB4\nD13 PB5\n\nRemark:\nPC4 as SDA and PC5 as SCL \nis conventional UNO pinout.\nSame for Rx and Tx."
- note removed: "Notes:\nArduino Pin to ATmega328\nA0 PC0\nA1 PC1\nA2 PC2\nA3 PC3\nA4 PC4\nA5 PC5\nD0 PD0\nD1 PD1\nD2 PD2\n'D3 PD3\nD4 PD4\n`D5 PD5\n`D6 PD6\nD7 PD7\nD8 PB0\n`D9 PB1\n`D10 PB2\n`D11 PB3\nD12 PB4\nD13 PB5"
- moved on the sheet: C101, C102, C105, C108, C109, C113, C114, D101, J101, J102, J103, J105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

Commit message: Update schottky symbol and part number. Import to PCB. Only the Arduino UNO symbol remains to connect.
Parts:
- removed D103: 1N5819WS, GeneralPurposeAlarmDevicePCB:D_SOD-323, symbol GPAD_SCH_LIB:1N5819WS
- added D103: Schottky 2A, Diode_SMD:D_SMB, symbol Device:D_Schottky
- added R108, R109: 1K, Resistor_SMD:R_0603_1608Metric, symbol Device:R
- F101: renamed from F?; footprint (none) -> Fuse:Fuse_0603_1608Metric; MPN (none) -> 0603L100SLYR; Manufacturier (none) -> Littelfuse
- gave numbers to parts that had none: 3
Connections:
- wire segments 224 -> 240
Other:
- moved on the sheet: C102, C110, R101, S101

Commit message: Add both UNO and NANO schematic and PCB foot print.  Zero schematic errors reported. This incorporates all of the updates from the review except the DO NOT FIX.
Parts:
- removed A101: Arduino_UNO_R3, Module:Arduino_UNO_R3, symbol MCU_Module:Arduino_UNO_R3
- added A101: Arduino_UNO_R3_Shield, Module:Arduino_UNO_R3, symbol GPAD_SCH_LIB:Arduino_UNO_R3_Shield
- added A102: Arduino_Nano_v2.x_Header, Module:Arduino_Nano, symbol GPAD_SCH_LIB:Arduino_Nano_v2.x_Header
Connections:
- net +5V: now also A101.2 (IOREF), A101.5 (+5V), A102.27 (+5V)
- net Attenuate: now also A101.19 (D4), A102.7 (D4)
- net CIPO: now also A101.27 (D12), A102.15 (D12)
- net COPI: now also A101.26 (D11), A102.14 (D11)
- net ControllerRX: now also A101.15 (D0/RX), A102.2 (D0/RX)
- net ControllerTX: now also A101.16 (D1/TX), A102.1 (D1/TX)
- net GND: now also U102.3 (GND), A101.29 (GND), A101.6 (GND), A101.7 (GND), A102.29 (GND), A102.4 (GND)
- net Light0: now also A101.18 (D3), A102.6 (D3)
- net Light1: now also A101.20 (D5), A102.8 (D5)
- net Light2: now also A101.21 (D6), A102.9 (D6)
- net Light3: now also A101.24 (D9), A102.12 (D9)
- net Light4: now also A101.25 (D10), A102.13 (D10)
- net SCL: now also A101.14 (SCL/A5), A101.32 (SCL/A5), A102.24 (A5)
- net SDA: now also A101.13 (SDA/A4), A101.31 (SDA/A4), A102.23 (A4)
- net SPI_SCK: now also A101.28 (D13), A102.16 (D13)
- net Switch_Mute: now also A101.17 (D2), A102.5 (D2)
- net Tone: now also A101.23 (D8), A102.11 (D8)
- net nCS: now also A101.22 (D7), A102.10 (D7)
- net ADC6: now reaches U102.19 (ADC6)
- net ADC6: now also A102.25 (A6)
- net ADC7: now reaches U102.22 (ADC7)
- net ADC7: now also A102.26 (A7)
- net PC0: now reaches U102.23 (PC0)
- net PC0: now also A101.9 (A0), A102.19 (A0)
- net PC1: now reaches U102.24 (PC1)
- net PC1: now also A101.10 (A1), A102.20 (A1)
- net PC2: now reaches U102.25 (PC2)
- net PC2: now also A101.11 (A2), A102.21 (A2)
- net PC3: now reaches U102.26 (PC3)
- net PC3: now also A101.12 (A3), A102.22 (A3)
- net nRESET: now reaches C110.1, D103.2 (A), R102.1, S101.1, S101.2, U102.29 (~RESET~/PC6)
- net nRESET: now also A101.3 (~RESET), A102.28 (~RESET), A102.3 (~RESET)
- net Vin: now reaches C102.1, C105.1, D101.1 (K), D104.1 (K), U101.3 (IN)
- net Vin: now also A101.8 (VIN), A102.30 (VIN)
- net VccControler renamed Aref
- net Aref: now also A101.30 (AREF), A102.18 (AREF)
- no-connect marks 7 -> 3
Other:
- note added: "NANO Headers"
- note added: "Notes:\nArduino Pin to ATmega328\nA0 PC0\nA1 PC1\nA2 PC2\nA3 PC3\nA4 PC4\nA5 PC5\nD0 PD0\nD1 PD1\nD2 PD2\n'D3 PD3\nD4 PD4\n`D5 PD5\n`D6 PD6\nD7 PD7\nD8 PB0\n`D9 PB1\n`D10 PB2\n`D11 PB3\nD12 PB4\nD13 PB5\n\nRemark:\nPC4 as SDA\nPC5 as SCL \nis conventional\n UNO pinout.\nSame for Rx and Tx."
- note added: "UNO Headers"
- note removed: "Notes:\nArduino Pin to ATmega328\nA0 PC0\nA1 PC1\nA2 PC2\nA3 PC3\nA4 PC4\nA5 PC5\nD0 PD0\nD1 PD1\nD2 PD2\n'D3 PD3\nD4 PD4\n`D5 PD5\n`D6 PD6\nD7 PD7\nD8 PB0\n`D9 PB1\n`D10 PB2\n`D11 PB3\nD12 PB4\nD13 PB5\n\nRemark:\nPC4 as SDA and PC5 as SCL \nis conventional UNO pinout.\nSame for Rx and Tx."
- moved on the sheet: C103, C104, C106, C107, C110, C111, C112, C113, C114, D102, D103, H101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

Commit message: Clean up a bunch of duplicate because of missspelled part field names. Still working on a few sch, pcb and 3D libraries.
Parts:
- C103, C105, C108, C110, C111, C113, C114: Manufacturer (none) -> YAGEO; Manufacturier YAGEO -> (none)
- D101, D103, D104: Distirbutor 1 PN C14996 -> (none); Distributor 1 PN (none) -> C14996
- F101: Manufacturer (none) -> Littelfuse; Manufacturier Littelfuse -> (none)
- J101: Manufacturer (none) -> XKB Connectivity / Tensility International Corp; Manufacturier XKB Connectivity / Tensility International Corp -> (none)
- J102, J103, J105, S101: Assembly Type (none) -> HAND
- XTAL101: Distributor 1 PN (none) -> TAXM16M2GLFBET2T; Distributor1 PN TAXM16M2GLFBET2T -> (none)
Changed lines of the file:
@@
 F 3 "http://www.ndk.com/images/products/catalog/c_NX3225GD-STD-CRA-3_e.pdf" H 2300 5100 60  0001 L CNN
 F 4 "JLCPCB" H 2100 4800 50  0001 C CNN "Distributor 1"
-F 5 "TAXM16M2GLFBET2T" H 2300 5200 60  0001 L CNN "Distributor1 PN"
+F 5 "TAXM16M2GLFBET2T" H 2300 5200 60  0001 L CNN "Distributor 1 PN"
 F 6 "NX3225GD-8MHZ-STD-CRA-3" H 2300 5300 60  0001 L CNN "MPN"
 F 7 "Crystals, Oscillators, Resonators" H 2300 5400 60  0001 L CNN "Category"
@@
 F 3 "~" H 1950 950 50  0001 C CNN
 F 4 "JLCPCB" H 1950 950 50  0001 C CNN "Distributor 1"
-F 5 "C14996" H 1950 950 50  0001 C CNN "Distirbutor 1 PN"
+F 5 "C14996" H 1950 950 50  0001 C CNN "Distributor 1 PN"
 F 6 "SS210" H 1950 950 50  0001 C CNN "MPN"
 F 7 "MDD（Microdiode Electronics）" H 1950 950 50  0001 C CNN "Manufacturer"
@@
 F 4 "JLCPCB" H 3650 1150 50  0001 C CNN "Distributor 1"
 F 5 "C14663" H 3650 1150 50  0001 C CNN "Distributor 1 PN"
-F 6 "YAGEO" H 3650 1150 50  0001 C CNN "Manufacturier"
+F 6 "YAGEO" H 3650 1150 50  0001 C CNN "Manufacturer"
 F 7 "CC0603KRX7R9BB104" H 3650 1150 50  0001 C CNN "MPN"
 F 8 "50V 100nF X7R ±10% 0603 Multilayer Ceramic Capacitors MLCC - SMD/SMT ROHS" H 3650 1150 50  0001 C CNN "Description"
@@
 F 4 "JLCPCB" H 850 1050 50  0001 C CNN "Distributor 1"
 F 5 "C319134" H 850 1050 50  0001 C CNN "Distributor 1 PN"
-F 6 "XKB Connectivity / Tensility International Corp" H 850 1050 50  0001 C CNN "Manufacturier"
+F 6 "XKB Connectivity / Tensility International Corp" H 850 1050 50  0001 C CNN "Manufacturer"
 F 7 "DC-005-5A-2.0-SMT / 54-00164" H 850 1050 50  0001 C CNN "MPN"
 F 8 "Power Barrel Connector Jack 2.10mm ID (0.083\"), 5.50mm OD (0.217\") Surface Mount, Right Angle" H 850 1050 50  0001 C CNN "Description"
@@
 F 4 "JLCPCB" H 1500 4050 50  0001 C CNN "Distributor 1"
 F 5 "C14663" H 1500 4050 50  0001 C CNN "Distributor 1 PN"
-F 6 "YAGEO" H 1500 4050 50  0001 C CNN "Manufacturier"
+F 6 "YAGEO" H 1500 4050 50  0001 C CNN "Manufacturer"
 F 7 "CC0603KRX7R9BB104" H 1500 4050 50  0001 C CNN "MPN"
 F 8 "50V 100nF X7R ±10% 0603 Multilayer Ceramic Capacitors MLCC - SMD/SMT ROHS" H 1500 4050 50  0001 C CNN "Description"
@@
 F 4 "JLCPCB" H 5000 4500 50  0001 C CNN "Distributor 1"
 F 5 "C14663" H 5000 4500 50  0001 C CNN "Distributor 1 PN"
-F 6 "YAGEO" H 5000 4500 50  0001 C CNN "Manufacturier"
+F 6 "YAGEO" H 5000 4500 50  0001 C CNN "Manufacturer"
 F 7 "CC0603KRX7R9BB104" H 5000 4500 50  0001 C CNN "MPN"
 F 8 "50V 100nF X7R ±10% 0603 Multilayer Ceramic Capacitors MLCC - SMD/SMT ROHS" H 5000 4500 50  0001 C CNN "Description"
@@
 F 14 "SWITCH TACTILE SPST-NO 0.05A 24V" H 5700 3700 60  0001 L CNN "Description"
 F 15 "Active" H 5700 3900 60  0001 L CNN "Status"
+F 16 "HAND" H 0   0   50  0001 C CNN "Assembly Type"
 	1    5500 2700
 	1    0    0    -1
@@
 F 4 "JLCPCB" H 4900 2800 50  0001 C CNN "Distributor 1"
 F 5 "C14663" H 4900 2800 50  0001 C CNN "Distributor 1 PN"
-F 6 "YAGEO" H 4900 2800 50  0001 C CNN "Manufacturier"
+F 6 "YAGEO" H 4900 2800 50  0001 C CNN "Manufacturer"
 F 7 "CC0603KRX7R9BB104" H 4900 2800 50  0001 C CNN "MPN"
 F 8 "50V 100nF X7R ±10% 0603 Multilayer Ceramic Capacitors MLCC - SMD/SMT ROHS" H 4900 2800 50  0001 C CNN "Description"
@@
 F 4 "JLCPCB" H 2600 1350 50  0001 C CNN "Distributor 1"
 F 5 "C14663" H 2600 1350 50  0001 C CNN "Distributor 1 PN"
-F 6 "YAGEO" H 2600 1350 50  0001 C CNN "Manufacturier"
+F 6 "YAGEO" H 2600 1350 50  0001 C CNN "Manufacturer"
 F 7 "CC0603KRX7R9BB104" H 2600 1350 50  0001 C CNN "MPN"
 F 8 "50V 100nF X7R ±10% 0603 Multilayer Ceramic Capacitors MLCC - SMD/SMT ROHS" H 2600 1350 50  0001 C CNN "Description"
@@
 F 11 "Molex" H 5300 1900 60  0001 L CNN "Manufacturer"
 F 12 "Active" H 5300 2000 60  0001 L CNN "Status"
+F 13 "HAND" H 0   0   50  0001 C CNN "Assembly Type"
 	1    5100 800
 	1    0    0    1
@@
 U 1 1 62D31EA3
 P 6550 800
-F 0 "J103" H 6463 762 50  0000 R CNN
-F 1 "22-23-2021" H 6463 853 50  0000 R CNN
+F 0 "J103" H 6450 650 50  0000 R CNN
+F 1 "22-23-2021" H 6450 750 50  0000 R CNN
 F 2 "Connector_Molex:Molex_KK-254_AE-6410-02A_1x02_P2.54mm_Vertical" H 6750 1000 60  0001 L CNN
 F 3 "https://media.digikey.com/pdf/Data%20Sheets/Molex%20PDFs/A-6373-N_Series_Dwg_2010-12-03.pdf" H 6750 1100 60  0001 L CNN
@@
 F 11 "Molex" H 6750 1900 60  0001 L CNN "Manufacturer"
 F 12 "Active" H 6750 2000 60  0001 L CNN "Status"
+F 13 "HAND" H 0   0   50  0001 C CNN "Assembly Type"
 	1    6550 800
 	1    0    0    1
@@
 F 12 "C265097" H 9800 2350 50  0001 C CNN "Distributor 1 PN"
 F 13 "DigiKey  " H 9800 2350 50  0001 C CNN "Distributor 2"
-F 14 "455-4090-ND" V 10036 2222 50  0000 R CNN "Distributor 2 PN"
+F 14 "455-4090-ND" V 10036 2222 50  0001 R CNN "Distributor 2 PN"
+F 15 "HAND" H 0   0   50  0001 C CNN "Assembly Type"
 	1    9800 2350
 	0    -1   1    0
@@
 F 4 "JLCPCB" H 9000 2950 50  0001 C CNN "Distributor 1"
 F 5 "C107047" H 9000 2950 50  0001 C CNN "Distributor 1 PN"
-F 6 "YAGEO" H 9000 2950 50  0001 C CNN "Manufacturier"
+F 6 "YAGEO" H 9000 2950 50  0001 C CNN "Manufacturer"
 F 7 "CC0603JRNPO9BN330" H 9000 2950 50  0001 C CNN "MPN"
 F 8 "50V 33pF NP0 ±5% 0603  Multilayer Ceramic Capacitors MLCC - SMD/SMT ROHS" H 9000 2950 50  0001 C CNN "Description"
@@
 F 4 "JLCPCB" H 9450 2950 50  0001 C CNN "Distributor 1"
 F 5 "C107047" H 9450 2950 50  0001 C CNN "Distributor 1 PN"
-F 6 "YAGEO" H 9450 2950 50  0001 C CNN "Manufacturier"
+F 6 "YAGEO" H 9450 2950 50  0001 C CNN "Manufacturer"
 F 7 "CC0603JRNPO9BN330" H 9450 2950 50  0001 C CNN "MPN"
 F 8 "50V 33pF NP0 ±5% 0603  Multilayer Ceramic Capacitors MLCC - SMD/SMT ROHS" H 9450 2950 50  0001 C CNN "Description"
@@
 F 2 "Fuse:Fuse_0603_1608Metric" H 1600 750 50  0001 L CNN
 F 3 "https://datasheet.lcsc.com/lcsc/1806131741_Littelfuse-0603L075SLYR_C207016.pdf" H 1550 950 50  0001 C CNN
-F 4 "Littelfuse" V 1550 950 50  0001 C CNN "Manufacturier"
+F 4 "Littelfuse" V 1550 950 50  0001 C CNN "Manufacturer"
 F 5 "0603L100SLYR" V 1550 950 50  0001 C CNN "MPN"
 	1    1550 950
@@
 U 1 1 62E0564A
 P 6250 1100
-F 0 "D104" H 6250 883 50  0000 C CNN
-F 1 "Schottky 2A" H 6250 974 50  0000 C CNN
+F 0 "D104" H 6100 1200 50  0000 C CNN
+F 1 "Schottky 2A" H 6050 1300 50  0000 C CNN
 F 2 "Diode_SMD:D_SMB" H 6250 1100 50  0001 C CNN
 F 3 "~" H 6250 1100 50  0001 C CNN
 F 4 "JLCPCB" H 6250 1100 50  0001 C CNN "Distributor 1"
-F 5 "C14996" H 6250 1100 50  0001 C CNN "Distirbutor 1 PN"
+F 5 "C14996" H 6250 1100 50  0001 C CNN "Distributor 1 PN"
 F 6 "SS210" H 6250 1100 50  0001 C CNN "MPN"
 F 7 "MDD（Microdiode Electronics）" H 6250 1100 50  0001 C CNN "Manufacturer"
@@
 F 3 "~" H 3350 2150 50  0001 C CNN
 F 4 "JLCPCB" H 3350 2150 50  0001 C CNN "Distributor 1"
-F 5 "C14996" H 3350 2150 50  0001 C CNN "Distirbutor 1 PN"
+F 5 "C14996" H 3350 2150 50  0001 C CNN "Distributor 1 PN"
 F 6 "SS210" H 3350 2150 50  0001 C CNN "MPN"
 F 7 "MDD（Microdiode Electronics）" H 3350 2150 50  0001 C CNN "Manufacturer"

Commit message: Add and LED indicating power on.
Parts:
- added D105: LTL2R3KEK, GeneralPurposeAlarmDevicePCB:LED_5mm_Radial, symbol dk_LED-Indication-Discrete:LTL2R3KEK
- added R110: 330R, Resistor_SMD:R_0603_1608Metric, symbol Device:R
Connections:
- net +5V: now also R110.2
- net GND: now also D105.2
- new net: D105.1, R110.1
Other:
- note added: "Power Indicator"
Changed lines of the file:
@@
 	2400 950  2500 950
 Wire Wire Line
-	4350 950  4900 950
+	4350 950  4750 950
 $Comp
 L Device:D_Schottky D104
@@
 	1    0    0    -1
 $EndComp
+$Comp
+L dk_LED-Indication-Discrete:LTL2R3KEK D105
+U 1 1 62D73675
+P 5700 1700
+F 0 "D105" H 5650 2037 60  0000 C CNN
+F 1 "LTL2R3KEK" H 5800 1950 60  0000 C CNN
+F 2 "GeneralPurposeAlarmDevicePCB:LED_5mm_Radial" H 5900 1900 60  0001 L CNN
+F 3 "http://optoelectronics.liteon.com/upload/download/DS-20-98-0286/LTL2R3KEK.pdf" H 5900 2000 60  0001 L CNN
+F 4 "160-1682-ND" H 5900 2100 60  0001 L CNN "Digi-Key_PN"
+F 5 "LTL2R3KEK" H 5900 2200 60  0001 L CNN "MPN"
+F 6 "Optoelectronics" H 5900 2300 60  0001 L CNN "Category"
+F 7 "LED Indication - Discrete" H 5900 2400 60  0001 L CNN "Family"
+F 8 "http://optoelectronics.liteon.com/upload/download/DS-20-98-0286/LTL2R3KEK.pdf" H 5900 2500 60  0001 L CNN "DK_Datasheet_Link"
+F 9 "/product-detail/en/lite-on-inc/LTL2R3KEK/160-1682-ND/573572" H 5900 2600 60  0001 L CNN "DK_Detail_Page"
+F 10 "LED RED CLEAR T-1 3/4 T/H" H 5900 2700 60  0001 L CNN "Description"
+F 11 "Lite-On Inc." H 5900 2800 60  0001 L CNN "Manufacturer"
+F 12 "Active" H 5900 2900 60  0001 L CNN "Status"
+	1    5700 1700
+	1    0    0    -1
+$EndComp
+$Comp
+L Device:R R110
+U 1 1 62D74668
+P 5000 1700
+F 0 "R110" V 4800 1650 50  0000 C CNN
+F 1 "330R" V 4900 1700 50  0000 C CNN
+F 2 "Resistor_SMD:R_0603_1608Metric" V 4930 1700 50  0001 C CNN
+F 3 "~" H 5000 1700 50  0001 C CNN
+F 4 "JLCPCB" V 5000 1700 50  0001 C CNN "Distributor 1"
+F 5 "C269711" V 5000 1700 50  0001 C CNN "Distributor 1 PN"
+F 6 "TyoHM" V 5000 1700 50  0001 C CNN "Manufacturer"
+F 7 "RMC06033301%N" V 5000 1700 50  0001 C CNN "MPN"
+F 8 "0.1W ±1% 330Ω 0603 Chip Resistor - Surface Mount ROHS" H 5000 1700 50  0001 C CNN "Description"
+	1    5000 1700
+	0    1    1    0
+$EndComp
+$Comp
+L power:GND #PWR0128
+U 1 1 62D74F16
+P 6050 1700
+F 0 "#PWR0128" H 6050 1450 50  0001 C CNN
+F 1 "GND" H 6055 1527 50  0000 C CNN
+F 2 "" H 6050 1700 50  0001 C CNN
+F 3 "" H 6050 1700 50  0001 C CNN
+	1    6050 1700
+	1    0    0    -1
+$EndComp
+Wire Wire Line
+	6050 1700 5800 1700
+Wire Wire Line
+	4850 1700 4750 1700
+Wire Wire Line
+	4750 1700 4750 950
+Connection ~ 4750 950
+Wire Wire Line
+	4750 950  4900 950
+Text Notes 4750 1900 0    50   ~ 0
+Power Indicator
+Wire Wire Line
+	5500 1700 5150 1700
 $EndSCHEMATC
