File: Hardware/GeneralPurposeAlarmDevicePCB/GeneralPurposeAlarmDevicePCB/LCD And I2C Interface.sch (KiCad schematic (older format))
At the start: 18 parts

Commit message: Add more parts drawings, buzzer. Add additional schematic sheet for AlarmAudio.
Connections:
- net labels added: SCL, SDA
- wire segments 94 -> 93
Changed lines of the file:
@@
 $Descr USLetter 11000 8500
 encoding utf-8
-Sheet 3 5
+Sheet 3 6
 Title "GeneralPurposeAlarmDevicePCB"
 Date "2022-06-20"
@@
 Wire Wire Line
 	4950 3050 3050 3050
-Wire Wire Line
-	3050 3050 3050 3000
 Connection ~ 4950 3050
 Connection ~ 5250 2950
@@
 Text Notes 3650 1750 0    50   ~ 0
 Wiring of I2C to LCD from:\nhttps://alselectro.wordpress.com/2016/05/12/serial-lcd-i2c-module-pcf8574/
+Text HLabel 2850 2950 0    50   Input ~ 0
+SCL
+Text HLabel 3050 3050 0    50   BiDi ~ 0
+SDA
 $EndSCHEMATC

Commit message: Annote reference designators.
Parts:
- U302: renamed from U?; symbol GeneralPurposeAlarmDevicePCB-rescue:LCD_20x4_Character-GPAD_SCH_LIB -> GeneralPurposeAlarmDevicePCB-rescue:LCD_20x4_Character-GPAD_SCH_LIB-GeneralPurposeAlarmDevicePCB-rescue
- gave numbers to parts that had none: 17
Changed lines of the file:
@@
 $EndDescr
 $Comp
-L GeneralPurposeAlarmDevicePCB-rescue:LCD_20x4_Character-GPAD_SCH_LIB U?
+L GeneralPurposeAlarmDevicePCB-rescue:LCD_20x4_Character-GPAD_SCH_LIB-GeneralPurposeAlarmDevicePCB-rescue U?
 U 1 1 62B90F17
 P 7300 3050
 AR Path="/62B90F17" Ref="U?"  Part="1"
-AR Path="/62B871EE/62B90F17" Ref="U?"  Part="1"
-F 0 "U?" H 6950 4200 50  0000 C CNN
+AR Path="/62B871EE/62B90F17" Ref="U302"  Part="1"
+F 0 "U302" H 6950 4200 50  0000 C CNN
 F 1 "LCD_20x4_Character" H 7300 4100 50  0000 C CNN
 F 2 "Display:NHD-0420H1Z" H 7300 2150 50  0001 C CNN
@@
 P 7300 3950
 AR Path="/62B90F1D" Ref="#PWR?"  Part="1"
-AR Path="/62B871EE/62B90F1D" Ref="#PWR?"  Part="1"
-F 0 "#PWR?" H 7300 3700 50  0001 C CNN
+AR Path="/62B871EE/62B90F1D" Ref="#PWR0304"  Part="1"
+F 0 "#PWR0304" H 7300 3700 50  0001 C CNN
 F 1 "GND" H 7305 3777 50  0000 C CNN
 F 2 "" H 7300 3950 50  0001 C CNN
@@
 P 6150 3350
 AR Path="/62B90F36" Ref="U?"  Part="1"
-AR Path="/62B871EE/62B90F36" Ref="U?"  Part="1"
-F 0 "U?" H 6150 4231 50  0000 C CNN
+AR Path="/62B871EE/62B90F36" Ref="U301"  Part="1"
+F 0 "U301" H 6150 4231 50  0000 C CNN
 F 1 "PCF8574AT" H 6150 4140 50  0000 C CNN
 F 2 "Package_SO:SOIC-16W_5.3x10.2mm_P1.27mm" H 6150 3350 50  0001 C CNN
@@
 P 4250 2500
 AR Path="/62B90F41" Ref="R?"  Part="1"
-AR Path="/62B871EE/62B90F41" Ref="R?"  Part="1"
-F 0 "R?" H 4150 2450 50  0000 C CNN
+AR Path="/62B871EE/62B90F41" Ref="R303"  Part="1"
+F 0 "R303" H 4150 2450 50  0000 C CNN
 F 1 "4K7" H 4100 2550 50  0000 C CNN
 F 2 "Resistor_SMD:R_0603_1608Metric" V 4180 2500 50  0001 C CNN
@@
 P 4600 2500
 AR Path="/62B90F4C" Ref="R?"  Part="1"
-AR Path="/62B871EE/62B90F4C" Ref="R?"  Part="1"
-F 0 "R?" H 4500 2450 50  0000 C CNN
+AR Path="/62B871EE/62B90F4C" Ref="R304"  Part="1"
+F 0 "R304" H 4500 2450 50  0000 C CNN
 F 1 "1K" H 4450 2550 50  0000 C CNN
 F 2 "Resistor_SMD:R_0603_1608Metric" V 4530 2500 50  0001 C CNN
@@
 P 4950 2500
 AR Path="/62B90F83" Ref="R?"  Part="1"
-AR Path="/62B871EE/62B90F83" Ref="R?"  Part="1"
-F 0 "R?" H 4850 2450 50  0000 C CNN
+AR Path="/62B871EE/62B90F83" Ref="R306"  Part="1"
+F 0 "R306" H 4850 2450 50  0000 C CNN
 F 1 "1K" H 4800 2550 50  0000 C CNN
 F 2 "Resistor_SMD:R_0603_1608Metric" V 4880 2500 50  0001 C CNN
@@
 P 5250 2500
 AR Path="/62B90F8E" Ref="R?"  Part="1"
-AR Path="/62B871EE/62B90F8E" Ref="R?"  Part="1"
-F 0 "R?" H 5150 2450 50  0000 C CNN
+AR Path="/62B871EE/62B90F8E" Ref="R308"  Part="1"
+F 0 "R308" H 5150 2450 50  0000 C CNN
 F 1 "1K" H 5100 2550 50  0000 C CNN
 F 2 "Resistor_SMD:R_0603_1608Metric" V 5180 2500 50  0001 C CNN
@@
 P 3850 2500
 AR Path="/62B90F99" Ref="R?"  Part="1"
-AR Path="/62B871EE/62B90F99" Ref="R?"  Part="1"
-F 0 "R?" H 3750 2450 50  0000 C CNN
+AR Path="/62B871EE/62B90F99" Ref="R302"  Part="1"
+F 0 "R302" H 3750 2450 50  0000 C CNN
 F 1 "4K7" H 3700 2550 50  0000 C CNN
 F 2 "Resistor_SMD:R_0603_1608Metric" V 3780 2500 50  0001 C CNN
@@
 P 3500 2500
 AR Path="/62B90FA4" Ref="R?"  Part="1"
-AR Path="/62B871EE/62B90FA4" Ref="R?"  Part="1"
-F 0 "R?" H 3400 2450 50  0000 C CNN
+AR Path="/62B871EE/62B90FA4" Ref="R301"  Part="1"
+F 0 "R301" H 3400 2450 50  0000 C CNN
 F 1 "4K7" H 3350 2550 50  0000 C CNN
 F 2 "Resistor_SMD:R_0603_1608Metric" V 3430 2500 50  0001 C CNN
@@
 P 6150 4150
 AR Path="/62B90FAA" Ref="#PWR?"  Part="1"
-AR Path="/62B871EE/62B90FAA" Ref="#PWR?"  Part="1"
-F 0 "#PWR?" H 6150 3900 50  0001 C CNN
+AR Path="/62B871EE/62B90FAA" Ref="#PWR0302"  Part="1"
+F 0 "#PWR0302" H 6150 3900 50  0001 C CNN
 F 1 "GND" H 6155 3977 50  0000 C CNN
 F 2 "" H 6150 4150 50  0001 C CNN
@@
 P 8500 1950
 AR Path="/62B90FB0" Ref="#PWR?"  Part="1"
-AR Path="/62B871EE/62B90FB0" Ref="#PWR?"  Part="1"
-F 0 "#PWR?" H 8500 1700 50  0001 C CNN
+AR Path="/62B871EE/62B90FB0" Ref="#PWR0307"  Part="1"
+F 0 "#PWR0307" H 8500 1700 50  0001 C CNN
 F 1 "GND" H 8505 1777 50  0000 C CNN
 F 2 "" H 8500 1950 50  0001 C CNN
@@
 P 7450 1600
 AR Path="/62B90FBB" Ref="R?"  Part="1"
-AR Path="/62B871EE/62B90FBB" Ref="R?"  Part="1"
-F 0 "R?" V 7250 1550 50  0000 C CNN
+AR Path="/62B871EE/62B90FBB" Ref="R310"  Part="1"
+F 0 "R310" V 7250 1550 50  0000 C CNN
 F 1 "1R0" V 7350 1600 50  0000 C CNN
 F 2 "Resistor_SMD:R_0603_1608Metric" V 7380 1600 50  0001 C CNN
@@
 P 8500 1750
 AR Path="/62B90FC5" Ref="C?"  Part="1"
-AR Path="/62B871EE/62B90FC5" Ref="C?"  Part="1"
-F 0 "C?" H 8618 1796 50  0000 L CNN
+AR Path="/62B871EE/62B90FC5" Ref="C302"  Part="1"
+F 0 "C302" H 8618 1796 50  0000 L CNN
 F 1 "47uF 16V" H 8618 1705 50  0000 L CNN
 F 2 "Capacitor_SMD:CP_Elec_5x5.4" H 8538 1600 50  0001 C CNN
@@
 P 8000 1750
 AR Path="/62B90FD0" Ref="C?"  Part="1"
-AR Path="/62B871EE/62B90FD0" Ref="C?"  Part="1"
-F 0 "C?" H 8115 1796 50  0000 L CNN
+AR Path="/62B871EE/62B90FD0" Ref="C301"  Part="1"
+F 0 "C301" H 8115 1796 50  0000 L CNN
 F 1 "100nF" H 8115 1705 50  0000 L CNN
 F 2 "Capacitor_SMD:C_0603_1608Metric_Pad1.08x0.95mm_HandSolder" H 8038 1600 50  0001 C CNN
@@
 P 8000 1950
 AR Path="/62B90FD6" Ref="#PWR?"  Part="1"
-AR Path="/62B871EE/62B90FD6" Ref="#PWR?"  Part="1"
-F 0 "#PWR?" H 8000 1700 50  0001 C CNN
+AR Path="/62B871EE/62B90FD6" Ref="#PWR0305"  Part="1"
+F 0 "#PWR0305" H 8000 1700 50  0001 C CNN
 F 1 "GND" H 8005 1777 50  0000 C CNN
 F 2 "" H 8000 1950 50  0001 C CNN
@@
 P 8700 4400
 AR Path="/62B90FDC" Ref="#PWR?"  Part="1"
-AR Path="/62B871EE/62B90FDC" Ref="#PWR?"  Part="1"
-F 0 "#PWR?" H 8700 4150 50  0001 C CNN
+AR Path="/62B871EE/62B90FDC" Ref="#PWR0308"  Part="1"
+F 0 "#PWR0308" H 8700 4150 50  0001 C CNN
 F 1 "GND" H 8705 4227 50  0000 C CNN
 F 2 "" H 8700 4400 50  0001 C CNN
@@
 P 8000 3950
 AR Path="/62B90FE7" Ref="R?"  Part="1"
-AR Path="/62B871EE/62B90FE7" Ref="R?"  Part="1"
-F 0 "R?" H 7900 3900 50  0000 C CNN
+AR Path="/62B871EE/62B90FE7" Ref="R311"  Part="1"
+F 0 "R311" H 7900 3900 50  0000 C CNN
 F 1 "4K7" H 7850 4000 50  0000 C CNN
 F 2 "Resistor_SMD:R_0603_1608Metric" V 7930 3950 50  0001 C CNN
@@
 P 8600 4100
 AR Path="/62B90FF3" Ref="Q?"  Part="1"
-AR Path="/62B871EE/62B90FF3" Ref="Q?"  Part="1"
-F 0 "Q?" H 8804 4146 50  0000 L CNN
+AR Path="/62B871EE/62B90FF3" Ref="Q301"  Part="1"
+F 0 "Q301" H 8804 4146 50  0000 L CNN
 F 1 "BSS138" H 8804 4055 50  0000 L CNN
 F 2 "Package_TO_SOT_SMD:SOT-23" H 8800 4025 50  0001 L CIN
@@
 P 7100 1600
 AR Path="/62B90FFA" Ref="#PWR?"  Part="1"
-AR Path="/62B871EE/62B90FFA" Ref="#PWR?"  Part="1"
-F 0 "#PWR?" H 7100 1450 50  0001 C CNN
+AR Path="/62B871EE/62B90FFA" Ref="#PWR0303"  Part="1"
+F 0 "#PWR0303" H 7100 1450 50  0001 C CNN
 F 1 "+5V" H 7115 1773 50  0000 C CNN
 F 2 "" H 7100 1600 50  0001 C CNN
@@
 P 8250 2950
 AR Path="/62B91000" Ref="#PWR?"  Part="1"
-AR Path="/62B871EE/62B91000" Ref="#PWR?"  Part="1"
-F 0 "#PWR?" H 8250 2700 50  0001 C CNN
+AR Path="/62B871EE/62B91000" Ref="#PWR0306"  Part="1"
+F 0 "#PWR0306" H 8250 2700 50  0001 C CNN
 F 1 "GND" H 8255 2777 50  0000 C CNN
 F 2 "" H 8250 2950 50  0001 C CNN
@@
 P 8250 2700
 AR Path="/62B9100B" Ref="RV?"  Part="1"
-AR Path="/62B871EE/62B9100B" Ref="RV?"  Part="1"
-F 0 "RV?" H 8180 2791 50  0000 R CNN
+AR Path="/62B871EE/62B9100B" Ref="RV301"  Part="1"
+F 0 "RV301" H 8180 2791 50  0000 R CNN
 F 1 "10K" H 8180 2700 50  0000 R CNN
 F 2 "digikey-footprints:Trimpot_3.8mmx3.6mm_TC33X-2-103E" H 8250 2700 50  0001 C CNN
@@
 P 5100 4100
 AR Path="/62C558F4" Ref="#PWR?"  Part="1"
-AR Path="/62B871EE/62C558F4" Ref="#PWR?"  Part="1"
-F 0 "#PWR?" H 5100 3850 50  0001 C CNN
+AR Path="/62B871EE/62C558F4" Ref="#PWR0301"  Part="1"
+F 0 "#PWR0301" H 5100 3850 50  0001 C CNN
 F 1 "GND" H 5105 3927 50  0000 C CNN
 F 2 "" H 5100 4100 50  0001 C CNN
@@
 P 4600 3750
 AR Path="/62C6D2FC" Ref="R?"  Part="1"
-AR Path="/62B871EE/62C6D2FC" Ref="R?"  Part="1"
-F 0 "R?" H 4700 3800 50  0000 C CNN
+AR Path="/62B871EE/62C6D2FC" Ref="R305"  Part="1"
+F 0 "R305" H 4700 3800 50  0000 C CNN
 F 1 "1R0" H 4750 3700 50  0000 C CNN
 F 2 "Resistor_SMD:R_0603_1608Metric" V 4530 3750 50  0001 C CNN
@@
 P 4950 3750
 AR Path="/62C73C08" Ref="R?"  Part="1"
-AR Path="/62B871EE/62C73C08" Ref="R?"  Part="1"
-F 0 "R?" H 5050 3800 50  0000 C CNN
+AR Path="/62B871EE/62C73C08" Ref="R307"  Part="1"
+F 0 "R307" H 5050 3800 50  0000 C CNN
 F 1 "1R0" H 5100 3700 50  0000 C CNN
 F 2 "Resistor_SMD:R_0603_1608Metric" V 4880 3750 50  0001 C CNN
@@
 P 5250 3750
 AR Path="/62C74117" Ref="R?"  Part="1"
-AR Path="/62B871EE/62C74117" Ref="R?"  Part="1"
-F 0 "R?" H 5350 3800 50  0000 C CNN
+AR Path="/62B871EE/62C74117" Ref="R309"  Part="1"
+F 0 "R309" H 5350 3800 50  0000 C CNN
 F 1 "1R0" H 5400 3700 50  0000 C CNN
 F 2 "Resistor_SMD:R_0603_1608Metric" V 5180 3750 50  0001 C CNN
@@
 	2850 2950 5250 2950
 $Comp
-L Connector:TestPoint TP?
+L Connector:TestPoint TP301
 U 1 1 62C8B28F
 P 5500 4200
-F 0 "TP?" H 5300 4250 50  0000 L CNN
+F 0 "TP301" H 5300 4250 50  0000 L CNN
 F 1 "TestPoint" H 5100 4350 50  0000 L CNN
 F 2 "" H 5700 4200 50  0001 C CNN

Commit message: Clear several DRC warnings.
Connections:
- net at C301.1, C302.1, R301.2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: now also U301.16 (VDD)
Changed lines of the file:
@@
 AR Path="/62B90F17" Ref="U?"  Part="1"
 AR Path="/62B871EE/62B90F17" Ref="U302"  Part="1"
-F 0 "U302" H 6950 4200 50  0000 C CNN
-F 1 "LCD_20x4_Character" H 7300 4100 50  0000 C CNN
+F 0 "U302" H 6550 3950 50  0000 C CNN
+F 1 "LCD_20x4_Character" H 6850 3850 50  0000 C CNN
 F 2 "Display:NHD-0420H1Z" H 7300 2150 50  0001 C CNN
 F 3 "http://www.newhavendisplay.com/specs/NHD-0420H1Z-FSW-GBW-33V3.pdf" H 7400 2950 50  0001 C CNN
@@
 AR Path="/62B90F36" Ref="U?"  Part="1"
 AR Path="/62B871EE/62B90F36" Ref="U301"  Part="1"
-F 0 "U301" H 6150 4231 50  0000 C CNN
-F 1 "PCF8574AT" H 6150 4140 50  0000 C CNN
+F 0 "U301" H 5800 4300 50  0000 C CNN
+F 1 "PCF8574AT" H 5900 4150 50  0000 C CNN
 F 2 "Package_SO:SOIC-16W_5.3x10.2mm_P1.27mm" H 6150 3350 50  0001 C CNN
 F 3 "http://www.nxp.com/documents/data_sheet/PCF8574_PCF8574A.pdf" H 6150 3350 50  0001 C CNN
@@
 	5250 2350 5250 2050
 Wire Wire Line
-	5250 2050 7300 2050
+	5250 2050 6150 2050
 Connection ~ 7300 2050
 Wire Wire Line
@@
 Text HLabel 3050 3050 0    50   BiDi ~ 0
 SDA
+Wire Wire Line
+	6150 2650 6150 2050
+Connection ~ 6150 2050
+Wire Wire Line
+	6150 2050 7300 2050
 $EndSCHEMATC

Commit message: Clear several more DRC warnings.
Changed lines of the file:
@@
 	6700 2950 6650 2950
-Wire Wire Line
-	6900 3250 6900 3150
-Wire Wire Line
-	6900 3050 6900 3150
-Connection ~ 6900 3150
-Wire Wire Line
-	6900 3050 6900 2950
-Connection ~ 6900 3050
 Wire Wire Line
 	6900 3250 6850 3250
@@
 Wire Wire Line
 	6850 3850 7300 3850
-Connection ~ 6900 3250
 Connection ~ 7300 3850
 Text Notes 3650 1750 0    50   ~ 0
@@
 Connection ~ 6150 2050
 Wire Wire Line
-	6150 2050 7300 2050
+	6150 2050 6600 2050
+$Comp
+L power:PWR_FLAG #FLG0103
+U 1 1 62E5EA08
+P 6600 1950
+F 0 "#FLG0103" H 6600 2025 50  0001 C CNN
+F 1 "PWR_FLAG" H 6600 2123 50  0000 C CNN
+F 2 "" H 6600 1950 50  0001 C CNN
+F 3 "~" H 6600 1950 50  0001 C CNN
+	1    6600 1950
+	1    0    0    -1
+$EndComp
+Wire Wire Line
+	6600 1950 6600 2050
+Connection ~ 6600 2050
+Wire Wire Line
+	6600 2050 7300 2050
+Wire Wire Line
+	6850 3250 6850 3150
+Wire Wire Line
+	6850 2950 6900 2950
+Connection ~ 6850 3250
+Wire Wire Line
+	6900 3050 6850 3050
+Connection ~ 6850 3050
+Wire Wire Line
+	6850 3050 6850 2950
+Wire Wire Line
+	6900 3150 6850 3150
+Connection ~ 6850 3150
+Wire Wire Line
+	6850 3150 6850 3050
 $EndSCHEMATC

Commit message: Pull parts into PCB Begin rough placement into groups.
Parts:
- TP301: footprint (none) -> TestPoint:TestPoint_Loop_D2.54mm_Drill1.5mm_Beaded
- U302: footprint Display:NHD-0420H1Z -> Display:LM16255
Changed lines of the file:
@@
 F 0 "U302" H 6550 3950 50  0000 C CNN
 F 1 "LCD_20x4_Character" H 6850 3850 50  0000 C CNN
-F 2 "Display:NHD-0420H1Z" H 7300 2150 50  0001 C CNN
+F 2 "Display:LM16255" H 7300 2150 50  0001 C CNN
 F 3 "http://www.newhavendisplay.com/specs/NHD-0420H1Z-FSW-GBW-33V3.pdf" H 7400 2950 50  0001 C CNN
 F 4 "Aliexpress" H 6220 2360 50  0001 C CNN "Distributor 1"
@@
 	7400 2200 7800 2200
 Wire Wire Line
-	7800 2200 7800 2700
+	7800 2200 7800 2350
 Wire Wire Line
 	7800 2700 8100 2700
@@
 F 0 "TP301" H 5300 4250 50  0000 L CNN
 F 1 "TestPoint" H 5100 4350 50  0000 L CNN
-F 2 "" H 5700 4200 50  0001 C CNN
+F 2 "TestPoint:TestPoint_Loop_D2.54mm_Drill1.5mm_Beaded" H 5700 4200 50  0001 C CNN
 F 3 "~" H 5700 4200 50  0001 C CNN
 	1    5500 4200
@@
 Connection ~ 6850 3250
 Wire Wire Line
-	6900 3050 6850 3050
-Connection ~ 6850 3050
-Wire Wire Line
-	6850 3050 6850 2950
-Wire Wire Line
 	6900 3150 6850 3150
 Connection ~ 6850 3150
+$Comp
+L power:PWR_FLAG #FLG0106
+U 1 1 62E7D140
+P 7800 2350
+F 0 "#FLG0106" H 7800 2425 50  0001 C CNN
+F 1 "PWR_FLAG" V 7800 2478 50  0000 L CNN
+F 2 "" H 7800 2350 50  0001 C CNN
+F 3 "~" H 7800 2350 50  0001 C CNN
+	1    7800 2350
+	0    1    1    0
+$EndComp
+Connection ~ 7800 2350
+Wire Wire Line
+	7800 2350 7800 2700
 Wire Wire Line
 	6850 3150 6850 3050
+Wire Wire Line
+	6850 3050 6850 2950
+Connection ~ 6850 3050
+Wire Wire Line
+	6900 3050 6850 3050
 $EndSCHEMATC

Commit message: Update LCD footprint for 2004A pcb and add STEP file found at Grabcad. Refresh PCB.
Parts:
- U302: footprint Display:LM16255 -> GeneralPurposeAlarmDevicePCB:LCD_2004A
Changed lines of the file:
@@
 F 0 "U302" H 6550 3950 50  0000 C CNN
 F 1 "LCD_20x4_Character" H 6850 3850 50  0000 C CNN
-F 2 "Display:LM16255" H 7300 2150 50  0001 C CNN
+F 2 "GeneralPurposeAlarmDevicePCB:LCD_2004A" H 7300 2150 50  0001 C CNN
 F 3 "http://www.newhavendisplay.com/specs/NHD-0420H1Z-FSW-GBW-33V3.pdf" H 7400 2950 50  0001 C CNN
 F 4 "Aliexpress" H 6220 2360 50  0001 C CNN "Distributor 1"

Commit message: Add new LED, RJ12 footprints to footprint library. Add STEP model.
Connections:
- net GND: now also RV301.1; no longer RV301.3
- net Vcc_LCD: now reaches C301.1, C302.1, R301.2, R302.2, R303.2, R304.2, R306.2, R308.2, R310.1, R311.2, U301.16 (VDD), U302.15 (A), U302.2 (VDD)
- net Vcc_LCD: now also RV301.3; no longer RV301.1
Changed lines of the file:
@@
 F 8 "HAND" H 8180 2609 50  0000 R CNN "Assembly Type"
 	1    8250 2700
-	-1   0    0    -1
+	-1   0    0    1
 $EndComp
 Text Notes 3650 1350 0    50   ~ 0
@@
 	6150 2050 6600 2050
 $Comp
-L power:PWR_FLAG #FLG0103
+L power:PWR_FLAG #FLG0301
 U 1 1 62E5EA08
 P 6600 1950
-F 0 "#FLG0103" H 6600 2025 50  0001 C CNN
+F 0 "#FLG0301" H 6600 2025 50  0001 C CNN
 F 1 "PWR_FLAG" H 6600 2123 50  0000 C CNN
 F 2 "" H 6600 1950 50  0001 C CNN
@@
 Connection ~ 6850 3150
 $Comp
-L power:PWR_FLAG #FLG0106
+L power:PWR_FLAG #FLG0302
 U 1 1 62E7D140
 P 7800 2350
-F 0 "#FLG0106" H 7800 2425 50  0001 C CNN
+F 0 "#FLG0302" H 7800 2425 50  0001 C CNN
 F 1 "PWR_FLAG" V 7800 2478 50  0000 L CNN
 F 2 "" H 7800 2350 50  0001 C CNN
@@
 Wire Wire Line
 	6900 3050 6850 3050
+Text Label 9150 1600 0    50   ~ 0
+Vcc_LCD
 $EndSCHEMATC

Commit message: Add JST connector for I2C and more.
Parts:
- RV301: footprint digikey-footprints:Trimpot_3.8mmx3.6mm_TC33X-2-103E -> GeneralPurposeAlarmDevicePCB:Potentiometer_Bourns_3386P_Vertical
Changed lines of the file:
@@
 	1    0    0    -1
-$EndComp
-$Comp
-L GPAD_SCH_LIB:10K RV?
-U 1 1 62B9100B
-P 8250 2700
-AR Path="/62B9100B" Ref="RV?"  Part="1"
-AR Path="/62B871EE/62B9100B" Ref="RV301"  Part="1"
-F 0 "RV301" H 8180 2791 50  0000 R CNN
-F 1 "10K" H 8180 2700 50  0000 R CNN
-F 2 "digikey-footprints:Trimpot_3.8mmx3.6mm_TC33X-2-103E" H 8250 2700 50  0001 C CNN
-F 3 "https://www.bourns.com/docs/Product-Datasheets/TC33.pdf" H 8250 2700 50  0001 C CNN
-F 4 "JLCPCB" H 8250 2700 50  0001 C CNN "Distributor 1"
-F 5 "C58159" H 8250 2700 50  0001 C CNN "Distributor 1 PN"
-F 6 "BOURNS" H 8250 2700 50  0001 C CNN "Manufacturier"
-F 7 "3362P-1-103LF" H 8250 2700 50  0001 C CNN "MPN"
-F 8 "HAND" H 8180 2609 50  0000 R CNN "Assembly Type"
-	1    8250 2700
-	-1   0    0    1
 $EndComp
 Text Notes 3650 1350 0    50   ~ 0
@@
 Text Label 9150 1600 0    50   ~ 0
 Vcc_LCD
+$Comp
+L GPAD_SCH_LIB:10K RV301
+U 1 1 62D26FDE
+P 8250 2700
+F 0 "RV301" H 8180 2609 50  0000 R CNN
+F 1 "10K" H 8180 2700 50  0000 R CNN
+F 2 "GeneralPurposeAlarmDevicePCB:Potentiometer_Bourns_3386P_Vertical" H 8250 2700 50  0001 C CNN
+F 3 "https://www.bourns.com/docs/Product-Datasheets/TC33.pdf" H 8250 2700 50  0001 C CNN
+F 4 "JLCPCB" H 8250 2700 50  0001 C CNN "Distributor 1"
+F 5 "C58159" H 8250 2700 50  0001 C CNN "Distributor 1 PN"
+F 6 "BOURNS" H 8250 2700 50  0001 C CNN "Manufacturier"
+F 7 "3362P-1-103LF" H 8250 2700 50  0001 C CNN "MPN"
+F 8 "HAND" H 8180 2791 50  0000 R CNN "Assembly Type"
+	1    8250 2700
+	-1   0    0    1
+$EndComp
 $EndSCHEMATC
