File: Hardware/GeneralPurposeAlarmDevicePCB/GeneralPurposeAlarmDevicePCB/LCD And I2C Interface.sch (KiCad schematic (older format))
At the start: 18 parts, among them Q301 BSS138, U301 PCF8574AT, U302 LCD_20x4_Character

Commit message: Update schottky symbol and part number. Import to PCB. Only the Arduino UNO symbol remains to connect.
Parts:
- R306, R308: value 1K -> DNI; Description 0.1W ±1% 1kΩ 0603 Chip Resistor - Surface Mount ROHS -> DNI; Distributor 1 PN C269704 -> DNI; MPN RMC06031K1%N -> DNI
Connections:
- net GND: now also R308.1
- net SCL: no longer R308.1
- net SDA: no longer R306.1
- net Vcc_LCD: no longer R308.2
- net at RV301.2, U302.3 (VO): now also R306.1, R308.2
Changed lines of the file:
@@
-$Comp
-L Device:R R?
-U 1 1 62B90F83
-P 4950 2500
-AR Path="/62B90F83" Ref="R?"  Part="1"
-AR Path="/62B871EE/62B90F83" Ref="R306"  Part="1"
-F 0 "R306" H 4850 2450 50  0000 C CNN
-F 1 "1K" H 4800 2550 50  0000 C CNN
-F 2 "Resistor_SMD:R_0603_1608Metric" V 4880 2500 50  0001 C CNN
-F 3 "~" H 4950 2500 50  0001 C CNN
-F 4 "JLCPCB" V 4950 2500 50  0001 C CNN "Distributor 1"
-F 5 "C269704" V 4950 2500 50  0001 C CNN "Distributor 1 PN"
-F 6 "TyoHM" V 4950 2500 50  0001 C CNN "Manufacturer"
-F 7 "RMC06031K1%N" V 4950 2500 50  0001 C CNN "MPN"
-F 8 "0.1W ±1% 1kΩ 0603 Chip Resistor - Surface Mount ROHS" H 4950 2500 50  0001 C CNN "Description"
-	1    4950 2500
-	-1   0    0    1
-$EndComp
-$Comp
-L Device:R R?
-U 1 1 62B90F8E
-P 5250 2500
-AR Path="/62B90F8E" Ref="R?"  Part="1"
-AR Path="/62B871EE/62B90F8E" Ref="R308"  Part="1"
-F 0 "R308" H 5150 2450 50  0000 C CNN
-F 1 "1K" H 5100 2550 50  0000 C CNN
-F 2 "Resistor_SMD:R_0603_1608Metric" V 5180 2500 50  0001 C CNN
-F 3 "~" H 5250 2500 50  0001 C CNN
-F 4 "JLCPCB" V 5250 2500 50  0001 C CNN "Distributor 1"
-F 5 "C269704" V 5250 2500 50  0001 C CNN "Distributor 1 PN"
-F 6 "TyoHM" V 5250 2500 50  0001 C CNN "Manufacturer"
-F 7 "RMC06031K1%N" V 5250 2500 50  0001 C CNN "MPN"
-F 8 "0.1W ±1% 1kΩ 0603 Chip Resistor - Surface Mount ROHS" H 5250 2500 50  0001 C CNN "Description"
-	1    5250 2500
-	-1   0    0    1
-$EndComp
 $Comp
 L Device:R R?
@@
 	8500 1600 9150 1600
 Wire Wire Line
-	9150 1600 9150 3350
+	9150 1600 9150 2000
 Wire Wire Line
 	9150 3350 8000 3350
@@
 Wire Wire Line
 	6150 4150 6150 4050
-Wire Wire Line
-	5650 2950 5250 2950
-Wire Wire Line
-	5250 2950 5250 2650
-Wire Wire Line
-	5650 3050 4950 3050
-Wire Wire Line
-	4950 3050 4950 2650
 Wire Wire Line
 	5450 3750 5450 3150
@@
 Wire Wire Line
 	7700 1600 8000 1600
-Wire Wire Line
-	5250 2350 5250 2050
-Wire Wire Line
-	5250 2050 6150 2050
 Connection ~ 7300 2050
 Wire Wire Line
-	4950 2350 4950 2050
-Wire Wire Line
-	4950 2050 5250 2050
-Connection ~ 5250 2050
-Wire Wire Line
 	4600 2350 4600 2050
-Wire Wire Line
-	4600 2050 4950 2050
-Connection ~ 4950 2050
 Wire Wire Line
 	4250 2350 4250 2050
@@
 Wire Wire Line
 	5450 3750 5500 3750
-Wire Wire Line
-	4950 3050 3050 3050
-Connection ~ 4950 3050
-Connection ~ 5250 2950
-Wire Wire Line
-	2850 2950 5250 2950
 $Comp
 L Connector:TestPoint TP301
@@
 	6850 3850 7300 3850
 Connection ~ 7300 3850
-Text Notes 3650 1750 0    50   ~ 0
+Text Notes 3650 1600 0    50   ~ 0
 Wiring of I2C to LCD from:\nhttps://alselectro.wordpress.com/2016/05/12/serial-lcd-i2c-module-pcf8574/
 Text HLabel 2850 2950 0    50   Input ~ 0
@@
 Connection ~ 7800 2350
 Wire Wire Line
-	7800 2350 7800 2700
+	7800 2350 7800 2450
 Wire Wire Line
 	6850 3150 6850 3050
@@
 EndData
 $EndBitmap
+$Comp
+L Device:R R?
+U 1 1 62E746DD
+P 8900 2350
+AR Path="/62E746DD" Ref="R?"  Part="1"
+AR Path="/62B871EE/62E746DD" Ref="R306"  Part="1"
+F 0 "R306" H 8800 2300 50  0000 C CNN
+F 1 "DNI" H 8750 2400 50  0000 C CNN
+F 2 "Resistor_SMD:R_0603_1608Metric" V 8830 2350 50  0001 C CNN
+F 3 "~" H 8900 2350 50  0001 C CNN
+F 4 "JLCPCB" V 8900 2350 50  0001 C CNN "Distributor 1"
+F 5 "DNI" V 8900 2350 50  0001 C CNN "Distributor 1 PN"
+F 6 "TyoHM" V 8900 2350 50  0001 C CNN "Manufacturer"
+F 7 "DNI" V 8900 2350 50  0001 C CNN "MPN"
+F 8 "DNI" H 8900 2350 50  0001 C CNN "Description"
+	1    8900 2350
+	-1   0    0    1
+$EndComp
+$Comp
+L power:GND #PWR?
+U 1 1 62E7558E
+P 8900 3050
+AR Path="/62E7558E" Ref="#PWR?"  Part="1"
+AR Path="/62B871EE/62E7558E" Ref="#PWR0309"  Part="1"
+F 0 "#PWR0309" H 8900 2800 50  0001 C CNN
+F 1 "GND" H 8905 2877 50  0000 C CNN
+F 2 "" H 8900 3050 50  0001 C CNN
+F 3 "" H 8900 3050 50  0001 C CNN
+	1    8900 3050
+	1    0    0    -1
+$EndComp
+Wire Wire Line
+	8900 3050 8900 3000
+Wire Wire Line
+	8900 2700 8900 2550
+Wire Wire Line
+	8900 2200 8900 2000
+Wire Wire Line
+	8900 2000 9150 2000
+Connection ~ 9150 2000
+Wire Wire Line
+	9150 2000 9150 3350
+Wire Wire Line
+	7800 2450 8700 2450
+Wire Wire Line
+	8700 2450 8700 2550
+Wire Wire Line
+	8700 2550 8900 2550
+Connection ~ 7800 2450
+Wire Wire Line
+	7800 2450 7800 2700
+Connection ~ 8900 2550
+Wire Wire Line
+	8900 2550 8900 2500
+$Comp
+L Device:R R?
+U 1 1 62E82D99
+P 8900 2850
+AR Path="/62E82D99" Ref="R?"  Part="1"
+AR Path="/62B871EE/62E82D99" Ref="R308"  Part="1"
+F 0 "R308" H 8800 2800 50  0000 C CNN
+F 1 "DNI" H 8750 2900 50  0000 C CNN
+F 2 "Resistor_SMD:R_0603_1608Metric" V 8830 2850 50  0001 C CNN
+F 3 "~" H 8900 2850 50  0001 C CNN
+F 4 "JLCPCB" V 8900 2850 50  0001 C CNN "Distributor 1"
+F 5 "DNI" V 8900 2850 50  0001 C CNN "Distributor 1 PN"
+F 6 "TyoHM" V 8900 2850 50  0001 C CNN "Manufacturer"
+F 7 "DNI" V 8900 2850 50  0001 C CNN "MPN"
+F 8 "DNI" H 8900 2850 50  0001 C CNN "Description"
+	1    8900 2850
+	-1   0    0    1
+$EndComp
+Wire Wire Line
+	2850 2950 5650 2950
+Wire Wire Line
+	3050 3050 5650 3050
+Wire Wire Line
+	4600 2050 6150 2050
 $EndSCHEMATC

Commit message: Clean up a bunch of duplicate because of missspelled part field names. Still working on a few sch, pcb and 3D libraries.
Parts:
- C301: Manufacturer (none) -> YAGEO; Manufacturier YAGEO -> (none)
- Q301: Distirbutor 1 JLCPCB -> (none); Distributor 1 (none) -> JLCPCB; Manufacturer (none) -> Yangzhou Yangjie Electronic Technology Co., Ltd; Manufacturier Yangzhou Yangjie Electronic Technology Co., Ltd -> (none)
- RV301: Manufacturer (none) -> BOURNS; Manufacturier BOURNS -> (none)
- U301: Descirption Remote 8-bit I/O expander for I2C-bus with interrupt -> (none); Description (none) -> Remote 8-bit I/O expander for I2C-bus with interrupt; Manufacturer (none) -> NXP Semicon; Manufacturier NXP Semicon -> (none)
Changed lines of the file:
@@
 F 4 "JLCPCB" H 6150 3350 50  0001 C CNN "Distributor 1"
 F 5 "C83193" H 6150 3350 50  0001 C CNN "Distributor 1 PN"
-F 6 "NXP Semicon" H 6150 3350 50  0001 C CNN "Manufacturier"
-F 7 "Remote 8-bit I/O expander for I2C-bus with interrupt" H 6150 3350 50  0001 C CNN "Descirption"
+F 6 "NXP Semicon" H 6150 3350 50  0001 C CNN "Manufacturer"
+F 7 "Remote 8-bit I/O expander for I2C-bus with interrupt" H 6150 3350 50  0001 C CNN "Description"
 F 8 "PCF8574AT/3,512" H 6150 3350 50  0001 C CNN "MPN"
 	1    6150 3350
@@
 F 4 "JLCPCB" H 8000 1750 50  0001 C CNN "Distributor 1"
 F 5 "C14663" H 8000 1750 50  0001 C CNN "Distributor 1 PN"
-F 6 "YAGEO" H 8000 1750 50  0001 C CNN "Manufacturier"
+F 6 "YAGEO" H 8000 1750 50  0001 C CNN "Manufacturer"
 F 7 "CC0603KRX7R9BB104" H 8000 1750 50  0001 C CNN "MPN"
 F 8 "50V 100nF X7R ±10% 0603 Multilayer Ceramic Capacitors MLCC - SMD/SMT ROHS" H 8000 1750 50  0001 C CNN "Description"
@@
 F 3 "https://www.onsemi.com/pub/Collateral/BSS138-D.PDF" H 8600 4100 50  0001 L CNN
 F 4 "N-Channel Enhancement Mode Field Effect Transistor" H 8600 4100 50  0001 C CNN "Description"
-F 5 "JLCPCB" H 8600 4100 50  0001 C CNN "Distirbutor 1"
+F 5 "JLCPCB" H 8600 4100 50  0001 C CNN "Distributor 1"
 F 6 "C400505" H 8600 4100 50  0001 C CNN "Distributor 1 PN"
 F 7 "" H 8600 4100 50  0001 C CNN "Field7"
-F 8 "Yangzhou Yangjie Electronic Technology Co., Ltd" H 8600 4100 50  0001 C CNN "Manufacturier"
+F 8 "Yangzhou Yangjie Electronic Technology Co., Ltd" H 8600 4100 50  0001 C CNN "Manufacturer"
 F 9 "BSS138" H 8600 4100 50  0001 C CNN "MPN"
 	1    8600 4100
@@
 F 4 "JLCPCB" H 8250 2700 50  0001 C CNN "Distributor 1"
 F 5 "C58159" H 8250 2700 50  0001 C CNN "Distributor 1 PN"
-F 6 "BOURNS" H 8250 2700 50  0001 C CNN "Manufacturier"
+F 6 "BOURNS" H 8250 2700 50  0001 C CNN "Manufacturer"
 F 7 "3362P-1-103LF" H 8250 2700 50  0001 C CNN "MPN"
 F 8 "HAND" H 8180 2791 50  0000 R CNN "Assembly Type"

Commit message: Remove NANO sheild foot print. Other changes per issue #23 notes of 20220712.
Parts:
- TP_nINT301: renamed from TP301; value TestPoint -> TestPoint_nINT
Changed lines of the file:
@@
 AR Path="/62B90F41" Ref="R?"  Part="1"
 AR Path="/62B871EE/62B90F41" Ref="R303"  Part="1"
-F 0 "R303" H 4150 2450 50  0000 C CNN
+F 0 "R303" H 4150 2350 50  0000 C CNN
 F 1 "4K7" H 4100 2550 50  0000 C CNN
 F 2 "Resistor_SMD:R_0603_1608Metric" V 4180 2500 50  0001 C CNN
@@
 AR Path="/62B90F4C" Ref="R?"  Part="1"
 AR Path="/62B871EE/62B90F4C" Ref="R304"  Part="1"
-F 0 "R304" H 4500 2450 50  0000 C CNN
+F 0 "R304" H 4500 2350 50  0000 C CNN
 F 1 "1K" H 4450 2550 50  0000 C CNN
 F 2 "Resistor_SMD:R_0603_1608Metric" V 4530 2500 50  0001 C CNN
@@
 AR Path="/62B90F99" Ref="R?"  Part="1"
 AR Path="/62B871EE/62B90F99" Ref="R302"  Part="1"
-F 0 "R302" H 3750 2450 50  0000 C CNN
+F 0 "R302" H 3750 2350 50  0000 C CNN
 F 1 "4K7" H 3700 2550 50  0000 C CNN
 F 2 "Resistor_SMD:R_0603_1608Metric" V 3780 2500 50  0001 C CNN
@@
 AR Path="/62B90FA4" Ref="R?"  Part="1"
 AR Path="/62B871EE/62B90FA4" Ref="R301"  Part="1"
-F 0 "R301" H 3400 2450 50  0000 C CNN
+F 0 "R301" H 3400 2350 50  0000 C CNN
 F 1 "4K7" H 3350 2550 50  0000 C CNN
 F 2 "Resistor_SMD:R_0603_1608Metric" V 3430 2500 50  0001 C CNN
@@
 Wire Wire Line
 	7600 1600 7700 1600
-Wire Wire Line
-	8500 1600 8250 1600
 Connection ~ 8000 1600
 Wire Wire Line
@@
 	8000 1950 8000 1900
 Wire Wire Line
-	8250 2550 8250 1600
-Connection ~ 8250 1600
-Wire Wire Line
-	8250 1600 8000 1600
+	8250 2550 8250 2250
 Wire Wire Line
 	8250 2850 8250 2950
@@
 AR Path="/62C6D2FC" Ref="R?"  Part="1"
 AR Path="/62B871EE/62C6D2FC" Ref="R305"  Part="1"
-F 0 "R305" H 4700 3800 50  0000 C CNN
+F 0 "R305" H 4700 3900 50  0000 C CNN
 F 1 "1R0" H 4750 3700 50  0000 C CNN
 F 2 "Resistor_SMD:R_0603_1608Metric" V 4530 3750 50  0001 C CNN
@@
 AR Path="/62C73C08" Ref="R?"  Part="1"
 AR Path="/62B871EE/62C73C08" Ref="R307"  Part="1"
-F 0 "R307" H 5050 3800 50  0000 C CNN
+F 0 "R307" H 5050 3900 50  0000 C CNN
 F 1 "1R0" H 5100 3700 50  0000 C CNN
 F 2 "Resistor_SMD:R_0603_1608Metric" V 4880 3750 50  0001 C CNN
@@
 AR Path="/62C74117" Ref="R?"  Part="1"
 AR Path="/62B871EE/62C74117" Ref="R309"  Part="1"
-F 0 "R309" H 5350 3800 50  0000 C CNN
+F 0 "R309" H 5350 3900 50  0000 C CNN
 F 1 "1R0" H 5400 3700 50  0000 C CNN
 F 2 "Resistor_SMD:R_0603_1608Metric" V 5180 3750 50  0001 C CNN
@@
 	5450 3750 5500 3750
 $Comp
-L Connector:TestPoint TP301
+L Connector:TestPoint TP_nINT301
 U 1 1 62C8B28F
 P 5500 4200
-F 0 "TP301" H 5300 4250 50  0000 L CNN
-F 1 "TestPoint" H 5100 4350 50  0000 L CNN
+F 0 "TP_nINT301" H 5200 4250 50  0000 L CNN
+F 1 "TestPoint_nINT" H 5100 4450 50  0000 L CNN
 F 2 "TestPoint:TestPoint_Loop_D2.54mm_Drill1.5mm_Beaded" H 5700 4200 50  0001 C CNN
 F 3 "~" H 5700 4200 50  0001 C CNN
@@
 AR Path="/62E746DD" Ref="R?"  Part="1"
 AR Path="/62B871EE/62E746DD" Ref="R306"  Part="1"
-F 0 "R306" H 8800 2300 50  0000 C CNN
+F 0 "R306" H 8800 2200 50  0000 C CNN
 F 1 "DNI" H 8750 2400 50  0000 C CNN
 F 2 "Resistor_SMD:R_0603_1608Metric" V 8830 2350 50  0001 C CNN
@@
 AR Path="/62E82D99" Ref="R?"  Part="1"
 AR Path="/62B871EE/62E82D99" Ref="R308"  Part="1"
-F 0 "R308" H 8800 2800 50  0000 C CNN
+F 0 "R308" H 8800 2700 50  0000 C CNN
 F 1 "DNI" H 8750 2900 50  0000 C CNN
 F 2 "Resistor_SMD:R_0603_1608Metric" V 8830 2850 50  0001 C CNN
@@
 Wire Wire Line
 	4600 2050 6150 2050
+Wire Wire Line
+	7700 2050 7900 2050
+Wire Wire Line
+	7900 2050 7900 2250
+Wire Wire Line
+	7900 2250 8250 2250
+Connection ~ 7700 2050
+Wire Wire Line
+	8000 1600 8500 1600
 $EndSCHEMATC
