File: Hardware/GeneralPurposeAlarmDevicePCB/GeneralPurposeAlarmDevicePCB/USB_UART.sch (KiCad schematic (older format))
At the start: 10 parts

Commit message: Add more parts drawings, buzzer. Add additional schematic sheet for AlarmAudio.
Connections:
- net GND: now also R?.1
- net at U?.4 (~RTS): no longer R?.1
- net at U?.5 (~CTS): now also R?.2
- net VBUS: now reaches C?.1, C?.1, J?.1 (VBUS), U?.7 (VCC)
- net VBUS: no longer R?.2
Changed lines of the file:
@@
 $Descr USLetter 11000 8500
 encoding utf-8
-Sheet 5 5
+Sheet 5 6
 Title "GeneralPurposeAlarmDevicePCB"
 Date "2022-06-20"
@@
 	0    1    1    0
 $EndComp
-Text Notes 7150 3150 0    50   ~ 0
+Text Notes 6500 3200 0    50   ~ 0
 NULL MODEM
 $Comp
@@
 	1    0    0    -1
 $EndComp
-Text GLabel 7150 3800 2    50   Input ~ 0
-ControllerTX
-Text GLabel 7100 3450 2    50   Input ~ 0
-ControllerRX
-Text Notes 6500 4750 0    50   ~ 0
+Text Notes 7300 4250 0    50   ~ 0
 TX is Output\nRX is Input\n/CTS is Input\n/RTS is Output
 $Comp
@@
 AR Path="/62BE31FB" Ref="D?"  Part="1"
 AR Path="/62BC4E7E/62BE31FB" Ref="D?"  Part="1"
-F 0 "D?" H 4700 4587 60  0000 C CNN
-F 1 "RED 0603" H 4700 4481 60  0000 C CNN
+F 0 "D?" H 4750 4100 60  0000 C CNN
+F 1 "RED 0603" H 4600 4450 60  0000 C CNN
 F 2 "LED_SMD:LED_0603_1608Metric" H 4950 4450 60  0001 L CNN
 F 3 "" H 4950 4550 60  0001 L CNN
@@
 $EndComp
 Wire Wire Line
-	6950 3450 7100 3450
-Wire Wire Line
 	6500 3450 6650 3450
 Wire Wire Line
@@
 	6650 3550 6650 3800
 Wire Wire Line
-	6950 3800 7150 3800
-Wire Wire Line
-	6500 4250 6700 4250
-Wire Wire Line
-	6700 4250 6700 4350
-Wire Wire Line
-	6700 4350 6900 4350
-Wire Wire Line
-	6100 4750 6100 4450
+	6100 4750 6100 4600
 Wire Wire Line
 	6000 3250 6000 3100
@@
 Connection ~ 4750 3000
 Wire Wire Line
-	6100 3000 7000 3000
-Wire Wire Line
-	7000 3000 7000 4000
-Wire Wire Line
-	7000 4000 6900 4000
-Wire Wire Line
-	6900 4000 6900 4050
-Connection ~ 6100 3000
-Wire Wire Line
 	5700 3950 5550 3950
 Wire Wire Line
@@
 	3650 4150 3650 4250
 Connection ~ 3650 4250
+Text HLabel 8400 3450 2    50   Output ~ 0
+ControllerRX
+Text HLabel 8350 3800 2    50   Input ~ 0
+ControllerTX
+Wire Wire Line
+	6950 3800 8350 3800
+Wire Wire Line
+	6950 3450 8400 3450
+Wire Wire Line
+	6500 3750 6550 3750
+Wire Wire Line
+	6900 4050 6550 4050
+Wire Wire Line
+	6550 4050 6550 3750
+Wire Wire Line
+	6100 4600 6900 4600
+Wire Wire Line
+	6900 4600 6900 4350
+Connection ~ 6100 4600
+Wire Wire Line
+	6100 4600 6100 4450
+Text HLabel 8350 3000 2    50   UnSpc ~ 0
+VBUS
+Wire Wire Line
+	6100 3000 8350 3000
+Connection ~ 6100 3000
 $EndSCHEMATC

Commit message: Annote reference designators.
Parts:
- gave numbers to parts that had none: 10
Changed lines of the file:
@@
 P 6100 3850
 AR Path="/62BE3184" Ref="U?"  Part="1"
-AR Path="/62BC4E7E/62BE3184" Ref="U?"  Part="1"
-F 0 "U?" H 6100 3161 50  0000 C CNN
+AR Path="/62BC4E7E/62BE3184" Ref="U501"  Part="1"
+F 0 "U501" H 6100 3161 50  0000 C CNN
 F 1 "CH340E" H 6100 3070 50  0000 C CNN
 F 2 "Package_SO:MSOP-10_3x3mm_P0.5mm" H 6150 3300 50  0001 L CNN
@@
 P 3650 3750
 AR Path="/62BE318A" Ref="J?"  Part="1"
-AR Path="/62BC4E7E/62BE318A" Ref="J?"  Part="1"
-F 0 "J?" H 3707 4217 50  0000 C CNN
+AR Path="/62BC4E7E/62BE318A" Ref="J501"  Part="1"
+F 0 "J501" H 3707 4217 50  0000 C CNN
 F 1 "USB_B_Micro" H 3707 4126 50  0000 C CNN
 F 2 "" H 3800 3700 50  0001 C CNN
@@
 P 6800 3450
 AR Path="/62BE3195" Ref="R?"  Part="1"
-AR Path="/62BC4E7E/62BE3195" Ref="R?"  Part="1"
-F 0 "R?" V 6600 3400 50  0000 C CNN
+AR Path="/62BC4E7E/62BE3195" Ref="R502"  Part="1"
+F 0 "R502" V 6600 3400 50  0000 C CNN
 F 1 "330R" V 6700 3450 50  0000 C CNN
 F 2 "Resistor_SMD:R_0603_1608Metric" V 6730 3450 50  0001 C CNN
@@
 P 6800 3800
 AR Path="/62BE31A0" Ref="R?"  Part="1"
-AR Path="/62BC4E7E/62BE31A0" Ref="R?"  Part="1"
-F 0 "R?" V 6600 3750 50  0000 C CNN
+AR Path="/62BC4E7E/62BE31A0" Ref="R503"  Part="1"
+F 0 "R503" V 6600 3750 50  0000 C CNN
 F 1 "330R" V 6700 3800 50  0000 C CNN
 F 2 "Resistor_SMD:R_0603_1608Metric" V 6730 3800 50  0001 C CNN
@@
 P 6100 4750
 AR Path="/62BE31A7" Ref="#PWR?"  Part="1"
-AR Path="/62BC4E7E/62BE31A7" Ref="#PWR?"  Part="1"
-F 0 "#PWR?" H 6100 4500 50  0001 C CNN
+AR Path="/62BC4E7E/62BE31A7" Ref="#PWR0506"  Part="1"
+F 0 "#PWR0506" H 6100 4500 50  0001 C CNN
 F 1 "GND" H 6105 4577 50  0000 C CNN
 F 2 "" H 6100 4750 50  0001 C CNN
@@
 P 5400 3250
 AR Path="/62BE31B2" Ref="C?"  Part="1"
-AR Path="/62BC4E7E/62BE31B2" Ref="C?"  Part="1"
-F 0 "C?" H 5515 3296 50  0000 L CNN
+AR Path="/62BC4E7E/62BE31B2" Ref="C503"  Part="1"
+F 0 "C503" H 5515 3296 50  0000 L CNN
 F 1 "100nF" H 5515 3205 50  0000 L CNN
 F 2 "Capacitor_SMD:C_0603_1608Metric_Pad1.08x0.95mm_HandSolder" H 5438 3100 50  0001 C CNN
@@
 P 5400 3450
 AR Path="/62BE31B8" Ref="#PWR?"  Part="1"
-AR Path="/62BC4E7E/62BE31B8" Ref="#PWR?"  Part="1"
-F 0 "#PWR?" H 5400 3200 50  0001 C CNN
+AR Path="/62BC4E7E/62BE31B8" Ref="#PWR0505"  Part="1"
+F 0 "#PWR0505" H 5400 3200 50  0001 C CNN
 F 1 "GND" H 5405 3277 50  0000 C CNN
 F 2 "" H 5400 3450 50  0001 C CNN
@@
 P 4750 3250
 AR Path="/62BE31C2" Ref="C?"  Part="1"
-AR Path="/62BC4E7E/62BE31C2" Ref="C?"  Part="1"
-F 0 "C?" H 4868 3296 50  0000 L CNN
+AR Path="/62BC4E7E/62BE31C2" Ref="C502"  Part="1"
+F 0 "C502" H 4868 3296 50  0000 L CNN
 F 1 "47uF 16V" H 4868 3205 50  0000 L CNN
 F 2 "Capacitor_SMD:CP_Elec_5x5.4" H 4788 3100 50  0001 C CNN
@@
 P 4200 3250
 AR Path="/62BE31CD" Ref="C?"  Part="1"
-AR Path="/62BC4E7E/62BE31CD" Ref="C?"  Part="1"
-F 0 "C?" H 4315 3296 50  0000 L CNN
+AR Path="/62BC4E7E/62BE31CD" Ref="C501"  Part="1"
+F 0 "C501" H 4315 3296 50  0000 L CNN
 F 1 "100nF" H 4315 3205 50  0000 L CNN
 F 2 "Capacitor_SMD:C_0603_1608Metric_Pad1.08x0.95mm_HandSolder" H 4238 3100 50  0001 C CNN
@@
 P 4200 3450
 AR Path="/62BE31D3" Ref="#PWR?"  Part="1"
-AR Path="/62BC4E7E/62BE31D3" Ref="#PWR?"  Part="1"
-F 0 "#PWR?" H 4200 3200 50  0001 C CNN
+AR Path="/62BC4E7E/62BE31D3" Ref="#PWR0502"  Part="1"
+F 0 "#PWR0502" H 4200 3200 50  0001 C CNN
 F 1 "GND" H 4205 3277 50  0000 C CNN
 F 2 "" H 4200 3450 50  0001 C CNN
@@
 P 4750 3450
 AR Path="/62BE31D9" Ref="#PWR?"  Part="1"
-AR Path="/62BC4E7E/62BE31D9" Ref="#PWR?"  Part="1"
-F 0 "#PWR?" H 4750 3200 50  0001 C CNN
+AR Path="/62BC4E7E/62BE31D9" Ref="#PWR0504"  Part="1"
+F 0 "#PWR0504" H 4750 3200 50  0001 C CNN
 F 1 "GND" H 4755 3277 50  0000 C CNN
 F 2 "" H 4750 3450 50  0001 C CNN
@@
 P 3650 4300
 AR Path="/62BE31DF" Ref="#PWR?"  Part="1"
-AR Path="/62BC4E7E/62BE31DF" Ref="#PWR?"  Part="1"
-F 0 "#PWR?" H 3650 4050 50  0001 C CNN
+AR Path="/62BC4E7E/62BE31DF" Ref="#PWR0501"  Part="1"
+F 0 "#PWR0501" H 3650 4050 50  0001 C CNN
 F 1 "GND" H 3655 4127 50  0000 C CNN
 F 2 "" H 3650 4300 50  0001 C CNN
@@
 P 5250 4250
 AR Path="/62BE31ED" Ref="R?"  Part="1"
-AR Path="/62BC4E7E/62BE31ED" Ref="R?"  Part="1"
-F 0 "R?" V 5050 4200 50  0000 C CNN
+AR Path="/62BC4E7E/62BE31ED" Ref="R501"  Part="1"
+F 0 "R501" V 5050 4200 50  0000 C CNN
 F 1 "330R" V 5150 4250 50  0000 C CNN
 F 2 "Resistor_SMD:R_0603_1608Metric" V 5180 4250 50  0001 C CNN
@@
 P 4750 4250
 AR Path="/62BE31FB" Ref="D?"  Part="1"
-AR Path="/62BC4E7E/62BE31FB" Ref="D?"  Part="1"
-F 0 "D?" H 4750 4100 60  0000 C CNN
+AR Path="/62BC4E7E/62BE31FB" Ref="D501"  Part="1"
+F 0 "D501" H 4750 4100 60  0000 C CNN
 F 1 "RED 0603" H 4600 4450 60  0000 C CNN
 F 2 "LED_SMD:LED_0603_1608Metric" H 4950 4450 60  0001 L CNN
@@
 P 4500 4300
 AR Path="/62BE3201" Ref="#PWR?"  Part="1"
-AR Path="/62BC4E7E/62BE3201" Ref="#PWR?"  Part="1"
-F 0 "#PWR?" H 4500 4050 50  0001 C CNN
+AR Path="/62BC4E7E/62BE3201" Ref="#PWR0503"  Part="1"
+F 0 "#PWR0503" H 4500 4050 50  0001 C CNN
 F 1 "GND" H 4505 4127 50  0000 C CNN
 F 2 "" H 4500 4300 50  0001 C CNN
@@
 AR Path="/62BE320C" Ref="R?"  Part="1"
 AR Path="/62B871EE/62BE320C" Ref="R?"  Part="1"
-AR Path="/62BC4E7E/62BE320C" Ref="R?"  Part="1"
-F 0 "R?" H 6800 4150 50  0000 C CNN
+AR Path="/62BC4E7E/62BE320C" Ref="R504"  Part="1"
+F 0 "R504" H 6800 4150 50  0000 C CNN
 F 1 "4K7" H 6750 4250 50  0000 C CNN
 F 2 "Resistor_SMD:R_0603_1608Metric" V 6830 4200 50  0001 C CNN

Commit message: Clear several DRC warnings.
Connections:
- no-connect marks 0 -> 2
Changed lines of the file:
@@
 AR Path="/62BE3184" Ref="U?"  Part="1"
 AR Path="/62BC4E7E/62BE3184" Ref="U501"  Part="1"
-F 0 "U501" H 6100 3161 50  0000 C CNN
-F 1 "CH340E" H 6100 3070 50  0000 C CNN
+F 0 "U501" H 5700 3250 50  0000 C CNN
+F 1 "CH340E" H 5750 3150 50  0000 C CNN
 F 2 "Package_SO:MSOP-10_3x3mm_P0.5mm" H 6150 3300 50  0001 L CNN
 F 3 "https://www.mpja.com/download/35227cpdata.pdf" H 5750 4650 50  0001 C CNN
@@
 	6100 3000 8350 3000
 Connection ~ 6100 3000
+NoConn ~ 6500 4250
+NoConn ~ 3950 3950
 $EndSCHEMATC

Commit message: Clear several more DRC warnings.
Changed lines of the file:
@@
 AR Path="/62B871EE/62BE320C" Ref="R?"  Part="1"
 AR Path="/62BC4E7E/62BE320C" Ref="R504"  Part="1"
-F 0 "R504" H 6800 4150 50  0000 C CNN
+F 0 "R504" H 6750 4150 50  0000 C CNN
 F 1 "4K7" H 6750 4250 50  0000 C CNN
 F 2 "Resistor_SMD:R_0603_1608Metric" V 6830 4200 50  0001 C CNN

Commit message: Pull parts into PCB Begin rough placement into groups.
Parts:
- J501: footprint (none) -> Connector_USB:USB_Micro-B_Amphenol_10118194_Horizontal; Distributor 1 (none) -> JLCPCB; Distributor 1 PN (none) -> C132563; MPN (none) -> 10118194-0001LF; Manufacturer (none) -> Amphenol ICC
Changed lines of the file:
@@
 F 0 "J501" H 3707 4217 50  0000 C CNN
 F 1 "USB_B_Micro" H 3707 4126 50  0000 C CNN
-F 2 "" H 3800 3700 50  0001 C CNN
+F 2 "Connector_USB:USB_Micro-B_Amphenol_10118194_Horizontal" H 3800 3700 50  0001 C CNN
 F 3 "~" H 3800 3700 50  0001 C CNN
+F 4 "JLCPCB" H 3650 3750 50  0001 C CNN "Distributor 1"
+F 5 "C132563" H 3650 3750 50  0001 C CNN "Distributor 1 PN"
+F 6 "Amphenol ICC" H 3650 3750 50  0001 C CNN "Manufacturer"
+F 7 "10118194-0001LF" H 3650 3750 50  0001 C CNN "MPN"
 	1    3650 3750
 	1    0    0    -1
@@
 F 3 "" H 4750 3450 50  0001 C CNN
 	1    4750 3450
-	1    0    0    -1
-$EndComp
-$Comp
-L power:GND #PWR?
-U 1 1 62BE31DF
-P 3650 4300
-AR Path="/62BE31DF" Ref="#PWR?"  Part="1"
-AR Path="/62BC4E7E/62BE31DF" Ref="#PWR0501"  Part="1"
-F 0 "#PWR0501" H 3650 4050 50  0001 C CNN
-F 1 "GND" H 3655 4127 50  0000 C CNN
-F 2 "" H 3650 4300 50  0001 C CNN
-F 3 "" H 3650 4300 50  0001 C CNN
-	1    3650 4300
 	1    0    0    -1
 $EndComp
@@
 	4050 3000 4200 3000
 Connection ~ 4200 3000
-Wire Wire Line
-	3550 4150 3550 4250
-Wire Wire Line
-	3550 4250 3650 4250
-Wire Wire Line
-	3650 4250 3650 4300
-Wire Wire Line
-	3650 4150 3650 4250
-Connection ~ 3650 4250
 Text HLabel 8400 3450 2    50   Output ~ 0
 ControllerRX
@@
 NoConn ~ 6500 4250
 NoConn ~ 3950 3950
+$Comp
+L power:GND #PWR?
+U 1 1 62E80326
+P 3550 4450
+AR Path="/62E80326" Ref="#PWR?"  Part="1"
+AR Path="/62BC4E7E/62E80326" Ref="#PWR0118"  Part="1"
+F 0 "#PWR0118" H 3550 4200 50  0001 C CNN
+F 1 "GND" H 3555 4277 50  0000 C CNN
+F 2 "" H 3550 4450 50  0001 C CNN
+F 3 "" H 3550 4450 50  0001 C CNN
+	1    3550 4450
+	1    0    0    -1
+$EndComp
+Wire Wire Line
+	3550 4450 3550 4150
+$Comp
+L power:GND #PWR?
+U 1 1 62E80FD9
+P 3700 4450
+AR Path="/62E80FD9" Ref="#PWR?"  Part="1"
+AR Path="/62BC4E7E/62E80FD9" Ref="#PWR0119"  Part="1"
+F 0 "#PWR0119" H 3700 4200 50  0001 C CNN
+F 1 "GND" H 3705 4277 50  0000 C CNN
+F 2 "" H 3700 4450 50  0001 C CNN
+F 3 "" H 3700 4450 50  0001 C CNN
+	1    3700 4450
+	1    0    0    -1
+$EndComp
+Wire Wire Line
+	3650 4150 3650 4300
+Wire Wire Line
+	3650 4300 3700 4300
+Wire Wire Line
+	3700 4300 3700 4450
 $EndSCHEMATC

Commit message: Add more parts including a place holder only for power jack 3D, USB micro is incomplete. Added I2C daisy chain connector.
Parts:
- removed J501: USB_B_Micro, Connector_USB:USB_Micro-B_Amphenol_10118194_Horizontal, symbol Connector:USB_B_Micro
- added J501: USB_B_Micro, Connector_USB:USB_Micro-B_Wuerth_629105150521, symbol GPAD_SCH_LIB:USB_B_Micro
Connections:
- net GND: now also J501.5 (GND), J501.6 (Shield)
- net VBUS: now also J501.1 (VBUS)
- net at U501.1 (UD+): now also J501.3 (D+)
- net at U501.2 (UD-): now also J501.2 (D-)
Changed lines of the file:
@@
-$EndComp
-$Comp
-L Connector:USB_B_Micro J?
-U 1 1 62BE318A
-P 3650 3750
-AR Path="/62BE318A" Ref="J?"  Part="1"
-AR Path="/62BC4E7E/62BE318A" Ref="J501"  Part="1"
-F 0 "J501" H 3707 4217 50  0000 C CNN
-F 1 "USB_B_Micro" H 3707 4126 50  0000 C CNN
-F 2 "Connector_USB:USB_Micro-B_Amphenol_10118194_Horizontal" H 3800 3700 50  0001 C CNN
-F 3 "~" H 3800 3700 50  0001 C CNN
-F 4 "JLCPCB" H 3650 3750 50  0001 C CNN "Distributor 1"
-F 5 "C132563" H 3650 3750 50  0001 C CNN "Distributor 1 PN"
-F 6 "Amphenol ICC" H 3650 3750 50  0001 C CNN "Manufacturer"
-F 7 "10118194-0001LF" H 3650 3750 50  0001 C CNN "MPN"
-	1    3650 3750
-	1    0    0    -1
 $EndComp
 $Comp
@@
 Wire Wire Line
 	3700 4300 3700 4450
+$Comp
+L GPAD_SCH_LIB:USB_B_Micro J501
+U 1 1 62E66B23
+P 3650 3750
+F 0 "J501" H 3707 4217 50  0000 C CNN
+F 1 "USB_B_Micro" H 3707 4126 50  0000 C CNN
+F 2 "Connector_USB:USB_Micro-B_Wuerth_629105150521" H 3800 3700 50  0001 C CNN
+F 3 "" H 3800 3700 50  0001 C CNN
+F 4 "JLCPCB" H 3650 3750 50  0001 C CNN "Distributor 1"
+F 5 "???   C132563" H 3650 3750 50  0001 C CNN "Distributor 1 PN"
+F 6 "Wuerth_629105150521  ???  Amphenol ICC" H 3650 3750 50  0001 C CNN "Manufacturer "
+F 7 "Wuerth_629105150521  ??? 10118194-0001LF" H 3650 3750 50  0001 C CNN "MPN "
+	1    3650 3750
+	1    0    0    -1
+$EndComp
 $EndSCHEMATC
