File: Hardware/GeneralPurposeAlarmDevicePCB/GeneralPurposeAlarmDevicePCB/USB_UART.sch (KiCad schematic (older format))
At the start: 10 parts, among them J501 USB_B_Micro, U501 CH340E

Commit message: Clean up a bunch of duplicate because of missspelled part field names. Still working on a few sch, pcb and 3D libraries.
Parts:
- C501, C503: Manufacturer (none) -> YAGEO; Manufacturier YAGEO -> (none)
- J501: MPN (none) -> Wuerth_629105150521 ??? 10118194-0001LF; MPN  Wuerth_629105150521 ??? 10118194-0001LF -> (none); Manufacturer (none) -> Wuerth_629105150521 ??? Amphenol ICC; Manufacturer  Wuerth_629105150521 ??? Amphenol ICC -> (none)
Changed lines of the file:
@@
 F 4 "JLCPCB" H 5400 3250 50  0001 C CNN "Distributor 1"
 F 5 "C14663" H 5400 3250 50  0001 C CNN "Distributor 1 PN"
-F 6 "YAGEO" H 5400 3250 50  0001 C CNN "Manufacturier"
+F 6 "YAGEO" H 5400 3250 50  0001 C CNN "Manufacturer"
 F 7 "CC0603KRX7R9BB104" H 5400 3250 50  0001 C CNN "MPN"
 F 8 "50V 100nF X7R ±10% 0603 Multilayer Ceramic Capacitors MLCC - SMD/SMT ROHS" H 5400 3250 50  0001 C CNN "Description"
@@
 F 4 "JLCPCB" H 4200 3250 50  0001 C CNN "Distributor 1"
 F 5 "C14663" H 4200 3250 50  0001 C CNN "Distributor 1 PN"
-F 6 "YAGEO" H 4200 3250 50  0001 C CNN "Manufacturier"
+F 6 "YAGEO" H 4200 3250 50  0001 C CNN "Manufacturer"
 F 7 "CC0603KRX7R9BB104" H 4200 3250 50  0001 C CNN "MPN"
 F 8 "50V 100nF X7R ±10% 0603 Multilayer Ceramic Capacitors MLCC - SMD/SMT ROHS" H 4200 3250 50  0001 C CNN "Description"
@@
 F 4 "JLCPCB" H 3650 3750 50  0001 C CNN "Distributor 1"
 F 5 "???   C132563" H 3650 3750 50  0001 C CNN "Distributor 1 PN"
-F 6 "Wuerth_629105150521  ???  Amphenol ICC" H 3650 3750 50  0001 C CNN "Manufacturer "
-F 7 "Wuerth_629105150521  ??? 10118194-0001LF" H 3650 3750 50  0001 C CNN "MPN "
+F 6 "Wuerth_629105150521  ???  Amphenol ICC" H 3650 3750 50  0001 C CNN "Manufacturer"
+F 7 "Wuerth_629105150521  ??? 10118194-0001LF" H 3650 3750 50  0001 C CNN "MPN"
 	1    3650 3750
 	1    0    0    -1
