File: Hardware/GeneralPurposeAlarmDevicePCB/GeneralPurposeAlarmDevicePCB/GeneralPurposeAlarmDevicePCB.kicad_pcb (KiCad board)
At the start: 2 copper layers, 137.2 x 152.4 mm, 83 parts, among them J101 Barrel_Jack_Switch_SMT, J102 22-23-2021, J103 22-23-2021, J401 RJ12, J501 USB_B_Micro, Q201 MMBT2222A-7-F, Q202 MMBT2222A-7-F, Q203 MMBT2222A-7-F, Q204 MMBT2222A-7-F, Q205 MMBT2222A-7-F, Q301 BSS138, Q601 MMBT2222A-7-F, Q602 MMBT2907ALT1G, U101 NCP1117ST50T3G, U102 PI_ATMEGA328P-AU-InOrder, U301 PCF8574AT, U302 LCD_20x4_Character, U501 CH340E

Commit message: Update LCD footprint for 2004A pcb and add STEP file found at Grabcad. Refresh PCB.
Parts:
- U302: footprint Display:LM16255 -> GeneralPurposeAlarmDevicePCB:LCD_2004A
- moved U302 34.1 mm to (123.2, 55.9)

Commit message: Add new LED, RJ12 footprints to footprint library. Add STEP model.
Parts:
- removed the C108 at (111.8, 152.4)
- removed R104: 1R0, Resistor_SMD:R_0603_1608Metric
- added C107: 39pF, Capacitor_SMD:C_0603_1608Metric_Pad1.08x0.95mm_HandSolder, F.Cu at (124.5, 61.0)
- added C112: 47uF 16V, Capacitor_SMD:CP_Elec_5x5.4, F.Cu at (119.4, 41.3)
- added H101: MountingHole_Pad_3.5mm, GeneralPurposeAlarmDevicePCB:MountingHole_3.5mm_Pad_Via, F.Cu at (61.0, 22.9)
- added H102: MountingHole_Pad_3.5mm, GeneralPurposeAlarmDevicePCB:MountingHole_3.5mm_Pad_Via, F.Cu at (188.0, 22.9)
- added H103: MountingHole_Pad_3.5mm, GeneralPurposeAlarmDevicePCB:MountingHole_3.5mm_Pad_Via, F.Cu at (61.0, 96.5)
- added H104: MountingHole_Pad_3.5mm, GeneralPurposeAlarmDevicePCB:MountingHole_3.5mm_Pad_Via, F.Cu at (188.0, 96.5)
- added R603: 10K, Resistor_SMD:R_0603_1608Metric, F.Cu at (86.4, 92.7)
- added S601: SWITCH_TACTILE_SPST-NO_0.05A_24V, GeneralPurposeAlarmDevicePCB:Switch_Tactile_THT_6x6mm, B.Cu at (81.3, 91.4)
- C105, C111: value 47uF 16V -> 100nF; footprint Capacitor_SMD:CP_Elec_5x5.4 -> Capacitor_SMD:C_0603_1608Metric_Pad1.08x0.95mm_HandSolder
- C106: value 39pF -> 47uF 16V; footprint Capacitor_SMD:C_0603_1608Metric_Pad1.08x0.95mm_HandSolder -> Capacitor_SMD:CP_Elec_5x5.4
- C109: value 100nF -> 47uF 16V; footprint Capacitor_SMD:C_0603_1608Metric_Pad1.08x0.95mm_HandSolder -> Capacitor_SMD:CP_Elec_5x5.4
- D102: footprint LED_SMD:LED_0603_1608Metric -> digikey-footprints:0805
- D201, D202, D203, D204, D205: value RED 0603 -> LED_T1.75_CLEAR_WHITE; footprint LED_SMD:LED_0603_1608Metric -> GeneralPurposeAlarmDevicePCB:LED_5mm_Radial; moved to B.Cu
- J101: footprint Connector_BarrelJack:BarrelJack_CLIFF_FC681465S_SMT_Horizontal -> GeneralPurposeAlarmDevicePCB:BarrelJack_CLIFF_FC681465S_SMT_Horizontal
- J401: value RJ12 -> RJ12_6P6C_HORZ; footprint Connector_RJ:RJ12_Amphenol_54601 -> GeneralPurposeAlarmDevicePCB:RJ12_Amphenol_54601
- R401, R402, R403, R404: value 330R -> R
- S101: footprint digikey-footprints:Switch_Tactile_THT_6x6mm -> GeneralPurposeAlarmDevicePCB:Switch_Tactile_THT_6x6mm
- XTAL101: footprint Crystal:Crystal_SMD_HC49-SD -> digikey-footprints:SMD-2_3.2x2.5mm
- moved J103 102.9 mm to (168.9, 43.2), turned to 270 degrees
- moved C108 102.2 mm to (95.2, 50.8), turned to 0 degrees
- moved D101 97.2 mm to (88.9, 52.1)
- moved R504 97.0 mm to (76.2, 38.1), turned to 270 degrees
- moved R502 96.7 mm to (92.1, 35.6)
- moved R503 96.7 mm to (92.1, 32.4)
- moved C503 96.4 mm to (81.3, 31.8), turned to 180 degrees
- moved U101 95.3 mm to (97.8, 57.1)
- moved C102 95.3 mm to (88.9, 62.2)
- moved D501 95.0 mm to (92.7, 40.6), turned to 0 degrees
- moved J501 94.9 mm to (72.4, 36.2)
- moved U501 94.9 mm to (81.1, 36.5)
- moved C109 94.7 mm to (95.2, 45.7)
- moved D102 93.6 mm to (129.5, 46.4), turned to 90 degrees
- moved J401 93.5 mm to (174.0, 58.4), turned to 90 degrees
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- renumbered C107 to C108
Connections:
- net Net-(C601-Pad1) renamed /AlarmAudio/VccBuzzer
- C105 pad 1: /VccControler -> Net-(C102-Pad1)
- C106 pad 1: Net-(C106-Pad1) -> /VccControler
- C109 pad 1: Net-(C109-Pad1) -> +5V
- C110 pad 1: /VccControler -> Net-(C110-Pad1)
- C301 pad 1: Net-(C301-Pad1) -> /LCD And I2C Interface/Vcc_LCD
- C302 pad 1: Net-(C301-Pad1) -> /LCD And I2C Interface/Vcc_LCD
- R102 pad 1: Net-(C109-Pad1) -> Net-(C110-Pad1)
- R301 pad 2: Net-(C301-Pad1) -> /LCD And I2C Interface/Vcc_LCD
- R302 pad 2: Net-(C301-Pad1) -> /LCD And I2C Interface/Vcc_LCD
- R303 pad 2: Net-(C301-Pad1) -> /LCD And I2C Interface/Vcc_LCD
- R304 pad 2: Net-(C301-Pad1) -> /LCD And I2C Interface/Vcc_LCD
- R306 pad 2: Net-(C301-Pad1) -> /LCD And I2C Interface/Vcc_LCD
- R308 pad 2: Net-(C301-Pad1) -> /LCD And I2C Interface/Vcc_LCD
- R310 pad 1: Net-(C301-Pad1) -> /LCD And I2C Interface/Vcc_LCD
- R311 pad 2: Net-(C301-Pad1) -> /LCD And I2C Interface/Vcc_LCD
- RV301 pad 1: Net-(C301-Pad1) -> GND
- RV301 pad 3: GND -> /LCD And I2C Interface/Vcc_LCD
- S101 pad 1: Net-(C109-Pad1) -> Net-(C110-Pad1)
- S101 pad 2: Net-(C109-Pad1) -> Net-(C110-Pad1)
- U101 pad 4: Net-(R104-Pad2) -> +5V
- U102 pad 29: Net-(C109-Pad1) -> Net-(C110-Pad1)
- U102 pad 32: Net-(U102-Pad32) -> Switch_Mute
- U102 pad 8: Net-(C106-Pad1) -> Net-(C107-Pad1)
- U301 pad 16: Net-(C301-Pad1) -> /LCD And I2C Interface/Vcc_LCD
- U302 pad 15: Net-(C301-Pad1) -> /LCD And I2C Interface/Vcc_LCD
- U302 pad 2: Net-(C301-Pad1) -> /LCD And I2C Interface/Vcc_LCD
- XTAL101 pad 2: Net-(C106-Pad1) -> Net-(C107-Pad1)
Other:
- board size 137.2 x 152.4 mm -> 137.2 x 83.8 mm

Commit message: Add JST connector for I2C and more.
Parts:
- added C113: 33pF, Capacitor_SMD:C_0603_1608Metric_Pad1.08x0.95mm_HandSolder, F.Cu at (175.3, 91.4)
- added C114: 33pF, Capacitor_SMD:C_0603_1608Metric_Pad1.08x0.95mm_HandSolder, F.Cu at (170.2, 91.4)
- added J105: S04B-XASK-1(LF)(SN), Connector_PinHeader_2.54mm:PinHeader_1x04_P2.54mm_Horizontal, F.Cu at (176.3, 96.7)
- added R104: 39R, Resistor_SMD:R_0603_1608Metric, F.Cu at (137.2, 45.7)
- added R105: 39R, Resistor_SMD:R_0603_1608Metric, F.Cu at (136.7, 48.3)
- J102, J103: footprint digikey-footprints:PinHeader_1x2_P2.54mm_Drill1.02mm -> Connector_Molex:Molex_KK-254_AE-6410-02A_1x02_P2.54mm_Vertical
- Q201, Q202, Q203, Q204, Q205, Q601, Q602: footprint digikey-footprints:SOT-23-3 -> Package_TO_SOT_SMD:SOT-23
- RV301: footprint digikey-footprints:Trimpot_3.8mmx3.6mm_TC33X-2-103E -> GeneralPurposeAlarmDevicePCB:Potentiometer_Bourns_3386P_Vertical
- moved J103 25.3 mm to (176.5, 67.3), turned to 0 degrees
- moved RV301 12.5 mm to (184.2, 38.1), turned to 90 degrees
- moved J102 10.2 mm to (63.5, 47.0), turned to 0 degrees
- moved R209 8.91 mm to (147.3, 78.7), turned to 90 degrees
- moved R207 7.65 mm to (137.2, 78.7), turned to 90 degrees
- moved Q205 7.24 mm to (148.6, 83.8)
- moved Q204 6.41 mm to (138.4, 83.8)
- moved Q201 5.46 mm to (104.1, 83.8)
- moved R205 5.08 mm to (125.7, 79.2), turned to 90 degrees
- moved Q203 5.07 mm to (127.0, 83.8)
- moved Q202 4.50 mm to (115.6, 83.8)
- moved R203 2.55 mm to (114.3, 79.2), turned to 90 degrees
- moved Q601 1.27 mm to (157.5, 74.9)
- turned R201 to 90 degrees

Commit message: Add more parts including a place holder only for power jack 3D, USB micro is incomplete. Added I2C daisy chain connector.
Parts:
- added D103: 1N5819WS, GeneralPurposeAlarmDevicePCB:D_SOD-323, F.Cu at (108.0, 59.7)
- J501: footprint Connector_USB:USB_Micro-B_Amphenol_10118194_Horizontal -> Connector_USB:USB_Micro-B_Wuerth_629105150521
- U102: footprint digikey-footprints:TQFP-32_7x7mm -> Package_QFP:TQFP-32_7x7mm_P0.8mm
- moved C109 47.6 mm to (62.2, 80.0), turned to 90 degrees
- moved J102 43.3 mm to (61.0, 90.2), turned to 90 degrees
- moved C108 40.4 mm to (67.3, 80.0), turned to 90 degrees
- moved J101 40.4 mm to (73.4, 97.0), turned to 90 degrees
- moved D101 39.9 mm to (68.6, 86.4), turned to 270 degrees
- moved S101 34.5 mm to (102.9, 55.9), turned to 180 degrees
- moved C101 34.5 mm to (73.4, 88.9), turned to 0 degrees
- moved C105 32.1 mm to (73.7, 83.8), turned to 270 degrees
- moved U101 31.5 mm to (73.7, 77.5), turned to 90 degrees
- moved C102 26.2 mm to (78.7, 86.4), turned to 270 degrees
- moved J501 23.1 mm to (58.4, 54.6)
- moved C501 20.8 mm to (68.6, 55.9)
- moved R503 20.8 mm to (79.4, 48.9)
- moved C502 20.8 mm to (69.8, 59.7)
- moved C503 20.8 mm to (68.6, 48.3)
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
Commit message: Add current limit to CongtollerVcc, and Barrel Input. Add jumper resistors for headers selecting VBus and ControllerVcc.
Parts:
- added A101: Arduino_UNO_R3, Module:Arduino_UNO_R3, F.Cu at (10.2, 41.9)
- added R602: 10K, Resistor_SMD:R_0603_1608Metric, F.Cu at (128.3, 54.6)
- added R604: 1R0, Resistor_SMD:R_0603_1608Metric, F.Cu at (161.3, 78.7)
- R401, R402, R403, R404: value R -> 330
- renumbered R602 to R605
Connections:
- net Net-(U102-Pad2) renamed Attenuate
- Q601 pad 2: Net-(BZ601-Pad1) -> Net-(Q601-Pad2)
- Q602 pad 2: Net-(BZ601-Pad1) -> Net-(Q601-Pad2)
- R605 pad 1: Tone -> Net-(R605-Pad1)

Commit message: Update schottky symbol and part number. Import to PCB. Only the Arduino UNO symbol remains to connect.
Parts:
- added C602: 100nF, Capacitor_SMD:C_0603_1608Metric_Pad1.08x0.95mm_HandSolder, F.Cu at (104.1, -8.89)
- added D104: Schottky 2A, Diode_SMD:D_SMB, F.Cu at (87.5, -7.37)
- added F101: Polyfuse_Small, Fuse:Fuse_0603_1608Metric, F.Cu at (57.1, -3.81)
- added F401: Polyfuse_Small, Fuse:Fuse_0603_1608Metric, F.Cu at (64.8, -3.81)
- added J601: 22-23-2021, Connector_Molex:Molex_KK-254_AE-6410-02A_1x02_P2.54mm_Vertical, F.Cu at (97.1, -6.20)
- added R106: DNI, Resistor_SMD:R_0603_1608Metric, F.Cu at (76.9, -3.34)
- added R107: DNI, Resistor_SMD:R_0603_1608Metric, F.Cu at (80.9, -3.34)
- added R108: 1K, Resistor_SMD:R_0603_1608Metric, F.Cu at (85.0, -3.34)
- added R109: 1K, Resistor_SMD:R_0603_1608Metric, F.Cu at (89.0, -3.34)
- D103: value 1N5819WS -> Schottky 2A; footprint GeneralPurposeAlarmDevicePCB:D_SOD-323 -> Diode_SMD:D_SMB
- R306, R308: value 1K -> DNI
- moved D103 73.0 mm to (79.1, -7.37)
- moved R306 70.7 mm to (76.9, 3.62), turned to 0 degrees
- moved R308 64.2 mm to (80.9, 3.62), turned to 0 degrees
Connections:
- D101 pad 2: Net-(C101-Pad1) -> Net-(D101-Pad2)
- J103 pad 1: +5V -> Net-(D104-Pad2)
- J401 pad 5: ControllerVcc -> Net-(F401-Pad2)
- R306 pad 1: SDA -> Net-(R306-Pad1)
- R308 pad 1: SCL -> GND
- R308 pad 2: /LCD And I2C Interface/Vcc_LCD -> Net-(R306-Pad1)
- RV301 pad 2: Net-(RV301-Pad2) -> Net-(R306-Pad1)
- U302 pad 3: Net-(RV301-Pad2) -> Net-(R306-Pad1)

Commit message: Add both UNO and NANO schematic and PCB foot print.  Zero schematic errors reported. This incorporates all of the updates from the review except the DO NOT FIX.
Parts:
- added A102: Arduino_Nano_v2.x_Header, Module:Arduino_Nano, F.Cu at (47.0, 55.9)
- A101: value Arduino_UNO_R3 -> Arduino_UNO_R3_Shield
- moved A101 1.80 mm to (8.89, 40.6)
Connections:
- A101 pad 10: Net-(A101-Pad10) -> PC1
- A101 pad 11: Net-(A101-Pad11) -> PC2
- A101 pad 12: Net-(A101-Pad12) -> PC3
- A101 pad 17: Net-(A101-Pad17) -> Switch_Mute
- A101 pad 18: Net-(A101-Pad18) -> Light0
- A101 pad 19: Net-(A101-Pad19) -> Attenuate
- A101 pad 2: Net-(A101-Pad2) -> +5V
- A101 pad 20: Net-(A101-Pad20) -> Light1
- A101 pad 21: Net-(A101-Pad21) -> Light2
- A101 pad 22: Net-(A101-Pad22) -> nCS
- A101 pad 23: Net-(A101-Pad23) -> Tone
- A101 pad 24: Net-(A101-Pad24) -> Light3
- A101 pad 25: Net-(A101-Pad25) -> Light4
- A101 pad 26: Net-(A101-Pad26) -> COPI
- A101 pad 27: Net-(A101-Pad27) -> CIPO
- A101 pad 28: Net-(A101-Pad28) -> SPI_SCK
- A101 pad 3: Net-(A101-Pad3) -> nRESET
- A101 pad 30: Net-(A101-Pad30) -> Aref
- A101 pad 31: Net-(A101-Pad31) -> SDA
- A101 pad 32: Net-(A101-Pad32) -> SCL
- A101 pad 5: Net-(A101-Pad5) -> +5V
- A101 pad 8: Net-(A101-Pad8) -> Vin
- A101 pad 9: Net-(A101-Pad9) -> PC0
- C102 pad 1: Net-(C102-Pad1) -> Vin
- C103 pad 1: /VccControler -> Aref
- C105 pad 1: Net-(C102-Pad1) -> Vin
- C106 pad 1: /VccControler -> Aref
- C110 pad 1: Net-(C110-Pad1) -> nRESET
- C111 pad 1: /VccControler -> Aref
- C112 pad 1: /VccControler -> Aref
- D101 pad 1: Net-(C102-Pad1) -> Vin
- D103 pad 1: /VccControler -> Aref
- D103 pad 2: Net-(C110-Pad1) -> nRESET
- D104 pad 1: Net-(C102-Pad1) -> Vin
- R101 pad 1: /VccControler -> Aref
- R102 pad 1: Net-(C110-Pad1) -> nRESET
- R102 pad 2: /VccControler -> Aref
- R108 pad 1: /VccControler -> Aref
- R109 pad 1: /VccControler -> Aref
- R605 pad 1: Net-(R605-Pad1) -> Attenuate
- S101 pad 1: Net-(C110-Pad1) -> nRESET
- S101 pad 2: Net-(C110-Pad1) -> nRESET
- U101 pad 3: Net-(C102-Pad1) -> Vin
- U102 pad 18: /VccControler -> Aref
- U102 pad 19: Net-(U102-Pad19) -> ADC6
- U102 pad 20: /VccControler -> Aref
- U102 pad 22: Net-(U102-Pad22) -> ADC7
- U102 pad 23: Net-(U102-Pad23) -> PC0
- U102 pad 24: Net-(U102-Pad24) -> PC1
- U102 pad 25: Net-(U102-Pad25) -> PC2
- U102 pad 26: Net-(U102-Pad26) -> PC3
- U102 pad 29: Net-(C110-Pad1) -> nRESET
- U102 pad 3: Net-(U102-Pad3) -> GND
- U102 pad 4: /VccControler -> Aref
- U102 pad 6: /VccControler -> Aref

Commit message: Clean up a bunch of duplicate because of missspelled part field names. Still working on a few sch, pcb and 3D libraries.
Parts:
- BZ601: value PKMCS0909E4000-R1 -> QMB-09B-03; footprint digikey-footprints:Piezo_9x9mm_PKMCS0909E4000-R1 -> GeneralPurposeAlarmDevicePCB:MagneticBuzzer_9mmx5.8mmP=4mm; moved to B.Cu
- C601: value 47uF 16V -> 47uF
- Q602: footprint Package_TO_SOT_SMD:SOT-23 -> digikey-footprints:SOT-23-3
- R601, R604: value 1R0 -> 1R
- R602: value 10K -> 1K
- R605: value 330R -> 330
- moved J601 121.8 mm to (162.6, 96.5), turned to 180 degrees
- moved F401 119.9 mm to (170.2, 53.3)
- moved R107 112.8 mm to (168.9, 67.3), turned to 180 degrees
- moved R306 111.2 mm to (180.3, 44.5), turned to 180 degrees
- moved R308 111.0 mm to (184.2, 44.5), turned to 180 degrees
- moved D104 101.4 mm to (160.0, 63.5)
- moved F101 95.7 mm to (66.0, 91.4)
- moved C602 90.9 mm to (92.7, 81.3), turned to 180 degrees
- moved R106 90.3 mm to (58.4, 85.1)
- moved D103 56.7 mm to (99.1, 45.7), turned to 180 degrees
- moved R108 53.4 mm to (107.8, 44.9)
- moved R109 53.4 mm to (111.8, 44.9)
- moved R602 31.5 mm to (152.4, 74.9), turned to 90 degrees
- moved J103 9.67 mm to (167.6, 63.5)
- moved BZ601 2.63 mm to (160.0, 87.6), turned to 0 degrees
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