File: Hardware/GeneralPurposeAlarmDevicePCB/GeneralPurposeAlarmDevicePCB/GeneralPurposeAlarmDevicePCB.kicad_pcb (KiCad board)
At the start: 2 copper layers, 137.2 x 83.8 mm, 110 parts, among them J101 Barrel_Jack_Switch_SMT, J102 22-23-2021, J103 22-23-2021, J105 S04B-XASK-1(LF)(SN), J401 RJ12_6P6C_HORZ, J501 USB_B_Micro, J601 22-23-2021, Q201 MMBT2222A-7-F, Q202 MMBT2222A-7-F, Q203 MMBT2222A-7-F, Q204 MMBT2222A-7-F, Q205 MMBT2222A-7-F, Q301 BSS138, Q601 MMBT2222A-7-F, Q602 MMBT2907ALT1G, U101 NCP1117ST50T3G, U102 PI_ATMEGA328P-AU-InOrder, U301 PCF8574AT, U302 LCD_20x4_Character, U501 CH340E

Commit message: updated PCB layout, most everything is connected.
Signed-off-by: lokimetasmith <lokimail@gmail.com>
Parts:
- moved R101 39.4 mm to (77.3, 79.6)
- moved R309 4.98 mm to (148.4, 48.1), turned to -90 degrees
- moved TP_3v3 2.10 mm to (91.6, 21.3)
- moved J103 2.08 mm to (165.9, 88.9), turned to 180 degrees
- moved R604 1.86 mm to (63.5, 79.7)
- moved R602 1.78 mm to (60.3, 80.4)
- moved R605 1.37 mm to (59.7, 78.8)
- moved C101 1.10 mm to (174.1, 87.8)
- moved R107 0.64 mm to (164.8, 93.3), turned to 0 degrees
- moved R504 0.40 mm to (101.8, 72.7)
- moved C108 0.37 mm to (182.8, 70.8)
- turned D104 to 180 degrees
- turned U101 to -90 degrees
Routing:
- net Vin: track 36.7 -> 135.9 mm, vias 0 -> 2
- net Tone: track 0.00 -> 84.1 mm, vias 0 -> 2
- net +5V: track 180.0 -> 254.3 mm, vias 2 -> 5
- net Aref: track 56.5 -> 121.5 mm, vias 2 -> 5
- net Attenuate: track 20.0 -> 78.3 mm, vias 1 -> 2
- net SPI_SCK: track 53.4 -> 103.3 mm, vias 0 -> 1
- net VBus: track 122.6 -> 74.1 mm, vias 4 -> 1
- net CIPO: track 51.5 -> 99.5 mm
- net Switch_Mute: track 29.4 -> 76.9 mm, vias 2 -> 3
- net COPI: track 44.4 -> 90.4 mm, vias 0 -> 1
- net Light4: track 12.9 -> 56.4 mm, vias 0 -> 1
- net Light3: track 8.35 -> 51.7 mm, vias 0 -> 1
- net nCS: track 40.9 -> 77.7 mm, vias 0 -> 1
- net Light2: track 7.82 -> 44.2 mm, vias 0 -> 1
- net Light1: track 13.4 -> 45.1 mm, vias 0 -> 1
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
Commit message: Update buzzer foot print. Fully connect all parts. Fix numerous silkscreen conflicts. Mix of metric and imperial grid.
Parts:
- added R111: 330R, Resistor_SMD:R_0603_1608Metric, F.Cu at (86.4, 21.0)
- BZ601: value QMB-09B-03 -> Buzzer_12.2mm_H6.5mm; footprint Buzzer_Beeper:MagneticBuzzer_PUI_AT-0927-TT-6-R -> Buzzer_Beeper:Buzzer_TDK_PS1240P02BT_D12.2mm_H6.5mm
- J501: footprint Connector_USB:USB_Micro-B_Wuerth_629105150521 -> GeneralPurposeAlarmDevicePCB:USB_Micro-B_Amphenol_10118194_Horizontal
- U302: value LCD_20x4_Character -> LCD_20x4_Character-GPAD_SCH_LIB
- moved J102 91.2 mm to (94.0, 96.5), turned to 180 degrees
- moved R106 84.1 mm to (92.7, 92.1), turned to 0 degrees
- moved S101 41.9 mm to (75.6, 24.1)
- moved C602 16.5 mm to (74.3, 95.2)
- moved R311 8.64 mm to (132.1, 28.6)
- moved R602 7.66 mm to (66.7, 76.2), turned to 0 degrees
- moved R605 6.97 mm to (66.7, 78.1), turned to 180 degrees
- moved R209 6.84 mm to (88.9, 80.0)
- moved R101 3.74 mm to (74.3, 77.5), turned to 180 degrees
- moved R309 3.73 mm to (149.2, 44.5), turned to 180 degrees
- moved R603 3.17 mm to (78.1, 94.0)
- moved BZ601 2.45 mm to (65.9, 85.7)
- moved D104 2.01 mm to (165.7, 80.6), turned to -90 degrees
- moved D101 1.42 mm to (182.2, 85.1)
- moved R108 1.39 mm to (111.7, 46.4)
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Connections:
- A101 pad 3: nRESET -> Net-(A101-Pad3)
Routing:
- net nRESET: track 56.2 -> 69.8 mm
- net Attenuate: track 78.3 -> 66.5 mm, vias 2 -> 3
- net +5V: track 254.3 -> 264.9 mm, vias 5 -> 6
- net VBus: track 74.1 -> 63.7 mm, vias 1 -> 2
- net Aref: track 121.5 -> 130.7 mm, vias 5 -> 3
- net Tone: track 84.1 -> 76.5 mm
- net Net-(A101-Pad3): track 0.00 -> 6.43 mm
- net GND: track 18.7 -> 23.4 mm, vias 10 -> 77
- net /LCD And I2C Interface/Vcc_LCD: track 135.9 -> 131.3 mm
- net Net-(Q205-Pad1): track 1.75 -> 5.65 mm
- net COPI: track 90.4 -> 94.2 mm
- net CIPO: track 99.5 -> 102.9 mm
- net Net-(Q601-Pad1): track 17.0 -> 13.7 mm
- net Vin: track 135.9 -> 132.7 mm, vias 2 -> 4
- net SDA: track 118.2 -> 121.0 mm
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
Commit message: Fix pot foot print, Add fifth mounting hole. Place all but UNO and test point.
Parts:
- added H105: MountingHole_Pad_3.5mm, GeneralPurposeAlarmDevicePCB:MountingHole_3.5mm_Pad_Via, F.Cu at (124.5, 96.5)
- RV301: value 10K -> POT 3/8 10K; moved to B.Cu
- S101: moved to B.Cu
- S601: value SWITCH_TACTILE_SPST-NO_0.05A_24V -> SWITCH_TACTILE_12mmx12mm_SPST-NO_0.05A_24V; footprint GeneralPurposeAlarmDevicePCB:Switch_Tactile_THT_6x6mm -> Button_Switch_THT:SW_PUSH-12mm
- moved TP_3v3 194.4 mm to (-72.4, 125.7), turned to 90 degrees
- moved A101 181.4 mm to (-66.0, 128.9), turned to 90 degrees
- moved S101 79.0 mm to (121.2, 88.6), turned to 0 degrees
- moved R210 70.6 mm to (71.1, 17.8), turned to 180 degrees
- moved D205 65.6 mm to (71.1, 24.1), turned to -90 degrees
- moved D201 63.5 mm to (71.1, 74.9), turned to -90 degrees
- moved R208 62.3 mm to (71.1, 29.2), turned to 180 degrees
- moved R209 62.3 mm to (76.2, 19.1), turned to 0 degrees
- moved Q205 60.3 mm to (76.2, 24.1), turned to -90 degrees
- moved R202 59.5 mm to (71.1, 67.3), turned to 180 degrees
- moved D204 58.0 mm to (71.1, 36.8), turned to -90 degrees
- moved D202 56.8 mm to (71.1, 62.2), turned to -90 degrees
- moved R207 56.6 mm to (74.9, 30.5), turned to 0 degrees
- moved Q201 56.6 mm to (76.2, 74.9), turned to -90 degrees
- moved R206 55.4 mm to (71.1, 43.2), turned to 180 degrees
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Routing:
- net +5V: track 264.9 -> 0.00 mm, vias 6 -> 0
- net Vin: track 132.7 -> 0.00 mm, vias 4 -> 0
- net /LCD And I2C Interface/Vcc_LCD: track 131.3 -> 0.00 mm
- net Aref: track 130.7 -> 0.00 mm, vias 3 -> 0
- net SCL: track 123.7 -> 0.00 mm, vias 5 -> 0
- net SDA: track 121.0 -> 0.00 mm, vias 5 -> 0
- net SPI_SCK: track 106.0 -> 0.00 mm, vias 1 -> 0
- net CIPO: track 102.9 -> 0.00 mm, vias 2 -> 0
- net COPI: track 94.2 -> 0.00 mm, vias 1 -> 0
- net nCS: track 77.7 -> 0.00 mm, vias 1 -> 0
- net Tone: track 76.5 -> 0.00 mm, vias 2 -> 0
- net Switch_Mute: track 75.1 -> 0.00 mm, vias 1 -> 0
- net nRESET: track 69.8 -> 0.00 mm
- net Attenuate: track 66.5 -> 0.00 mm, vias 3 -> 0
- net VBus: track 63.7 -> 0.00 mm, vias 2 -> 0
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- removed copper zone on B.Cu, net GND
- removed copper zone on F.Cu, net GND

Commit message: Tweek POT and power LED. UNO placed.
Parts:
- moved A101 164.6 mm to (88.9, 73.4)
- moved TP_3v3 164.6 mm to (82.5, 70.2)
- moved RV301 3.85 mm to (182.9, 41.3)
- moved TP_nINT301 2.62 mm to (136.5, 31.8)
- moved D105 2.54 mm to (189.2, 54.6)
Changed lines of the file:
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@@
   )
   (footprint "TestPoint:TestPoint_Loop_D2.54mm_Drill1.5mm_Beaded" (layer "F.Cu")
-    (at 137.16 34.29)
+    (at 136.525 31.75)
     (descr "wire loop with bead as test point, loop diameter2.548mm, hole diameter 1.5mm")
     (tags "test point wire loop bead")
@@
   )
   (footprint "Module:Arduino_UNO_R3" (layer "F.Cu")
-    (at -66.04 128.905 90)
+    (at 88.9 73.41 90)
     (descr "Arduino UNO R3, http://www.mouser.com/pdfdocs/Gravitech_Arduino_Nano3_0.pdf")
     (tags "Arduino UNO R3")
@@
   )
   (footprint "TestPoint:TestPoint_Loop_D2.54mm_Drill1.5mm_Beaded" (layer "F.Cu")
-    (at -72.39 125.73 90)
+    (at 82.55 70.235 90)
     (descr "wire loop with bead as test point, loop diameter2.548mm, hole diameter 1.5mm")
     (tags "test point wire loop bead")
@@
   )
   (footprint "GeneralPurposeAlarmDevicePCB:LED_5mm_Radial" (layer "B.Cu")
-    (at 189.23 57.15)
+    (at 189.23 54.61)
     (descr "http://optoelectronics.liteon.com/upload/download/DS20-2000-343/1CHKxKNN.pdf")
     (property "Category" "Optoelectronics")
@@
   )
   (footprint "GeneralPurposeAlarmDevicePCB:Potentiometer_Bourns_3386P_Vertical" (layer "B.Cu")
-    (at 182.245 45.07 90)
+    (at 182.88 41.275 90)
     (descr "Potentiometer, vertical, Bourns 3386P, https://www.bourns.com/pdfs/3386.pdf")
     (tags "Potentiometer vertical Bourns 3386P")

Commit message: Fixed library and schematic broken due to POT description including a "/" in symbol name.
Parts:
- RV301: value POT 3/8 10K -> POT 0.375 10K
Changed lines of the file:
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@@
     (property "Sheetname" "LCD And I2C Interface")
     (attr through_hole)
-    (fp_text reference "RV301" (at -0.015 8.555 90) (layer "B.SilkS")
+    (fp_text reference "RV301" (at -6.35 2.54 180) (layer "B.SilkS")
       (effects (font (size 1 1) (thickness 0.15)) (justify mirror))
     )
-    (fp_text value "POT 3/8 10K" (at -0.015 -3.475 90) (layer "B.Fab")
+    (fp_text value "POT 0.375 10K" (at -0.015 -3.475 90) (layer "B.Fab")
       (effects (font (size 1 1) (thickness 0.15)) (justify mirror))
     )
@@
       (effects (font (size 1 1) (thickness 0.15)) (justify mirror))
     )
+    (fp_line (start 4.87 7.425) (end 4.87 -2.345) (layer "B.SilkS") (width 0.12))
+    (fp_line (start -4.9 7.425) (end 4.87 7.425) (layer "B.SilkS") (width 0.12))
+    (fp_line (start -4.9 7.425) (end -4.9 -2.345) (layer "B.SilkS") (width 0.12))
+    (fp_line (start -0.891 0.98) (end -0.89 4.099) (layer "B.SilkS") (width 0.1))
     (fp_line (start -4.9 -2.345) (end 4.87 -2.345) (layer "B.SilkS") (width 0.12))
-    (fp_line (start -4.9 7.425) (end 4.87 7.425) (layer "B.SilkS") (width 0.12))
-    (fp_line (start -0.891 0.98) (end -0.89 4.099) (layer "B.SilkS") (width 0.1))
-    (fp_line (start -4.9 7.425) (end -4.9 -2.345) (layer "B.SilkS") (width 0.12))
-    (fp_line (start 4.87 7.425) (end 4.87 -2.345) (layer "B.SilkS") (width 0.12))
     (fp_circle (center -0.8905 2.5395) (end 0.6845 2.5395) (layer "B.SilkS") (width 0.1) (fill none))
     (fp_line (start -5.03 -2.48) (end 5 -2.48) (layer "B.CrtYd") (width 0.05))
+    (fp_line (start 5 7.56) (end -5.03 7.56) (layer "B.CrtYd") (width 0.05))
     (fp_line (start -5.03 7.56) (end -5.03 -2.48) (layer "B.CrtYd") (width 0.05))
     (fp_line (start 5 -2.48) (end 5 7.56) (layer "B.CrtYd") (width 0.05))
-    (fp_line (start 5 7.56) (end -5.03 7.56) (layer "B.CrtYd") (width 0.05))
+    (fp_line (start -0.891 0.98) (end -0.89 4.099) (layer "B.Fab") (width 0.1))
+    (fp_line (start 4.75 -2.225) (end 4.75 7.305) (layer "B.Fab") (width 0.1))
     (fp_line (start -4.78 -2.225) (end 4.75 -2.225) (layer "B.Fab") (width 0.1))
-    (fp_line (start -0.891 0.98) (end -0.89 4.099) (layer "B.Fab") (width 0.1))
+    (fp_line (start -4.78 7.305) (end -4.78 -2.225) (layer "B.Fab") (width 0.1))
     (fp_line (start 4.75 7.305) (end -4.78 7.305) (layer "B.Fab") (width 0.1))
-    (fp_line (start 4.75 -2.225) (end 4.75 7.305) (layer "B.Fab") (width 0.1))
-    (fp_line (start -4.78 7.305) (end -4.78 -2.225) (layer "B.Fab") (width 0.1))
     (fp_circle (center -0.891 2.54) (end 0.684 2.54) (layer "B.Fab") (width 0.1) (fill none))
     (pad "1" thru_hole circle (at 0 0 90) (size 1.44 1.44) (drill 0.8) (layers *.Cu *.Mask)

Commit message: Tweek to placement of the I2C connector.
Parts:
- moved R105 6.93 mm to (142.9, 51.4)
- moved R104 5.85 mm to (142.9, 47.0)
- moved J105 0.29 mm to (141.0, 96.5)
Changed lines of the file:
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@@
   )
   (footprint "Connector_PinHeader_2.54mm:PinHeader_1x04_P2.54mm_Horizontal" (layer "F.Cu")
-    (at 140.72 96.67 -90)
+    (at 140.97 96.52 -90)
     (descr "Through hole angled pin header, 1x04, 2.54mm pitch, 6mm pin length, single row")
     (tags "Through hole angled pin header THT 1x04 2.54mm single row")
@@
   )
   (footprint "Resistor_SMD:R_0603_1608Metric" (layer "F.Cu")
-    (at 137.16 45.72 180)
+    (at 142.875 46.99 180)
     (descr "Resistor SMD 0603 (1608 Metric), square (rectangular) end terminal, IPC_7351 nominal, (Body size source: IPC-SM-782 page 72, https://www.pcb-3d.com/wordpress/wp-content/uploads/ipc-sm-782a_amendment_1_and_2.pdf), generated with kicad-footprint-generator")
     (tags "resistor")
@@
   )
   (footprint "Resistor_SMD:R_0603_1608Metric" (layer "F.Cu")
-    (at 136.715 48.26 180)
+    (at 142.875 51.435 180)
     (descr "Resistor SMD 0603 (1608 Metric), square (rectangular) end terminal, IPC_7351 nominal, (Body size source: IPC-SM-782 page 72, https://www.pcb-3d.com/wordpress/wp-content/uploads/ipc-sm-782a_amendment_1_and_2.pdf), generated with kicad-footprint-generator")
     (tags "resistor")

Commit message: Add an Arduino UNO footprint to the PDB and make a PCB footprint with same.
Parts:
- A101: moved to B.Cu
- moved TP_3v3 57.9 mm to (140.3, 66.7)
- moved A101 45.7 mm to (134.6, 73.4)
- moved R101 40.0 mm to (120.7, 74.3), turned to 0 degrees
- moved XTAL101 33.7 mm to (101.0, 43.8), turned to -90 degrees
- moved D102 33.2 mm to (99.7, 61.0), turned to -90 degrees
- moved D103 31.9 mm to (120.7, 69.2), turned to 0 degrees
- moved C104 31.6 mm to (104.8, 41.3), turned to 90 degrees
- moved J102 27.9 mm to (76.2, 96.5)
- moved R103 27.7 mm to (102.9, 61.0), turned to -90 degrees
- moved C106 27.3 mm to (110.5, 40.6), turned to 0 degrees
- moved C112 26.5 mm to (109.9, 66.0), turned to 180 degrees
- moved R111 26.0 mm to (127.6, 54.0), turned to 180 degrees
- moved C107 24.5 mm to (104.8, 46.4), turned to -90 degrees
- moved R109 22.0 mm to (121.4, 62.4), turned to 180 degrees
- moved C103 17.9 mm to (110.5, 45.7), turned to 0 degrees
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
Commit message: Add12mmx12mmSwitc.
Parts:
- S601: footprint Button_Switch_THT:SW_PUSH-12mm -> GeneralPurposeAlarmDevicePCB:SW_PUSH-12mm_WithCap_Green
- moved R603 47.6 mm to (81.9, 43.2), turned to 180 degrees
- moved R605 45.6 mm to (81.3, 48.3)
- moved R602 33.6 mm to (81.3, 59.7)
- moved C602 10.5 mm to (81.3, 83.8), turned to 0 degrees
Changed lines of the file:
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@@
     )
     (pad_to_mask_clearance 0)
-    (grid_origin 48.26 38.1)
+    (grid_origin 55.88 101.6)
     (pcbplotparams
       (layerselection 0x00010fc_ffffffff)
@@
   )
   (footprint "Resistor_SMD:R_0603_1608Metric" (layer "F.Cu")
-    (at 64.77 90.805 180)
+    (at 81.28 48.26 180)
     (descr "Resistor SMD 0603 (1608 Metric), square (rectangular) end terminal, IPC_7351 nominal, (Body size source: IPC-SM-782 page 72, https://www.pcb-3d.com/wordpress/wp-content/uploads/ipc-sm-782a_amendment_1_and_2.pdf), generated with kicad-footprint-generator")
     (tags "resistor")
@@
     (property "Sheetname" "AlarmAudio")
     (attr smd)
-    (fp_text reference "R605" (at -3.175 0) (layer "F.SilkS")
+    (fp_text reference "R605" (at 0 1.27) (layer "F.SilkS")
       (effects (font (size 1 1) (thickness 0.15)))
     )
@@
   )
   (footprint "Resistor_SMD:R_0603_1608Metric" (layer "F.Cu")
-    (at 70.950785 89.535)
+    (at 81.915 43.18 180)
     (descr "Resistor SMD 0603 (1608 Metric), square (rectangular) end terminal, IPC_7351 nominal, (Body size source: IPC-SM-782 page 72, https://www.pcb-3d.com/wordpress/wp-content/uploads/ipc-sm-782a_amendment_1_and_2.pdf), generated with kicad-footprint-generator")
     (tags "resistor")
@@
     (property "Sheetname" "AlarmAudio")
     (attr smd)
-    (fp_text reference "R603" (at 0 -1.43) (layer "F.SilkS")
+    (fp_text reference "R603" (at 0.237258 1.905) (layer "F.SilkS")
       (effects (font (size 1 1) (thickness 0.15)))
     )
@@
     (fp_line (start -0.8 -0.4125) (end 0.8 -0.4125) (layer "F.Fab") (width 0.1))
     (fp_line (start 0.8 0.4125) (end -0.8 0.4125) (layer "F.Fab") (width 0.1))
-    (pad "1" smd roundrect locked (at -0.825 0) (size 0.8 0.95) (layers "F.Cu" "F.Paste" "F.Mask") (roundrect_rratio 0.25)
+    (pad "1" smd roundrect locked (at -0.825 0 180) (size 0.8 0.95) (layers "F.Cu" "F.Paste" "F.Mask") (roundrect_rratio 0.25)
       (net 69 "Switch_Mute") (pintype "passive"))
-    (pad "2" smd roundrect locked (at 0.825 0) (size 0.8 0.95) (layers "F.Cu" "F.Paste" "F.Mask") (roundrect_rratio 0.25)
+    (pad "2" smd roundrect locked (at 0.825 0 180) (size 0.8 0.95) (layers "F.Cu" "F.Paste" "F.Mask") (roundrect_rratio 0.25)
       (net 5 "+5V") (pintype "passive"))
     (model "${KISYS3DMOD}/Resistor_SMD.3dshapes/R_0603_1608Metric.wrl"
@@
   )
   (footprint "Capacitor_SMD:C_0603_1608Metric_Pad1.08x0.95mm_HandSolder" (layer "F.Cu")
-    (at 70.950785 81.915 180)
+    (at 81.28 83.82)
     (descr "Capacitor SMD 0603 (1608 Metric), square (rectangular) end terminal, IPC_7351 nominal with elongated pad for handsoldering. (Body size source: IPC-SM-782 page 76, https://www.pcb-3d.com/wordpress/wp-content/uploads/ipc-sm-782a_amendment_1_and_2.pdf), generated with kicad-footprint-generator")
     (tags "capacitor handsolder")
@@
     (fp_line (start 0.8 -0.4) (end 0.8 0.4) (layer "F.Fab") (width 0.1))
     (fp_line (start -0.8 0.4) (end -0.8 -0.4) (layer "F.Fab") (width 0.1))
-    (pad "1" smd roundrect locked (at -0.8625 0 180) (size 1.075 0.95) (layers "F.Cu" "F.Paste" "F.Mask") (roundrect_rratio 0.25)
+    (pad "1" smd roundrect locked (at -0.8625 0) (size 1.075 0.95) (layers "F.Cu" "F.Paste" "F.Mask") (roundrect_rratio 0.25)
       (net 69 "Switch_Mute") (pintype "passive"))
-    (pad "2" smd roundrect locked (at 0.8625 0 180) (size 1.075 0.95) (layers "F.Cu" "F.Paste" "F.Mask") (roundrect_rratio 0.25)
+    (pad "2" smd roundrect locked (at 0.8625 0) (size 1.075 0.95) (layers "F.Cu" "F.Paste" "F.Mask") (roundrect_rratio 0.25)
       (net 2 "GND") (pintype "passive"))
     (model "${KISYS3DMOD}/Capacitor_SMD.3dshapes/C_0603_1608Metric.wrl"
@@
   )
   (footprint "Resistor_SMD:R_0603_1608Metric" (layer "F.Cu")
-    (at 64.77 88.9)
+    (at 81.28 59.69)
     (descr "Resistor SMD 0603 (1608 Metric), square (rectangular) end terminal, IPC_7351 nominal, (Body size source: IPC-SM-782 page 72, https://www.pcb-3d.com/wordpress/wp-content/uploads/ipc-sm-782a_amendment_1_and_2.pdf), generated with kicad-footprint-generator")
     (tags "resistor")
@@
     (property "Sheetname" "AlarmAudio")
     (attr smd)
-    (fp_text reference "R602" (at 3.81 0) (layer "F.SilkS")
+    (fp_text reference "R602" (at 0 -1.27) (layer "F.SilkS")
       (effects (font (size 1 1) (thickness 0.15)))
     )
@@
     )
   )
-  (footprint "Button_Switch_THT:SW_PUSH-12mm" (layer "B.Cu")
+  (footprint "GeneralPurposeAlarmDevicePCB:SW_PUSH-12mm_WithCap_Green" (layer "B.Cu")
     (at 93.98 88.9 180)
     (descr "SW PUSH 12mm https://www.e-switch.com/system/asset/product_line/data_sheet/143/TL1100.pdf")
@@
     )
     (fp_line (start 12.4 -8.65) (end 0.1 -8.65) (layer "B.SilkS") (width 0.12))
-    (fp_line (start 0.1 0.93) (end 0.1 3.65) (layer "B.SilkS") (width 0.12))
-    (fp_line (start 0.1 -4.07) (end 0.1 -0.93) (layer "B.SilkS") (width 0.12))
     (fp_line (start 12.4 -5.93) (end 12.4 -8.65) (layer "B.SilkS") (width 0.12))
     (fp_line (start 12.4 3.65) (end 12.4 0.93) (layer "B.SilkS") (width 0.12))
+    (fp_line (start 0.1 3.65) (end 12.4 3.65) (layer "B.SilkS") (width 0.12))
     (fp_line (start 12.4 -0.93) (end 12.4 -4.07) (layer "B.SilkS") (width 0.12))
     (fp_line (start 0.1 -8.65) (end 0.1 -5.93) (layer "B.SilkS") (width 0.12))
-    (fp_line (start 0.1 3.65) (end 12.4 3.65) (layer "B.SilkS") (width 0.12))
+    (fp_line (start 0.1 -4.07) (end 0.1 -0.93) (layer "B.SilkS") (width 0.12))
+    (fp_line (start 0.1 0.93) (end 0.1 3.65) (layer "B.SilkS") (width 0.12))
     (fp_circle (center 6.35 -2.54) (end 10.16 -5.08) (layer "B.SilkS") (width 0.12) (fill none))
-    (fp_line (start 14.25 -8.75) (end -1.77 -8.75) (layer "B.CrtYd") (width 0.05))
+    (fp_line (start -1.77 3.75) (end 14.25 3.75) (layer "B.CrtYd") (width 0.05))
     (fp_line (start 14.25 -8.75) (end 14.25 3.75) (layer "B.CrtYd") (width 0.05))
     (fp_line (start -1.77 3.75) (end -1.77 -8.75) (layer "B.CrtYd") (width 0.05))
-    (fp_line (start -1.77 3.75) (end 14.25 3.75) (layer "B.CrtYd") (width 0.05))
+    (fp_line (start 14.25 -8.75) (end -1.77 -8.75) (layer "B.CrtYd") (width 0.05))
+    (fp_line (start 0.25 -8.5) (end 12.25 -8.5) (layer "B.Fab") (width 0.1))
     (fp_line (start 0.25 3.5) (end 0.25 -8.5) (layer "B.Fab") (width 0.1))
-    (fp_line (start 0.25 3.5) (end 12.25 3.5) (layer "B.Fab") (width 0.1))
     (fp_line (start 12.25 3.5) (end 12.25 -8.5) (layer "B.Fab") (width 0.1))
-    (fp_line (start 0.25 -8.5) (end 12.25 -8.5) (layer "B.Fab") (width 0.1))
+    (fp_line (start 0.25 3.5) (end 12.25 3.5) (layer "B.Fab") (width 0.1))
     (pad "1" thru_hole oval (at 0 0 180) (size 3.048 1.85) (drill 1.3) (layers *.Cu *.Mask)
       (net 69 "Switch_Mute") (pintype "passive"))
-    (pad "1" thru_hole oval (at 12.5 0 180) (size 3.048 1.85) (drill 1.3) (layers *.Cu *.Mask)
-      (net 69 "Switch_Mute") (pintype "passive"))
-    (pad "2" thru_hole oval (at 0 -5 180) (size 3.048 1.85) (drill 1.3) (layers *.Cu *.Mask)
-      (net 69 "Switch_Mute") (pintype "passive"))
-    (pad "2" thru_hole oval (at 12.5 -5 180) (size 3.048 1.85) (drill 1.3) (layers *.Cu *.Mask)
+    (pad "2" thru_hole oval (at 12.5 0 180) (size 3.048 1.85) (drill 1.3) (layers *.Cu *.Mask)
       (net 69 "Switch_Mute") (pintype "passive"))
-    (model "${KICAD6_3DMODEL_DIR}/Button_Switch_THT.3dshapes/SW_PUSH-12mm.wrl"
-      (offset (xyz 0 0 0))
+    (pad "3" thru_hole oval (at 0 -5 180) (size 3.048 1.85) (drill 1.3) (layers *.Cu *.Mask)
+      (net 2 "GND") (pintype "passive"))
+    (pad "4" thru_hole oval (at 12.5 -5 180) (size 3.048 1.85) (drill 1.3) (layers *.Cu *.Mask)
+      (net 2 "GND") (pintype "passive"))
+    (model "${KIPRJMOD}/Parts/12mmx12mm With Green cap.stp"
+      (offset (xyz 6.25 -2.5 0))
       (scale (xyz 1 1 1))
       (rotate (xyz 0 0 0))
