File: Hardware/GeneralPurposeAlarmDevicePCB/GeneralPurposeAlarmDevicePCB/GeneralPurposeAlarmDevicePCB.kicad_pcb (KiCad board)
At the start: 2 copper layers, 137.2 x 83.8 mm, 123 parts, among them J101 Barrel_Jack_Switch_SMT, J102 0.100_2Pin, J103 0.100_2Pin, J105 S04B-XASK-1(LF)(SN), J401 RJ12_6P6C_HORZ, J501 USB_B_Micro, J601 22-23-2021, Q201 MMBT2222A-7-F, Q202 MMBT2222A-7-F, Q203 MMBT2222A-7-F, Q204 MMBT2222A-7-F, Q205 MMBT2222A-7-F, Q301 BSS138, Q601 MMBT2222A-7-F, Q602 MMBT2907ALT1G, U101 LM7805_TO220, U102 PI_ATMEGA328P-AU-InOrder, U301 PCF8574AT, U302 LCD_20x4_Character-GPAD_SCH_L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, U501 CH340E

Commit message: Route some power. Move transistors and resistors near LEDs for signall access.
Parts:
- moved R310 37.4 mm to (171.4, 27.9), turned to 0 degrees
- moved R503 35.3 mm to (118.7, 51.4), turned to 0 degrees
- moved D102 18.9 mm to (81.3, 65.4), turned to 90 degrees
- moved R101 14.2 mm to (127.0, 61.6)
- moved TP103 12.1 mm to (190.5, 49.5)
- moved R207 10.2 mm to (73.7, 40.6), turned to 90 degrees
- moved R203 9.25 mm to (73.7, 66.0), turned to 90 degrees
- moved R209 9.25 mm to (73.7, 27.9), turned to 90 degrees
- moved R205 9.05 mm to (73.7, 53.3), turned to 90 degrees
- moved R201 8.98 mm to (73.7, 78.7), turned to 90 degrees
- moved R202 8.03 mm to (73.7, 74.9), turned to -90 degrees
- moved R204 8.03 mm to (73.7, 62.2), turned to -90 degrees
- moved R208 7.43 mm to (73.7, 36.2), turned to -90 degrees
- moved Q202 6.87 mm to (70.5, 66.0), turned to 180 degrees
- moved Q203 6.87 mm to (70.5, 53.3), turned to 180 degrees
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Routing:
- net +5V: track 0.00 -> 352.8 mm
- net VccController: track 0.00 -> 30.1 mm
- net GND: track 0.00 -> 27.3 mm, vias 0 -> 6
- net VBus: track 0.00 -> 9.61 mm
- net Net-(D105-Pad2): track 0.00 -> 7.58 mm

Commit message: Update crystal footprint for proper SMT. Position compoonents for routing. Add resistor to attenuate audio.
Parts:
- added R505: 10K, Resistor_SMD:R_0603_1608Metric_Pad0.98x0.95mm_HandSolder, F.Cu at (59.1, 89.5)
- C104: footprint Capacitor_SMD:C_0603_1608Metric -> Capacitor_SMD:C_0603_1608Metric_Pad1.08x0.95mm_HandSolder
- C113, C114: value 33pF -> 39pF
- C601: value 47uF -> 47uF 16V
- J501: value USB_B_Micro -> USB_B_Micro_Local
- R101, R102, R103, R104, R105, R106, R107, R108, R109, R110, R111, R201, R202, R203, R204, R205, R206, R207, R208, R209, R210, R301, R302, R303, R304, R305, R306, R307, R308, R309, R310, R311, R401, R402, R403, R404, R501, R502, R503, R504, R601, R602, R603, R604, R605: footprint Resistor_SMD:R_0603_1608Metric -> Resistor_SMD:R_0603_1608Metric_Pad0.98x0.95mm_HandSolder
- XTAL101: footprint digikey-footprints:SMD-2_3.2x2.5mm -> Crystal:Crystal_SMD_HC49-SD
- moved G*** 40.4 mm to (92.7, 29.2)
- moved Graphic1 27.7 mm to (82.5, 28.6)
- moved R103 23.1 mm to (83.2, 72.4)
- moved J102 21.0 mm to (97.2, 98.4), turned to 90 degrees
- moved R111 12.1 mm to (127.0, 67.9)
- moved R308 10.5 mm to (178.4, 38.7)
- moved R306 10.5 mm to (178.4, 42.0)
- moved R601 9.25 mm to (62.9, 73.0)
- moved C105 7.01 mm to (181.6, 83.8)
- moved C108 4.96 mm to (185.4, 83.8), turned to 180 degrees
- moved XTAL101 4.62 mm to (99.1, 41.9), turned to 180 degrees
- moved C113 4.26 mm to (137.8, 85.7), turned to 180 degrees
- moved R109 4.05 mm to (117.5, 63.5)
- moved C114 3.86 mm to (134.0, 85.7)
- moved R102 3.81 mm to (121.9, 59.7)
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Routing:
- net +5V: track 352.8 -> 372.6 mm
- net VBus: track 9.61 -> 14.0 mm
Other:
- board text added: "CERN Open Hardware License Version 2 - Strongly Reciprocal"
- board text added: "SN:______________________"
- board text removed: "SN:"

Commit message: Begining routing near uController and LCD.
Parts:
- moved R105 7.67 mm to (139.7, 44.5)
- moved D103 7.04 mm to (121.5, 74.9)
- moved R104 6.54 mm to (139.7, 41.3)
- moved R102 6.14 mm to (122.8, 65.8)
- moved C110 6.14 mm to (125.2, 65.8)
- moved R111 4.32 mm to (127.9, 72.2)
- moved C104 4.32 mm to (108.8, 50.6)
- moved XTAL101 4.32 mm to (99.9, 46.1)
- moved C103 4.32 mm to (111.4, 50.0)
- moved C106 4.32 mm to (111.4, 45.5)
- moved C107 4.32 mm to (105.7, 52.5)
- moved C112 4.32 mm to (110.7, 69.0)
- moved R101 4.32 mm to (127.9, 67.7)
- moved R108 4.32 mm to (118.5, 64.6)
- moved R109 4.32 mm to (118.3, 67.7)
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Routing:
- net /LCD And I2C Interface/Vcc_LCD: track 0.00 -> 123.0 mm, vias 0 -> 2
- net ControllerRX: track 0.00 -> 56.7 mm
- net SDA: track 0.00 -> 52.5 mm, vias 0 -> 1
- net ControllerTX: track 0.00 -> 50.9 mm
- net SCL: track 0.00 -> 50.3 mm
- net Vin: track 0.00 -> 48.2 mm, vias 0 -> 1
- net Switch_Mute: track 0.00 -> 47.2 mm
- net Attenuate: track 0.00 -> 46.7 mm
- net Light0: track 0.00 -> 45.3 mm
- net Net-(Q301-Pad1): track 0.00 -> 44.0 mm, vias 0 -> 2
- net Net-(R306-Pad1): track 0.00 -> 43.9 mm, vias 0 -> 2
- net VccController: track 30.1 -> 71.8 mm
- net PC3: track 0.00 -> 34.1 mm
- net PC0: track 0.00 -> 32.6 mm
- net PC2: track 0.00 -> 31.9 mm
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
Commit message: Begining routing near bottom connectors.
Parts:
- moved R403 3.17 mm to (148.6, 83.2)
- moved R404 3.17 mm to (151.8, 83.2)
- moved D103 2.17 mm to (122.6, 73.0)
- moved R108 1.48 mm to (118.5, 66.0)
- moved C101 1.40 mm to (172.7, 87.8)
- moved R503 0.63 mm to (119.6, 54.0)
- turned F401 to 90 degrees
Routing:
- net nCS: track 21.1 -> 120.4 mm
- net CIPO: track 24.7 -> 97.7 mm, vias 0 -> 2
- net COPI: track 24.0 -> 89.1 mm, vias 0 -> 2
- net +5V: track 358.2 -> 421.7 mm, vias 0 -> 3
- net SPI_SCK: track 26.8 -> 89.2 mm
- net Net-(C114-Pad1): track 0.00 -> 61.6 mm, vias 0 -> 5
- net Net-(C113-Pad1): track 0.00 -> 60.8 mm, vias 0 -> 6
- net GND: track 55.1 -> 99.9 mm, vias 18 -> 31
- net Net-(R503-Pad2): track 0.00 -> 44.4 mm, vias 0 -> 6
- net Vin: track 48.2 -> 88.3 mm
- net ControllerRX: track 56.7 -> 89.0 mm, vias 0 -> 6
- net nRESET: track 22.7 -> 52.3 mm, vias 2 -> 7
- net Net-(C101-Pad1): track 0.00 -> 16.1 mm
- net VccController: track 71.8 -> 86.4 mm, vias 0 -> 2
- net ControllerVcc: track 0.00 -> 12.2 mm, vias 0 -> 1
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
Commit message: Almost all routed. The LEDs next.
Parts:
- moved R603 47.4 mm to (98.4, 87.6), turned to 0 degrees
- moved R109 27.1 mm to (140.0, 51.4)
- moved R108 27.1 mm to (140.1, 49.7)
- moved R605 3.59 mm to (83.8, 50.8), turned to -90 degrees
- moved R602 2.84 mm to (83.8, 58.4), turned to -90 degrees
- moved D102 1.80 mm to (82.5, 67.9), turned to -90 degrees
- moved R103 0.64 mm to (83.2, 71.8)
Routing:
- net SCL: track 50.3 -> 170.1 mm, vias 0 -> 2
- net SDA: track 52.5 -> 159.6 mm, vias 1 -> 2
- net Switch_Mute: track 47.2 -> 126.4 mm, vias 0 -> 3
- net Light0: track 45.3 -> 120.3 mm, vias 0 -> 2
- net VccController: track 86.4 -> 151.5 mm, vias 2 -> 5
- net Net-(Q601-Pad1): track 0.00 -> 63.5 mm, vias 0 -> 3
- net +5V: track 421.7 -> 463.7 mm
- net Net-(BZ601-Pad1): track 0.00 -> 19.8 mm, vias 0 -> 1
- net /AlarmAudio/VccBuzzer: track 0.00 -> 19.4 mm
- net Net-(C503-Pad1): track 0.00 -> 10.3 mm
- net VBus: track 14.0 -> 23.7 mm
- net Net-(R504-Pad2): track 0.00 -> 8.38 mm
- net GND: track 99.9 -> 108.2 mm, vias 31 -> 35
- net Net-(Q601-Pad2): track 0.00 -> 6.76 mm
- net Net-(J501-Pad3): track 0.00 -> 6.36 mm, vias 0 -> 2
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
Commit message: Almost all but ground pours.
Routing:
- net Light4: track 23.2 -> 90.3 mm, vias 0 -> 5
- net Light1: track 22.5 -> 72.8 mm, vias 0 -> 3
- net Light3: track 22.5 -> 56.6 mm, vias 0 -> 3
- net Light2: track 21.8 -> 35.8 mm, vias 0 -> 1
- net Net-(D202-Pad2): track 0.00 -> 4.49 mm
- net Net-(Q601-Pad1): track 63.5 -> 63.6 mm, vias 3 -> 4

Commit message: Add ground pours. ABout 7 DRC reported.
Parts:
- moved C501 1.50 mm to (106.7, 90.2), turned to -90 degrees
- moved C502 1.37 mm to (116.8, 90.8), turned to -90 degrees
Routing:
- net GND: track 108.2 -> 120.3 mm, vias 35 -> 71
- net VBus: track 23.7 -> 31.3 mm
- net +5V: track 463.7 -> 459.4 mm
- net Net-(Q601-Pad1): track 63.6 -> 67.6 mm
- net VccController: track 151.5 -> 148.4 mm, vias 5 -> 4
- net nCS: track 123.3 -> 126.3 mm
- net Light4: track 90.3 -> 88.0 mm, vias 5 -> 3
- net Light3: track 56.6 -> 58.8 mm
- net /LCD And I2C Interface/Vcc_LCD: track 123.0 -> 121.2 mm
- net Net-(A101-Pad3): track 8.35 -> 9.19 mm
- net Net-(C114-Pad1): track 61.6 -> 60.9 mm
- net Net-(C113-Pad1): track 60.8 -> 60.1 mm, vias 6 -> 5
- net Net-(R503-Pad2): track 44.4 -> 45.1 mm
- net Net-(Q301-Pad1): track 44.0 -> 43.4 mm
- net PC0: track 30.4 -> 31.0 mm
- added copper zone on B.Cu, net GND
- added copper zone on F.Cu, net GND

Commit message: PCB routed and no DRC errors not waved. One warning about the open hardware on the silk screen.
Parts:
- moved R105 1.90 mm to (139.7, 46.4)
Routing:
- net GND: track 120.3 -> 148.4 mm, vias 71 -> 93
- net Light0: track 120.3 -> 116.2 mm
- net VccController: track 148.4 -> 151.5 mm
- net SDA: track 159.9 -> 157.3 mm
- net Net-(C114-Pad1): track 60.9 -> 59.2 mm
- net Light4: track 88.0 -> 86.8 mm
- net SCL: track 170.2 -> 169.5 mm
- net ControllerRX: track 89.3 -> 89.9 mm
- net PC3: track 34.1 -> 33.5 mm
- net ControllerTX: track 50.9 -> 50.4 mm
- net Light1: track 73.1 -> 73.7 mm
