File: Hardware/GeneralPurposeAlarmDevicePCB/GeneralPurposeAlarmDevicePCB/SPI Peripherial.sch (KiCad schematic (older format))
At the start: 5 parts

Commit message: Add more parts drawings, buzzer. Add additional schematic sheet for AlarmAudio.
Connections:
- net CIPO: now reaches R?.1
- net SCK: now reaches R?.1
- net COPI: now reaches R?.1
- net nCS: now reaches R?.1
- net ControllerVcc: now reaches J?.5
Other:
- moved on the sheet: R?
Changed lines of the file:
@@
 $Descr USLetter 11000 8500
 encoding utf-8
-Sheet 4 5
+Sheet 4 6
 Title "GeneralPurposeAlarmDevicePCB"
 Date "2022-06-20"
@@
 L Device:R R?
 U 1 1 62B96D7C
-P 7100 4550
+P 7300 4850
 AR Path="/62B96D7C" Ref="R?"  Part="1"
 AR Path="/62B93801/62B96D7C" Ref="R?"  Part="1"
-F 0 "R?" V 6900 4500 50  0000 C CNN
-F 1 "330R" V 7000 4550 50  0000 C CNN
-F 2 "Resistor_SMD:R_0603_1608Metric" V 7030 4550 50  0001 C CNN
-F 3 "~" H 7100 4550 50  0001 C CNN
-F 4 "JLCPCB" V 7100 4550 50  0001 C CNN "Distributor 1"
-F 5 "C269711" V 7100 4550 50  0001 C CNN "Distributor 1 PN"
-F 6 "TyoHM" V 7100 4550 50  0001 C CNN "Manufacturer"
-F 7 "RMC06033301%N" V 7100 4550 50  0001 C CNN "MPN"
-F 8 "0.1W ±1% 330Ω 0603 Chip Resistor - Surface Mount ROHS" H 7100 4550 50  0001 C CNN "Description"
-	1    7100 4550
+F 0 "R?" V 7100 4800 50  0000 C CNN
+F 1 "330R" V 7200 4850 50  0000 C CNN
+F 2 "Resistor_SMD:R_0603_1608Metric" V 7230 4850 50  0001 C CNN
+F 3 "~" H 7300 4850 50  0001 C CNN
+F 4 "JLCPCB" V 7300 4850 50  0001 C CNN "Distributor 1"
+F 5 "C269711" V 7300 4850 50  0001 C CNN "Distributor 1 PN"
+F 6 "TyoHM" V 7300 4850 50  0001 C CNN "Manufacturer"
+F 7 "RMC06033301%N" V 7300 4850 50  0001 C CNN "MPN"
+F 8 "0.1W ±1% 330Ω 0603 Chip Resistor - Surface Mount ROHS" H 7300 4850 50  0001 C CNN "Description"
+	1    7300 4850
 	0    1    1    0
 $EndComp
@@
 Wire Wire Line
 	4500 3950 5050 3950
+Text HLabel 7750 4450 2    50   Input ~ 0
+COPI
+Text HLabel 7800 3850 2    50   Output ~ 0
+CIPO
+Text HLabel 7750 4300 2    50   Input ~ 0
+SCK
+Text HLabel 7750 4850 2    50   Input ~ 0
+nCS
 Wire Wire Line
-	4500 4550 6950 4550
+	5750 4200 7500 4200
+Wire Wire Line
+	7500 4200 7500 4300
+Wire Wire Line
+	7500 4300 7750 4300
+Wire Wire Line
+	5350 3950 7500 3950
+Wire Wire Line
+	6200 4450 7750 4450
+Wire Wire Line
+	7000 4550 7000 4850
+Wire Wire Line
+	7000 4850 7150 4850
+Wire Wire Line
+	4500 4550 7000 4550
+Wire Wire Line
+	7450 4850 7750 4850
+Wire Wire Line
+	7500 3950 7500 3850
+Wire Wire Line
+	7500 3850 7800 3850
+Wire Wire Line
+	4500 4050 7800 4050
+Text HLabel 7800 4050 2    50   UnSpc ~ 0
+ControllerVcc
 $EndSCHEMATC

Commit message: Annote reference designators.
Parts:
- gave numbers to parts that had none: 5
Changed lines of the file:
@@
 P 5200 3950
 AR Path="/62B96D5B" Ref="R?"  Part="1"
-AR Path="/62B93801/62B96D5B" Ref="R?"  Part="1"
-F 0 "R?" V 5000 3900 50  0000 C CNN
+AR Path="/62B93801/62B96D5B" Ref="R401"  Part="1"
+F 0 "R401" V 5000 3900 50  0000 C CNN
 F 1 "330R" V 5100 3950 50  0000 C CNN
 F 2 "Resistor_SMD:R_0603_1608Metric" V 5130 3950 50  0001 C CNN
@@
 P 5600 4200
 AR Path="/62B96D66" Ref="R?"  Part="1"
-AR Path="/62B93801/62B96D66" Ref="R?"  Part="1"
-F 0 "R?" V 5400 4150 50  0000 C CNN
+AR Path="/62B93801/62B96D66" Ref="R402"  Part="1"
+F 0 "R402" V 5400 4150 50  0000 C CNN
 F 1 "330R" V 5500 4200 50  0000 C CNN
 F 2 "Resistor_SMD:R_0603_1608Metric" V 5530 4200 50  0001 C CNN
@@
 P 6050 4450
 AR Path="/62B96D71" Ref="R?"  Part="1"
-AR Path="/62B93801/62B96D71" Ref="R?"  Part="1"
-F 0 "R?" V 5850 4400 50  0000 C CNN
+AR Path="/62B93801/62B96D71" Ref="R403"  Part="1"
+F 0 "R403" V 5850 4400 50  0000 C CNN
 F 1 "330R" V 5950 4450 50  0000 C CNN
 F 2 "Resistor_SMD:R_0603_1608Metric" V 5980 4450 50  0001 C CNN
@@
 P 7300 4850
 AR Path="/62B96D7C" Ref="R?"  Part="1"
-AR Path="/62B93801/62B96D7C" Ref="R?"  Part="1"
-F 0 "R?" V 7100 4800 50  0000 C CNN
+AR Path="/62B93801/62B96D7C" Ref="R404"  Part="1"
+F 0 "R404" V 7100 4800 50  0000 C CNN
 F 1 "330R" V 7200 4850 50  0000 C CNN
 F 2 "Resistor_SMD:R_0603_1608Metric" V 7230 4850 50  0001 C CNN
@@
 P 4100 4250
 AR Path="/62B96D82" Ref="J?"  Part="1"
-AR Path="/62B93801/62B96D82" Ref="J?"  Part="1"
-F 0 "J?" H 4157 4817 50  0000 C CNN
+AR Path="/62B93801/62B96D82" Ref="J401"  Part="1"
+F 0 "J401" H 4157 4817 50  0000 C CNN
 F 1 "RJ12" H 4157 4726 50  0000 C CNN
 F 2 "" V 4100 4275 50  0001 C CNN
@@
 P 4850 4250
 AR Path="/62B96D89" Ref="#PWR?"  Part="1"
-AR Path="/62B93801/62B96D89" Ref="#PWR?"  Part="1"
-F 0 "#PWR?" H 4850 4000 50  0001 C CNN
+AR Path="/62B93801/62B96D89" Ref="#PWR0401"  Part="1"
+F 0 "#PWR0401" H 4850 4000 50  0001 C CNN
 F 1 "GND" H 4950 4250 50  0000 C CNN
 F 2 "" H 4850 4250 50  0001 C CNN

Commit message: Pull parts into PCB Begin rough placement into groups.
Parts:
- J401: footprint (none) -> Connector_RJ:RJ12_Amphenol_54601; Distributor 1 (none) -> JLCPCB; Distributor 1 PN (none) -> C305981; MPN (none) -> 5555165-1; Manufacturer (none) -> TE Connectivity
Changed lines of the file:
@@
 F 0 "J401" H 4157 4817 50  0000 C CNN
 F 1 "RJ12" H 4157 4726 50  0000 C CNN
-F 2 "" V 4100 4275 50  0001 C CNN
-F 3 "~" V 4100 4275 50  0001 C CNN
+F 2 "Connector_RJ:RJ12_Amphenol_54601" V 4100 4275 50  0001 C CNN
+F 3 "https://datasheet.lcsc.com/lcsc/1811141146_TE-Connectivity-5555165-1_C305981.pdf" V 4100 4275 50  0001 C CNN
+F 4 "TE Connectivity" H 4100 4250 50  0001 C CNN "Manufacturer"
+F 5 "JLCPCB" H 4100 4250 50  0001 C CNN "Distributor 1"
+F 6 "C305981" H 4100 4250 50  0001 C CNN "Distributor 1 PN"
+F 7 "5555165-1" H 4100 4250 50  0001 C CNN "MPN"
 	1    4100 4250
 	1    0    0    -1

Commit message: Add new LED, RJ12 footprints to footprint library. Add STEP model.
Parts:
- removed J401: RJ12, Connector_RJ:RJ12_Amphenol_54601, symbol Connector:RJ12
- added J401: RJ12_6P6C_HORZ, GeneralPurposeAlarmDevicePCB:RJ12_Amphenol_54601, symbol GPAD_SCH_LIB:RJ12_6P6C_HORZ
- R401, R402, R403, R404: value 330R -> R
Connections:
- net ControllerVcc: now also J401.5
- net GND: now also J401.3
- net at R401.2: now also J401.6
- net at R402.2: now also J401.4
- net at R403.2: now also J401.2
- net at R404.2: now also J401.1
Changed lines of the file:
@@
 AR Path="/62B93801/62B96D5B" Ref="R401"  Part="1"
 F 0 "R401" V 5000 3900 50  0000 C CNN
-F 1 "330R" V 5100 3950 50  0000 C CNN
+F 1 "R" V 5100 3950 50  0000 C CNN
 F 2 "Resistor_SMD:R_0603_1608Metric" V 5130 3950 50  0001 C CNN
 F 3 "~" H 5200 3950 50  0001 C CNN
@@
 AR Path="/62B93801/62B96D66" Ref="R402"  Part="1"
 F 0 "R402" V 5400 4150 50  0000 C CNN
-F 1 "330R" V 5500 4200 50  0000 C CNN
+F 1 "R" V 5500 4200 50  0000 C CNN
 F 2 "Resistor_SMD:R_0603_1608Metric" V 5530 4200 50  0001 C CNN
 F 3 "~" H 5600 4200 50  0001 C CNN
@@
 AR Path="/62B93801/62B96D71" Ref="R403"  Part="1"
 F 0 "R403" V 5850 4400 50  0000 C CNN
-F 1 "330R" V 5950 4450 50  0000 C CNN
+F 1 "R" V 5950 4450 50  0000 C CNN
 F 2 "Resistor_SMD:R_0603_1608Metric" V 5980 4450 50  0001 C CNN
 F 3 "~" H 6050 4450 50  0001 C CNN
@@
 AR Path="/62B93801/62B96D7C" Ref="R404"  Part="1"
 F 0 "R404" V 7100 4800 50  0000 C CNN
-F 1 "330R" V 7200 4850 50  0000 C CNN
+F 1 "R" V 7200 4850 50  0000 C CNN
 F 2 "Resistor_SMD:R_0603_1608Metric" V 7230 4850 50  0001 C CNN
 F 3 "~" H 7300 4850 50  0001 C CNN
@@
 	1    7300 4850
 	0    1    1    0
-$EndComp
-$Comp
-L Connector:RJ12 J?
-U 1 1 62B96D82
-P 4100 4250
-AR Path="/62B96D82" Ref="J?"  Part="1"
-AR Path="/62B93801/62B96D82" Ref="J401"  Part="1"
-F 0 "J401" H 4157 4817 50  0000 C CNN
-F 1 "RJ12" H 4157 4726 50  0000 C CNN
-F 2 "Connector_RJ:RJ12_Amphenol_54601" V 4100 4275 50  0001 C CNN
-F 3 "https://datasheet.lcsc.com/lcsc/1811141146_TE-Connectivity-5555165-1_C305981.pdf" V 4100 4275 50  0001 C CNN
-F 4 "TE Connectivity" H 4100 4250 50  0001 C CNN "Manufacturer"
-F 5 "JLCPCB" H 4100 4250 50  0001 C CNN "Distributor 1"
-F 6 "C305981" H 4100 4250 50  0001 C CNN "Distributor 1 PN"
-F 7 "5555165-1" H 4100 4250 50  0001 C CNN "MPN"
-	1    4100 4250
-	1    0    0    -1
 $EndComp
 Text Notes 3800 3600 0    50   ~ 0
@@
 Text HLabel 7800 4050 2    50   UnSpc ~ 0
 ControllerVcc
+$Comp
+L GPAD_SCH_LIB:RJ12_6P6C_HORZ J401
+U 1 1 62D0D90D
+P 4100 4250
+F 0 "J401" H 4157 4907 50  0000 C CNN
+F 1 "RJ12_6P6C_HORZ" H 4157 4816 50  0000 C CNN
+F 2 "GeneralPurposeAlarmDevicePCB:RJ12_Amphenol_54601" V 4100 4275 50  0001 C CNN
+F 3 "https://datasheet.lcsc.com/lcsc/1811141146_TE-Connectivity-5555165-1_C305981.pdf" V 4100 4275 50  0001 C CNN
+F 4 "JLCPCB" H 4100 4250 50  0001 C CNN "Distributor 1"
+F 5 "C305981" H 4100 4250 50  0001 C CNN "Distributor 1 PN"
+F 6 "Digikey" H 4100 4250 50  0001 C CNN "Distributor 2"
+F 7 "A31422-ND" H 4100 4250 50  0001 C CNN "Distributor 2 PN"
+F 8 "TE Connectivity" H 4100 4250 50  0001 C CNN "Manufacturer"
+F 9 "Jack Modular Connector 6p6c (RJ11, RJ12, RJ14, RJ25) 90° Angle (Right) Unshielded Cat3" H 4100 4250 50  0001 C CNN "Description"
+F 10 "HAND" H 4157 4725 50  0000 C CNN "AssemblyType"
+F 11 "5555165-1" H 4100 4250 50  0001 C CNN "MPN"
+	1    4100 4250
+	1    0    0    -1
+$EndComp
 $EndSCHEMATC

Commit message: Add current limit to CongtollerVcc, and Barrel Input. Add jumper resistors for headers selecting VBus and ControllerVcc.
Parts:
- R401, R402, R403, R404: value R -> 330

Commit message: Update schottky symbol and part number. Import to PCB. Only the Arduino UNO symbol remains to connect.
Parts:
- added F401: Polyfuse_Small, Fuse:Fuse_0603_1608Metric, symbol Device:Polyfuse_Small
Connections:
- net ControllerVcc: now also F401.1; no longer J401.5
- new net: F401.2, J401.5
Changed lines of the file:
@@
 Wire Wire Line
 	7500 3850 7800 3850
-Wire Wire Line
-	4500 4050 7800 4050
 Text HLabel 7800 4050 2    50   UnSpc ~ 0
 ControllerVcc
@@
 EndData
 $EndBitmap
+Wire Wire Line
+	7450 4050 7800 4050
+Wire Wire Line
+	7250 4050 4500 4050
+$Comp
+L Device:Polyfuse_Small F?
+U 1 1 630AB448
+P 7350 4050
+AR Path="/630AB448" Ref="F?"  Part="1"
+AR Path="/62B93801/630AB448" Ref="F401"  Part="1"
+F 0 "F401" V 7145 4050 50  0000 C CNN
+F 1 "Polyfuse_Small" V 7450 4100 50  0000 C CNN
+F 2 "Fuse:Fuse_0603_1608Metric" H 7400 3850 50  0001 L CNN
+F 3 "https://datasheet.lcsc.com/lcsc/1806131741_Littelfuse-0603L075SLYR_C207016.pdf" H 7350 4050 50  0001 C CNN
+F 4 "Littelfuse" V 7350 4050 50  0001 C CNN "Manufacturier"
+F 5 "0603L100SLYR" V 7350 4050 50  0001 C CNN "MPN"
+	1    7350 4050
+	0    1    1    0
+$EndComp
 $EndSCHEMATC

Commit message: Clean up a bunch of duplicate because of missspelled part field names. Still working on a few sch, pcb and 3D libraries.
Parts:
- F401: Manufacturer (none) -> Littelfuse; Manufacturier Littelfuse -> (none)
- J401: Assembly Type (none) -> HAND; AssemblyType HAND -> (none)
Changed lines of the file:
@@
 F 8 "TE Connectivity" H 4100 4250 50  0001 C CNN "Manufacturer"
 F 9 "Jack Modular Connector 6p6c (RJ11, RJ12, RJ14, RJ25) 90° Angle (Right) Unshielded Cat3" H 4100 4250 50  0001 C CNN "Description"
-F 10 "HAND" H 4157 4725 50  0000 C CNN "AssemblyType"
+F 10 "HAND" H 4157 4725 50  0000 C CNN "Assembly Type"
 F 11 "5555165-1" H 4100 4250 50  0001 C CNN "MPN"
 	1    4100 4250
@@
 F 2 "Fuse:Fuse_0603_1608Metric" H 7400 3850 50  0001 L CNN
 F 3 "https://datasheet.lcsc.com/lcsc/1806131741_Littelfuse-0603L075SLYR_C207016.pdf" H 7350 4050 50  0001 C CNN
-F 4 "Littelfuse" V 7350 4050 50  0001 C CNN "Manufacturier"
+F 4 "Littelfuse" V 7350 4050 50  0001 C CNN "Manufacturer"
 F 5 "0603L100SLYR" V 7350 4050 50  0001 C CNN "MPN"
 	1    7350 4050
