File: Hardware/GeneralPurposeAlarmDevicePCB/GeneralPurposeAlarmDevicePCB/AlarmAudio.sch (KiCad schematic (older format))
At the start: 6 parts

Commit message: Annote reference designators.
Parts:
- gave numbers to parts that had none: 6
Changed lines of the file:
@@
 $EndDescr
 $Comp
-L dk_Alarms-Buzzers-and-Sirens:PKMCS0909E4000-R1 BZ?
+L dk_Alarms-Buzzers-and-Sirens:PKMCS0909E4000-R1 BZ601
 U 1 1 62DD9B52
 P 7500 3550
-F 0 "BZ?" H 7840 3658 60  0000 L CNN
+F 0 "BZ601" H 7840 3658 60  0000 L CNN
 F 1 "PKMCS0909E4000-R1" H 7840 3552 60  0000 L CNN
 F 2 "digikey-footprints:Piezo_9x9mm_PKMCS0909E4000-R1" H 7700 3750 60  0001 L CNN
@@
 P 4550 2800
 AR Path="/62B3AC2F/62DE23F8" Ref="R?"  Part="1"
-AR Path="/62DD8E5F/62DE23F8" Ref="R?"  Part="1"
-F 0 "R?" V 4650 2850 50  0000 C CNN
+AR Path="/62DD8E5F/62DE23F8" Ref="R602"  Part="1"
+F 0 "R602" V 4650 2850 50  0000 C CNN
 F 1 "330R" V 4400 2800 50  0000 C CNN
 F 2 "Resistor_SMD:R_0603_1608Metric" V 4480 2800 50  0001 C CNN
@@
 P 5300 2400
 AR Path="/62B3AC2F/62DE2407" Ref="Q?"  Part="1"
-AR Path="/62DD8E5F/62DE2407" Ref="Q?"  Part="1"
-F 0 "Q?" H 5488 2453 60  0000 L CNN
+AR Path="/62DD8E5F/62DE2407" Ref="Q601"  Part="1"
+F 0 "Q601" H 5488 2453 60  0000 L CNN
 F 1 "MMBT2222A-7-F" H 5488 2347 60  0000 L CNN
 F 2 "digikey-footprints:SOT-23-3" H 5500 2600 60  0001 L CNN
@@
 $EndComp
 $Comp
-L dk_Transistors-Bipolar-BJT-Single:MMBT2907ALT1G Q?
+L dk_Transistors-Bipolar-BJT-Single:MMBT2907ALT1G Q602
 U 1 1 62DE3E9B
 P 5300 3050
-F 0 "Q?" H 5488 3103 60  0000 L CNN
+F 0 "Q602" H 5488 3103 60  0000 L CNN
 F 1 "MMBT2907ALT1G" H 5488 2997 60  0000 L CNN
 F 2 "digikey-footprints:SOT-23-3" H 5500 3250 60  0001 L CNN
@@
 P 2850 2100
 AR Path="/62DE752C" Ref="C?"  Part="1"
-AR Path="/62DD8E5F/62DE752C" Ref="C?"  Part="1"
-F 0 "C?" H 2968 2146 50  0000 L CNN
+AR Path="/62DD8E5F/62DE752C" Ref="C601"  Part="1"
+F 0 "C601" H 2968 2146 50  0000 L CNN
 F 1 "47uF 16V" H 2968 2055 50  0000 L CNN
 F 2 "Capacitor_SMD:CP_Elec_5x5.4" H 2888 1950 50  0001 C CNN
@@
 P 2850 2300
 AR Path="/62DE7532" Ref="#PWR?"  Part="1"
-AR Path="/62DD8E5F/62DE7532" Ref="#PWR?"  Part="1"
-F 0 "#PWR?" H 2850 2050 50  0001 C CNN
+AR Path="/62DD8E5F/62DE7532" Ref="#PWR0602"  Part="1"
+F 0 "#PWR0602" H 2850 2050 50  0001 C CNN
 F 1 "GND" H 2855 2127 50  0000 C CNN
 F 2 "" H 2850 2300 50  0001 C CNN
@@
 P 5400 3400
 AR Path="/62DE76BB" Ref="#PWR?"  Part="1"
-AR Path="/62DD8E5F/62DE76BB" Ref="#PWR?"  Part="1"
-F 0 "#PWR?" H 5400 3150 50  0001 C CNN
+AR Path="/62DD8E5F/62DE76BB" Ref="#PWR0603"  Part="1"
+F 0 "#PWR0603" H 5400 3150 50  0001 C CNN
 F 1 "GND" H 5405 3227 50  0000 C CNN
 F 2 "" H 5400 3400 50  0001 C CNN
@@
 AR Path="/62DEA4D3" Ref="R?"  Part="1"
 AR Path="/62B871EE/62DEA4D3" Ref="R?"  Part="1"
-AR Path="/62DD8E5F/62DEA4D3" Ref="R?"  Part="1"
-F 0 "R?" V 1950 1850 50  0000 C CNN
+AR Path="/62DD8E5F/62DEA4D3" Ref="R601"  Part="1"
+F 0 "R601" V 1950 1850 50  0000 C CNN
 F 1 "1R0" V 2050 1900 50  0000 C CNN
 F 2 "Resistor_SMD:R_0603_1608Metric" V 2080 1900 50  0001 C CNN
@@
 AR Path="/62DEA4D9" Ref="#PWR?"  Part="1"
 AR Path="/62B871EE/62DEA4D9" Ref="#PWR?"  Part="1"
-AR Path="/62DD8E5F/62DEA4D9" Ref="#PWR?"  Part="1"
-F 0 "#PWR?" H 1400 1750 50  0001 C CNN
+AR Path="/62DD8E5F/62DEA4D9" Ref="#PWR0601"  Part="1"
+F 0 "#PWR0601" H 1400 1750 50  0001 C CNN
 F 1 "+5V" H 1415 2073 50  0000 C CNN
 F 2 "" H 1400 1900 50  0001 C CNN
@@
 P 6900 3750
 AR Path="/62DECBDB" Ref="#PWR?"  Part="1"
-AR Path="/62DD8E5F/62DECBDB" Ref="#PWR?"  Part="1"
-F 0 "#PWR?" H 6900 3500 50  0001 C CNN
+AR Path="/62DD8E5F/62DECBDB" Ref="#PWR0604"  Part="1"
+F 0 "#PWR0604" H 6900 3500 50  0001 C CNN
 F 1 "GND" H 6905 3577 50  0000 C CNN
 F 2 "" H 6900 3750 50  0001 C CNN

Commit message: Add new LED, RJ12 footprints to footprint library. Add STEP model.
Parts:
- added R603: 10K, Resistor_SMD:R_0603_1608Metric, symbol Device:R
- added S601: SWITCH_TACTILE_SPST-NO_0.05A_24V, GeneralPurposeAlarmDevicePCB:Switch_Tactile_THT_6x6mm, symbol GPAD_SCH_LIB:SWITCH_TACTILE_SPST-NO_0.05A_24V
Connections:
- net labels added: Switch_Mute, VccBuzzer
- wire segments 20 -> 31
Changed lines of the file:
@@
 L power:+5V #PWR?
 U 1 1 62DEA4D9
-P 1400 1900
+P 1400 1800
 AR Path="/62DEA4D9" Ref="#PWR?"  Part="1"
 AR Path="/62B871EE/62DEA4D9" Ref="#PWR?"  Part="1"
 AR Path="/62DD8E5F/62DEA4D9" Ref="#PWR0601"  Part="1"
-F 0 "#PWR0601" H 1400 1750 50  0001 C CNN
-F 1 "+5V" H 1415 2073 50  0000 C CNN
-F 2 "" H 1400 1900 50  0001 C CNN
-F 3 "" H 1400 1900 50  0001 C CNN
-	1    1400 1900
+F 0 "#PWR0601" H 1400 1650 50  0001 C CNN
+F 1 "+5V" H 1415 1973 50  0000 C CNN
+F 2 "" H 1400 1800 50  0001 C CNN
+F 3 "" H 1400 1800 50  0001 C CNN
+	1    1400 1800
 	1    0    0    -1
 $EndComp
@@
 Wire Wire Line
 	3400 2800 4400 2800
+Wire Wire Line
+	1400 1900 1400 1800
+Text Label 2600 1900 0    50   ~ 0
+VccBuzzer
+$Comp
+L GPAD_SCH_LIB:SWITCH_TACTILE_SPST-NO_0.05A_24V S?
+U 1 1 62C80308
+P 3500 4750
+AR Path="/62C80308" Ref="S?"  Part="1"
+AR Path="/62DD8E5F/62C80308" Ref="S601"  Part="1"
+F 0 "S601" H 3500 5097 60  0000 C CNN
+F 1 "SWITCH_TACTILE_SPST-NO_0.05A_24V" H 3500 4991 60  0000 C CNN
+F 2 "GeneralPurposeAlarmDevicePCB:Switch_Tactile_THT_6x6mm" H 3700 4950 60  0001 L CNN
+F 3 "https://www.te.com/commerce/DocumentDelivery/DDEController?Action=srchrtrv&DocNm=1825910&DocType=Customer+Drawing&DocLang=English" H 3700 5050 60  0001 L CNN
+F 4 "JLCPCB" H 3500 4750 50  0001 C CNN "Distributor 1"
+F 5 "C592982" H 3500 4750 50  0001 C CNN "Distributor 1 PN"
+F 6 "Digikey" H 3500 4750 50  0001 C CNN "Distributor 2"
+F 7 "450-1804-ND" H 3700 5150 60  0001 L CNN "Distributor 2 PN"
+F 8 "TE Connectivity ALCOSWITCH Switches" H 3700 5850 60  0001 L CNN "Manufacturer"
+F 9 "1825910-7" H 3700 5250 60  0001 L CNN "MPN"
+F 10 "Switches" H 3700 5350 60  0001 L CNN "Category"
+F 11 "Tactile Switches" H 3700 5450 60  0001 L CNN "Family"
+F 12 "https://www.te.com/commerce/DocumentDelivery/DDEController?Action=srchrtrv&DocNm=1825910&DocType=Customer+Drawing&DocLang=English" H 3700 5550 60  0001 L CNN "DK_Datasheet_Link"
+F 13 "/product-detail/en/te-connectivity-alcoswitch-switches/1825910-7/450-1804-ND/1731414" H 3700 5650 60  0001 L CNN "DK_Detail_Page"
+F 14 "SWITCH TACTILE SPST-NO 0.05A 24V" H 3700 5750 60  0001 L CNN "Description"
+F 15 "Active" H 3700 5950 60  0001 L CNN "Status"
+	1    3500 4750
+	1    0    0    -1
+$EndComp
+$Comp
+L power:GND #PWR?
+U 1 1 62C8131C
+P 3750 5050
+AR Path="/62C8131C" Ref="#PWR?"  Part="1"
+AR Path="/62DD8E5F/62C8131C" Ref="#PWR0606"  Part="1"
+F 0 "#PWR0606" H 3750 4800 50  0001 C CNN
+F 1 "GND" H 3755 4877 50  0000 C CNN
+F 2 "" H 3750 5050 50  0001 C CNN
+F 3 "" H 3750 5050 50  0001 C CNN
+	1    3750 5050
+	1    0    0    -1
+$EndComp
+Wire Wire Line
+	3700 4650 3750 4650
+Wire Wire Line
+	3750 4650 3750 4850
+Wire Wire Line
+	3700 4850 3750 4850
+Connection ~ 3750 4850
+Wire Wire Line
+	3750 4850 3750 5050
+Wire Wire Line
+	3300 4850 2450 4850
+Wire Wire Line
+	2450 4850 2450 4650
+Wire Wire Line
+	2450 4650 3300 4650
+$Comp
+L Device:R R?
+U 1 1 62C8BE9A
+P 2150 4650
+AR Path="/62C8BE9A" Ref="R?"  Part="1"
+AR Path="/62DD8E5F/62C8BE9A" Ref="R603"  Part="1"
+F 0 "R603" V 1950 4600 50  0000 C CNN
+F 1 "10K" V 2050 4650 50  0000 C CNN
+F 2 "Resistor_SMD:R_0603_1608Metric" V 2080 4650 50  0001 C CNN
+F 3 "~" H 2150 4650 50  0001 C CNN
+F 4 "JLCPCB" V 2150 4650 50  0001 C CNN "Distributor 1"
+F 5 "C269701" V 2150 4650 50  0001 C CNN "Distributor 1 PN"
+F 6 "TyoHM" V 2150 4650 50  0001 C CNN "Manufacturer"
+F 7 "RMC 0603 10K F N" V 2150 4650 50  0001 C CNN "MPN"
+F 8 "0.1W ±1% 10kΩ 0603  Chip Resistor - Surface Mount ROHS" H 2150 4650 50  0001 C CNN "Description"
+	1    2150 4650
+	0    1    1    0
+$EndComp
+$Comp
+L power:+5V #PWR?
+U 1 1 62C8CF60
+P 1600 4500
+AR Path="/62C8CF60" Ref="#PWR?"  Part="1"
+AR Path="/62B871EE/62C8CF60" Ref="#PWR?"  Part="1"
+AR Path="/62DD8E5F/62C8CF60" Ref="#PWR0605"  Part="1"
+F 0 "#PWR0605" H 1600 4350 50  0001 C CNN
+F 1 "+5V" H 1615 4673 50  0000 C CNN
+F 2 "" H 1600 4500 50  0001 C CNN
+F 3 "" H 1600 4500 50  0001 C CNN
+	1    1600 4500
+	1    0    0    -1
+$EndComp
+Wire Wire Line
+	2450 4650 2300 4650
+Connection ~ 2450 4650
+Wire Wire Line
+	2000 4650 1600 4650
+Wire Wire Line
+	1600 4650 1600 4500
+Text HLabel 2450 4850 0    50   Input ~ 0
+Switch_Mute
 $EndSCHEMATC

Commit message: Add JST connector for I2C and more.
Parts:
- removed Q601: MMBT2222A-7-F, digikey-footprints:SOT-23-3, symbol dk_Transistors-Bipolar-BJT-Single:MMBT2222A-7-F
- added Q601: MMBT2222A-7-F, Package_TO_SOT_SMD:SOT-23, symbol GPAD_SCH_LIB:MMBT2222A-7-F
- Q602: footprint digikey-footprints:SOT-23-3 -> Package_TO_SOT_SMD:SOT-23
Changed lines of the file:
@@
-$EndComp
-$Comp
-L dk_Transistors-Bipolar-BJT-Single:MMBT2222A-7-F Q?
-U 1 1 62DE2407
-P 5300 2400
-AR Path="/62B3AC2F/62DE2407" Ref="Q?"  Part="1"
-AR Path="/62DD8E5F/62DE2407" Ref="Q601"  Part="1"
-F 0 "Q601" H 5488 2453 60  0000 L CNN
-F 1 "MMBT2222A-7-F" H 5488 2347 60  0000 L CNN
-F 2 "digikey-footprints:SOT-23-3" H 5500 2600 60  0001 L CNN
-F 3 "https://www.diodes.com/assets/Datasheets/ds30041.pdf" H 5500 2700 60  0001 L CNN
-F 4 "MMBT2222A-FDICT-ND" H 5500 2800 60  0001 L CNN "Digi-Key_PN"
-F 5 "MMBT2222A-7-F" H 5500 2900 60  0001 L CNN "MPN"
-F 6 "Discrete Semiconductor Products" H 5500 3000 60  0001 L CNN "Category"
-F 7 "Transistors - Bipolar (BJT) - Single" H 5500 3100 60  0001 L CNN "Family"
-F 8 "https://www.diodes.com/assets/Datasheets/ds30041.pdf" H 5500 3200 60  0001 L CNN "DK_Datasheet_Link"
-F 9 "/product-detail/en/diodes-incorporated/MMBT2222A-7-F/MMBT2222A-FDICT-ND/815723" H 5500 3300 60  0001 L CNN "DK_Detail_Page"
-F 10 "TRANS NPN 40V 0.6A SMD SOT23-3" H 5500 3400 60  0001 L CNN "Description"
-F 11 "Diodes Incorporated" H 5500 3500 60  0001 L CNN "Manufacturer"
-F 12 "Active" H 5500 3600 60  0001 L CNN "Status"
-	1    5300 2400
-	1    0    0    -1
 $EndComp
 $Comp
@@
 F 0 "Q602" H 5488 3103 60  0000 L CNN
 F 1 "MMBT2907ALT1G" H 5488 2997 60  0000 L CNN
-F 2 "digikey-footprints:SOT-23-3" H 5500 3250 60  0001 L CNN
+F 2 "Package_TO_SOT_SMD:SOT-23" H 5500 3250 60  0001 L CNN
 F 3 "http://www.onsemi.com/pub/Collateral/MMBT2907ALT1-D.PDF" H 5500 3350 60  0001 L CNN
 F 4 "MMBT2907ALT1GOSCT-ND" H 5500 3450 60  0001 L CNN "Digi-Key_PN"
@@
 Text HLabel 2450 4850 0    50   Input ~ 0
 Switch_Mute
+$Comp
+L GPAD_SCH_LIB:MMBT2222A-7-F Q601
+U 1 1 62D2B660
+P 5300 2400
+F 0 "Q601" H 5488 2453 60  0000 L CNN
+F 1 "MMBT2222A-7-F" H 5488 2347 60  0000 L CNN
+F 2 "Package_TO_SOT_SMD:SOT-23" H 5500 2600 60  0001 L CNN
+F 3 "https://www.diodes.com/assets/Datasheets/ds30041.pdf" H 5500 2700 60  0001 L CNN
+F 4 "MMBT2222A-FDICT-ND" H 5500 2800 60  0001 L CNN "Digi-Key_PN"
+F 5 "MMBT2222A-7-F" H 5500 2900 60  0001 L CNN "MPN"
+F 6 "Discrete Semiconductor Products" H 5500 3000 60  0001 L CNN "Category"
+F 7 "Transistors - Bipolar (BJT) - Single" H 5500 3100 60  0001 L CNN "Family"
+F 8 "https://www.diodes.com/assets/Datasheets/ds30041.pdf" H 5500 3200 60  0001 L CNN "DK_Datasheet_Link"
+F 9 "/product-detail/en/diodes-incorporated/MMBT2222A-7-F/MMBT2222A-FDICT-ND/815723" H 5500 3300 60  0001 L CNN "DK_Detail_Page"
+F 10 "TRANS NPN 40V 0.6A SMD SOT23-3" H 5500 3400 60  0001 L CNN "Description"
+F 11 "Diodes Incorporated" H 5500 3500 60  0001 L CNN "Manufacturer"
+F 12 "Active" H 5500 3600 60  0001 L CNN "Status"
+	1    5300 2400
+	1    0    0    -1
+$EndComp
 $EndSCHEMATC

Commit message: Add current limit to CongtollerVcc, and Barrel Input. Add jumper resistors for headers selecting VBus and ControllerVcc.
Parts:
- added R602: 10K, Resistor_SMD:R_0603_1608Metric, symbol Device:R
- added R604: 1R0, Resistor_SMD:R_0603_1608Metric, symbol Device:R
- renumbered R602 to R605
Connections:
- net labels added: Attenuate
- wire segments 31 -> 36
Other:
- moved on the sheet: R605

Commit message: Update schottky symbol and part number. Import to PCB. Only the Arduino UNO symbol remains to connect.
Parts:
- added C602: 100nF, Capacitor_SMD:C_0603_1608Metric_Pad1.08x0.95mm_HandSolder, symbol Device:C
- added J601: 22-23-2021, Connector_Molex:Molex_KK-254_AE-6410-02A_1x02_P2.54mm_Vertical, symbol GPAD_SCH_LIB:22-23-2021
Connections:
- wire segments 36 -> 47
Other:
- note added: "For external "speaker"."
Changed lines of the file:
@@
 	6900 2700 6900 3450
 Wire Wire Line
-	6900 3450 7400 3450
+	6900 3450 7100 3450
 Connection ~ 5400 2700
 Wire Wire Line
@@
 	3750 4850 3750 5050
 Wire Wire Line
-	3300 4850 2450 4850
-Wire Wire Line
-	2450 4850 2450 4650
-Wire Wire Line
-	2450 4650 3300 4650
+	3300 4850 3200 4850
+Wire Wire Line
+	2450 4650 2550 4650
 $Comp
 L Device:R R?
@@
 Wire Wire Line
 	1600 4650 1600 4500
-Text HLabel 2450 4850 0    50   Input ~ 0
+Text HLabel 2450 4050 0    50   Input ~ 0
 Switch_Mute
 $Comp
@@
 Wire Wire Line
 	3450 3550 3750 3550
+Wire Wire Line
+	2450 4050 2550 4050
+Wire Wire Line
+	2550 4050 2550 4650
+Connection ~ 2550 4650
+Wire Wire Line
+	2550 4650 3200 4650
+$Comp
+L Device:C C?
+U 1 1 62FF8897
+P 2450 5150
+AR Path="/62FF8897" Ref="C?"  Part="1"
+AR Path="/62DD8E5F/62FF8897" Ref="C602"  Part="1"
+F 0 "C602" H 2565 5196 50  0000 L CNN
+F 1 "100nF" H 2565 5105 50  0000 L CNN
+F 2 "Capacitor_SMD:C_0603_1608Metric_Pad1.08x0.95mm_HandSolder" H 2488 5000 50  0001 C CNN
+F 3 "~" H 2450 5150 50  0001 C CNN
+F 4 "JLCPCB" H 2450 5150 50  0001 C CNN "Distributor 1"
+F 5 "C14663" H 2450 5150 50  0001 C CNN "Distributor 1 PN"
+F 6 "YAGEO" H 2450 5150 50  0001 C CNN "Manufacturier"
+F 7 "CC0603KRX7R9BB104" H 2450 5150 50  0001 C CNN "MPN"
+F 8 "50V 100nF X7R ±10% 0603 Multilayer Ceramic Capacitors MLCC - SMD/SMT ROHS" H 2450 5150 50  0001 C CNN "Description"
+	1    2450 5150
+	1    0    0    -1
+$EndComp
+$Comp
+L power:GND #PWR?
+U 1 1 62FF8F7F
+P 2450 5400
+AR Path="/62FF8F7F" Ref="#PWR?"  Part="1"
+AR Path="/62DD8E5F/62FF8F7F" Ref="#PWR0607"  Part="1"
+F 0 "#PWR0607" H 2450 5150 50  0001 C CNN
+F 1 "GND" H 2455 5227 50  0000 C CNN
+F 2 "" H 2450 5400 50  0001 C CNN
+F 3 "" H 2450 5400 50  0001 C CNN
+	1    2450 5400
+	1    0    0    -1
+$EndComp
+Wire Wire Line
+	2450 5300 2450 5400
+Wire Wire Line
+	3200 4650 3200 4850
+Connection ~ 3200 4650
+Wire Wire Line
+	3200 4650 3300 4650
+Wire Wire Line
+	2450 4650 2450 5000
+$Comp
+L GPAD_SCH_LIB:22-23-2021 J?
+U 1 1 6301024B
+P 7650 4400
+AR Path="/6301024B" Ref="J?"  Part="1"
+AR Path="/62DD8E5F/6301024B" Ref="J601"  Part="1"
+F 0 "J601" V 7550 4250 50  0000 R CNN
+F 1 "22-23-2021" V 7900 4550 50  0000 R CNN
+F 2 "Connector_Molex:Molex_KK-254_AE-6410-02A_1x02_P2.54mm_Vertical" H 7850 4600 60  0001 L CNN
+F 3 "https://media.digikey.com/pdf/Data%20Sheets/Molex%20PDFs/A-6373-N_Series_Dwg_2010-12-03.pdf" H 7850 4700 60  0001 L CNN
+F 4 "WM4200-ND" H 7850 4800 60  0001 L CNN "Digi-Key_PN"
+F 5 "22-23-2021" H 7850 4900 60  0001 L CNN "MPN"
+F 6 "Connectors, Interconnects" H 7850 5000 60  0001 L CNN "Category"
+F 7 "Rectangular Connectors - Headers, Male Pins" H 7850 5100 60  0001 L CNN "Family"
+F 8 "https://media.digikey.com/pdf/Data%20Sheets/Molex%20PDFs/A-6373-N_Series_Dwg_2010-12-03.pdf" H 7850 5200 60  0001 L CNN "DK_Datasheet_Link"
+F 9 "/product-detail/en/molex/22-23-2021/WM4200-ND/26667" H 7850 5300 60  0001 L CNN "DK_Detail_Page"
+F 10 "CONN HEADER VERT 2POS 2.54MM" H 7850 5400 60  0001 L CNN "Description"
+F 11 "Molex" H 7850 5500 60  0001 L CNN "Manufacturer"
+F 12 "Active" H 7850 5600 60  0001 L CNN "Status"
+	1    7650 4400
+	0    -1   1    0
+$EndComp
+Wire Wire Line
+	7100 3450 7100 4400
+Wire Wire Line
+	7100 4400 7550 4400
+Connection ~ 7100 3450
+Wire Wire Line
+	7100 3450 7400 3450
+$Comp
+L power:GND #PWR?
+U 1 1 6301310E
+P 7250 4550
+AR Path="/6301310E" Ref="#PWR?"  Part="1"
+AR Path="/62DD8E5F/6301310E" Ref="#PWR0608"  Part="1"
+F 0 "#PWR0608" H 7250 4300 50  0001 C CNN
+F 1 "GND" H 7255 4377 50  0000 C CNN
+F 2 "" H 7250 4550 50  0001 C CNN
+F 3 "" H 7250 4550 50  0001 C CNN
+	1    7250 4550
+	1    0    0    -1
+$EndComp
+Wire Wire Line
+	7250 4550 7250 4500
+Wire Wire Line
+	7250 4500 7550 4500
+Text Notes 7600 4200 0    50   ~ 0
+For external "speaker".
 $EndSCHEMATC

Commit message: Add both UNO and NANO schematic and PCB foot print.  Zero schematic errors reported. This incorporates all of the updates from the review except the DO NOT FIX.
Connections:
- net Attenuate: now also R605.1
Changed lines of the file:
@@
 Attenuate
-Wire Wire Line
-	3450 3550 3750 3550
 Wire Wire Line
 	2450 4050 2550 4050
@@
 Text Notes 7600 4200 0    50   ~ 0
 For external "speaker".
+Wire Wire Line
+	3400 3550 3750 3550
 $EndSCHEMATC
