File: Hardware/GeneralPurposeAlarmDevicePCB/GeneralPurposeAlarmDevicePCB/AlarmAudio.sch (KiCad schematic (older format))
At the start: 12 parts, among them J601 22-23-2021, Q601 MMBT2222A-7-F, Q602 MMBT2907ALT1G

Commit message: Clean up a bunch of duplicate because of missspelled part field names. Still working on a few sch, pcb and 3D libraries.
Parts:
- removed BZ601: PKMCS0909E4000-R1, digikey-footprints:Piezo_9x9mm_PKMCS0909E4000-R1, symbol dk_Alarms-Buzzers-and-Sirens:PKMCS0909E4000-R1
- added BZ601: QMB-09B-03, GeneralPurposeAlarmDevicePCB:MagneticBuzzer_9mmx5.8mmP=4mm, symbol GPAD_SCH_LIB:QMB-09B-03
- C601: value 47uF 16V -> 47uF
- C602: Manufacturer (none) -> YAGEO; Manufacturier YAGEO -> (none)
- J601: Assembly Type (none) -> HAND
- Q602: footprint Package_TO_SOT_SMD:SOT-23 -> digikey-footprints:SOT-23-3
- R601, R604: value 1R0 -> 1R
- R602: value 10K -> 1K; Description 0.1W ±1% 10kΩ 0603 Chip Resistor - Surface Mount ROHS -> 0.1W ±1% 1kΩ 0603 Chip Resistor - Surface Mount ROHS; Distributor 1 PN C269701 -> C269704; MPN RMC 0603 10K F N -> RMC06031K1%N
- R605: value 330R -> 330
- S601: Assembly Type (none) -> HAND; Distributor 1 PN C592982 -> C13828; MPN 1825910-7 -> TE Connectivity 1825910-7, Dongguan Guangzhu Industrial C13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
Connections:
- net GND: now also BZ601.2
- net at J601.1, R604.1: now also BZ601.1
Changed lines of the file:
@@
 $EndDescr
-$Comp
-L dk_Alarms-Buzzers-and-Sirens:PKMCS0909E4000-R1 BZ601
-U 1 1 62DD9B52
-P 7500 3550
-F 0 "BZ601" H 7840 3658 60  0000 L CNN
-F 1 "PKMCS0909E4000-R1" H 7840 3552 60  0000 L CNN
-F 2 "digikey-footprints:Piezo_9x9mm_PKMCS0909E4000-R1" H 7700 3750 60  0001 L CNN
-F 3 "https://www.murata.com/~/media/webrenewal/products/sound/sounder/vppt-buzj083-d.ashx" H 7700 3850 60  0001 L CNN
-F 4 "490-9647-1-ND" H 7700 3950 60  0001 L CNN "Digi-Key_PN"
-F 5 "PKMCS0909E4000-R1" H 7700 4050 60  0001 L CNN "MPN"
-F 6 "Audio Products" H 7700 4150 60  0001 L CNN "Category"
-F 7 "Alarms, Buzzers, and Sirens" H 7700 4250 60  0001 L CNN "Family"
-F 8 "https://www.murata.com/~/media/webrenewal/products/sound/sounder/vppt-buzj083-d.ashx" H 7700 4350 60  0001 L CNN "DK_Datasheet_Link"
-F 9 "/product-detail/en/murata-electronics-north-america/PKMCS0909E4000-R1/490-9647-1-ND/4878401" H 7700 4450 60  0001 L CNN "DK_Detail_Page"
-F 10 "AUDIO PIEZO TRANSDUCER 12.5V SMD" H 7700 4550 60  0001 L CNN "Description"
-F 11 "Murata Electronics North America" H 7700 4650 60  0001 L CNN "Manufacturer"
-F 12 "Active" H 7700 4750 60  0001 L CNN "Status"
-	1    7500 3550
-	1    0    0    -1
-$EndComp
 $Comp
 L Device:R R?
@@
 AR Path="/62DD8E5F/62DE23F8" Ref="R605"  Part="1"
 F 0 "R605" V 4000 3600 50  0000 C CNN
-F 1 "330R" V 3750 3550 50  0000 C CNN
+F 1 "330" V 3750 3550 50  0000 C CNN
 F 2 "Resistor_SMD:R_0603_1608Metric" V 3830 3550 50  0001 C CNN
 F 3 "~" H 3900 3550 50  0001 C CNN
@@
 F 0 "Q602" H 5488 3103 60  0000 L CNN
 F 1 "MMBT2907ALT1G" H 5488 2997 60  0000 L CNN
-F 2 "Package_TO_SOT_SMD:SOT-23" H 5500 3250 60  0001 L CNN
+F 2 "digikey-footprints:SOT-23-3" H 5500 3250 60  0001 L CNN
 F 3 "http://www.onsemi.com/pub/Collateral/MMBT2907ALT1-D.PDF" H 5500 3350 60  0001 L CNN
 F 4 "MMBT2907ALT1GOSCT-ND" H 5500 3450 60  0001 L CNN "Digi-Key_PN"
@@
 AR Path="/62DD8E5F/62DE752C" Ref="C601"  Part="1"
 F 0 "C601" H 2968 2146 50  0000 L CNN
-F 1 "47uF 16V" H 2968 2055 50  0000 L CNN
+F 1 "47uF" H 2968 2055 50  0000 L CNN
 F 2 "Capacitor_SMD:CP_Elec_5x5.4" H 2888 1950 50  0001 C CNN
 F 3 "~" H 2850 2100 50  0001 C CNN
@@
 AR Path="/62DD8E5F/62DEA4D3" Ref="R601"  Part="1"
 F 0 "R601" V 1950 1850 50  0000 C CNN
-F 1 "1R0" V 2050 1900 50  0000 C CNN
+F 1 "1R" V 2050 1900 50  0000 C CNN
 F 2 "Resistor_SMD:R_0603_1608Metric" V 2080 1900 50  0001 C CNN
 F 3 "~" H 2150 1900 50  0001 C CNN
@@
 F 3 "https://www.te.com/commerce/DocumentDelivery/DDEController?Action=srchrtrv&DocNm=1825910&DocType=Customer+Drawing&DocLang=English" H 3700 5050 60  0001 L CNN
 F 4 "JLCPCB" H 3500 4750 50  0001 C CNN "Distributor 1"
-F 5 "C592982" H 3500 4750 50  0001 C CNN "Distributor 1 PN"
+F 5 "C13828" H 3500 4750 50  0001 C CNN "Distributor 1 PN"
 F 6 "Digikey" H 3500 4750 50  0001 C CNN "Distributor 2"
 F 7 "450-1804-ND" H 3700 5150 60  0001 L CNN "Distributor 2 PN"
 F 8 "TE Connectivity ALCOSWITCH Switches" H 3700 5850 60  0001 L CNN "Manufacturer"
-F 9 "1825910-7" H 3700 5250 60  0001 L CNN "MPN"
+F 9 "TE Connectivity 1825910-7,   Dongguan Guangzhu Industrial C13828" H 3700 5250 60  0001 L CNN "MPN"
 F 10 "Switches" H 3700 5350 60  0001 L CNN "Category"
 F 11 "Tactile Switches" H 3700 5450 60  0001 L CNN "Family"
@@
 F 14 "SWITCH TACTILE SPST-NO 0.05A 24V" H 3700 5750 60  0001 L CNN "Description"
 F 15 "Active" H 3700 5950 60  0001 L CNN "Status"
+F 16 "HAND" H 0   0   50  0001 C CNN "Assembly Type"
 	1    3500 4750
 	1    0    0    -1
@@
 AR Path="/62DD8E5F/62C9323E" Ref="R604"  Part="1"
 F 0 "R604" V 6300 2650 50  0000 C CNN
-F 1 "1R0" V 6400 2700 50  0000 C CNN
+F 1 "1R" V 6400 2700 50  0000 C CNN
 F 2 "Resistor_SMD:R_0603_1608Metric" V 6430 2700 50  0001 C CNN
 F 3 "~" H 6500 2700 50  0001 C CNN
@@
 Wire Wire Line
 	4050 2800 4350 2800
-$Comp
-L Device:R R?
-U 1 1 62C9ABF4
-P 3900 2800
-AR Path="/62C9ABF4" Ref="R?"  Part="1"
-AR Path="/62DD8E5F/62C9ABF4" Ref="R602"  Part="1"
-F 0 "R602" V 3700 2750 50  0000 C CNN
-F 1 "10K" V 3800 2800 50  0000 C CNN
-F 2 "Resistor_SMD:R_0603_1608Metric" V 3830 2800 50  0001 C CNN
-F 3 "~" H 3900 2800 50  0001 C CNN
-F 4 "JLCPCB" V 3900 2800 50  0001 C CNN "Distributor 1"
-F 5 "C269701" V 3900 2800 50  0001 C CNN "Distributor 1 PN"
-F 6 "TyoHM" V 3900 2800 50  0001 C CNN "Manufacturer"
-F 7 "RMC 0603 10K F N" V 3900 2800 50  0001 C CNN "MPN"
-F 8 "0.1W ±1% 10kΩ 0603  Chip Resistor - Surface Mount ROHS" H 3900 2800 50  0001 C CNN "Description"
-	1    3900 2800
-	0    1    1    0
-$EndComp
 Wire Wire Line
 	4050 3550 4350 3550
@@
 F 4 "JLCPCB" H 2450 5150 50  0001 C CNN "Distributor 1"
 F 5 "C14663" H 2450 5150 50  0001 C CNN "Distributor 1 PN"
-F 6 "YAGEO" H 2450 5150 50  0001 C CNN "Manufacturier"
+F 6 "YAGEO" H 2450 5150 50  0001 C CNN "Manufacturer"
 F 7 "CC0603KRX7R9BB104" H 2450 5150 50  0001 C CNN "MPN"
 F 8 "50V 100nF X7R ±10% 0603 Multilayer Ceramic Capacitors MLCC - SMD/SMT ROHS" H 2450 5150 50  0001 C CNN "Description"
@@
 F 11 "Molex" H 7850 5500 60  0001 L CNN "Manufacturer"
 F 12 "Active" H 7850 5600 60  0001 L CNN "Status"
+F 13 "HAND" H 0   0   50  0001 C CNN "Assembly Type"
 	1    7650 4400
 	0    -1   1    0
@@
 Wire Wire Line
 	3400 3550 3750 3550
+$Comp
+L GPAD_SCH_LIB:QMB-09B-03 BZ601
+U 1 1 63A1E0DF
+P 7500 3550
+F 0 "BZ601" H 7840 3658 60  0000 L CNN
+F 1 "QMB-09B-03" H 7840 3552 60  0000 L CNN
+F 2 "GeneralPurposeAlarmDevicePCB:MagneticBuzzer_9mmx5.8mmP=4mm" H 7700 3750 60  0001 L CNN
+F 3 "2104011834_Jiangsu-Huaneng-Elec-QMB-09B-03_C96256.pdf" H 7700 3850 60  0001 L CNN
+F 4 "" H 7700 3950 60  0001 L CNN "Digi-Key_PN"
+F 5 "QMB-09B-03" H 7700 4050 60  0001 L CNN "MPN"
+F 6 "Audio Products" H 7700 4150 60  0001 L CNN "Category"
+F 7 "Alarms, Buzzers, and Sirens" H 7700 4250 60  0001 L CNN "Family"
+F 8 "https://www.murata.com/~/media/webrenewal/products/sound/sounder/vppt-buzj083-d.ashx" H 7700 4350 60  0001 L CNN "DK_Datasheet_Link"
+F 9 "/product-detail/en/murata-electronics-north-america/PKMCS0909E4000-R1/490-9647-1-ND/4878401" H 7700 4450 60  0001 L CNN "DK_Detail_Page"
+F 10 "5.7mm 9mm Externally Driven 85dB@3V,10cm 2V~5V Magnetic 3V 2700Hz Plugin,P=4mm Buzzers ROHS" H 7700 4550 60  0001 L CNN "Description"
+F 11 "Jiangsu Huaneng Elec" H 7700 4650 60  0001 L CNN "Manufacturer"
+F 12 "Active" H 7700 4750 60  0001 L CNN "Status"
+F 13 "JLCPCB" H 7500 3550 50  0001 C CNN "Distirbutor 1"
+F 14 "C96256" H 7500 3550 50  0001 C CNN "Distirbutor 1 PN"
+	1    7500 3550
+	1    0    0    -1
+$EndComp
+$Comp
+L Device:R R?
+U 1 1 63A4299B
+P 3900 2800
+AR Path="/63A4299B" Ref="R?"  Part="1"
+AR Path="/62B871EE/63A4299B" Ref="R?"  Part="1"
+AR Path="/62DD8E5F/63A4299B" Ref="R602"  Part="1"
+F 0 "R602" V 3700 2750 50  0000 C CNN
+F 1 "1K" V 3800 2750 50  0000 C CNN
+F 2 "Resistor_SMD:R_0603_1608Metric" V 3830 2800 50  0001 C CNN
+F 3 "~" H 3900 2800 50  0001 C CNN
+F 4 "JLCPCB" V 3900 2800 50  0001 C CNN "Distributor 1"
+F 5 "C269704" V 3900 2800 50  0001 C CNN "Distributor 1 PN"
+F 6 "TyoHM" V 3900 2800 50  0001 C CNN "Manufacturer"
+F 7 "RMC06031K1%N" V 3900 2800 50  0001 C CNN "MPN"
+F 8 "0.1W ±1% 1kΩ 0603 Chip Resistor - Surface Mount ROHS" H 3900 2800 50  0001 C CNN "Description"
+	1    3900 2800
+	0    1    1    0
+$EndComp
 $EndSCHEMATC

Commit message: Still have to make a 3D for buzzer and for USB connector. Still have to make PubInv logo and other Open Source logos. Experimental PCB placement tightned up.
Parts:
- removed BZ601: QMB-09B-03, GeneralPurposeAlarmDevicePCB:MagneticBuzzer_9mmx5.8mmP=4mm, symbol GPAD_SCH_LIB:QMB-09B-03
- added BZ601: QMB-09B-03, QMB-09B-03:QMB09B03, symbol QMB-09B-03:QMB-09B-03
Connections:
- net GND: now also BZ601.2
- net at J601.1, R604.1: now also BZ601.1
Changed lines of the file:
@@
 $EndComp
-Wire Wire Line
-	7400 3550 6900 3550
 Wire Wire Line
 	6900 3550 6900 3750
@@
 	3400 3550 3750 3550
 $Comp
-L GPAD_SCH_LIB:QMB-09B-03 BZ601
-U 1 1 63A1E0DF
-P 7500 3550
-F 0 "BZ601" H 7840 3658 60  0000 L CNN
-F 1 "QMB-09B-03" H 7840 3552 60  0000 L CNN
-F 2 "GeneralPurposeAlarmDevicePCB:MagneticBuzzer_9mmx5.8mmP=4mm" H 7700 3750 60  0001 L CNN
-F 3 "2104011834_Jiangsu-Huaneng-Elec-QMB-09B-03_C96256.pdf" H 7700 3850 60  0001 L CNN
-F 4 "" H 7700 3950 60  0001 L CNN "Digi-Key_PN"
-F 5 "QMB-09B-03" H 7700 4050 60  0001 L CNN "MPN"
-F 6 "Audio Products" H 7700 4150 60  0001 L CNN "Category"
-F 7 "Alarms, Buzzers, and Sirens" H 7700 4250 60  0001 L CNN "Family"
-F 8 "https://www.murata.com/~/media/webrenewal/products/sound/sounder/vppt-buzj083-d.ashx" H 7700 4350 60  0001 L CNN "DK_Datasheet_Link"
-F 9 "/product-detail/en/murata-electronics-north-america/PKMCS0909E4000-R1/490-9647-1-ND/4878401" H 7700 4450 60  0001 L CNN "DK_Detail_Page"
-F 10 "5.7mm 9mm Externally Driven 85dB@3V,10cm 2V~5V Magnetic 3V 2700Hz Plugin,P=4mm Buzzers ROHS" H 7700 4550 60  0001 L CNN "Description"
-F 11 "Jiangsu Huaneng Elec" H 7700 4650 60  0001 L CNN "Manufacturer"
-F 12 "Active" H 7700 4750 60  0001 L CNN "Status"
-F 13 "JLCPCB" H 7500 3550 50  0001 C CNN "Distirbutor 1"
-F 14 "C96256" H 7500 3550 50  0001 C CNN "Distirbutor 1 PN"
-	1    7500 3550
-	1    0    0    -1
-$EndComp
-$Comp
 L Device:R R?
 U 1 1 63A4299B
@@
 	0    1    1    0
 $EndComp
+Wire Wire Line
+	7400 3550 6900 3550
+$Comp
+L QMB-09B-03:QMB-09B-03 BZ601
+U 1 1 62CCB6C9
+P 7400 3550
+F 0 "BZ601" H 7692 3185 50  0000 C CNN
+F 1 "QMB-09B-03" H 7692 3276 50  0000 C CNN
+F 2 "QMB-09B-03:QMB09B03" H 8050 3650 50  0001 L CNN
+F 3 "https://datasheet.lcsc.com/szlcsc/Jiangsu-Huaneng-Elec-QMB-09B-03_C96256.pdf" H 8050 3550 50  0001 L CNN
+F 4 "Magnetic NO 2700Hz 3V 2 ~ 5V 9mm 9*5.5mm Buzzers" H 8050 3450 50  0001 L CNN "Description"
+F 5 "Jiangsu Huaneng Elec" H 8050 3250 50  0001 L CNN "Manufacturer"
+F 6 "QMB-09B-03" H 8050 3150 50  0001 L CNN "MPN"
+F 7 "JLCPCB" H 7400 3550 50  0001 C CNN "Distributor 1"
+F 8 "C96256" H 7400 3550 50  0001 C CNN "Distributor 1 PN"
+	1    7400 3550
+	1    0    0    1
+$EndComp
 $EndSCHEMATC
