File: Hardware/GeneralPurposeAlarmDevicePCB/GeneralPurposeAlarmDevicePCB/AlarmLights5.sch (KiCad schematic (older format))
At the start: 20 parts

Commit message: Add more parts drawings, buzzer. Add additional schematic sheet for AlarmAudio.
Connections:
- net GND: now also Q?.2 (E), Q?.2 (E), Q?.2 (E), Q?.2 (E), Q?.2 (E)
- net at R?.1: now also Q?.1 (B) (x5)
- net Light0: now reaches R?.2
- net at R?.1: now also D?.1 (x5)
- net +5V: now reaches R?.2
- net +5V: now also R?.2, R?.2, R?.2, R?.2
- net at Q?.3 (C): now also D?.2 (x5)
- net Light1: now reaches R?.2
- net Light2: now reaches R?.2
- net Light3: now reaches R?.2
- net Light4: now reaches R?.2
Changed lines of the file:
@@
 $Descr USLetter 11000 8500
 encoding utf-8
-Sheet 2 5
+Sheet 2 6
 Title "GeneralPurposeAlarmDevicePCB"
 Date "2022-06-20"
@@
 Text Notes 5050 2750 0    50   ~ 0
 Alarm lights, 5 Levels
+Wire Wire Line
+	8300 4200 8300 4150
+Wire Wire Line
+	7100 4200 7100 4150
+Wire Wire Line
+	5900 4150 5900 4200
+Wire Wire Line
+	4700 4200 4700 4150
+Wire Wire Line
+	3500 4200 3500 4150
+Wire Wire Line
+	3000 3850 3000 3950
+Wire Wire Line
+	3000 3950 3200 3950
+Wire Wire Line
+	3500 3750 3500 3650
+Wire Wire Line
+	3500 3400 3500 3350
+Connection ~ 3500 3350
+Wire Wire Line
+	3500 3350 3500 3250
+Wire Wire Line
+	4200 3850 4200 3950
+Wire Wire Line
+	4200 3950 4400 3950
+Wire Wire Line
+	4700 3750 4700 3650
+Wire Wire Line
+	4700 3350 4700 3250
+Wire Wire Line
+	5400 3850 5400 3950
+Wire Wire Line
+	5400 3950 5600 3950
+Wire Wire Line
+	5900 3750 5900 3650
+Wire Wire Line
+	5900 3350 5900 3250
+Wire Wire Line
+	6600 3850 6600 3950
+Wire Wire Line
+	6600 3950 6800 3950
+Wire Wire Line
+	7100 3750 7100 3650
+Wire Wire Line
+	7100 3350 7100 3250
+Wire Wire Line
+	7800 3850 7800 3950
+Wire Wire Line
+	7800 3950 8000 3950
+Wire Wire Line
+	8300 3750 8300 3650
+Wire Wire Line
+	8300 3350 8300 3250
+Wire Wire Line
+	3500 2950 3500 2800
+Wire Wire Line
+	8250 2800 8250 2950
+Wire Wire Line
+	8250 2950 8300 2950
+Wire Wire Line
+	7100 2950 7100 2800
+Connection ~ 7100 2800
+Wire Wire Line
+	7100 2800 8250 2800
+Wire Wire Line
+	5900 2950 5900 2800
+Wire Wire Line
+	3500 2800 4700 2800
+Connection ~ 5900 2800
+Wire Wire Line
+	5900 2800 7100 2800
+Wire Wire Line
+	4700 2950 4700 2800
+Connection ~ 4700 2800
+Wire Wire Line
+	4700 2800 5900 2800
+$Comp
+L power:+5V #PWR?
+U 1 1 62CBF69C
+P 3500 2350
+AR Path="/62CBF69C" Ref="#PWR?"  Part="1"
+AR Path="/62B3AC2F/62CBF69C" Ref="#PWR?"  Part="1"
+F 0 "#PWR?" H 3500 2200 50  0001 C CNN
+F 1 "+5V" H 3515 2523 50  0000 C CNN
+F 2 "" H 3500 2350 50  0001 C CNN
+F 3 "" H 3500 2350 50  0001 C CNN
+	1    3500 2350
+	1    0    0    -1
+$EndComp
+Wire Wire Line
+	3500 2800 3500 2350
+Connection ~ 3500 2800
+Text HLabel 3000 3200 0    50   Input ~ 0
+Light0
+Wire Wire Line
+	3000 3200 3000 3550
+Text HLabel 4200 3200 0    50   Input ~ 0
+Light1
+Wire Wire Line
+	4200 3200 4200 3550
+Text HLabel 5400 3200 0    50   Input ~ 0
+Light2
+Wire Wire Line
+	5400 3200 5400 3550
+Text HLabel 6600 3200 0    50   Input ~ 0
+Light3
+Wire Wire Line
+	6600 3200 6600 3550
+Text HLabel 7800 3200 0    50   Input ~ 0
+Light4
+Wire Wire Line
+	7800 3200 7800 3550
 $EndSCHEMATC

Commit message: Annote reference designators.
Parts:
- gave numbers to parts that had none: 20
Changed lines of the file:
@@
 $EndDescr
 $Comp
-L Device:R R?
+L Device:R R201
 U 1 1 62B5A2AE
 P 3000 3700
-F 0 "R?" H 2900 3650 50  0000 C CNN
+F 0 "R201" H 2900 3650 50  0000 C CNN
 F 1 "4K7" H 2850 3750 50  0000 C CNN
 F 2 "Resistor_SMD:R_0603_1608Metric" V 2930 3700 50  0001 C CNN
@@
 $EndComp
 $Comp
-L power:GND #PWR?
+L power:GND #PWR0202
 U 1 1 62B5A2B4
 P 3500 4200
-F 0 "#PWR?" H 3500 3950 50  0001 C CNN
+F 0 "#PWR0202" H 3500 3950 50  0001 C CNN
 F 1 "GND" H 3505 4027 50  0000 C CNN
 F 2 "" H 3500 4200 50  0001 C CNN
@@
 $EndComp
 $Comp
-L Device:R R?
+L Device:R R202
 U 1 1 62B5A2BF
 P 3500 3100
-F 0 "R?" H 3400 3050 50  0000 C CNN
+F 0 "R202" H 3400 3050 50  0000 C CNN
 F 1 "330R" H 3350 3150 50  0000 C CNN
 F 2 "Resistor_SMD:R_0603_1608Metric" V 3430 3100 50  0001 C CNN
@@
 $EndComp
 $Comp
-L dk_Transistors-Bipolar-BJT-Single:MMBT2222A-7-F Q?
+L dk_Transistors-Bipolar-BJT-Single:MMBT2222A-7-F Q201
 U 1 1 62B5A2CE
 P 3400 3950
-F 0 "Q?" H 3588 4003 60  0000 L CNN
+F 0 "Q201" H 3588 4003 60  0000 L CNN
 F 1 "MMBT2222A-7-F" H 3588 3897 60  0000 L CNN
 F 2 "digikey-footprints:SOT-23-3" H 3600 4150 60  0001 L CNN
@@
 $EndComp
 $Comp
-L dk_LED-Indication-Discrete:LTST-C171KRKT D?
+L dk_LED-Indication-Discrete:LTST-C171KRKT D201
 U 1 1 62B5A2DC
 P 3500 3550
-F 0 "D?" V 3450 3800 60  0000 C CNN
+F 0 "D201" V 3450 3800 60  0000 C CNN
 F 1 "RED 0603" V 3600 3850 60  0000 C CNN
 F 2 "LED_SMD:LED_0603_1608Metric" H 3700 3750 60  0001 L CNN
@@
 $EndComp
 $Comp
-L Device:R R?
+L Device:R R203
 U 1 1 62B5A2E7
 P 4200 3700
-F 0 "R?" H 4100 3650 50  0000 C CNN
+F 0 "R203" H 4100 3650 50  0000 C CNN
 F 1 "4K7" H 4050 3750 50  0000 C CNN
 F 2 "Resistor_SMD:R_0603_1608Metric" V 4130 3700 50  0001 C CNN
@@
 $EndComp
 $Comp
-L power:GND #PWR?
+L power:GND #PWR0203
 U 1 1 62B5A2ED
 P 4700 4200
-F 0 "#PWR?" H 4700 3950 50  0001 C CNN
+F 0 "#PWR0203" H 4700 3950 50  0001 C CNN
 F 1 "GND" H 4705 4027 50  0000 C CNN
 F 2 "" H 4700 4200 50  0001 C CNN
@@
 $EndComp
 $Comp
-L Device:R R?
+L Device:R R204
 U 1 1 62B5A2F8
 P 4700 3100
-F 0 "R?" H 4600 3050 50  0000 C CNN
+F 0 "R204" H 4600 3050 50  0000 C CNN
 F 1 "330R" H 4550 3150 50  0000 C CNN
 F 2 "Resistor_SMD:R_0603_1608Metric" V 4630 3100 50  0001 C CNN
@@
 $EndComp
 $Comp
-L dk_Transistors-Bipolar-BJT-Single:MMBT2222A-7-F Q?
+L dk_Transistors-Bipolar-BJT-Single:MMBT2222A-7-F Q202
 U 1 1 62B5A307
 P 4600 3950
-F 0 "Q?" H 4788 4003 60  0000 L CNN
+F 0 "Q202" H 4788 4003 60  0000 L CNN
 F 1 "MMBT2222A-7-F" H 4788 3897 60  0000 L CNN
 F 2 "digikey-footprints:SOT-23-3" H 4800 4150 60  0001 L CNN
@@
 $EndComp
 $Comp
-L dk_LED-Indication-Discrete:LTST-C171KRKT D?
+L dk_LED-Indication-Discrete:LTST-C171KRKT D202
 U 1 1 62B5A315
 P 4700 3550
-F 0 "D?" V 4650 3800 60  0000 C CNN
+F 0 "D202" V 4650 3800 60  0000 C CNN
 F 1 "RED 0603" V 4800 3850 60  0000 C CNN
 F 2 "LED_SMD:LED_0603_1608Metric" H 4900 3750 60  0001 L CNN
@@
 $EndComp
 $Comp
-L Device:R R?
+L Device:R R205
 U 1 1 62B5A320
 P 5400 3700
-F 0 "R?" H 5300 3650 50  0000 C CNN
+F 0 "R205" H 5300 3650 50  0000 C CNN
 F 1 "4K7" H 5250 3750 50  0000 C CNN
 F 2 "Resistor_SMD:R_0603_1608Metric" V 5330 3700 50  0001 C CNN
@@
 $EndComp
 $Comp
-L power:GND #PWR?
+L power:GND #PWR0204
 U 1 1 62B5A326
 P 5900 4200
-F 0 "#PWR?" H 5900 3950 50  0001 C CNN
+F 0 "#PWR0204" H 5900 3950 50  0001 C CNN
 F 1 "GND" H 5905 4027 50  0000 C CNN
 F 2 "" H 5900 4200 50  0001 C CNN
@@
 $EndComp
 $Comp
-L Device:R R?
+L Device:R R206
 U 1 1 62B5A331
 P 5900 3100
-F 0 "R?" H 5800 3050 50  0000 C CNN
+F 0 "R206" H 5800 3050 50  0000 C CNN
 F 1 "330R" H 5750 3150 50  0000 C CNN
 F 2 "Resistor_SMD:R_0603_1608Metric" V 5830 3100 50  0001 C CNN
@@
 $EndComp
 $Comp
-L dk_Transistors-Bipolar-BJT-Single:MMBT2222A-7-F Q?
+L dk_Transistors-Bipolar-BJT-Single:MMBT2222A-7-F Q203
 U 1 1 62B5A340
 P 5800 3950
-F 0 "Q?" H 5988 4003 60  0000 L CNN
+F 0 "Q203" H 5988 4003 60  0000 L CNN
 F 1 "MMBT2222A-7-F" H 5988 3897 60  0000 L CNN
 F 2 "digikey-footprints:SOT-23-3" H 6000 4150 60  0001 L CNN
@@
 $EndComp
 $Comp
-L dk_LED-Indication-Discrete:LTST-C171KRKT D?
+L dk_LED-Indication-Discrete:LTST-C171KRKT D203
 U 1 1 62B5A34E
 P 5900 3550
-F 0 "D?" V 5850 3800 60  0000 C CNN
+F 0 "D203" V 5850 3800 60  0000 C CNN
 F 1 "RED 0603" V 6000 3850 60  0000 C CNN
 F 2 "LED_SMD:LED_0603_1608Metric" H 6100 3750 60  0001 L CNN
@@
 $EndComp
 $Comp
-L Device:R R?
+L Device:R R207
 U 1 1 62B5A359
 P 6600 3700
-F 0 "R?" H 6500 3650 50  0000 C CNN
+F 0 "R207" H 6500 3650 50  0000 C CNN
 F 1 "4K7" H 6450 3750 50  0000 C CNN
 F 2 "Resistor_SMD:R_0603_1608Metric" V 6530 3700 50  0001 C CNN
@@
 $EndComp
 $Comp
-L power:GND #PWR?
+L power:GND #PWR0205
 U 1 1 62B5A35F
 P 7100 4200
-F 0 "#PWR?" H 7100 3950 50  0001 C CNN
+F 0 "#PWR0205" H 7100 3950 50  0001 C CNN
 F 1 "GND" H 7105 4027 50  0000 C CNN
 F 2 "" H 7100 4200 50  0001 C CNN
@@
 $EndComp
 $Comp
-L Device:R R?
+L Device:R R208
 U 1 1 62B5A36A
 P 7100 3100
-F 0 "R?" H 7000 3050 50  0000 C CNN
+F 0 "R208" H 7000 3050 50  0000 C CNN
 F 1 "330R" H 6950 3150 50  0000 C CNN
 F 2 "Resistor_SMD:R_0603_1608Metric" V 7030 3100 50  0001 C CNN
@@
 $EndComp
 $Comp
-L dk_Transistors-Bipolar-BJT-Single:MMBT2222A-7-F Q?
+L dk_Transistors-Bipolar-BJT-Single:MMBT2222A-7-F Q204
 U 1 1 62B5A379
 P 7000 3950
-F 0 "Q?" H 7188 4003 60  0000 L CNN
+F 0 "Q204" H 7188 4003 60  0000 L CNN
 F 1 "MMBT2222A-7-F" H 7188 3897 60  0000 L CNN
 F 2 "digikey-footprints:SOT-23-3" H 7200 4150 60  0001 L CNN
@@
 $EndComp
 $Comp
-L dk_LED-Indication-Discrete:LTST-C171KRKT D?
+L dk_LED-Indication-Discrete:LTST-C171KRKT D204
 U 1 1 62B5A387
 P 7100 3550
-F 0 "D?" V 7050 3800 60  0000 C CNN
+F 0 "D204" V 7050 3800 60  0000 C CNN
 F 1 "RED 0603" V 7200 3850 60  0000 C CNN
 F 2 "LED_SMD:LED_0603_1608Metric" H 7300 3750 60  0001 L CNN
@@
 $EndComp
 $Comp
-L Device:R R?
+L Device:R R209
 U 1 1 62B5A392
 P 7800 3700
-F 0 "R?" H 7700 3650 50  0000 C CNN
+F 0 "R209" H 7700 3650 50  0000 C CNN
 F 1 "4K7" H 7650 3750 50  0000 C CNN
 F 2 "Resistor_SMD:R_0603_1608Metric" V 7730 3700 50  0001 C CNN
@@
 $EndComp
 $Comp
-L power:GND #PWR?
+L power:GND #PWR0206
 U 1 1 62B5A398
 P 8300 4200
-F 0 "#PWR?" H 8300 3950 50  0001 C CNN
+F 0 "#PWR0206" H 8300 3950 50  0001 C CNN
 F 1 "GND" H 8305 4027 50  0000 C CNN
 F 2 "" H 8300 4200 50  0001 C CNN
@@
 $EndComp
 $Comp
-L Device:R R?
+L Device:R R210
 U 1 1 62B5A3A3
 P 8300 3100
-F 0 "R?" H 8200 3050 50  0000 C CNN
+F 0 "R210" H 8200 3050 50  0000 C CNN
 F 1 "330R" H 8150 3150 50  0000 C CNN
 F 2 "Resistor_SMD:R_0603_1608Metric" V 8230 3100 50  0001 C CNN
@@
 $EndComp
 $Comp
-L dk_Transistors-Bipolar-BJT-Single:MMBT2222A-7-F Q?
+L dk_Transistors-Bipolar-BJT-Single:MMBT2222A-7-F Q205
 U 1 1 62B5A3B2
 P 8200 3950
-F 0 "Q?" H 8388 4003 60  0000 L CNN
+F 0 "Q205" H 8388 4003 60  0000 L CNN
 F 1 "MMBT2222A-7-F" H 8388 3897 60  0000 L CNN
 F 2 "digikey-footprints:SOT-23-3" H 8400 4150 60  0001 L CNN
@@
 $EndComp
 $Comp
-L dk_LED-Indication-Discrete:LTST-C171KRKT D?
+L dk_LED-Indication-Discrete:LTST-C171KRKT D205
 U 1 1 62B5A3C0
 P 8300 3550
-F 0 "D?" V 8250 3800 60  0000 C CNN
+F 0 "D205" V 8250 3800 60  0000 C CNN
 F 1 "RED 0603" V 8400 3850 60  0000 C CNN
 F 2 "LED_SMD:LED_0603_1608Metric" H 8500 3750 60  0001 L CNN
@@
 P 3500 2350
 AR Path="/62CBF69C" Ref="#PWR?"  Part="1"
-AR Path="/62B3AC2F/62CBF69C" Ref="#PWR?"  Part="1"
-F 0 "#PWR?" H 3500 2200 50  0001 C CNN
+AR Path="/62B3AC2F/62CBF69C" Ref="#PWR0201"  Part="1"
+F 0 "#PWR0201" H 3500 2200 50  0001 C CNN
 F 1 "+5V" H 3515 2523 50  0000 C CNN
 F 2 "" H 3500 2350 50  0001 C CNN

Commit message: Add new LED, RJ12 footprints to footprint library. Add STEP model.
Parts:
- removed D201, D202, D203, D204, D205: RED 0603, LED_SMD:LED_0603_1608Metric, symbol dk_LED-Indication-Discrete:LTST-C171KRKT
- added D201, D202, D203, D204, D205: LED_T1.75_CLEAR_WHITE, GeneralPurposeAlarmDevicePCB:LED_5mm_Radial, symbol GPAD_SCH_LIB:LED_T1.75_CLEAR_WHITE
Connections:
- net at R202.1: now also D201.1
- net at Q201.3 (C): now also D201.2
- net at R204.1: now also D202.1
- net at Q202.3 (C): now also D202.2
- net at R206.1: now also D203.1
- net at Q203.3 (C): now also D203.2
- net at R208.1: now also D204.1
- net at Q204.3 (C): now also D204.2
- net at R210.1: now also D205.1
- net at Q205.3 (C): now also D205.2

Commit message: Add JST connector for I2C and more.
Parts:
- removed Q201, Q202, Q203, Q204, Q205: MMBT2222A-7-F, digikey-footprints:SOT-23-3, symbol dk_Transistors-Bipolar-BJT-Single:MMBT2222A-7-F
- added Q201, Q202, Q203, Q204, Q205: MMBT2222A-7-F, Package_TO_SOT_SMD:SOT-23, symbol GPAD_SCH_LIB:MMBT2222A-7-F
Connections:
- net GND: now also Q201.2 (E), Q202.2 (E), Q203.2 (E), Q204.2 (E), Q205.2 (E)
- net at R201.1: now also Q201.1 (B)
- net at D201.2: now also Q201.3 (C)
- net at R203.1: now also Q202.1 (B)
- net at D202.2: now also Q202.3 (C)
- net at R205.1: now also Q203.1 (B)
- net at D203.2: now also Q203.3 (C)
- net at R207.1: now also Q204.1 (B)
- net at D204.2: now also Q204.3 (C)
- net at R209.1: now also Q205.1 (B)
- net at D205.2: now also Q205.3 (C)

Commit message: Remove NANO sheild foot print. Other changes per issue #23 notes of 20220712.
Changed lines of the file:
@@
 U 1 1 62B5A2AE
 P 3000 3700
-F 0 "R201" H 2900 3650 50  0000 C CNN
+F 0 "R201" H 2900 3550 50  0000 C CNN
 F 1 "4K7" H 2850 3750 50  0000 C CNN
 F 2 "Resistor_SMD:R_0603_1608Metric" V 2930 3700 50  0001 C CNN
@@
 U 1 1 62B5A2BF
 P 3500 3100
-F 0 "R202" H 3400 3050 50  0000 C CNN
+F 0 "R202" H 3400 2950 50  0000 C CNN
 F 1 "330R" H 3350 3150 50  0000 C CNN
 F 2 "Resistor_SMD:R_0603_1608Metric" V 3430 3100 50  0001 C CNN
@@
 U 1 1 62B5A2F8
 P 4700 3100
-F 0 "R204" H 4600 3050 50  0000 C CNN
+F 0 "R204" H 4600 2950 50  0000 C CNN
 F 1 "330R" H 4550 3150 50  0000 C CNN
 F 2 "Resistor_SMD:R_0603_1608Metric" V 4630 3100 50  0001 C CNN
@@
 U 1 1 62B5A331
 P 5900 3100
-F 0 "R206" H 5800 3050 50  0000 C CNN
+F 0 "R206" H 5800 2950 50  0000 C CNN
 F 1 "330R" H 5750 3150 50  0000 C CNN
 F 2 "Resistor_SMD:R_0603_1608Metric" V 5830 3100 50  0001 C CNN
@@
 U 1 1 62B5A36A
 P 7100 3100
-F 0 "R208" H 7000 3050 50  0000 C CNN
+F 0 "R208" H 7000 2950 50  0000 C CNN
 F 1 "330R" H 6950 3150 50  0000 C CNN
 F 2 "Resistor_SMD:R_0603_1608Metric" V 7030 3100 50  0001 C CNN
@@
 U 1 1 62B5A3A3
 P 8300 3100
-F 0 "R210" H 8200 3050 50  0000 C CNN
+F 0 "R210" H 8200 2950 50  0000 C CNN
 F 1 "330R" H 8150 3150 50  0000 C CNN
 F 2 "Resistor_SMD:R_0603_1608Metric" V 8230 3100 50  0001 C CNN
