File: Hardware/GeneralPurposeAlarmDevicePCB/GeneralPurposeAlarmDevicePCB/GeneralPurposeAlarmDevicePCB.kicad_sch (KiCad schematic)
At the start: 44 parts

Commit message: Updated footprints and schematic Signed-off-by: lokimetasmith <lokimail@gmail.com>
Parts:
- A101: value (none) -> Arduino_UNO_R3_Shield; footprint (none) -> Module:Arduino_UNO_R3
- C101, C107: value (none) -> 39pF; footprint (none) -> Capacitor_SMD:C_0603_1608Metric_Pad1.08x0.95mm_HandSolder
- C102, C106, C109, C112: value (none) -> 47uF 16V; footprint (none) -> Capacitor_SMD:CP_Elec_5x5.4; symbol GeneralPurposeAlarmDevicePCB-rescue:CP-Device -> Device:C_Polarized
- C103, C105, C108, C110, C111: value (none) -> 100nF; footprint (none) -> Capacitor_SMD:C_0603_1608Metric_Pad1.08x0.95mm_HandSolder
- C104: value (none) -> 39pF; footprint (none) -> Capacitor_SMD:C_0603_1608Metric
- C113, C114: value (none) -> 33pF; footprint (none) -> Capacitor_SMD:C_0603_1608Metric_Pad1.08x0.95mm_HandSolder
- D101, D103, D104: value (none) -> Schottky 2A; footprint (none) -> Diode_SMD:D_SMB
- D102: value (none) -> RED 0603; footprint (none) -> digikey-footprints:0805; symbol GeneralPurposeAlarmDevicePCB-rescue:LTST-C171KRKT-dk_LED-Indication-Discrete -> Device:LED
- D105: value (none) -> LTL2R3KEK; footprint (none) -> GeneralPurposeAlarmDevicePCB:LED_5mm_Radial; symbol GeneralPurposeAlarmDevicePCB-rescue:LTL2R3KEK-dk_LED-Indication-Discrete -> Device:LED
- F101: value (none) -> Polyfuse_Small; footprint (none) -> Fuse:Fuse_0603_1608Metric
- H101, H102, H103, H104: value (none) -> MountingHole_Pad_3.5mm; footprint (none) -> GeneralPurposeAlarmDevicePCB:MountingHole_3.5mm_Pad_Via
- J101: value (none) -> Barrel_Jack_Switch_SMT; footprint (none) -> GeneralPurposeAlarmDevicePCB:BarrelJack_CLIFF_FC681465S_SMT_Horizontal
- J102, J103: value (none) -> 22-23-2021; footprint (none) -> Connector_Molex:Molex_KK-254_AE-6410-02A_1x02_P2.54mm_Vertical
- J105: value (none) -> S04B-XASK-1(LF)(SN); footprint (none) -> Connector_PinHeader_2.54mm:PinHeader_1x04_P2.54mm_Horizontal
- R101: value (none) -> 1R0; footprint (none) -> Resistor_SMD:R_0603_1608Metric
- R102: value (none) -> 10K; footprint (none) -> Resistor_SMD:R_0603_1608Metric
- R103, R110: value (none) -> 330R; footprint (none) -> Resistor_SMD:R_0603_1608Metric
- R104, R105: value (none) -> 39R; footprint (none) -> Resistor_SMD:R_0603_1608Metric
- R106, R107: value (none) -> DNI; footprint (none) -> Resistor_SMD:R_0603_1608Metric
- R108, R109: value (none) -> 1K; footprint (none) -> Resistor_SMD:R_0603_1608Metric
- S101: value (none) -> SWITCH_TACTILE_SPST-NO_0.05A_24V; footprint (none) -> GeneralPurposeAlarmDevicePCB:Switch_Tactile_THT_6x6mm
- TP_3v3: value (none) -> TestPoint 3.3V; footprint (none) -> TestPoint:TestPoint_Loop_D2.54mm_Drill1.5mm_Beaded
- U101: value (none) -> NCP1117ST50T3G; footprint (none) -> Package_TO_SOT_SMD:SOT-223
- U102: value (none) -> PI_ATMEGA328P-AU-InOrder; footprint (none) -> Package_QFP:TQFP-32_7x7mm_P0.8mm
- XTAL101: value (none) -> 16MHZ 20PF HC-49S/SMD; footprint (none) -> digikey-footprints:SMD-2_3.2x2.5mm; symbol GeneralPurposeAlarmDevicePCB-rescue:NX3225GD-8MHZ-STD-CRA-3-dk_Crystals -> Device:Crystal
Connections:
- net +5V: now also C109.1
- net Aref: now also C106.1, C112.1
- net GND: now also C102.2, C106.2, C109.2, C112.2, D102.2 (A), D105.2 (A)
- net Vin: now also C102.1
- net at C104.1, U102.7 (XTAL1/PB6): now also XTAL101.1
- net at C107.1, U102.8 (XTAL2/PB7): now also XTAL101.2
- net at R103.1: now also D102.1 (K)
- net at R110.1: now also D105.1 (K)
- no-connect marks 3 -> 2

Commit message: Update buzzer foot print. Fully connect all parts. Fix numerous silkscreen conflicts. Mix of metric and imperial grid.
Parts:
- added R111: 330R, Resistor_SMD:R_0603_1608Metric, symbol Device:R
- J101: Manufacturier (none) -> XKB Connectivity / Tensility International Corp
Connections:
- net nRESET: now also R111.1; no longer A101.3 (~{RESET})
- new net: A101.3 (~{RESET}), R111.2
Other:
- sheet USB_UART ports: added VBus; removed VBUS
Changed lines of the file:
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@@
     (stroke (width 0) (type default) (color 0 0 0 0))
   )
+  (wire (pts (xy 218.44 118.11) (xy 217.17 118.11))
+    (stroke (width 0) (type default) (color 0 0 0 0))
+  )
   (wire (pts (xy 120.65 87.63) (xy 140.97 87.63))
     (stroke (width 0) (type default) (color 0 0 0 0))
@@
     (stroke (width 0) (type default) (color 0 0 0 0))
   )
+  (wire (pts (xy 219.71 113.03) (xy 218.44 113.03))
+    (stroke (width 0) (type default) (color 0 0 0 0))
+  )
   (wire (pts (xy 85.09 24.13) (xy 88.9 24.13))
     (stroke (width 0) (type default) (color 0 0 0 0))
@@
     (stroke (width 0) (type default) (color 0 0 0 0))
   )
+  (wire (pts (xy 218.44 113.03) (xy 218.44 118.11))
+    (stroke (width 0) (type default) (color 0 0 0 0))
+  )
   (wire (pts (xy 52.07 36.83) (xy 52.07 39.37))
     (stroke (width 0) (type default) (color 0 0 0 0))
@@
     )
   )
-  (global_label "nRESET" (shape passive) (at 209.55 118.11 0) (fields_autoplaced)
+  (global_label "nRESET" (shape passive) (at 219.71 113.03 0) (fields_autoplaced)
     (effects (font (size 1.27 1.27)) (justify left))
-    (property "Intersheet References" "${INTERSHEET_REFS}" (id 0) (at 0 0 0)
+    (property "Intersheet References" "${INTERSHEET_REFS}" (id 0) (at 10.16 -5.08 0)
       (effects (font (size 1.27 1.27)) hide)
     )
@@
       (effects (font (size 1.27 1.27)) hide)
     )
+    (property "Manufacturier" "XKB Connectivity / Tensility International Corp" (id 11) (at 21.59 26.67 0)
+      (effects (font (size 1.27 1.27)) hide)
+    )
     (pin "1")
     (pin "2")
@@
       (effects (font (size 1.27 1.27)) (justify left) hide)
     )
-    (property "Datasheet" "https://datasheet.lcsc.com/lcsc/1806131741_Littelfuse-0603L075SLYR_C207016.pdf" (id 3) (at 39.37 24.13 0)
+    (property "Datasheet" "~" (id 3) (at 39.37 24.13 0)
       (effects (font (size 1.27 1.27)) hide)
     )
@@
     (pin "9")
   )
+  (symbol (lib_id "Device:R") (at 213.36 118.11 270) (unit 1)
+    (in_bom yes) (on_board yes)
+    (property "Reference" "R111" (id 0) (at 212.09 113.03 90))
+    (property "Value" "330R" (id 1) (at 213.36 115.57 90))
+    (property "Footprint" "Resistor_SMD:R_0603_1608Metric" (id 2) (at 213.36 116.332 90)
+      (effects (font (size 1.27 1.27)) hide)
+    )
+    (property "Datasheet" "~" (id 3) (at 213.36 118.11 0)
+      (effects (font (size 1.27 1.27)) hide)
+    )
+    (property "Distributor 1" "JLCPCB" (id 4) (at 213.36 118.11 90)
+      (effects (font (size 1.27 1.27)) hide)
+    )
+    (property "Distributor 1 PN" "C269711" (id 5) (at 213.36 118.11 90)
+      (effects (font (size 1.27 1.27)) hide)
+    )
+    (property "Manufacturer" "TyoHM" (id 6) (at 213.36 118.11 90)
+      (effects (font (size 1.27 1.27)) hide)
+    )
+    (property "MPN" "RMC06033301%N" (id 7) (at 213.36 118.11 90)
+      (effects (font (size 1.27 1.27)) hide)
+    )
+    (property "Description" "0.1W ±1% 330Ω 0603 Chip Resistor - Surface Mount ROHS" (id 8) (at 213.36 118.11 0)
+      (effects (font (size 1.27 1.27)) hide)
+    )
+    (pin "1")
+    (pin "2")
+  )
   (sheet (at 243.84 135.89) (size 20.32 29.21) (fields_autoplaced)
     (stroke (width 0) (type solid) (color 0 0 0 0))
@@
       (effects (font (size 1.27 1.27)) (justify right))
     )
-    (pin "VBUS" passive (at 46.99 177.8 0)
+    (pin "VBus" passive (at 46.99 177.8 0)
       (effects (font (size 1.27 1.27)) (justify right))
     )
@@
       (reference "A101") (unit 1) (value "Arduino_UNO_R3_Shield") (footprint "Module:Arduino_UNO_R3")
     )
-    (path "/00000000-0000-0000-0000-000062dd8e5f/00000000-0000-0000-0000-000062ccb6c9"
-      (reference "BZ601") (unit 1) (value "QMB-09B-03") (footprint "Buzzer_Beeper:MagneticBuzzer_PUI_AT-0927-TT-6-R")
+    (path "/00000000-0000-0000-0000-000062dd8e5f/5897491e-9402-49c5-a894-b7415b30b227"
+      (reference "BZ601") (unit 1) (value "Buzzer_12.2mm_H6.5mm") (footprint "Buzzer_Beeper:Buzzer_TDK_PS1240P02BT_D12.2mm_H6.5mm")
     )
     (path "/00000000-0000-0000-0000-000062b4bd4b"
@@
     )
     (path "/00000000-0000-0000-0000-000062bc4e7e/00000000-0000-0000-0000-000062e66b23"
-      (reference "J501") (unit 1) (value "USB_B_Micro") (footprint "Connector_USB:USB_Micro-B_Wuerth_629105150521")
+      (reference "J501") (unit 1) (value "USB_B_Micro") (footprint "GeneralPurposeAlarmDevicePCB:USB_Micro-B_Amphenol_10118194_Horizontal")
     )
     (path "/00000000-0000-0000-0000-000062dd8e5f/00000000-0000-0000-0000-00006301024b"
@@
       (reference "R110") (unit 1) (value "330R") (footprint "Resistor_SMD:R_0603_1608Metric")
     )
+    (path "/5716d05c-8ea0-453d-90d5-7f037f812389"
+      (reference "R111") (unit 1) (value "330R") (footprint "Resistor_SMD:R_0603_1608Metric")
+    )
     (path "/00000000-0000-0000-0000-000062b3ac2f/00000000-0000-0000-0000-000062b5a2ae"
       (reference "R201") (unit 1) (value "4K7") (footprint "Resistor_SMD:R_0603_1608Metric")
@@
       (reference "U301") (unit 1) (value "PCF8574AT") (footprint "Package_SO:SOIC-16W_5.3x10.2mm_P1.27mm")
     )
-    (path "/00000000-0000-0000-0000-000062b871ee/00000000-0000-0000-0000-000062b90f17"
-      (reference "U302") (unit 1) (value "LCD_20x4_Character") (footprint "GeneralPurposeAlarmDevicePCB:LCD_2004A")
+    (path "/00000000-0000-0000-0000-000062b871ee/2ab4402c-7d6e-4745-b7e2-2505e19e98be"
+      (reference "U302") (unit 1) (value "LCD_20x4_Character-GPAD_SCH_LIB") (footprint "GeneralPurposeAlarmDevicePCB:LCD_2004A")
     )
     (path "/00000000-0000-0000-0000-000062bc4e7e/00000000-0000-0000-0000-000062be3184"

Commit message: Fix pot foot print, Add fifth mounting hole. Place all but UNO and test point.
Parts:
- added H105: MountingHole_Pad_3.5mm, GeneralPurposeAlarmDevicePCB:MountingHole_3.5mm_Pad_Via, symbol GPAD_SCH_LIB:MountingHole_Pad_3.5mm
Connections:
- net GND: now also H105.1
Other:
- moved on the sheet: H101, H102, H103, H104

Commit message: Add 7805 alternative for linear regulator, Add test points on power supply nets, add MechanicalPartsPlacement.pdf.
Parts:
- added TP101: TP_GND, TestPoint:TestPoint_Loop_D2.54mm_Drill1.5mm_Beaded, symbol Connector:TestPoint
- added TP102: TP_Vin, TestPoint:TestPoint_Loop_D2.54mm_Drill1.5mm_Beaded, symbol Connector:TestPoint
- added TP103: TP_+5V, TestPoint:TestPoint_Loop_D2.54mm_Drill1.5mm_Beaded, symbol Connector:TestPoint
- added TP104: TP_VccController, TestPoint:TestPoint_Loop_D2.54mm_Drill1.5mm_Beaded, symbol Connector:TestPoint
- added U103: LM7805_TO220, Package_TO_SOT_THT:TO-220-3_Vertical, symbol Regulator_Linear:LM7805_TO220
- U101: value NCP1117ST50T3G -> DNI
Connections:
- net +5V: now also TP103.1, U103.3 (VO)
- net GND: now also D102.1 (K), D105.1 (K), TP101.1, U103.2 (GND); no longer D102.2 (A), D105.2 (A)
- net Vin: now also TP102.1, U103.1 (VI)
- net at R103.1: now also D102.2 (A); no longer D102.1 (K)
- net at R110.1: now also D105.2 (A); no longer D105.1 (K)
- net Aref renamed VccController
- net VccController: now also TP104.1
Other:
- moved on the sheet: C108, C109, D102, D104, D105, J102, J103, R106, R107, R110, TP_3v3
