File: Hardware/GeneralPurposeAlarmDevicePCB/GeneralPurposeAlarmDevicePCB/GeneralPurposeAlarmDevicePCB.kicad_sch (KiCad schematic)
At the start: 51 parts, among them J101 Barrel_Jack_Switch_SMT, J102 22-23-2021, J103 22-23-2021, J105 S04B-XASK-1(LF)(SN), U101 DNI, U102 PI_ATMEGA328P-AU-InOrder, U103 LM7805_TO220

Commit message: Make JST footprint for J105 in porject library. Change schematic for JST footprint. Import to PCB. Position at exactly 3200. Update User.Drawing.
Parts:
- J105: footprint Connector_PinHeader_2.54mm:PinHeader_1x04_P2.54mm_Horizontal -> GeneralPurposeAlarmDevicePCB:S04B-XASK-1(LF)(SN)
Changed lines of the file:
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@@
       (effects (font (size 1.27 1.27)) (justify right))
     )
-    (property "Footprint" "Connector_PinHeader_2.54mm:PinHeader_1x04_P2.54mm_Horizontal" (id 2) (at 243.84 64.77 0)
+    (property "Footprint" "GeneralPurposeAlarmDevicePCB:S04B-XASK-1(LF)(SN)" (id 2) (at 243.84 64.77 0)
       (effects (font (size 1.524 1.524)) (justify left) hide)
     )
@@
     )
     (path "/00000000-0000-0000-0000-000062d4a7fc"
-      (reference "J105") (unit 1) (value "S04B-XASK-1(LF)(SN)") (footprint "Connector_PinHeader_2.54mm:PinHeader_1x04_P2.54mm_Horizontal")
+      (reference "J105") (unit 1) (value "S04B-XASK-1(LF)(SN)") (footprint "GeneralPurposeAlarmDevicePCB:S04B-XASK-1(LF)(SN)")
     )
     (path "/00000000-0000-0000-0000-000062b93801/00000000-0000-0000-0000-000062d0d90d"

Commit message: Change to LM7805 regulator. Delete the smaller more expensive SMT regulator.
Parts:
- removed U101: DNI, Package_TO_SOT_SMD:SOT-223, symbol GPAD_SCH_LIB:NCP1117ST50T3G
- J101: Manufacturier XKB Connectivity / Tensility International Corp -> (none)
- J102, J103: value 22-23-2021 -> 0.100_2Pin; footprint Connector_Molex:Molex_KK-254_AE-6410-02A_1x02_P2.54mm_Vertical -> Connector_PinHeader_2.54mm:PinHeader_1x02_P2.54mm_Vertical; Cost (none) -> 0.1458; DK_Datasheet_Link https://media.digikey.com/pdf/Data%20Sheets/Molex%20PDFs/A-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 -> (none); DK_Detail_Page /product-detail/en/molex/22-23-2021/WM4200-ND/26667 -> (none); Digi-Key_PN WM4200-ND -> (none); Distributor 1 (none) -> JLCPCB; Distributor 1 PN (none) -> C168673; MPN 22-23-2021 -> 68000-102HLF; Manufacturer Molex -> Amphenol ICC
- U101: renamed from U103; footprint Package_TO_SOT_THT:TO-220-3_Vertical -> Package_TO_SOT_THT:TO-220-3_Horizontal_TabDown; Assembly Type (none) -> HAND; Cost (none) -> 0.1164; Distributor 1 (none) -> JLCPCB; Distributor 1 PN (none) -> C2977083; MPN  (none) -> LM7805CTG; Manufacturer (none) -> HANSCHIP semiconductor
Other:
- moved on the sheet: U101

Commit message: Change TP to show value on F silk screen. Make REF DES smaller.
Parts:
- TP102: value TP_Vin -> Vin
- TP103: value TP_+5V -> +5V
- TP104: value TP_VccController -> VccController
- TP105: renamed from TP_3v3; value TestPoint 3.3V -> 3.3V
Changed lines of the file:
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@@
   (symbol (lib_id "Connector:TestPoint") (at 194.31 101.6 0) (unit 1)
     (in_bom yes) (on_board yes)
-    (property "Reference" "TP_3v3" (id 0) (at 184.15 93.98 0)
-      (effects (font (size 1.27 1.27)) (justify left))
-    )
-    (property "Value" "TestPoint 3.3V" (id 1) (at 184.15 96.52 0)
+    (property "Reference" "TP105" (id 0) (at 184.15 93.98 0)
+      (effects (font (size 1.27 1.27)) (justify left))
+    )
+    (property "Value" "3.3V" (id 1) (at 184.15 96.52 0)
       (effects (font (size 1.27 1.27)) (justify left))
     )
@@
       (effects (font (size 1.27 1.27)) (justify left))
     )
-    (property "Value" "TP_Vin" (id 1) (at 49.53 16.51 0)
+    (property "Value" "Vin" (id 1) (at 49.53 16.51 0)
       (effects (font (size 1.27 1.27)) (justify left))
     )
@@
       (effects (font (size 1.27 1.27)) (justify left))
     )
-    (property "Value" "TP_VccController" (id 1) (at 36.83 83.82 0)
+    (property "Value" "VccController" (id 1) (at 36.83 83.82 0)
       (effects (font (size 1.27 1.27)) (justify left))
     )
@@
       (effects (font (size 1.27 1.27)) (justify left))
     )
-    (property "Value" "TP_+5V" (id 1) (at 105.41 20.32 0)
+    (property "Value" "+5V" (id 1) (at 105.41 20.32 0)
       (effects (font (size 1.27 1.27)) (justify left))
     )
@@
     )
     (path "/03b31824-c9ec-4eb2-b379-23f077cd8439"
-      (reference "TP102") (unit 1) (value "TP_Vin") (footprint "TestPoint:TestPoint_Loop_D2.54mm_Drill1.5mm_Beaded")
+      (reference "TP102") (unit 1) (value "Vin") (footprint "TestPoint:TestPoint_Loop_D2.54mm_Drill1.5mm_Beaded")
     )
     (path "/6fcee3b3-4e61-4f69-8b79-bd71e045ce39"
-      (reference "TP103") (unit 1) (value "TP_+5V") (footprint "TestPoint:TestPoint_Loop_D2.54mm_Drill1.5mm_Beaded")
+      (reference "TP103") (unit 1) (value "+5V") (footprint "TestPoint:TestPoint_Loop_D2.54mm_Drill1.5mm_Beaded")
     )
     (path "/30ce955d-1a78-456a-8adc-fb5342ef2400"
-      (reference "TP104") (unit 1) (value "TP_VccController") (footprint "TestPoint:TestPoint_Loop_D2.54mm_Drill1.5mm_Beaded")
+      (reference "TP104") (unit 1) (value "VccController") (footprint "TestPoint:TestPoint_Loop_D2.54mm_Drill1.5mm_Beaded")
+    )
+    (path "/00000000-0000-0000-0000-000062ddd6fe"
+      (reference "TP105") (unit 1) (value "3.3V") (footprint "TestPoint:TestPoint_Loop_D2.54mm_Drill1.5mm_Beaded")
     )
     (path "/00000000-0000-0000-0000-000062bc4e7e/4d49e72a-82c3-4f7f-a0d6-3ebdc8952d81"
-      (reference "TP201") (unit 1) (value "TP_VBus") (footprint "TestPoint:TestPoint_Loop_D2.54mm_Drill1.5mm_Beaded")
+      (reference "TP201") (unit 1) (value "VBus") (footprint "TestPoint:TestPoint_Loop_D2.54mm_Drill1.5mm_Beaded")
     )
     (path "/00000000-0000-0000-0000-000062bc4e7e/5d43196d-d659-4f19-9c48-4fbf1939a3e8"
-      (reference "TP202") (unit 1) (value "TP_V3") (footprint "TestPoint:TestPoint_Loop_D2.54mm_Drill1.5mm_Beaded")
+      (reference "TP202") (unit 1) (value "V3") (footprint "TestPoint:TestPoint_Loop_D2.54mm_Drill1.5mm_Beaded")
+    )
+    (path "/00000000-0000-0000-0000-000062bc4e7e/addc1ab8-8672-45af-ab9e-760bc1b60a98"
+      (reference "TP203") (unit 1) (value "nCTS") (footprint "TestPoint:TestPoint_Loop_D2.54mm_Drill1.5mm_Beaded")
     )
     (path "/00000000-0000-0000-0000-000062b871ee/dab85703-edaf-43d3-9499-41b59d9a43e0"
-      (reference "TP401") (unit 1) (value "TP_Vcc_LCD") (footprint "TestPoint:TestPoint_Loop_D2.54mm_Drill1.5mm_Beaded")
+      (reference "TP401") (unit 1) (value "Vcc_LCD") (footprint "TestPoint:TestPoint_Loop_D2.54mm_Drill1.5mm_Beaded")
+    )
+    (path "/00000000-0000-0000-0000-000062b871ee/00000000-0000-0000-0000-000062c8b28f"
+      (reference "TP402") (unit 1) (value "nINT") (footprint "TestPoint:TestPoint_Loop_D2.54mm_Drill1.5mm_Beaded")
     )
     (path "/00000000-0000-0000-0000-000062dd8e5f/7dcf7fcf-935c-48c9-afab-acdf96e81919"
-      (reference "TP501") (unit 1) (value "TP_VccBuzzer") (footprint "TestPoint:TestPoint_Loop_D2.54mm_Drill1.5mm_Beaded")
-    )
-    (path "/00000000-0000-0000-0000-000062ddd6fe"
-      (reference "TP_3v3") (unit 1) (value "TestPoint 3.3V") (footprint "TestPoint:TestPoint_Loop_D2.54mm_Drill1.5mm_Beaded")
-    )
-    (path "/00000000-0000-0000-0000-000062bc4e7e/addc1ab8-8672-45af-ab9e-760bc1b60a98"
-      (reference "TP_nCTS201") (unit 1) (value "TestPoint_nCTS") (footprint "TestPoint:TestPoint_Loop_D2.54mm_Drill1.5mm_Beaded")
-    )
-    (path "/00000000-0000-0000-0000-000062b871ee/00000000-0000-0000-0000-000062c8b28f"
-      (reference "TP_nINT301") (unit 1) (value "TestPoint_nINT") (footprint "TestPoint:TestPoint_Loop_D2.54mm_Drill1.5mm_Beaded")
+      (reference "TP501") (unit 1) (value "VccBuzzer") (footprint "TestPoint:TestPoint_Loop_D2.54mm_Drill1.5mm_Beaded")
     )
     (path "/c7a20d25-3819-4e4f-aecf-c5b601fc3576"

Commit message: Mature the BOM parts. Remove misspelled fields. Add some costs.
Parts:
- A101, D102, D105, TP101, TP102, TP103, TP104, TP105: AssemblyType (none) -> HAND
- C104: footprint Capacitor_SMD:C_0603_1608Metric -> Capacitor_SMD:C_0603_1608Metric_Pad1.08x0.95mm_HandSolder
- H101, H102, H103, H104, H105: AssemblyType (none) -> NA
- J101: AssemblyType (none) -> HAND; Cost (none) -> 0.205
- J102, J103, J105, S101: Assembly Type HAND -> (none); AssemblyType (none) -> HAND
- R101, R102, R103, R104, R105, R106, R107, R108, R109, R110, R111: footprint Resistor_SMD:R_0603_1608Metric -> Resistor_SMD:R_0603_1608Metric_Pad0.98x0.95mm_HandSolder
- U101: Assembly Type HAND -> (none); AssemblyType (none) -> HAND; MPN (none) -> LM7805CTG; MPN  LM7805CTG -> (none)

Commit message: Update a lot of cost and PNs from JLCPCB and some Digikey.
Parts:
- A101: Cost (none) -> 1000000
- C101, C104, C107: AssemblyType (none) -> SMT; Cost (none) -> 0.003; Distributor 1 (none) -> JLCPCB; Distributor 1 PN (none) -> C107049; MPN (none) -> CC0603JRNPO9BN390; Manufacturer (none) -> YAGEO
- C102, C106, C109, C112: AssemblyType (none) -> SMT; Cost (none) -> 0.038
- C103, C105, C108, C110, C111: AssemblyType (none) -> SMT; Cost (none) -> 0.0021
- C113, C114: value 33pF -> 39pF; AssemblyType (none) -> SMT; Cost (none) -> 0.003; Distributor 1 PN C107047 -> C107049; MPN CC0603JRNPO9BN330 -> CC0603JRNPO9BN390
- D101, D103, D104: AssemblyType (none) -> SMT; Cost (none) -> 0.0343
- D102: Cost (none) -> 0.0054
- D105: Cost (none) -> 0.36000; Distributor 1 (none) -> DigiKey; Distributor 1 PN (none) -> 160-1682-ND
- F101: AssemblyType (none) -> SMT; Cost (none) -> 0.2448; Distributor 1 (none) -> JLCPCB; Distributor 1 PN (none) -> C207017
- H101, H102, H103, H104, H105: Cost (none) -> 0; Distributor 1 (none) -> NA; Distributor 1 PN (none) -> NA
- J105: Cost (none) -> 0.1517
- R101, R102, R103, R104, R105, R106, R107, R108, R109, R110, R111: AssemblyType (none) -> SMT; Cost (none) -> 0.0015
- S101: Cost (none) -> 0.0315
- U102: AssemblyType (none) -> SMT; Cost (none) -> 6.0206; Distributor 1 DigiKey -> JLCPCB; Distributor 1 PN ATMEGA328P-AU-ND -> C14877; Distributor 2 (none) -> DigiKey; Distributor 2 PN (none) -> ATMEGA328P-AU-ND
- XTAL101: AssemblyType (none) -> SMT; Cost (none) -> 0.0853

Commit message: Update with a place holder for cost of PCB.
Parts:
- added MF101: PCB_GPAD_VER1, NA, symbol GPAD_SCH_LIB:PCB_GPAD_VER1
Changed lines of the file:
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@@
     (pin "1")
+  )
+  (symbol (lib_id "GPAD_SCH_LIB:PCB_GPAD_VER1") (at 177.8 71.12 0) (unit 1)
+    (in_bom yes) (on_board no)
+    (property "Reference" "MF101" (id 0) (at 175.26 59.69 0)
+      (effects (font (size 1.27 1.27)) (justify left))
+    )
+    (property "Value" "PCB_GPAD_VER1" (id 1) (at 171.45 76.2 0)
+      (effects (font (size 1.27 1.27)) (justify left))
+    )
+    (property "Footprint" "NA" (id 2) (at 177.8 71.12 0)
+      (effects (font (size 1.27 1.27)) hide)
+    )
+    (property "Datasheet" "https://www.mcmaster.com/catalog/128/3306" (id 3) (at 177.8 71.12 0)
+      (effects (font (size 1.27 1.27)) hide)
+    )
+    (property "Distributor 1" "PublicInvention" (id 4) (at 177.8 71.12 0)
+      (effects (font (size 1.27 1.27)) hide)
+    )
+    (property "Distributor 1 PN" "PCB_GPAD_V1" (id 5) (at 177.8 71.12 0)
+      (effects (font (size 1.27 1.27)) hide)
+    )
+    (property "Cost" "1000000" (id 6) (at 177.8 71.12 0)
+      (effects (font (size 1.27 1.27)) hide)
+    )
+    (property "AssemblyType" "HAND" (id 7) (at 177.8 71.12 0)
+      (effects (font (size 1.27 1.27)) hide)
+    )
+    (property "Description" "PCB for GPAD Version 1" (id 8) (at 177.8 71.12 0)
+      (effects (font (size 1.27 1.27)) hide)
+    )
+    (property "MPN" "PCB_GPAD_V1" (id 9) (at 177.8 71.12 0)
+      (effects (font (size 1.27 1.27)) hide)
+    )
   )
   (symbol (lib_id "GPAD_SCH_LIB:MountingHole_Pad_3.5mm") (at 130.81 190.5 0) (unit 1)
@@
       (reference "J601") (unit 1) (value "22-23-2021") (footprint "Connector_Molex:Molex_KK-254_AE-6410-02A_1x02_P2.54mm_Vertical")
     )
+    (path "/1ac3cf10-4c07-4a47-a37c-e10545089899"
+      (reference "MF101") (unit 1) (value "PCB_GPAD_VER1") (footprint "NA")
+    )
     (path "/00000000-0000-0000-0000-000062b871ee/fbcd2f6c-e85f-48ea-bb94-218dde6e448f"
