File: Hardware/GeneralPurposeAlarmDevicePCB/GeneralPurposeAlarmDevicePCB/GeneralPurposeAlarmDevicePCB.kicad_sch (KiCad schematic)
At the start: 51 parts, among them J101 Barrel_Jack_Switch_SMT, J102 0.100_2Pin, J103 0.100_2Pin, J105 S04B-XASK-1(LF)(SN), U101 LM7805_TO220, U102 PI_ATMEGA328P-AU-InOrder

Commit message: Update with a place holder for cost of enclosure.
Parts:
- added MF102: ENCLOSURE_GPAD_VER1, symbol GPAD_SCH_LIB:ENCLOSURE_GPAD_VER1
Other:
- moved on the sheet: MF101
Changed lines of the file:
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@@
     (effects (font (size 1.27 1.27)) (justify left bottom))
   )
-  (text "UNO Headers" (at 168.91 92.71 0)
+  (text "UNO Headers" (at 163.83 100.33 0)
     (effects (font (size 1.27 1.27)) (justify left bottom))
   )
@@
   (symbol (lib_id "Connector:TestPoint") (at 194.31 101.6 0) (unit 1)
     (in_bom yes) (on_board yes)
-    (property "Reference" "TP105" (id 0) (at 184.15 93.98 0)
+    (property "Reference" "TP105" (id 0) (at 186.69 99.06 0)
       (effects (font (size 1.27 1.27)) (justify left))
     )
-    (property "Value" "3.3V" (id 1) (at 184.15 96.52 0)
+    (property "Value" "3.3V" (id 1) (at 189.23 101.6 0)
       (effects (font (size 1.27 1.27)) (justify left))
     )
@@
     (pin "1")
   )
-  (symbol (lib_id "GPAD_SCH_LIB:PCB_GPAD_VER1") (at 177.8 71.12 0) (unit 1)
+  (symbol (lib_id "GPAD_SCH_LIB:PCB_GPAD_VER1") (at 190.5 80.01 0) (unit 1)
     (in_bom yes) (on_board no)
-    (property "Reference" "MF101" (id 0) (at 175.26 59.69 0)
+    (property "Reference" "MF101" (id 0) (at 187.96 68.58 0)
       (effects (font (size 1.27 1.27)) (justify left))
     )
-    (property "Value" "PCB_GPAD_VER1" (id 1) (at 171.45 76.2 0)
+    (property "Value" "PCB_GPAD_VER1" (id 1) (at 184.15 78.74 0)
       (effects (font (size 1.27 1.27)) (justify left))
     )
-    (property "Footprint" "NA" (id 2) (at 177.8 71.12 0)
+    (property "Footprint" "NA" (id 2) (at 190.5 80.01 0)
       (effects (font (size 1.27 1.27)) hide)
     )
-    (property "Datasheet" "https://www.mcmaster.com/catalog/128/3306" (id 3) (at 177.8 71.12 0)
+    (property "Datasheet" "https://www.mcmaster.com/catalog/128/3306" (id 3) (at 190.5 80.01 0)
       (effects (font (size 1.27 1.27)) hide)
     )
-    (property "Distributor 1" "PublicInvention" (id 4) (at 177.8 71.12 0)
+    (property "Distributor 1" "PublicInvention" (id 4) (at 190.5 80.01 0)
       (effects (font (size 1.27 1.27)) hide)
     )
-    (property "Distributor 1 PN" "PCB_GPAD_V1" (id 5) (at 177.8 71.12 0)
+    (property "Distributor 1 PN" "PCB_GPAD_V1" (id 5) (at 190.5 80.01 0)
       (effects (font (size 1.27 1.27)) hide)
     )
-    (property "Cost" "1000000" (id 6) (at 177.8 71.12 0)
+    (property "Cost" "1000000" (id 6) (at 190.5 80.01 0)
       (effects (font (size 1.27 1.27)) hide)
     )
-    (property "AssemblyType" "HAND" (id 7) (at 177.8 71.12 0)
+    (property "AssemblyType" "HAND" (id 7) (at 190.5 80.01 0)
       (effects (font (size 1.27 1.27)) hide)
     )
-    (property "Description" "PCB for GPAD Version 1" (id 8) (at 177.8 71.12 0)
+    (property "Description" "PCB for GPAD Version 1" (id 8) (at 190.5 80.01 0)
       (effects (font (size 1.27 1.27)) hide)
     )
-    (property "MPN" "PCB_GPAD_V1" (id 9) (at 177.8 71.12 0)
+    (property "MPN" "PCB_GPAD_V1" (id 9) (at 190.5 80.01 0)
       (effects (font (size 1.27 1.27)) hide)
     )
@@
     (pin "2")
   )
+  (symbol (lib_id "GPAD_SCH_LIB:ENCLOSURE_GPAD_VER1") (at 190.5 53.34 0) (unit 1)
+    (in_bom yes) (on_board no)
+    (property "Reference" "MF102" (id 0) (at 186.69 41.91 0)
+      (effects (font (size 1.27 1.27)) (justify left))
+    )
+    (property "Value" "ENCLOSURE_GPAD_VER1" (id 1) (at 180.34 50.8 0)
+      (effects (font (size 1.27 1.27)) (justify left))
+    )
+    (property "Footprint" "" (id 2) (at 190.5 53.34 0)
+      (effects (font (size 1.27 1.27)) hide)
+    )
+    (property "Datasheet" "https://www.mcmaster.com/catalog/128/3306" (id 3) (at 190.5 53.34 0)
+      (effects (font (size 1.27 1.27)) hide)
+    )
+    (property "Distributor 1" "PublicInvention" (id 4) (at 190.5 53.34 0)
+      (effects (font (size 1.27 1.27)) hide)
+    )
+    (property "Distributor 1 PN" "ENCLOSURE_GPAD_VER1" (id 5) (at 190.5 53.34 0)
+      (effects (font (size 1.27 1.27)) hide)
+    )
+    (property "Cost" "1000000" (id 6) (at 190.5 53.34 0)
+      (effects (font (size 1.27 1.27)) hide)
+    )
+  )
   (symbol (lib_id "Connector:TestPoint") (at 22.86 40.64 0) (unit 1)
     (in_bom yes) (on_board yes)
@@
       (reference "MF101") (unit 1) (value "PCB_GPAD_VER1") (footprint "NA")
     )
+    (path "/609751d7-2460-4a48-8bd6-11c461bf85a7"
+      (reference "MF102") (unit 1) (value "ENCLOSURE_GPAD_VER1") (footprint "")
+    )
     (path "/00000000-0000-0000-0000-000062b871ee/fbcd2f6c-e85f-48ea-bb94-218dde6e448f"

Commit message: Update crystal footprint for proper SMT. Position compoonents for routing. Add resistor to attenuate audio.
Parts:
- XTAL101: footprint digikey-footprints:SMD-2_3.2x2.5mm -> Crystal:Crystal_SMD_HC49-SD
Changed lines of the file:
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@@
     (property "Reference" "XTAL101" (id 0) (at 53.34 115.824 0))
     (property "Value" "16MHZ 20PF HC-49S/SMD" (id 1) (at 55.88 118.11 0))
-    (property "Footprint" "digikey-footprints:SMD-2_3.2x2.5mm" (id 2) (at 53.34 121.92 0)
+    (property "Footprint" "Crystal:Crystal_SMD_HC49-SD" (id 2) (at 53.34 121.92 0)
       (effects (font (size 1.27 1.27)) hide)
     )
@@
       (reference "#PWR0507") (unit 1) (value "GND") (footprint "")
     )
+    (path "/00000000-0000-0000-0000-000062dd8e5f/fa5ebd36-5f6b-4b8c-867f-a63bd41bbb22"
+      (reference "#PWR0508") (unit 1) (value "GND") (footprint "")
+    )
     (path "/00000000-0000-0000-0000-000062dd8e5f/00000000-0000-0000-0000-000062dea4d9"
       (reference "#PWR0601") (unit 1) (value "+5V") (footprint "")
@@
       (reference "R504") (unit 1) (value "4K7") (footprint "Resistor_SMD:R_0603_1608Metric_Pad0.98x0.95mm_HandSolder")
     )
+    (path "/00000000-0000-0000-0000-000062dd8e5f/10551ca1-d6a7-406a-82bf-3bf09f7bf6ac"
+      (reference "R505") (unit 1) (value "10K") (footprint "Resistor_SMD:R_0603_1608Metric_Pad0.98x0.95mm_HandSolder")
+    )
     (path "/00000000-0000-0000-0000-000062dd8e5f/00000000-0000-0000-0000-000062dea4d3"
       (reference "R601") (unit 1) (value "1R") (footprint "Resistor_SMD:R_0603_1608Metric_Pad0.98x0.95mm_HandSolder")
@@
     )
     (path "/00000000-0000-0000-0000-000062b3a927"
-      (reference "XTAL101") (unit 1) (value "16MHZ 20PF HC-49S/SMD") (footprint "digikey-footprints:SMD-2_3.2x2.5mm")
-    )
-  )
+      (reference "XTAL101") (unit 1) (value "16MHZ 20PF HC-49S/SMD") (footprint "Crystal:Crystal_SMD_HC49-SD")
+    )
+  )
