File: Hardware/GeneralPurposeAlarmDevicePCB/GeneralPurposeAlarmDevicePCB/LCD And I2C Interface.kicad_sch (KiCad schematic)
At the start: 19 parts, among them Q301 BSS138, U301 PCF8574AT, U302 LCD_20x4_Character-GPAD_SCH_L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

Commit message: Change TP to show value on F silk screen. Make REF DES smaller.
Parts:
- TP401: value TP_Vcc_LCD -> Vcc_LCD
- TP402: renamed from TP_nINT301; value TestPoint_nINT -> nINT
Changed lines of the file:
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@@
   (symbol (lib_id "Connector:TestPoint") (at 139.7 106.68 180) (unit 1)
     (in_bom yes) (on_board yes)
-    (property "Reference" "TP_nINT301" (id 0) (at 147.32 107.95 0)
-      (effects (font (size 1.27 1.27)) (justify left))
-    )
-    (property "Value" "TestPoint_nINT" (id 1) (at 149.86 113.03 0)
+    (property "Reference" "TP402" (id 0) (at 143.51 107.95 0)
+      (effects (font (size 1.27 1.27)) (justify left))
+    )
+    (property "Value" "nINT" (id 1) (at 144.78 113.03 0)
       (effects (font (size 1.27 1.27)) (justify left))
     )
@@
       (effects (font (size 1.27 1.27)) (justify left))
     )
-    (property "Value" "TP_Vcc_LCD" (id 1) (at 224.79 34.29 0)
-      (effects (font (size 1.27 1.27)) (justify left))
-    )
+    (property "Value" "Vcc_LCD" (id 1) (at 224.79 34.29 0)
+      (effects (font (size 1.27 1.27)) (justify left))
+    )

Commit message: Add cost LCD, Add screw, spacer and nut to symbol library. Add screw and nut to schematic.
Parts:
- added MF? (x4): Screw_4-40_0.375_Phillips, symbol GPAD_SCH_LIB:Screw_4-40_0.375_Phillips
- added MF?: Nut_4-40_Lock,_External-Tooth, symbol GPAD_SCH_LIB:Nut_4-40_Lock,_External-Tooth
Changed lines of the file:
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@@
     (pin "9")
+  )
+  (symbol (lib_id "GPAD_SCH_LIB:Screw_4-40_0.375_Phillips") (at 55.88 123.19 0) (unit 1)
+    (in_bom yes) (on_board no) (fields_autoplaced)
+    (property "Reference" "MF?" (id 0) (at 59.69 121.9199 0)
+      (effects (font (size 1.27 1.27)) (justify left))
+    )
+    (property "Value" "Screw_4-40_0.375_Phillips" (id 1) (at 59.69 124.4599 0)
+      (effects (font (size 1.27 1.27)) (justify left))
+    )
+    (property "Footprint" "" (id 2) (at 55.88 123.19 0)
+      (effects (font (size 1.27 1.27)) hide)
+    )
+    (property "Datasheet" "https://www.mcmaster.com/catalog/128/3306" (id 3) (at 55.88 123.19 0)
+      (effects (font (size 1.27 1.27)) hide)
+    )
+    (property "Distributor 1" "McMaster-Carr" (id 4) (at 55.88 123.19 0)
+      (effects (font (size 1.27 1.27)) hide)
+    )
+    (property "Distributor 1 PN" "90272A108" (id 5) (at 55.88 123.19 0)
+      (effects (font (size 1.27 1.27)) hide)
+    )
+    (property "Cost" "0.0182" (id 6) (at 55.88 123.19 0)
+      (effects (font (size 1.27 1.27)) hide)
+    )
   )
   (symbol (lib_id "GPAD_SCH_LIB:POT 0.375 10K") (at 209.55 68.58 180) (unit 1)
@@
     (pin "3")
   )
+  (symbol (lib_id "GPAD_SCH_LIB:Screw_4-40_0.375_Phillips") (at 90.17 123.19 0) (unit 1)
+    (in_bom yes) (on_board no) (fields_autoplaced)
+    (property "Reference" "MF?" (id 0) (at 93.98 121.9199 0)
+      (effects (font (size 1.27 1.27)) (justify left))
+    )
+    (property "Value" "Screw_4-40_0.375_Phillips" (id 1) (at 93.98 124.4599 0)
+      (effects (font (size 1.27 1.27)) (justify left))
+    )
+    (property "Footprint" "" (id 2) (at 90.17 123.19 0)
+      (effects (font (size 1.27 1.27)) hide)
+    )
+    (property "Datasheet" "https://www.mcmaster.com/catalog/128/3306" (id 3) (at 90.17 123.19 0)
+      (effects (font (size 1.27 1.27)) hide)
+    )
+    (property "Distributor 1" "McMaster-Carr" (id 4) (at 90.17 123.19 0)
+      (effects (font (size 1.27 1.27)) hide)
+    )
+    (property "Distributor 1 PN" "90272A108" (id 5) (at 90.17 123.19 0)
+      (effects (font (size 1.27 1.27)) hide)
+    )
+    (property "Cost" "0.0182" (id 6) (at 90.17 123.19 0)
+      (effects (font (size 1.27 1.27)) hide)
+    )
+  )
+  (symbol (lib_id "GPAD_SCH_LIB:Screw_4-40_0.375_Phillips") (at 124.46 123.19 0) (unit 1)
+    (in_bom yes) (on_board no) (fields_autoplaced)
+    (property "Reference" "MF?" (id 0) (at 128.27 121.9199 0)
+      (effects (font (size 1.27 1.27)) (justify left))
+    )
+    (property "Value" "Screw_4-40_0.375_Phillips" (id 1) (at 128.27 124.4599 0)
+      (effects (font (size 1.27 1.27)) (justify left))
+    )
+    (property "Footprint" "" (id 2) (at 124.46 123.19 0)
+      (effects (font (size 1.27 1.27)) hide)
+    )
+    (property "Datasheet" "https://www.mcmaster.com/catalog/128/3306" (id 3) (at 124.46 123.19 0)
+      (effects (font (size 1.27 1.27)) hide)
+    )
+    (property "Distributor 1" "McMaster-Carr" (id 4) (at 124.46 123.19 0)
+      (effects (font (size 1.27 1.27)) hide)
+    )
+    (property "Distributor 1 PN" "90272A108" (id 5) (at 124.46 123.19 0)
+      (effects (font (size 1.27 1.27)) hide)
+    )
+    (property "Cost" "0.0182" (id 6) (at 124.46 123.19 0)
+      (effects (font (size 1.27 1.27)) hide)
+    )
+  )
+  (symbol (lib_id "GPAD_SCH_LIB:Nut_4-40_Lock,_External-Tooth") (at 19.05 157.48 0) (unit 1)
+    (in_bom yes) (on_board no) (fields_autoplaced)
+    (property "Reference" "MF?" (id 0) (at 25.4 156.2099 0)
+      (effects (font (size 1.27 1.27)) (justify left))
+    )
+    (property "Value" "Nut_4-40_Lock,_External-Tooth" (id 1) (at 25.4 158.7499 0)
+      (effects (font (size 1.27 1.27)) (justify left))
+    )
+    (property "Footprint" "" (id 2) (at 19.05 157.48 0)
+      (effects (font (size 1.27 1.27)) hide)
+    )
+    (property "Datasheet" "https://www.mcmaster.com/catalog/128/3306" (id 3) (at 19.05 157.48 0)
+      (effects (font (size 1.27 1.27)) hide)
+    )
+    (property "Distributor 1" "McMaster-Carr" (id 4) (at 19.05 157.48 0)
+      (effects (font (size 1.27 1.27)) hide)
+    )
+    (property "Distributor 1 PN" "93590A107" (id 5) (at 19.05 157.48 0)
+      (effects (font (size 1.27 1.27)) hide)
+    )
+    (property "Cost" "0.0392" (id 6) (at 19.05 157.48 0)
+      (effects (font (size 1.27 1.27)) hide)
+    )
+  )
   (symbol (lib_id "Connector:TestPoint") (at 223.52 35.56 0) (unit 1)
     (in_bom yes) (on_board yes)
@@
     (pin "1")
   )
+  (symbol (lib_id "GPAD_SCH_LIB:Screw_4-40_0.375_Phillips") (at 19.05 123.19 0) (unit 1)
+    (in_bom yes) (on_board no) (fields_autoplaced)
+    (property "Reference" "MF?" (id 0) (at 22.86 121.9199 0)
+      (effects (font (size 1.27 1.27)) (justify left))
+    )
+    (property "Value" "Screw_4-40_0.375_Phillips" (id 1) (at 22.86 124.4599 0)
+      (effects (font (size 1.27 1.27)) (justify left))
+    )
+    (property "Footprint" "" (id 2) (at 19.05 123.19 0)
+      (effects (font (size 1.27 1.27)) hide)
+    )
+    (property "Datasheet" "https://www.mcmaster.com/catalog/128/3306" (id 3) (at 19.05 123.19 0)
+      (effects (font (size 1.27 1.27)) hide)
+    )
+    (property "Distributor 1" "McMaster-Carr" (id 4) (at 19.05 123.19 0)
+      (effects (font (size 1.27 1.27)) hide)
+    )
+    (property "Distributor 1 PN" "90272A108" (id 5) (at 19.05 123.19 0)
+      (effects (font (size 1.27 1.27)) hide)
+    )
+    (property "Cost" "0.0182" (id 6) (at 19.05 123.19 0)
+      (effects (font (size 1.27 1.27)) hide)
+    )
+  )
 )

Commit message: Add again nuts and spacers to schematic. Fix cost in Symbol library.
Parts:
- added MF402, MF405, MF408, MF411: Spacer_0.0182x0.125 inch, symbol GPAD_SCH_LIB:Spacer_0.0182x0.125 inch
- added MF406, MF409, MF412: Nut_4-40_Lock,_External-Tooth, symbol GPAD_SCH_LIB:Nut_4-40_Lock,_External-Tooth
- gave numbers to parts that had none: 5
Changed lines of the file:
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@@
     (pin "2")
+  )
+  (symbol (lib_id "GPAD_SCH_LIB:Nut_4-40_Lock,_External-Tooth") (at 90.17 157.48 0) (unit 1)
+    (in_bom yes) (on_board no) (fields_autoplaced)
+    (property "Reference" "MF409" (id 0) (at 96.52 156.2099 0)
+      (effects (font (size 1.27 1.27)) (justify left))
+    )
+    (property "Value" "Nut_4-40_Lock,_External-Tooth" (id 1) (at 96.52 158.7499 0)
+      (effects (font (size 1.27 1.27)) (justify left))
+    )
+    (property "Footprint" "" (id 2) (at 90.17 157.48 0)
+      (effects (font (size 1.27 1.27)) hide)
+    )
+    (property "Datasheet" "https://www.mcmaster.com/catalog/128/3306" (id 3) (at 90.17 157.48 0)
+      (effects (font (size 1.27 1.27)) hide)
+    )
+    (property "Distributor 1" "McMaster-Carr" (id 4) (at 90.17 157.48 0)
+      (effects (font (size 1.27 1.27)) hide)
+    )
+    (property "Distributor 1 PN" "93590A107" (id 5) (at 90.17 157.48 0)
+      (effects (font (size 1.27 1.27)) hide)
+    )
+    (property "Cost" "0.0392" (id 6) (at 90.17 157.48 0)
+      (effects (font (size 1.27 1.27)) hide)
+    )
+  )
+  (symbol (lib_id "GPAD_SCH_LIB:Spacer_0.0182x0.125 inch") (at 90.17 139.7 0) (unit 1)
+    (in_bom yes) (on_board no) (fields_autoplaced)
+    (property "Reference" "MF408" (id 0) (at 96.52 138.4299 0)
+      (effects (font (size 1.27 1.27)) (justify left))
+    )
+    (property "Value" "Spacer_0.0182x0.125 inch" (id 1) (at 96.52 140.9699 0)
+      (effects (font (size 1.27 1.27)) (justify left))
+    )
+    (property "Footprint" "" (id 2) (at 90.17 139.7 0)
+      (effects (font (size 1.27 1.27)) hide)
+    )
+    (property "Datasheet" "https://www.mcmaster.com/catalog/128/3306" (id 3) (at 90.17 139.7 0)
+      (effects (font (size 1.27 1.27)) hide)
+    )
+    (property "Distributor 1" "McMaster-Carr" (id 4) (at 90.17 139.7 0)
+      (effects (font (size 1.27 1.27)) hide)
+    )
+    (property "Distributor 1 PN" "94639A702" (id 5) (at 90.17 139.7 0)
+      (effects (font (size 1.27 1.27)) hide)
+    )
+    (property "Cost" "0.0392" (id 6) (at 90.17 139.7 0)
+      (effects (font (size 1.27 1.27)) hide)
+    )
   )
   (symbol (lib_id "GPAD_SCH_LIB:LCD_20x4_Character-GPAD_SCH_LIB") (at 185.42 77.47 0) (unit 1)
@@
     (pin "9")
   )
+  (symbol (lib_id "GPAD_SCH_LIB:Nut_4-40_Lock,_External-Tooth") (at 55.88 156.21 0) (unit 1)
+    (in_bom yes) (on_board no) (fields_autoplaced)
+    (property "Reference" "MF406" (id 0) (at 62.23 154.9399 0)
+      (effects (font (size 1.27 1.27)) (justify left))
+    )
+    (property "Value" "Nut_4-40_Lock,_External-Tooth" (id 1) (at 62.23 157.4799 0)
+      (effects (font (size 1.27 1.27)) (justify left))
+    )
+    (property "Footprint" "" (id 2) (at 55.88 156.21 0)
+      (effects (font (size 1.27 1.27)) hide)
+    )
+    (property "Datasheet" "https://www.mcmaster.com/catalog/128/3306" (id 3) (at 55.88 156.21 0)
+      (effects (font (size 1.27 1.27)) hide)
+    )
+    (property "Distributor 1" "McMaster-Carr" (id 4) (at 55.88 156.21 0)
+      (effects (font (size 1.27 1.27)) hide)
+    )
+    (property "Distributor 1 PN" "93590A107" (id 5) (at 55.88 156.21 0)
+      (effects (font (size 1.27 1.27)) hide)
+    )
+    (property "Cost" "0.0392" (id 6) (at 55.88 156.21 0)
+      (effects (font (size 1.27 1.27)) hide)
+    )
+  )
   (symbol (lib_id "GPAD_SCH_LIB:Screw_4-40_0.375_Phillips") (at 55.88 123.19 0) (unit 1)
     (in_bom yes) (on_board no) (fields_autoplaced)
-    (property "Reference" "MF?" (id 0) (at 59.69 121.9199 0)
+    (property "Reference" "MF404" (id 0) (at 59.69 121.9199 0)
       (effects (font (size 1.27 1.27)) (justify left))
     )
@@
     (pin "3")
   )
+  (symbol (lib_id "GPAD_SCH_LIB:Spacer_0.0182x0.125 inch") (at 19.05 138.43 0) (unit 1)
+    (in_bom yes) (on_board no) (fields_autoplaced)
+    (property "Reference" "MF402" (id 0) (at 25.4 137.1599 0)
+      (effects (font (size 1.27 1.27)) (justify left))
+    )
+    (property "Value" "Spacer_0.0182x0.125 inch" (id 1) (at 25.4 139.6999 0)
+      (effects (font (size 1.27 1.27)) (justify left))
+    )
+    (property "Footprint" "" (id 2) (at 19.05 138.43 0)
+      (effects (font (size 1.27 1.27)) hide)
+    )
+    (property "Datasheet" "https://www.mcmaster.com/catalog/128/3306" (id 3) (at 19.05 138.43 0)
+      (effects (font (size 1.27 1.27)) hide)
+    )
+    (property "Distributor 1" "McMaster-Carr" (id 4) (at 19.05 138.43 0)
+      (effects (font (size 1.27 1.27)) hide)
+    )
+    (property "Distributor 1 PN" "94639A702" (id 5) (at 19.05 138.43 0)
+      (effects (font (size 1.27 1.27)) hide)
+    )
+    (property "Cost" "0.0392" (id 6) (at 19.05 138.43 0)
+      (effects (font (size 1.27 1.27)) hide)
+    )
+  )
   (symbol (lib_id "GPAD_SCH_LIB:Screw_4-40_0.375_Phillips") (at 90.17 123.19 0) (unit 1)
     (in_bom yes) (on_board no) (fields_autoplaced)
-    (property "Reference" "MF?" (id 0) (at 93.98 121.9199 0)
+    (property "Reference" "MF407" (id 0) (at 93.98 121.9199 0)
       (effects (font (size 1.27 1.27)) (justify left))
     )
@@
   (symbol (lib_id "GPAD_SCH_LIB:Screw_4-40_0.375_Phillips") (at 124.46 123.19 0) (unit 1)
     (in_bom yes) (on_board no) (fields_autoplaced)
-    (property "Reference" "MF?" (id 0) (at 128.27 121.9199 0)
+    (property "Reference" "MF410" (id 0) (at 128.27 121.9199 0)
       (effects (font (size 1.27 1.27)) (justify left))
     )
@@
     )
   )
+  (symbol (lib_id "GPAD_SCH_LIB:Spacer_0.0182x0.125 inch") (at 55.88 138.43 0) (unit 1)
+    (in_bom yes) (on_board no) (fields_autoplaced)
+    (property "Reference" "MF405" (id 0) (at 62.23 137.1599 0)
+      (effects (font (size 1.27 1.27)) (justify left))
+    )
+    (property "Value" "Spacer_0.0182x0.125 inch" (id 1) (at 62.23 139.6999 0)
+      (effects (font (size 1.27 1.27)) (justify left))
+    )
+    (property "Footprint" "" (id 2) (at 55.88 138.43 0)
+      (effects (font (size 1.27 1.27)) hide)
+    )
+    (property "Datasheet" "https://www.mcmaster.com/catalog/128/3306" (id 3) (at 55.88 138.43 0)
+      (effects (font (size 1.27 1.27)) hide)
+    )
+    (property "Distributor 1" "McMaster-Carr" (id 4) (at 55.88 138.43 0)
+      (effects (font (size 1.27 1.27)) hide)
+    )
+    (property "Distributor 1 PN" "94639A702" (id 5) (at 55.88 138.43 0)
+      (effects (font (size 1.27 1.27)) hide)
+    )
+    (property "Cost" "0.0392" (id 6) (at 55.88 138.43 0)
+      (effects (font (size 1.27 1.27)) hide)
+    )
+  )
+  (symbol (lib_id "GPAD_SCH_LIB:Nut_4-40_Lock,_External-Tooth") (at 127 156.21 0) (unit 1)
+    (in_bom yes) (on_board no) (fields_autoplaced)
+    (property "Reference" "MF412" (id 0) (at 133.35 154.9399 0)
+      (effects (font (size 1.27 1.27)) (justify left))
+    )
+    (property "Value" "Nut_4-40_Lock,_External-Tooth" (id 1) (at 133.35 157.4799 0)
+      (effects (font (size 1.27 1.27)) (justify left))
+    )
+    (property "Footprint" "" (id 2) (at 127 156.21 0)
+      (effects (font (size 1.27 1.27)) hide)
+    )
+    (property "Datasheet" "https://www.mcmaster.com/catalog/128/3306" (id 3) (at 127 156.21 0)
+      (effects (font (size 1.27 1.27)) hide)
+    )
+    (property "Distributor 1" "McMaster-Carr" (id 4) (at 127 156.21 0)
+      (effects (font (size 1.27 1.27)) hide)
+    )
+    (property "Distributor 1 PN" "93590A107" (id 5) (at 127 156.21 0)
+      (effects (font (size 1.27 1.27)) hide)
+    )
+    (property "Cost" "0.0392" (id 6) (at 127 156.21 0)
+      (effects (font (size 1.27 1.27)) hide)
+    )
+  )
   (symbol (lib_id "GPAD_SCH_LIB:Nut_4-40_Lock,_External-Tooth") (at 19.05 157.48 0) (unit 1)
     (in_bom yes) (on_board no) (fields_autoplaced)
-    (property "Reference" "MF?" (id 0) (at 25.4 156.2099 0)
+    (property "Reference" "MF403" (id 0) (at 25.4 156.2099 0)
       (effects (font (size 1.27 1.27)) (justify left))
     )
@@
     (pin "1")
   )
+  (symbol (lib_id "GPAD_SCH_LIB:Spacer_0.0182x0.125 inch") (at 125.73 138.43 0) (unit 1)
+    (in_bom yes) (on_board no) (fields_autoplaced)
+    (property "Reference" "MF411" (id 0) (at 132.08 137.1599 0)
+      (effects (font (size 1.27 1.27)) (justify left))
+    )
+    (property "Value" "Spacer_0.0182x0.125 inch" (id 1) (at 132.08 139.6999 0)
+      (effects (font (size 1.27 1.27)) (justify left))
+    )
+    (property "Footprint" "" (id 2) (at 125.73 138.43 0)
+      (effects (font (size 1.27 1.27)) hide)
+    )
+    (property "Datasheet" "https://www.mcmaster.com/catalog/128/3306" (id 3) (at 125.73 138.43 0)
+      (effects (font (size 1.27 1.27)) hide)
+    )
+    (property "Distributor 1" "McMaster-Carr" (id 4) (at 125.73 138.43 0)
+      (effects (font (size 1.27 1.27)) hide)
+    )
+    (property "Distributor 1 PN" "94639A702" (id 5) (at 125.73 138.43 0)
+      (effects (font (size 1.27 1.27)) hide)
+    )
+    (property "Cost" "0.0392" (id 6) (at 125.73 138.43 0)
+      (effects (font (size 1.27 1.27)) hide)
+    )
+  )
   (symbol (lib_id "GPAD_SCH_LIB:Screw_4-40_0.375_Phillips") (at 19.05 123.19 0) (unit 1)
     (in_bom yes) (on_board no) (fields_autoplaced)
-    (property "Reference" "MF?" (id 0) (at 22.86 121.9199 0)
-      (effects (font (size 1.27 1.27)) (justify left))
-    )
+    (property "Reference" "MF401" (id 0) (at 22.86 121.9199 0)
+      (effects (font (size 1.27 1.27)) (justify left))
+    )

Commit message: Add to schematic, again nuts and spacers to schematic. Fix cost in Symbol library.
Parts:
- MF401, MF403, MF404, MF406, MF407, MF409, MF410, MF412: AssemblyType (none) -> HAND
- MF402, MF405, MF408, MF411: AssemblyType (none) -> HAND; Cost 0.0392 -> 0.1145
Changed lines of the file:
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@@
+      (effects (font (size 1.27 1.27)) hide)
+    )
+    (property "AssemblyType" "HAND" (id 7) (at 90.17 157.48 0)
       (effects (font (size 1.27 1.27)) hide)
     )
@@
       (effects (font (size 1.27 1.27)) hide)
     )
-    (property "Cost" "0.0392" (id 6) (at 90.17 139.7 0)
+    (property "Cost" "0.1145" (id 6) (at 90.17 139.7 0)
+      (effects (font (size 1.27 1.27)) hide)
+    )
+    (property "AssemblyType" "HAND" (id 7) (at 90.17 139.7 0)
       (effects (font (size 1.27 1.27)) hide)
     )
@@
       (effects (font (size 1.27 1.27)) hide)
     )
+    (property "AssemblyType" "HAND" (id 7) (at 55.88 156.21 0)
+      (effects (font (size 1.27 1.27)) hide)
+    )
   )
   (symbol (lib_id "GPAD_SCH_LIB:Screw_4-40_0.375_Phillips") (at 55.88 123.19 0) (unit 1)
@@
     )
     (property "Cost" "0.0182" (id 6) (at 55.88 123.19 0)
+      (effects (font (size 1.27 1.27)) hide)
+    )
+    (property "AssemblyType" "HAND" (id 7) (at 55.88 123.19 0)
       (effects (font (size 1.27 1.27)) hide)
     )
@@
       (effects (font (size 1.27 1.27)) hide)
     )
-    (property "Cost" "0.0392" (id 6) (at 19.05 138.43 0)
+    (property "Cost" "0.1145" (id 6) (at 19.05 138.43 0)
+      (effects (font (size 1.27 1.27)) hide)
+    )
+    (property "AssemblyType" "HAND" (id 7) (at 19.05 138.43 0)
       (effects (font (size 1.27 1.27)) hide)
     )
@@
       (effects (font (size 1.27 1.27)) hide)
     )
+    (property "AssemblyType" "HAND" (id 7) (at 90.17 123.19 0)
+      (effects (font (size 1.27 1.27)) hide)
+    )
   )
   (symbol (lib_id "GPAD_SCH_LIB:Screw_4-40_0.375_Phillips") (at 124.46 123.19 0) (unit 1)
@@
       (effects (font (size 1.27 1.27)) hide)
     )
+    (property "AssemblyType" "HAND" (id 7) (at 124.46 123.19 0)
+      (effects (font (size 1.27 1.27)) hide)
+    )
   )
   (symbol (lib_id "GPAD_SCH_LIB:Spacer_0.0182x0.125 inch") (at 55.88 138.43 0) (unit 1)
@@
       (effects (font (size 1.27 1.27)) hide)
     )
-    (property "Cost" "0.0392" (id 6) (at 55.88 138.43 0)
+    (property "Cost" "0.1145" (id 6) (at 55.88 138.43 0)
+      (effects (font (size 1.27 1.27)) hide)
+    )
+    (property "AssemblyType" "HAND" (id 7) (at 55.88 138.43 0)
       (effects (font (size 1.27 1.27)) hide)
     )
@@
       (effects (font (size 1.27 1.27)) hide)
     )
+    (property "AssemblyType" "HAND" (id 7) (at 127 156.21 0)
+      (effects (font (size 1.27 1.27)) hide)
+    )
   )
   (symbol (lib_id "GPAD_SCH_LIB:Nut_4-40_Lock,_External-Tooth") (at 19.05 157.48 0) (unit 1)
@@
     )
     (property "Cost" "0.0392" (id 6) (at 19.05 157.48 0)
+      (effects (font (size 1.27 1.27)) hide)
+    )
+    (property "AssemblyType" "HAND" (id 7) (at 19.05 157.48 0)
       (effects (font (size 1.27 1.27)) hide)
     )
@@
       (effects (font (size 1.27 1.27)) hide)
     )
-    (property "Cost" "0.0392" (id 6) (at 125.73 138.43 0)
+    (property "Cost" "0.1145" (id 6) (at 125.73 138.43 0)
+      (effects (font (size 1.27 1.27)) hide)
+    )
+    (property "AssemblyType" "HAND" (id 7) (at 125.73 138.43 0)
       (effects (font (size 1.27 1.27)) hide)
     )
@@
       (effects (font (size 1.27 1.27)) hide)
     )
+    (property "AssemblyType" "HAND" (id 7) (at 19.05 123.19 0)
+      (effects (font (size 1.27 1.27)) hide)
+    )
