File: Hardware/GeneralPurposeAlarmDevicePCB/GeneralPurposeAlarmDevicePCB/LCD And I2C Interface.kicad_sch (KiCad schematic)
At the start: 31 parts, among them Q301 BSS138, U301 PCF8574AT, U302 LCD_20x4_Character-GPAD_SCH_L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

Commit message: Mature the BOM parts. Remove misspelled fields. Add some costs.
Parts:
- MF401, MF402, MF403, MF404, MF405, MF406, MF407, MF408, MF409, MF410, MF411, MF412: footprint (none) -> NA
- R301, R302, R303, R304, R305, R306, R307, R308, R309, R310, R311: footprint Resistor_SMD:R_0603_1608Metric -> Resistor_SMD:R_0603_1608Metric_Pad0.98x0.95mm_HandSolder
- RV301: Assembly Type HAND -> (none); Cost (none) -> 0.6963; Manufacturer  BOURNS -> (none)
- TP401, TP402: AssemblyType (none) -> HAND
- U302: Assembly Type HAND -> (none); AssemblyType (none) -> HAND
Changed lines of the file:
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@@
     (property "Reference" "R303" (id 0) (at 110.49 59.69 0))
     (property "Value" "4K7" (id 1) (at 111.76 64.77 0))
-    (property "Footprint" "Resistor_SMD:R_0603_1608Metric" (id 2) (at 109.728 63.5 90)
+    (property "Footprint" "Resistor_SMD:R_0603_1608Metric_Pad0.98x0.95mm_HandSolder" (id 2) (at 109.728 63.5 90)
       (effects (font (size 1.27 1.27)) hide)
     )
@@
     (property "Reference" "R304" (id 0) (at 119.38 59.69 0))
     (property "Value" "1K" (id 1) (at 120.65 64.77 0))
-    (property "Footprint" "Resistor_SMD:R_0603_1608Metric" (id 2) (at 118.618 63.5 90)
+    (property "Footprint" "Resistor_SMD:R_0603_1608Metric_Pad0.98x0.95mm_HandSolder" (id 2) (at 118.618 63.5 90)
       (effects (font (size 1.27 1.27)) hide)
     )
@@
     (property "Reference" "R302" (id 0) (at 100.33 59.69 0))
     (property "Value" "4K7" (id 1) (at 101.6 64.77 0))
-    (property "Footprint" "Resistor_SMD:R_0603_1608Metric" (id 2) (at 99.568 63.5 90)
+    (property "Footprint" "Resistor_SMD:R_0603_1608Metric_Pad0.98x0.95mm_HandSolder" (id 2) (at 99.568 63.5 90)
       (effects (font (size 1.27 1.27)) hide)
     )
@@
     (property "Reference" "R301" (id 0) (at 91.44 59.69 0))
     (property "Value" "4K7" (id 1) (at 92.71 64.77 0))
-    (property "Footprint" "Resistor_SMD:R_0603_1608Metric" (id 2) (at 90.678 63.5 90)
+    (property "Footprint" "Resistor_SMD:R_0603_1608Metric_Pad0.98x0.95mm_HandSolder" (id 2) (at 90.678 63.5 90)
       (effects (font (size 1.27 1.27)) hide)
     )
@@
     (property "Reference" "R310" (id 0) (at 187.96 35.56 90))
     (property "Value" "1R0" (id 1) (at 189.23 38.1 90))
-    (property "Footprint" "Resistor_SMD:R_0603_1608Metric" (id 2) (at 189.23 38.862 90)
+    (property "Footprint" "Resistor_SMD:R_0603_1608Metric_Pad0.98x0.95mm_HandSolder" (id 2) (at 189.23 38.862 90)
       (effects (font (size 1.27 1.27)) hide)
     )
@@
     (property "Reference" "R311" (id 0) (at 208.28 99.06 0))
     (property "Value" "4K7" (id 1) (at 207.01 101.6 0))
-    (property "Footprint" "Resistor_SMD:R_0603_1608Metric" (id 2) (at 204.978 100.33 90)
+    (property "Footprint" "Resistor_SMD:R_0603_1608Metric_Pad0.98x0.95mm_HandSolder" (id 2) (at 204.978 100.33 90)
       (effects (font (size 1.27 1.27)) hide)
     )
@@
     (property "Reference" "R305" (id 0) (at 119.38 91.44 0))
     (property "Value" "1R0" (id 1) (at 120.65 96.52 0))
-    (property "Footprint" "Resistor_SMD:R_0603_1608Metric" (id 2) (at 115.062 95.25 90)
+    (property "Footprint" "Resistor_SMD:R_0603_1608Metric_Pad0.98x0.95mm_HandSolder" (id 2) (at 115.062 95.25 90)
       (effects (font (size 1.27 1.27)) hide)
     )
@@
     (property "Reference" "R307" (id 0) (at 128.27 91.44 0))
     (property "Value" "1R0" (id 1) (at 129.54 96.52 0))
-    (property "Footprint" "Resistor_SMD:R_0603_1608Metric" (id 2) (at 123.952 95.25 90)
+    (property "Footprint" "Resistor_SMD:R_0603_1608Metric_Pad0.98x0.95mm_HandSolder" (id 2) (at 123.952 95.25 90)
       (effects (font (size 1.27 1.27)) hide)
     )
@@
     (property "Reference" "R309" (id 0) (at 135.89 91.44 0))
     (property "Value" "1R0" (id 1) (at 137.16 96.52 0))
-    (property "Footprint" "Resistor_SMD:R_0603_1608Metric" (id 2) (at 131.572 95.25 90)
+    (property "Footprint" "Resistor_SMD:R_0603_1608Metric_Pad0.98x0.95mm_HandSolder" (id 2) (at 131.572 95.25 90)
       (effects (font (size 1.27 1.27)) hide)
     )
@@
     )
     (property "Datasheet" "~" (id 3) (at 134.62 106.68 0)
+      (effects (font (size 1.27 1.27)) hide)
+    )
+    (property "AssemblyType" "HAND" (id 4) (at 139.7 106.68 0)
       (effects (font (size 1.27 1.27)) hide)
     )
@@
     (property "Reference" "R306" (id 0) (at 228.6 55.88 0))
     (property "Value" "DNI" (id 1) (at 229.87 60.96 0))
-    (property "Footprint" "Resistor_SMD:R_0603_1608Metric" (id 2) (at 227.838 59.69 90)
+    (property "Footprint" "Resistor_SMD:R_0603_1608Metric_Pad0.98x0.95mm_HandSolder" (id 2) (at 227.838 59.69 90)
       (effects (font (size 1.27 1.27)) hide)
     )
@@
     (property "Reference" "R308" (id 0) (at 228.6 68.58 0))
     (property "Value" "DNI" (id 1) (at 229.87 73.66 0))
-    (property "Footprint" "Resistor_SMD:R_0603_1608Metric" (id 2) (at 227.838 72.39 90)
+    (property "Footprint" "Resistor_SMD:R_0603_1608Metric_Pad0.98x0.95mm_HandSolder" (id 2) (at 227.838 72.39 90)
       (effects (font (size 1.27 1.27)) hide)
     )
@@
       (effects (font (size 1.27 1.27)) (justify left))
     )
-    (property "Footprint" "" (id 2) (at 90.17 157.48 0)
+    (property "Footprint" "NA" (id 2) (at 90.17 157.48 0)
       (effects (font (size 1.27 1.27)) hide)
     )
@@
       (effects (font (size 1.27 1.27)) (justify left))
     )
-    (property "Footprint" "" (id 2) (at 90.17 139.7 0)
+    (property "Footprint" "NA" (id 2) (at 90.17 139.7 0)
       (effects (font (size 1.27 1.27)) hide)
     )
@@
       (effects (font (size 1.27 1.27)) hide)
     )
-    (property "Assembly Type" "HAND" (id 8) (at 185.42 77.47 0)
+    (property "Assembly Type" "" (id 8) (at 185.42 77.47 0)
       (effects (font (size 1.27 1.27)) hide)
     )
@@
     )
     (property "Manufacturer " "" (id 14) (at 185.42 77.47 0)
+      (effects (font (size 1.27 1.27)) hide)
+    )
+    (property "AssemblyType" "HAND" (id 15) (at 185.42 77.47 0)
       (effects (font (size 1.27 1.27)) hide)
     )
@@
       (effects (font (size 1.27 1.27)) (justify left))
     )
-    (property "Footprint" "" (id 2) (at 55.88 156.21 0)
+    (property "Footprint" "NA" (id 2) (at 55.88 156.21 0)
       (effects (font (size 1.27 1.27)) hide)
     )
@@
       (effects (font (size 1.27 1.27)) (justify left))
     )
-    (property "Footprint" "" (id 2) (at 55.88 123.19 0)
+    (property "Footprint" "NA" (id 2) (at 55.88 123.19 0)
       (effects (font (size 1.27 1.27)) hide)
     )
@@
   (symbol (lib_id "GPAD_SCH_LIB:POT 0.375 10K") (at 209.55 68.58 180) (unit 1)
     (in_bom yes) (on_board yes) (fields_autoplaced)
-    (property "Reference" "RV301" (id 0) (at 212.09 64.6429 0)
+    (property "Reference" "RV301" (id 0) (at 207.01 72.5171 0)
       (effects (font (size 1.27 1.27)) (justify right))
     )
-    (property "Value" "POT 0.375 10K" (id 1) (at 212.09 67.1829 0)
+    (property "Value" "POT 0.375 10K" (id 1) (at 207.01 69.9771 0)
       (effects (font (size 1.27 1.27)) (justify right))
     )
@@
       (effects (font (size 1.27 1.27)) hide)
     )
-    (property "Manufacturier" "" (id 6) (at 209.55 68.58 0)
-      (effects (font (size 1.27 1.27)) hide)
-    )
     (property "MPN" "3386P-1-103LF" (id 7) (at 209.55 68.58 0)
       (effects (font (size 1.27 1.27)) hide)
     )
-    (property "Assembly Type" "HAND" (id 8) (at 212.09 69.7229 0)
+    (property "Assembly Type" "" (id 8) (at 207.01 67.4371 0)
       (effects (font (size 1.27 1.27)) (justify right))
     )
@@
       (effects (font (size 1.27 1.27)) hide)
     )
-    (property "Distributor 2 PN" "3386P-103LF-ND" (id 10) (at 212.09 72.2629 0)
+    (property "Distributor 2 PN" "3386P-103LF-ND" (id 10) (at 207.01 64.8971 0)
       (effects (font (size 1.27 1.27)) (justify right))
     )
-    (property "Cost" "" (id 11) (at 209.55 68.58 0))
+    (property "Cost" "0.6963" (id 11) (at 209.55 68.58 0))
     (property "Manufacturer" "BOURNS" (id 12) (at 209.55 68.58 0)
       (effects (font (size 1.27 1.27)) hide)
     )
-    (property "Manufacturer " "BOURNS" (id 13) (at 209.55 68.58 0)
-      (effects (font (size 1.27 1.27)) hide)
-    )
     (pin "1")
     (pin "2")
@@
       (effects (font (size 1.27 1.27)) (justify left))
     )
-    (property "Footprint" "" (id 2) (at 19.05 138.43 0)
+    (property "Footprint" "NA" (id 2) (at 19.05 138.43 0)
       (effects (font (size 1.27 1.27)) hide)
     )
@@
       (effects (font (size 1.27 1.27)) (justify left))
     )
-    (property "Footprint" "" (id 2) (at 90.17 123.19 0)
+    (property "Footprint" "NA" (id 2) (at 90.17 123.19 0)
       (effects (font (size 1.27 1.27)) hide)
     )
@@
       (effects (font (size 1.27 1.27)) (justify left))
     )
-    (property "Footprint" "" (id 2) (at 124.46 123.19 0)
+    (property "Footprint" "NA" (id 2) (at 124.46 123.19 0)
       (effects (font (size 1.27 1.27)) hide)
     )
@@
       (effects (font (size 1.27 1.27)) (justify left))
     )
-    (property "Footprint" "" (id 2) (at 55.88 138.43 0)
+    (property "Footprint" "NA" (id 2) (at 55.88 138.43 0)
       (effects (font (size 1.27 1.27)) hide)
     )
@@
       (effects (font (size 1.27 1.27)) (justify left))
     )
-    (property "Footprint" "" (id 2) (at 127 156.21 0)
+    (property "Footprint" "NA" (id 2) (at 127 156.21 0)
       (effects (font (size 1.27 1.27)) hide)
     )
@@
       (effects (font (size 1.27 1.27)) (justify left))
     )
-    (property "Footprint" "" (id 2) (at 19.05 157.48 0)
+    (property "Footprint" "NA" (id 2) (at 19.05 157.48 0)
       (effects (font (size 1.27 1.27)) hide)
     )
@@
       (effects (font (size 1.27 1.27)) hide)
     )
+    (property "AssemblyType" "HAND" (id 4) (at 223.52 35.56 0)
+      (effects (font (size 1.27 1.27)) hide)
+    )
     (pin "1")
   )
@@
       (effects (font (size 1.27 1.27)) (justify left))
     )
-    (property "Footprint" "" (id 2) (at 125.73 138.43 0)
+    (property "Footprint" "NA" (id 2) (at 125.73 138.43 0)
       (effects (font (size 1.27 1.27)) hide)
     )
@@
       (effects (font (size 1.27 1.27)) (justify left))
     )
-    (property "Footprint" "" (id 2) (at 19.05 123.19 0)
-      (effects (font (size 1.27 1.27)) hide)
-    )
+    (property "Footprint" "NA" (id 2) (at 19.05 123.19 0)
+      (effects (font (size 1.27 1.27)) hide)
+    )

Commit message: Update a lot of cost and PNs from JLCPCB and some Digikey.
Parts:
- C301: AssemblyType (none) -> SMT; Cost (none) -> 0.0021
- C302: AssemblyType (none) -> SMT; Cost (none) -> 0.038
- Q301: AssemblyType (none) -> SMT; Cost (none) -> 0.0196
- R301, R302, R303, R304, R305, R306, R307, R308, R309, R310, R311: AssemblyType (none) -> SMT; Cost (none) -> 0.0015
- RV301: AssemblyType (none) -> SMT
- U301: AssemblyType (none) -> SMT; Cost (none) -> 0.6414
- U302: Cost (none) -> 4.99; Distributor 1 (none) -> Aliexpress; Distributor 1 PN (none) -> https://www.aliexpress.com/item/3256803213374992.html; Distributor 2 (none) -> Amazon; Distributor 2 PN (none) -> https://www.amazon.com/GeeekPi-Interface-Adapter-Backlight-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
Changed lines of the file:
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@@
+      (effects (font (size 1.27 1.27)) hide)
+    )
+    (property "AssemblyType" "SMT" (id 9) (at 156.21 85.09 0)
+      (effects (font (size 1.27 1.27)) hide)
+    )
+    (property "Cost" "0.6414" (id 10) (at 156.21 85.09 0)
       (effects (font (size 1.27 1.27)) hide)
     )
@@
       (effects (font (size 1.27 1.27)) hide)
     )
+    (property "AssemblyType" "SMT" (id 9) (at 107.95 63.5 0)
+      (effects (font (size 1.27 1.27)) hide)
+    )
+    (property "Cost" "0.0015" (id 10) (at 107.95 63.5 0)
+      (effects (font (size 1.27 1.27)) hide)
+    )
     (pin "1")
     (pin "2")
@@
       (effects (font (size 1.27 1.27)) hide)
     )
+    (property "AssemblyType" "SMT" (id 9) (at 116.84 63.5 0)
+      (effects (font (size 1.27 1.27)) hide)
+    )
+    (property "Cost" "0.0015" (id 10) (at 116.84 63.5 0)
+      (effects (font (size 1.27 1.27)) hide)
+    )
     (pin "1")
     (pin "2")
@@
       (effects (font (size 1.27 1.27)) hide)
     )
+    (property "AssemblyType" "SMT" (id 9) (at 97.79 63.5 0)
+      (effects (font (size 1.27 1.27)) hide)
+    )
+    (property "Cost" "0.0015" (id 10) (at 97.79 63.5 0)
+      (effects (font (size 1.27 1.27)) hide)
+    )
     (pin "1")
     (pin "2")
@@
       (effects (font (size 1.27 1.27)) hide)
     )
+    (property "AssemblyType" "SMT" (id 9) (at 88.9 63.5 0)
+      (effects (font (size 1.27 1.27)) hide)
+    )
+    (property "Cost" "0.0015" (id 10) (at 88.9 63.5 0)
+      (effects (font (size 1.27 1.27)) hide)
+    )
     (pin "1")
     (pin "2")
@@
       (effects (font (size 1.27 1.27)) hide)
     )
+    (property "AssemblyType" "SMT" (id 9) (at 189.23 40.64 0)
+      (effects (font (size 1.27 1.27)) hide)
+    )
+    (property "Cost" "0.0015" (id 10) (at 189.23 40.64 0)
+      (effects (font (size 1.27 1.27)) hide)
+    )
     (pin "1")
     (pin "2")
@@
       (effects (font (size 1.27 1.27)) hide)
     )
+    (property "AssemblyType" "SMT" (id 8) (at 215.9 44.45 0)
+      (effects (font (size 1.27 1.27)) hide)
+    )
+    (property "Cost" "0.038" (id 9) (at 215.9 44.45 0)
+      (effects (font (size 1.27 1.27)) hide)
+    )
     (pin "1")
     (pin "2")
@@
     )
     (property "Description" "50V 100nF X7R ±10% 0603 Multilayer Ceramic Capacitors MLCC - SMD/SMT ROHS" (id 8) (at 203.2 44.45 0)
+      (effects (font (size 1.27 1.27)) hide)
+    )
+    (property "AssemblyType" "SMT" (id 9) (at 203.2 44.45 0)
+      (effects (font (size 1.27 1.27)) hide)
+    )
+    (property "Cost" "0.0021" (id 10) (at 203.2 44.45 0)
       (effects (font (size 1.27 1.27)) hide)
     )
@@
       (effects (font (size 1.27 1.27)) hide)
     )
+    (property "AssemblyType" "SMT" (id 9) (at 203.2 100.33 0)
+      (effects (font (size 1.27 1.27)) hide)
+    )
+    (property "Cost" "0.0015" (id 10) (at 203.2 100.33 0)
+      (effects (font (size 1.27 1.27)) hide)
+    )
     (pin "1")
     (pin "2")
@@
     )
     (property "MPN" "BSS138" (id 9) (at 218.44 104.14 0)
+      (effects (font (size 1.27 1.27)) hide)
+    )
+    (property "AssemblyType" "SMT" (id 10) (at 218.44 104.14 0)
+      (effects (font (size 1.27 1.27)) hide)
+    )
+    (property "Cost" "0.0196" (id 11) (at 218.44 104.14 0)
       (effects (font (size 1.27 1.27)) hide)
     )
@@
       (effects (font (size 1.27 1.27)) hide)
     )
+    (property "AssemblyType" "SMT" (id 9) (at 116.84 95.25 0)
+      (effects (font (size 1.27 1.27)) hide)
+    )
+    (property "Cost" "0.0015" (id 10) (at 116.84 95.25 0)
+      (effects (font (size 1.27 1.27)) hide)
+    )
     (pin "1")
     (pin "2")
@@
       (effects (font (size 1.27 1.27)) hide)
     )
+    (property "AssemblyType" "SMT" (id 9) (at 125.73 95.25 0)
+      (effects (font (size 1.27 1.27)) hide)
+    )
+    (property "Cost" "0.0015" (id 10) (at 125.73 95.25 0)
+      (effects (font (size 1.27 1.27)) hide)
+    )
     (pin "1")
     (pin "2")
@@
       (effects (font (size 1.27 1.27)) hide)
     )
+    (property "AssemblyType" "SMT" (id 9) (at 133.35 95.25 0)
+      (effects (font (size 1.27 1.27)) hide)
+    )
+    (property "Cost" "0.0015" (id 10) (at 133.35 95.25 0)
+      (effects (font (size 1.27 1.27)) hide)
+    )
     (pin "1")
     (pin "2")
@@
       (effects (font (size 1.27 1.27)) hide)
     )
+    (property "AssemblyType" "SMT" (id 9) (at 226.06 59.69 0)
+      (effects (font (size 1.27 1.27)) hide)
+    )
+    (property "Cost" "0.0015" (id 10) (at 226.06 59.69 0)
+      (effects (font (size 1.27 1.27)) hide)
+    )
     (pin "1")
     (pin "2")
@@
       (effects (font (size 1.27 1.27)) hide)
     )
+    (property "AssemblyType" "SMT" (id 9) (at 226.06 72.39 0)
+      (effects (font (size 1.27 1.27)) hide)
+    )
+    (property "Cost" "0.0015" (id 10) (at 226.06 72.39 0)
+      (effects (font (size 1.27 1.27)) hide)
+    )
     (pin "1")
     (pin "2")
@@
       (effects (font (size 1.27 1.27)) hide)
     )
-    (property "Distributor 1" "" (id 4) (at 157.988 94.996 0)
-      (effects (font (size 1.27 1.27)) hide)
-    )
-    (property "Distributor 1 PN" "" (id 5) (at 182.88 97.536 0)
-      (effects (font (size 1.27 1.27)) hide)
-    )
-    (property "Distributor 2" "" (id 6) (at 156.972 100.584 0)
-      (effects (font (size 1.27 1.27)) hide)
-    )
-    (property "Distributor 2 PN" "" (id 7) (at 205.486 102.87 0)
+    (property "Distributor 1" "Aliexpress" (id 4) (at 157.988 94.996 0)
+      (effects (font (size 1.27 1.27)) hide)
+    )
+    (property "Distributor 1 PN" "https://www.aliexpress.com/item/3256803213374992.html" (id 5) (at 182.88 97.536 0)
+      (effects (font (size 1.27 1.27)) hide)
+    )
+    (property "Distributor 2" "Amazon" (id 6) (at 156.972 100.584 0)
+      (effects (font (size 1.27 1.27)) hide)
+    )
+    (property "Distributor 2 PN" "https://www.amazon.com/GeeekPi-Interface-Adapter-Backlight-Raspberry/dp/B07QLRD3TM/ref=sr_1_2" (id 7) (at 205.486 102.87 0)
       (effects (font (size 1.27 1.27)) hide)
     )
@@
       (effects (font (size 1.27 1.27)) hide)
     )
-    (property "Cost" "" (id 9) (at 185.42 77.47 0)
+    (property "Cost" "4.99" (id 9) (at 185.42 77.47 0)
       (effects (font (size 1.27 1.27)) hide)
     )
@@
       (effects (font (size 1.27 1.27)) hide)
     )
+    (property "AssemblyType" "SMT" (id 13) (at 209.55 68.58 0)
+      (effects (font (size 1.27 1.27)) hide)
+    )
+    (property "Description" "±10% ±100ppm/℃ 10kΩ Plugin Variable Resistors/Potentiometers ROHS" (id 14) (at 209.55 68.58 0)
+      (effects (font (size 1.27 1.27)) hide)
+    )
