File: Hardware/GeneralPurposeAlarmDevicePCB/GeneralPurposeAlarmDevicePCB/AlarmAudio.kicad_sch (KiCad schematic)
At the start: 12 parts

Commit message: Updated footprints and schematic Signed-off-by: lokimetasmith <lokimail@gmail.com>
Parts:
- BZ601: value (none) -> QMB-09B-03; footprint (none) -> QMB-09B-03:QMB09B03; symbol GeneralPurposeAlarmDevicePCB-rescue:QMB-09B-03-QMB-09B-03 -> Device:Buzzer
- C601: renamed from C?; value (none) -> 47uF; footprint (none) -> Capacitor_SMD:CP_Elec_5x5.4; symbol GeneralPurposeAlarmDevicePCB-rescue:CP-Device -> Device:C_Polarized
- C602: renamed from C?; value (none) -> 100nF; footprint (none) -> Capacitor_SMD:C_0603_1608Metric_Pad1.08x0.95mm_HandSolder
- J601: renamed from J?; value (none) -> 22-23-2021; footprint (none) -> Connector_Molex:Molex_KK-254_AE-6410-02A_1x02_P2.54mm_Vertical
- Q601: value (none) -> MMBT2222A-7-F; footprint (none) -> Package_TO_SOT_SMD:SOT-23
- Q602: value (none) -> MMBT2907ALT1G; footprint (none) -> digikey-footprints:SOT-23-3; symbol GeneralPurposeAlarmDevicePCB-rescue:MMBT2907ALT1G-dk_Transistors-Bipolar-BJT-Single -> Device:Q_PNP_BEC
- R601, R604: renamed from R?; value (none) -> 1R; footprint (none) -> Resistor_SMD:R_0603_1608Metric
- R602: renamed from R?; value (none) -> 1K; footprint (none) -> Resistor_SMD:R_0603_1608Metric
- R603: renamed from R?; value (none) -> 10K; footprint (none) -> Resistor_SMD:R_0603_1608Metric
- R605: renamed from R?; value (none) -> 330; footprint (none) -> Resistor_SMD:R_0603_1608Metric
- S601: renamed from S?; value (none) -> SWITCH_TACTILE_SPST-NO_0.05A_24V; footprint (none) -> GeneralPurposeAlarmDevicePCB:Switch_Tactile_THT_6x6mm
Connections:
- net GND: now also BZ601.2 (+), C601.2, Q602.2 (E)
- net VccBuzzer: now also C601.1
- net at J601.1, R604.1: now also BZ601.1 (-)
- net at Q601.2 (E), R604.2: now also Q602.3 (C)
- net at Q601.1 (B), R602.1, R605.2: now also Q602.1 (B)

Commit message: updated buzzer footprint to a generic compatible one
Signed-off-by: lokimetasmith <lokimail@gmail.com>
Parts:
- BZ601: footprint QMB-09B-03:QMB09B03 -> Buzzer_Beeper:MagneticBuzzer_PUI_AT-0927-TT-6-R
Changed lines of the file:
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@@
     (property "Reference" "BZ601" (id 0) (at 197.9168 99.441 0))
     (property "Value" "QMB-09B-03" (id 1) (at 197.9168 97.1296 0))
-    (property "Footprint" "QMB-09B-03:QMB09B03" (id 2) (at 189.865 87.63 90)
+    (property "Footprint" "Buzzer_Beeper:MagneticBuzzer_PUI_AT-0927-TT-6-R" (id 2) (at 189.865 87.63 90)
       (effects (font (size 1.27 1.27)) hide)
     )

Commit message: Update buzzer foot print. Fully connect all parts. Fix numerous silkscreen conflicts. Mix of metric and imperial grid.
Parts:
- BZ601: value QMB-09B-03 -> Buzzer_12.2mm_H6.5mm; footprint Buzzer_Beeper:MagneticBuzzer_PUI_AT-0927-TT-6-R -> Buzzer_Beeper:Buzzer_TDK_PS1240P02BT_D12.2mm_H6.5mm; Cost (none) -> 0.62000; Distributor 1 PN C96256 -> C76871; Distributor 2 (none) -> Digi-Key; Distributor 2 PN (none) -> 445-2525-1-ND; MPN QMB-09B-03 -> PS1240P02BT; Manufacturer Jiangsu Huaneng Elec -> TDK Corporation
Changed lines of the file:
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@@
-    (pin "2")
-  )
-  (symbol (lib_id "Device:Buzzer") (at 190.5 90.17 0) (unit 1)
-    (in_bom yes) (on_board yes)
-    (property "Reference" "BZ601" (id 0) (at 197.9168 99.441 0))
-    (property "Value" "QMB-09B-03" (id 1) (at 197.9168 97.1296 0))
-    (property "Footprint" "Buzzer_Beeper:MagneticBuzzer_PUI_AT-0927-TT-6-R" (id 2) (at 189.865 87.63 90)
-      (effects (font (size 1.27 1.27)) hide)
-    )
-    (property "Datasheet" "~" (id 3) (at 189.865 87.63 90)
-      (effects (font (size 1.27 1.27)) hide)
-    )
-    (property "Description" "Magnetic NO 2700Hz 3V 2 ~ 5V 9mm 9*5.5mm Buzzers" (id 4) (at 207.01 92.71 0)
-      (effects (font (size 1.27 1.27)) (justify left) hide)
-    )
-    (property "Manufacturer" "Jiangsu Huaneng Elec" (id 5) (at 207.01 97.79 0)
-      (effects (font (size 1.27 1.27)) (justify left) hide)
-    )
-    (property "MPN" "QMB-09B-03" (id 6) (at 207.01 100.33 0)
-      (effects (font (size 1.27 1.27)) (justify left) hide)
-    )
-    (property "Distributor 1" "JLCPCB" (id 7) (at 190.5 90.17 0)
-      (effects (font (size 1.27 1.27)) hide)
-    )
-    (property "Distributor 1 PN" "C96256" (id 8) (at 190.5 90.17 0)
-      (effects (font (size 1.27 1.27)) hide)
-    )
-    (pin "1")
     (pin "2")
   )
@@
       (effects (font (size 1.27 1.27)) hide)
     )
+    (pin "1")
+    (pin "2")
+  )
+  (symbol (lib_id "Device:Buzzer") (at 190.5 90.17 0) (unit 1)
+    (in_bom yes) (on_board yes) (fields_autoplaced)
+    (property "Reference" "BZ601" (id 0) (at 194.31 88.8999 0)
+      (effects (font (size 1.27 1.27)) (justify left))
+    )
+    (property "Value" "Buzzer_12.2mm_H6.5mm" (id 1) (at 194.31 91.4399 0)
+      (effects (font (size 1.27 1.27)) (justify left))
+    )
+    (property "Footprint" "Buzzer_Beeper:Buzzer_TDK_PS1240P02BT_D12.2mm_H6.5mm" (id 2) (at 189.865 87.63 90)
+      (effects (font (size 1.27 1.27)) hide)
+    )
+    (property "Datasheet" "~" (id 3) (at 189.865 87.63 90)
+      (effects (font (size 1.27 1.27)) hide)
+    )
+    (property "Distributor 1" "JLCPCB" (id 9) (at 190.5 90.17 0)
+      (effects (font (size 1.27 1.27)) hide)
+    )
+    (property "Distributor 1 PN" "C76871" (id 10) (at 190.5 90.17 0)
+      (effects (font (size 1.27 1.27)) hide)
+    )
+    (property "Distributor 2" "Digi-Key" (id 5) (at 190.5 90.17 0)
+      (effects (font (size 1.27 1.27)) hide)
+    )
+    (property "Distributor 2 PN" "445-2525-1-ND" (id 6) (at 190.5 90.17 0)
+      (effects (font (size 1.27 1.27)) hide)
+    )
+    (property "Manufacturer" "TDK Corporation" (id 7) (at 190.5 90.17 0)
+      (effects (font (size 1.27 1.27)) hide)
+    )
+    (property "MPN" "PS1240P02BT" (id 8) (at 190.5 90.17 0)
+      (effects (font (size 1.27 1.27)) hide)
+    )
+    (property "Cost" "0.62000" (id 9) (at 190.5 90.17 0)
+      (effects (font (size 1.27 1.27)) hide)
+    )

Commit message: Fix pot foot print, Add fifth mounting hole. Place all but UNO and test point.
Parts:
- removed S601: SWITCH_TACTILE_SPST-NO_0.05A_24V, GeneralPurposeAlarmDevicePCB:Switch_Tactile_THT_6x6mm, symbol GPAD_SCH_LIB:SWITCH_TACTILE_SPST-NO_0.05A_24V
- added S601: SWITCH_TACTILE_12mmx12mm_SPST-NO_0.05A_24V, Button_Switch_THT:SW_PUSH-12mm, symbol GPAD_SCH_LIB:SWITCH_TACTILE_12mmx12mm_SPST-NO_0.05A_24V
Connections:
- net GND: now also S601.3, S601.4
- net Switch_Mute: now also S601.1, S601.2
Changed lines of the file:
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@@
     (effects (font (size 1.27 1.27)) (justify right))
-  )
-  (symbol (lib_id "GPAD_SCH_LIB:SWITCH_TACTILE_SPST-NO_0.05A_24V") (at 88.9 120.65 0) (unit 1)
-    (in_bom yes) (on_board yes)
-    (property "Reference" "S601" (id 0) (at 88.9 111.8362 0)
-      (effects (font (size 1.524 1.524)))
-    )
-    (property "Value" "SWITCH_TACTILE_SPST-NO_0.05A_24V" (id 1) (at 88.9 114.5286 0)
-      (effects (font (size 1.524 1.524)))
-    )
-    (property "Footprint" "GeneralPurposeAlarmDevicePCB:Switch_Tactile_THT_6x6mm" (id 2) (at 93.98 115.57 0)
-      (effects (font (size 1.524 1.524)) (justify left) hide)
-    )
-    (property "Datasheet" "https://www.te.com/commerce/DocumentDelivery/DDEController?Action=srchrtrv&DocNm=1825910&DocType=Customer+Drawing&DocLang=English" (id 3) (at 93.98 113.03 0)
-      (effects (font (size 1.524 1.524)) (justify left) hide)
-    )
-    (property "Distributor 1" "JLCPCB" (id 4) (at 88.9 120.65 0)
-      (effects (font (size 1.27 1.27)) hide)
-    )
-    (property "Distributor 1 PN" "C13828" (id 5) (at 88.9 120.65 0)
-      (effects (font (size 1.27 1.27)) hide)
-    )
-    (property "Distributor 2" "Digikey" (id 6) (at 88.9 120.65 0)
-      (effects (font (size 1.27 1.27)) hide)
-    )
-    (property "Distributor 2 PN" "450-1804-ND" (id 7) (at 93.98 110.49 0)
-      (effects (font (size 1.524 1.524)) (justify left) hide)
-    )
-    (property "Manufacturer" "TE Connectivity ALCOSWITCH Switches" (id 8) (at 93.98 92.71 0)
-      (effects (font (size 1.524 1.524)) (justify left) hide)
-    )
-    (property "MPN" "TE Connectivity 1825910-7,   Dongguan Guangzhu Industrial C13828" (id 9) (at 93.98 107.95 0)
-      (effects (font (size 1.524 1.524)) (justify left) hide)
-    )
-    (property "Category" "Switches" (id 10) (at 93.98 105.41 0)
-      (effects (font (size 1.524 1.524)) (justify left) hide)
-    )
-    (property "Family" "Tactile Switches" (id 11) (at 93.98 102.87 0)
-      (effects (font (size 1.524 1.524)) (justify left) hide)
-    )
-    (property "DK_Datasheet_Link" "https://www.te.com/commerce/DocumentDelivery/DDEController?Action=srchrtrv&DocNm=1825910&DocType=Customer+Drawing&DocLang=English" (id 12) (at 93.98 100.33 0)
-      (effects (font (size 1.524 1.524)) (justify left) hide)
-    )
-    (property "DK_Detail_Page" "/product-detail/en/te-connectivity-alcoswitch-switches/1825910-7/450-1804-ND/1731414" (id 13) (at 93.98 97.79 0)
-      (effects (font (size 1.524 1.524)) (justify left) hide)
-    )
-    (property "Description" "SWITCH TACTILE SPST-NO 0.05A 24V" (id 14) (at 93.98 95.25 0)
-      (effects (font (size 1.524 1.524)) (justify left) hide)
-    )
-    (property "Status" "Active" (id 15) (at 93.98 90.17 0)
-      (effects (font (size 1.524 1.524)) (justify left) hide)
-    )
-    (property "Assembly Type" "HAND" (id 16) (at 0 241.3 0)
-      (effects (font (size 1.27 1.27)) hide)
-    )
-    (pin "1")
-    (pin "2")
-    (pin "3")
-    (pin "4")
   )
   (symbol (lib_id "power:GND") (at 95.25 128.27 0) (unit 1)
@@
       (effects (font (size 1.27 1.27)) hide)
     )
-    (property "Cost" "0.62000" (id 9) (at 190.5 90.17 0)
-      (effects (font (size 1.27 1.27)) hide)
-    )
-    (pin "1")
-    (pin "2")
+    (property "Cost" "0.62000" (id 11) (at 190.5 90.17 0)
+      (effects (font (size 1.27 1.27)) hide)
+    )
+    (pin "1")
+    (pin "2")
+  )
+  (symbol (lib_id "GPAD_SCH_LIB:SWITCH_TACTILE_12mmx12mm_SPST-NO_0.05A_24V") (at 88.9 120.65 0) (unit 1)
+    (in_bom yes) (on_board yes) (fields_autoplaced)
+    (property "Reference" "S601" (id 0) (at 88.9 111.76 0)
+      (effects (font (size 1.524 1.524)))
+    )
+    (property "Value" "SWITCH_TACTILE_12mmx12mm_SPST-NO_0.05A_24V" (id 1) (at 88.9 115.57 0)
+      (effects (font (size 1.524 1.524)))
+    )
+    (property "Footprint" "Button_Switch_THT:SW_PUSH-12mm" (id 2) (at 93.98 115.57 0)
+      (effects (font (size 1.524 1.524)) (justify left) hide)
+    )
+    (property "Datasheet" "" (id 3) (at 93.98 113.03 0)
+      (effects (font (size 1.524 1.524)) (justify left) hide)
+    )
+    (property "Distributor 1" "JLCPCB" (id 4) (at 88.9 120.65 0)
+      (effects (font (size 1.27 1.27)) hide)
+    )
+    (property "Distributor 1 PN" "C84931" (id 5) (at 88.9 120.65 0)
+      (effects (font (size 1.27 1.27)) hide)
+    )
+    (property "Distributor 2" "Digikey" (id 6) (at 88.9 120.65 0)
+      (effects (font (size 1.27 1.27)) hide)
+    )
+    (property "Distributor 2 PN" "SW414-ND" (id 7) (at 93.98 110.49 0)
+      (effects (font (size 1.524 1.524)) (justify left) hide)
+    )
+    (property "Manufacturer" "Omron Electronics" (id 8) (at 93.98 92.71 0)
+      (effects (font (size 1.524 1.524)) (justify left) hide)
+    )
+    (property "MPN" "B3F-4055" (id 9) (at 93.98 107.95 0)
+      (effects (font (size 1.524 1.524)) (justify left) hide)
+    )
+    (property "Category" "Switches" (id 10) (at 93.98 105.41 0)
+      (effects (font (size 1.524 1.524)) (justify left) hide)
+    )
+    (property "Family" "Tactile Switches" (id 11) (at 93.98 102.87 0)
+      (effects (font (size 1.524 1.524)) (justify left) hide)
+    )
+    (property "Cost" "0.1181" (id 12) (at 93.98 100.33 0)
+      (effects (font (size 0 0)) (justify left) hide)
+    )
+    (property "DK_Detail_Page" "" (id 13) (at 93.98 97.79 0)
+      (effects (font (size 1.524 1.524)) (justify left) hide)
+    )
+    (property "Description" "SWITCH_TACTILE_12mmx12mm_SPST-NO_0.05A_24V" (id 14) (at 93.98 95.25 0)
+      (effects (font (size 1.524 1.524)) (justify left) hide)
+    )
+    (property "Status" "Active" (id 15) (at 93.98 90.17 0)
+      (effects (font (size 1.524 1.524)) (justify left) hide)
+    )
+    (property "Assembly Type" "HAND" (id 16) (at 88.9 120.65 0)
+      (effects (font (size 1.27 1.27)) hide)
+    )
+    (pin "1")
+    (pin "2")
+    (pin "3")
+    (pin "4")
   )
 )

Commit message: Add12mmx12mmSwitc.
Parts:
- S601: footprint Button_Switch_THT:SW_PUSH-12mm -> GeneralPurposeAlarmDevicePCB:SW_PUSH-12mm_WithCap_Green
Changed lines of the file:
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@@
       (effects (font (size 1.524 1.524)))
     )
-    (property "Footprint" "Button_Switch_THT:SW_PUSH-12mm" (id 2) (at 93.98 115.57 0)
+    (property "Footprint" "GeneralPurposeAlarmDevicePCB:SW_PUSH-12mm_WithCap_Green" (id 2) (at 93.98 115.57 0)
       (effects (font (size 1.524 1.524)) (justify left) hide)
     )

Commit message: Add 7805 alternative for linear regulator, Add test points on power supply nets, add MechanicalPartsPlacement.pdf.
Parts:
- added TP501: TP_VccBuzzer, TestPoint:TestPoint_Loop_D2.54mm_Drill1.5mm_Beaded, symbol Connector:TestPoint
Connections:
- net VccBuzzer: now also TP501.1
Changed lines of the file:
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@@
   (junction (at 137.16 68.58) (diameter 0) (color 0 0 0 0)
   )
+  (junction (at 101.6 48.26) (diameter 0) (color 0 0 0 0)
+  )
   (junction (at 123.19 71.12) (diameter 0) (color 0 0 0 0)
   )
@@
     (stroke (width 0) (type default) (color 0 0 0 0))
   )
-  (wire (pts (xy 72.39 48.26) (xy 137.16 48.26))
+  (wire (pts (xy 72.39 48.26) (xy 101.6 48.26))
     (stroke (width 0) (type default) (color 0 0 0 0))
   )
@@
   )
   (wire (pts (xy 83.82 123.19) (xy 81.28 123.19))
+    (stroke (width 0) (type default) (color 0 0 0 0))
+  )
+  (wire (pts (xy 101.6 48.26) (xy 137.16 48.26))
+    (stroke (width 0) (type default) (color 0 0 0 0))
+  )
+  (wire (pts (xy 101.6 43.18) (xy 101.6 48.26))
     (stroke (width 0) (type default) (color 0 0 0 0))
   )
@@
     (pin "2")
   )
+  (symbol (lib_id "Connector:TestPoint") (at 101.6 43.18 0) (unit 1)
+    (in_bom yes) (on_board yes)
+    (property "Reference" "TP501" (id 0) (at 102.87 39.37 0)
+      (effects (font (size 1.27 1.27)) (justify left))
+    )
+    (property "Value" "TP_VccBuzzer" (id 1) (at 102.87 41.91 0)
+      (effects (font (size 1.27 1.27)) (justify left))
+    )
+    (property "Footprint" "TestPoint:TestPoint_Loop_D2.54mm_Drill1.5mm_Beaded" (id 2) (at 106.68 43.18 0)
+      (effects (font (size 1.27 1.27)) hide)
+    )
+    (property "Datasheet" "~" (id 3) (at 106.68 43.18 0)
+      (effects (font (size 1.27 1.27)) hide)
+    )
+    (pin "1")
+  )
   (symbol (lib_id "GPAD_SCH_LIB:SWITCH_TACTILE_12mmx12mm_SPST-NO_0.05A_24V") (at 88.9 120.65 0) (unit 1)

Commit message: Fix incorrect Q602 emiter collector orientation.
Connections:
- net GND: now also Q602.3 (C); no longer Q602.2 (E)
- net at Q601.2 (E), R604.2: now also Q602.2 (E); no longer Q602.3 (C)
Changed lines of the file:
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@@
     (pin "2")
   )
-  (symbol (lib_id "Device:Q_PNP_BEC") (at 134.62 77.47 0) (unit 1)
+  (symbol (lib_id "Device:Q_PNP_BEC") (at 134.62 77.47 0) (mirror x) (unit 1)
     (in_bom yes) (on_board yes)
-    (property "Reference" "Q602" (id 0) (at 139.3952 76.1238 0)
+    (property "Reference" "Q602" (id 0) (at 139.3952 78.8162 0)
       (effects (font (size 1.524 1.524)) (justify left))
     )
-    (property "Value" "MMBT2907ALT1G" (id 1) (at 139.3952 78.8162 0)
+    (property "Value" "MMBT2907ALT1G" (id 1) (at 139.3952 76.1238 0)
       (effects (font (size 1.524 1.524)) (justify left))
     )
-    (property "Footprint" "digikey-footprints:SOT-23-3" (id 2) (at 139.7 74.93 0)
+    (property "Footprint" "digikey-footprints:SOT-23-3" (id 2) (at 139.7 80.01 0)
       (effects (font (size 1.27 1.27)) hide)
     )
@@
       (effects (font (size 1.27 1.27)) hide)
     )
-    (property "Digi-Key_PN" "MMBT2907ALT1GOSCT-ND" (id 4) (at 139.7 67.31 0)
+    (property "Digi-Key_PN" "MMBT2907ALT1GOSCT-ND" (id 4) (at 139.7 87.63 0)
       (effects (font (size 1.524 1.524)) (justify left) hide)
     )
-    (property "MPN" "MMBT2907ALT1G" (id 5) (at 139.7 64.77 0)
+    (property "MPN" "MMBT2907ALT1G" (id 5) (at 139.7 90.17 0)
       (effects (font (size 1.524 1.524)) (justify left) hide)
     )
-    (property "Category" "Discrete Semiconductor Products" (id 6) (at 139.7 62.23 0)
+    (property "Category" "Discrete Semiconductor Products" (id 6) (at 139.7 92.71 0)
       (effects (font (size 1.524 1.524)) (justify left) hide)
     )
-    (property "Family" "Transistors - Bipolar (BJT) - Single" (id 7) (at 139.7 59.69 0)
+    (property "Family" "Transistors - Bipolar (BJT) - Single" (id 7) (at 139.7 95.25 0)
       (effects (font (size 1.524 1.524)) (justify left) hide)
     )
-    (property "DK_Datasheet_Link" "http://www.onsemi.com/pub/Collateral/MMBT2907ALT1-D.PDF" (id 8) (at 139.7 57.15 0)
+    (property "DK_Datasheet_Link" "http://www.onsemi.com/pub/Collateral/MMBT2907ALT1-D.PDF" (id 8) (at 139.7 97.79 0)
       (effects (font (size 1.524 1.524)) (justify left) hide)
     )
-    (property "DK_Detail_Page" "/product-detail/en/on-semiconductor/MMBT2907ALT1G/MMBT2907ALT1GOSCT-ND/1139812" (id 9) (at 139.7 54.61 0)
+    (property "DK_Detail_Page" "/product-detail/en/on-semiconductor/MMBT2907ALT1G/MMBT2907ALT1GOSCT-ND/1139812" (id 9) (at 139.7 100.33 0)
       (effects (font (size 1.524 1.524)) (justify left) hide)
     )
-    (property "Description" "TRANS PNP 60V 0.6A SOT23" (id 10) (at 139.7 52.07 0)
+    (property "Description" "TRANS PNP 60V 0.6A SOT23" (id 10) (at 139.7 102.87 0)
       (effects (font (size 1.524 1.524)) (justify left) hide)
     )
-    (property "Manufacturer" "ON Semiconductor" (id 11) (at 139.7 49.53 0)
+    (property "Manufacturer" "ON Semiconductor" (id 11) (at 139.7 105.41 0)
       (effects (font (size 1.524 1.524)) (justify left) hide)
     )
-    (property "Status" "Active" (id 12) (at 139.7 46.99 0)
+    (property "Status" "Active" (id 12) (at 139.7 107.95 0)
       (effects (font (size 1.524 1.524)) (justify left) hide)
     )

Commit message: Change TP to show value on F silk screen. Make REF DES smaller.
Parts:
- TP501: value TP_VccBuzzer -> VccBuzzer
Changed lines of the file:
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@@
       (effects (font (size 1.27 1.27)) (justify left))
     )
-    (property "Value" "TP_VccBuzzer" (id 1) (at 102.87 41.91 0)
+    (property "Value" "VccBuzzer" (id 1) (at 102.87 41.91 0)
       (effects (font (size 1.27 1.27)) (justify left))
     )
