File: Hardware/GeneralPurposeAlarmDevicePCB/GeneralPurposeAlarmDevicePCB/AlarmAudio.kicad_sch (KiCad schematic)
At the start: 13 parts, among them J601 22-23-2021, Q601 MMBT2222A-7-F, Q602 MMBT2907ALT1G

Commit message: Mature the BOM parts. Remove misspelled fields. Add some costs.
Parts:
- BZ601, TP501: AssemblyType (none) -> HAND
- J601, S601: Assembly Type HAND -> (none); AssemblyType (none) -> HAND
- R601, R602, R603, R604, R605: footprint Resistor_SMD:R_0603_1608Metric -> Resistor_SMD:R_0603_1608Metric_Pad0.98x0.95mm_HandSolder
Changed lines of the file:
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@@
     (property "Reference" "R603" (id 0) (at 53.34 113.03 90))
     (property "Value" "10K" (id 1) (at 54.61 115.57 90))
-    (property "Footprint" "Resistor_SMD:R_0603_1608Metric" (id 2) (at 54.61 116.332 90)
+    (property "Footprint" "Resistor_SMD:R_0603_1608Metric_Pad0.98x0.95mm_HandSolder" (id 2) (at 54.61 116.332 90)
       (effects (font (size 1.27 1.27)) hide)
     )
@@
     (property "Reference" "R604" (id 0) (at 163.83 63.5 90))
     (property "Value" "1R" (id 1) (at 165.1 66.04 90))
-    (property "Footprint" "Resistor_SMD:R_0603_1608Metric" (id 2) (at 165.1 66.802 90)
+    (property "Footprint" "Resistor_SMD:R_0603_1608Metric_Pad0.98x0.95mm_HandSolder" (id 2) (at 165.1 66.802 90)
       (effects (font (size 1.27 1.27)) hide)
     )
@@
     (property "Reference" "R605" (id 0) (at 97.79 87.63 90))
     (property "Value" "330" (id 1) (at 99.06 93.98 90))
-    (property "Footprint" "Resistor_SMD:R_0603_1608Metric" (id 2) (at 99.06 91.948 90)
+    (property "Footprint" "Resistor_SMD:R_0603_1608Metric_Pad0.98x0.95mm_HandSolder" (id 2) (at 99.06 91.948 90)
       (effects (font (size 1.27 1.27)) hide)
     )
@@
     (property "Reference" "R601" (id 0) (at 53.34 43.18 90))
     (property "Value" "1R" (id 1) (at 54.61 45.72 90))
-    (property "Footprint" "Resistor_SMD:R_0603_1608Metric" (id 2) (at 54.61 46.482 90)
+    (property "Footprint" "Resistor_SMD:R_0603_1608Metric_Pad0.98x0.95mm_HandSolder" (id 2) (at 54.61 46.482 90)
       (effects (font (size 1.27 1.27)) hide)
     )
@@
       (effects (font (size 1.524 1.524)) (justify left) hide)
     )
-    (property "Assembly Type" "HAND" (id 13) (at 306.07 -82.55 0)
+    (property "Assembly Type" "" (id 13) (at 306.07 -82.55 0)
+      (effects (font (size 1.27 1.27)) hide)
+    )
+    (property "AssemblyType" "HAND" (id 14) (at 194.31 111.76 0)
       (effects (font (size 1.27 1.27)) hide)
     )
@@
     (property "Reference" "R602" (id 0) (at 97.79 66.04 90))
     (property "Value" "1K" (id 1) (at 97.79 68.58 90))
-    (property "Footprint" "Resistor_SMD:R_0603_1608Metric" (id 2) (at 99.06 69.342 90)
+    (property "Footprint" "Resistor_SMD:R_0603_1608Metric_Pad0.98x0.95mm_HandSolder" (id 2) (at 99.06 69.342 90)
       (effects (font (size 1.27 1.27)) hide)
     )
@@
       (effects (font (size 1.27 1.27)) hide)
     )
+    (property "AssemblyType" "HAND" (id 12) (at 190.5 90.17 0)
+      (effects (font (size 1.27 1.27)) hide)
+    )
     (pin "1")
     (pin "2")
@@
     )
     (property "Datasheet" "~" (id 3) (at 106.68 43.18 0)
+      (effects (font (size 1.27 1.27)) hide)
+    )
+    (property "AssemblyType" "HAND" (id 4) (at 101.6 43.18 0)
       (effects (font (size 1.27 1.27)) hide)
     )
@@
       (effects (font (size 1.524 1.524)) (justify left) hide)
     )
-    (property "Assembly Type" "HAND" (id 16) (at 88.9 120.65 0)
-      (effects (font (size 1.27 1.27)) hide)
-    )
+    (property "Assembly Type" "" (id 16) (at 88.9 120.65 0)
+      (effects (font (size 1.27 1.27)) hide)
+    )
+    (property "AssemblyType" "HAND" (id 17) (at 88.9 120.65 0)
+      (effects (font (size 1.27 1.27)) hide)
+    )

Commit message: Update a lot of cost and PNs from JLCPCB and some Digikey.
Parts:
- C601: value 47uF -> 47uF 16V; AssemblyType (none) -> SMT; Cost (none) -> 0.038
- C602: AssemblyType (none) -> SMT; Cost (none) -> 0.0021
- J601: Cost (none) -> 0.22000; Distributor 1 (none) -> DigiKey; Distributor 1 PN (none) -> 900-0022232021-ND
- Q601: AssemblyType (none) -> SMT; Cost (none) -> 0.0475; Distributor 1 (none) -> JLCPCB; Distributor 1 PN (none) -> C94515
- Q602: AssemblyType (none) -> SMT; Cost (none) -> 0.0374; Distributor 1 (none) -> JCLPCB; Distributor 1 PN (none) -> C40752
- R601, R602, R603, R604, R605: AssemblyType (none) -> SMT; Cost (none) -> 0.0015
Changed lines of the file:
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@@
+      (effects (font (size 1.27 1.27)) hide)
+    )
+    (property "AssemblyType" "SMT" (id 9) (at 54.61 118.11 0)
+      (effects (font (size 1.27 1.27)) hide)
+    )
+    (property "Cost" "0.0015" (id 10) (at 54.61 118.11 0)
       (effects (font (size 1.27 1.27)) hide)
     )
@@
       (effects (font (size 1.27 1.27)) hide)
     )
+    (property "AssemblyType" "SMT" (id 9) (at 165.1 68.58 0)
+      (effects (font (size 1.27 1.27)) hide)
+    )
+    (property "Cost" "0.0015" (id 10) (at 165.1 68.58 0)
+      (effects (font (size 1.27 1.27)) hide)
+    )
     (pin "1")
     (pin "2")
@@
     (property "Status" "Active" (id 12) (at 139.7 30.48 0)
       (effects (font (size 1.524 1.524)) (justify left) hide)
+    )
+    (property "AssemblyType" "SMT" (id 13) (at 134.62 60.96 0)
+      (effects (font (size 1.27 1.27)) hide)
+    )
+    (property "Distributor 1" "JLCPCB" (id 14) (at 134.62 60.96 0)
+      (effects (font (size 1.27 1.27)) hide)
+    )
+    (property "Distributor 1 PN" "C94515" (id 15) (at 134.62 60.96 0)
+      (effects (font (size 1.27 1.27)) hide)
+    )
+    (property "Cost" "0.0475" (id 16) (at 134.62 60.96 0)
+      (effects (font (size 1.27 1.27)) hide)
     )
     (pin "1")
@@
       (effects (font (size 1.27 1.27)) hide)
     )
+    (property "AssemblyType" "SMT" (id 9) (at 99.06 90.17 0)
+      (effects (font (size 1.27 1.27)) hide)
+    )
+    (property "Cost" "0.0015" (id 10) (at 99.06 90.17 0)
+      (effects (font (size 1.27 1.27)) hide)
+    )
     (pin "1")
     (pin "2")
@@
       (effects (font (size 1.524 1.524)) (justify left) hide)
     )
+    (property "AssemblyType" "SMT" (id 13) (at 134.62 77.47 0)
+      (effects (font (size 1.27 1.27)) hide)
+    )
+    (property "Distributor 1" "JCLPCB" (id 14) (at 134.62 77.47 0)
+      (effects (font (size 1.27 1.27)) hide)
+    )
+    (property "Distributor 1 PN" "C40752" (id 15) (at 134.62 77.47 0)
+      (effects (font (size 1.27 1.27)) hide)
+    )
+    (property "Cost" "0.0374" (id 16) (at 134.62 77.47 0)
+      (effects (font (size 1.27 1.27)) hide)
+    )
     (pin "1")
     (pin "2")
@@
       (effects (font (size 1.27 1.27)) (justify left))
     )
-    (property "Value" "47uF" (id 1) (at 75.3872 54.483 0)
+    (property "Value" "47uF 16V" (id 1) (at 75.3872 54.483 0)
       (effects (font (size 1.27 1.27)) (justify left))
     )
@@
     )
     (property "MPN" "RVT47UF16V67RV0019" (id 7) (at 72.39 53.34 0)
+      (effects (font (size 1.27 1.27)) hide)
+    )
+    (property "AssemblyType" "SMT" (id 8) (at 72.39 53.34 0)
+      (effects (font (size 1.27 1.27)) hide)
+    )
+    (property "Cost" "0.038" (id 9) (at 72.39 53.34 0)
+      (effects (font (size 1.27 1.27)) hide)
+    )
+    (property "Description" "16V 47uF SMD,5x5.4mm Aluminum Electrolytic Capacitors - SMD ROHS" (id 10) (at 72.39 53.34 0)
       (effects (font (size 1.27 1.27)) hide)
     )
@@
       (effects (font (size 1.27 1.27)) hide)
     )
+    (property "AssemblyType" "SMT" (id 9) (at 54.61 48.26 0)
+      (effects (font (size 1.27 1.27)) hide)
+    )
+    (property "Cost" "0.0015" (id 10) (at 54.61 48.26 0)
+      (effects (font (size 1.27 1.27)) hide)
+    )
     (pin "1")
     (pin "2")
@@
       (effects (font (size 1.27 1.27)) hide)
     )
+    (property "AssemblyType" "SMT" (id 9) (at 62.23 130.81 0)
+      (effects (font (size 1.27 1.27)) hide)
+    )
+    (property "Cost" "0.0021" (id 10) (at 62.23 130.81 0)
+      (effects (font (size 1.27 1.27)) hide)
+    )
     (pin "1")
     (pin "2")
@@
     )
     (property "AssemblyType" "HAND" (id 14) (at 194.31 111.76 0)
+      (effects (font (size 1.27 1.27)) hide)
+    )
+    (property "Cost" "0.22000" (id 15) (at 194.31 111.76 0)
+      (effects (font (size 1.27 1.27)) hide)
+    )
+    (property "Distributor 1" "DigiKey" (id 16) (at 194.31 111.76 0)
+      (effects (font (size 1.27 1.27)) hide)
+    )
+    (property "Distributor 1 PN" "900-0022232021-ND" (id 17) (at 194.31 111.76 0)
       (effects (font (size 1.27 1.27)) hide)
     )
@@
       (effects (font (size 1.27 1.27)) hide)
     )
+    (property "AssemblyType" "SMT" (id 9) (at 99.06 71.12 0)
+      (effects (font (size 1.27 1.27)) hide)
+    )
+    (property "Cost" "0.0015" (id 10) (at 99.06 71.12 0)
+      (effects (font (size 1.27 1.27)) hide)
+    )

Commit message: Update crystal footprint for proper SMT. Position compoonents for routing. Add resistor to attenuate audio.
Parts:
- added R505: 10K, Resistor_SMD:R_0603_1608Metric_Pad0.98x0.95mm_HandSolder, symbol Device:R
Connections:
- net GND: now also R505.1
- net at Q601.1 (B), Q602.1 (B), R602.1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: now also R505.2
Changed lines of the file:
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@@
   (junction (at 81.28 118.11) (diameter 0) (color 0 0 0 0)
   )
+  (junction (at 110.49 90.17) (diameter 0) (color 0 0 0 0)
+  )
   (junction (at 110.49 71.12) (diameter 0) (color 0 0 0 0)
   )
@@
     (stroke (width 0) (type default) (color 0 0 0 0))
   )
+  (wire (pts (xy 110.49 97.79) (xy 116.84 97.79))
+    (stroke (width 0) (type default) (color 0 0 0 0))
+  )
   (wire (pts (xy 64.77 118.11) (xy 81.28 118.11))
     (stroke (width 0) (type default) (color 0 0 0 0))
@@
     (stroke (width 0) (type default) (color 0 0 0 0))
   )
+  (wire (pts (xy 132.08 97.79) (xy 132.08 99.06))
+    (stroke (width 0) (type default) (color 0 0 0 0))
+  )
   (wire (pts (xy 180.34 87.63) (xy 180.34 111.76))
     (stroke (width 0) (type default) (color 0 0 0 0))
@@
     (stroke (width 0) (type default) (color 0 0 0 0))
   )
+  (wire (pts (xy 124.46 97.79) (xy 132.08 97.79))
+    (stroke (width 0) (type default) (color 0 0 0 0))
+  )
   (wire (pts (xy 62.23 118.11) (xy 64.77 118.11))
     (stroke (width 0) (type default) (color 0 0 0 0))
   )
   (wire (pts (xy 187.96 92.71) (xy 175.26 92.71))
+    (stroke (width 0) (type default) (color 0 0 0 0))
+  )
+  (wire (pts (xy 110.49 90.17) (xy 110.49 97.79))
     (stroke (width 0) (type default) (color 0 0 0 0))
   )
@@
     (pin "2")
   )
+  (symbol (lib_id "Device:R") (at 120.65 97.79 270) (unit 1)
+    (in_bom yes) (on_board yes)
+    (property "Reference" "R505" (id 0) (at 119.38 92.71 90))
+    (property "Value" "10K" (id 1) (at 120.65 95.25 90))
+    (property "Footprint" "Resistor_SMD:R_0603_1608Metric_Pad0.98x0.95mm_HandSolder" (id 2) (at 120.65 96.012 90)
+      (effects (font (size 1.27 1.27)) hide)
+    )
+    (property "Datasheet" "~" (id 3) (at 120.65 97.79 0)
+      (effects (font (size 1.27 1.27)) hide)
+    )
+    (property "Distributor 1" "JLCPCB" (id 4) (at 120.65 97.79 90)
+      (effects (font (size 1.27 1.27)) hide)
+    )
+    (property "Distributor 1 PN" "C269701" (id 5) (at 120.65 97.79 90)
+      (effects (font (size 1.27 1.27)) hide)
+    )
+    (property "Manufacturer" "TyoHM" (id 6) (at 120.65 97.79 90)
+      (effects (font (size 1.27 1.27)) hide)
+    )
+    (property "MPN" "RMC 0603 10K F N" (id 7) (at 120.65 97.79 90)
+      (effects (font (size 1.27 1.27)) hide)
+    )
+    (property "Description" "0.1W ±1% 10kΩ 0603  Chip Resistor - Surface Mount ROHS" (id 8) (at 120.65 97.79 0)
+      (effects (font (size 1.27 1.27)) hide)
+    )
+    (property "AssemblyType" "SMT" (id 9) (at 120.65 97.79 0)
+      (effects (font (size 1.27 1.27)) hide)
+    )
+    (property "Cost" "0.0015" (id 10) (at 120.65 97.79 0)
+      (effects (font (size 1.27 1.27)) hide)
+    )
+    (pin "1")
+    (pin "2")
+  )
   (symbol (lib_id "Device:Buzzer") (at 190.5 90.17 0) (unit 1)
     (in_bom yes) (on_board yes) (fields_autoplaced)
@@
     (pin "4")
   )
+  (symbol (lib_id "power:GND") (at 132.08 99.06 0) (unit 1)
+    (in_bom yes) (on_board yes)
+    (property "Reference" "#PWR0508" (id 0) (at 132.08 105.41 0)
+      (effects (font (size 1.27 1.27)) hide)
+    )
+    (property "Value" "GND" (id 1) (at 132.207 103.4542 0))
+    (property "Footprint" "" (id 2) (at 132.08 99.06 0)
+      (effects (font (size 1.27 1.27)) hide)
+    )
+    (property "Datasheet" "" (id 3) (at 132.08 99.06 0)
+      (effects (font (size 1.27 1.27)) hide)
+    )
+    (pin "1")
+  )
 )
