File: Hardware/GeneralPurposeAlarmDevicePCB/GeneralPurposeAlarmDevicePCB/AlarmLights5.kicad_sch (KiCad schematic)
At the start: 20 parts

Commit message: Updated footprints and schematic Signed-off-by: lokimetasmith <lokimail@gmail.com>
Parts:
- D201, D202, D203, D204, D205: value (none) -> LED_T1.75_CLEAR_WHITE; footprint (none) -> GeneralPurposeAlarmDevicePCB:LED_5mm_Radial
- Q201, Q202, Q203, Q204, Q205: value (none) -> MMBT2222A-7-F; footprint (none) -> Package_TO_SOT_SMD:SOT-23
- R201, R203, R205, R207, R209: value (none) -> 4K7; footprint (none) -> Resistor_SMD:R_0603_1608Metric
- R202, R204, R206, R208, R210: value (none) -> 330R; footprint (none) -> Resistor_SMD:R_0603_1608Metric

Commit message: Mature the BOM parts. Remove misspelled fields. Add some costs.
Parts:
- D201, D202, D203, D204, D205: AssemblyType (none) -> HAND
- R201, R202, R203, R204, R205, R206, R207, R208, R209, R210: footprint Resistor_SMD:R_0603_1608Metric -> Resistor_SMD:R_0603_1608Metric_Pad0.98x0.95mm_HandSolder
Changed lines of the file:
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@@
     (property "Reference" "R201" (id 0) (at 78.74 90.17 0))
     (property "Value" "4K7" (id 1) (at 80.01 95.25 0))
-    (property "Footprint" "Resistor_SMD:R_0603_1608Metric" (id 2) (at 77.978 93.98 90)
+    (property "Footprint" "Resistor_SMD:R_0603_1608Metric_Pad0.98x0.95mm_HandSolder" (id 2) (at 77.978 93.98 90)
       (effects (font (size 1.27 1.27)) hide)
     )
@@
     (property "Reference" "R202" (id 0) (at 91.44 74.93 0))
     (property "Value" "330R" (id 1) (at 92.71 80.01 0))
-    (property "Footprint" "Resistor_SMD:R_0603_1608Metric" (id 2) (at 90.678 78.74 90)
+    (property "Footprint" "Resistor_SMD:R_0603_1608Metric_Pad0.98x0.95mm_HandSolder" (id 2) (at 90.678 78.74 90)
       (effects (font (size 1.27 1.27)) hide)
     )
@@
     (property "Reference" "R203" (id 0) (at 109.22 92.71 0))
     (property "Value" "4K7" (id 1) (at 110.49 95.25 0))
-    (property "Footprint" "Resistor_SMD:R_0603_1608Metric" (id 2) (at 108.458 93.98 90)
+    (property "Footprint" "Resistor_SMD:R_0603_1608Metric_Pad0.98x0.95mm_HandSolder" (id 2) (at 108.458 93.98 90)
       (effects (font (size 1.27 1.27)) hide)
     )
@@
     (property "Reference" "R204" (id 0) (at 121.92 74.93 0))
     (property "Value" "330R" (id 1) (at 123.19 80.01 0))
-    (property "Footprint" "Resistor_SMD:R_0603_1608Metric" (id 2) (at 121.158 78.74 90)
+    (property "Footprint" "Resistor_SMD:R_0603_1608Metric_Pad0.98x0.95mm_HandSolder" (id 2) (at 121.158 78.74 90)
       (effects (font (size 1.27 1.27)) hide)
     )
@@
     (property "Reference" "R205" (id 0) (at 139.7 92.71 0))
     (property "Value" "4K7" (id 1) (at 140.97 95.25 0))
-    (property "Footprint" "Resistor_SMD:R_0603_1608Metric" (id 2) (at 138.938 93.98 90)
+    (property "Footprint" "Resistor_SMD:R_0603_1608Metric_Pad0.98x0.95mm_HandSolder" (id 2) (at 138.938 93.98 90)
       (effects (font (size 1.27 1.27)) hide)
     )
@@
     (property "Reference" "R206" (id 0) (at 152.4 74.93 0))
     (property "Value" "330R" (id 1) (at 153.67 80.01 0))
-    (property "Footprint" "Resistor_SMD:R_0603_1608Metric" (id 2) (at 151.638 78.74 90)
+    (property "Footprint" "Resistor_SMD:R_0603_1608Metric_Pad0.98x0.95mm_HandSolder" (id 2) (at 151.638 78.74 90)
       (effects (font (size 1.27 1.27)) hide)
     )
@@
     (property "Reference" "R207" (id 0) (at 170.18 92.71 0))
     (property "Value" "4K7" (id 1) (at 171.45 95.25 0))
-    (property "Footprint" "Resistor_SMD:R_0603_1608Metric" (id 2) (at 169.418 93.98 90)
+    (property "Footprint" "Resistor_SMD:R_0603_1608Metric_Pad0.98x0.95mm_HandSolder" (id 2) (at 169.418 93.98 90)
       (effects (font (size 1.27 1.27)) hide)
     )
@@
     (property "Reference" "R208" (id 0) (at 182.88 74.93 0))
     (property "Value" "330R" (id 1) (at 184.15 80.01 0))
-    (property "Footprint" "Resistor_SMD:R_0603_1608Metric" (id 2) (at 182.118 78.74 90)
+    (property "Footprint" "Resistor_SMD:R_0603_1608Metric_Pad0.98x0.95mm_HandSolder" (id 2) (at 182.118 78.74 90)
       (effects (font (size 1.27 1.27)) hide)
     )
@@
     (property "Reference" "R209" (id 0) (at 200.66 92.71 0))
     (property "Value" "4K7" (id 1) (at 201.93 95.25 0))
-    (property "Footprint" "Resistor_SMD:R_0603_1608Metric" (id 2) (at 199.898 93.98 90)
+    (property "Footprint" "Resistor_SMD:R_0603_1608Metric_Pad0.98x0.95mm_HandSolder" (id 2) (at 199.898 93.98 90)
       (effects (font (size 1.27 1.27)) hide)
     )
@@
     (property "Reference" "R210" (id 0) (at 213.36 74.93 0))
     (property "Value" "330R" (id 1) (at 214.63 80.01 0))
-    (property "Footprint" "Resistor_SMD:R_0603_1608Metric" (id 2) (at 212.598 78.74 90)
+    (property "Footprint" "Resistor_SMD:R_0603_1608Metric_Pad0.98x0.95mm_HandSolder" (id 2) (at 212.598 78.74 90)
       (effects (font (size 1.27 1.27)) hide)
     )
@@
       (effects (font (size 1.524 1.524)) (justify left) hide)
     )
+    (property "AssemblyType" "HAND" (id 13) (at 119.38 90.17 0)
+      (effects (font (size 1.27 1.27)) hide)
+    )
     (pin "1")
     (pin "2")
@@
       (effects (font (size 1.524 1.524)) (justify left) hide)
     )
+    (property "AssemblyType" "HAND" (id 13) (at 149.86 90.17 0)
+      (effects (font (size 1.27 1.27)) hide)
+    )
     (pin "1")
     (pin "2")
@@
       (effects (font (size 1.524 1.524)) (justify left) hide)
     )
+    (property "AssemblyType" "HAND" (id 13) (at 180.34 90.17 0)
+      (effects (font (size 1.27 1.27)) hide)
+    )
     (pin "1")
     (pin "2")
@@
       (effects (font (size 1.524 1.524)) (justify left) hide)
     )
+    (property "AssemblyType" "HAND" (id 13) (at 210.82 90.17 0)
+      (effects (font (size 1.27 1.27)) hide)
+    )
     (pin "1")
     (pin "2")
@@
       (effects (font (size 1.524 1.524)) (justify left) hide)
     )
-    (pin "1")
+    (property "AssemblyType" "HAND" (id 13) (at 88.9 90.17 0)
+      (effects (font (size 1.27 1.27)) hide)
+    )
+    (pin "1")

Commit message: Update a lot of cost and PNs from JLCPCB and some Digikey.
Parts:
- D201, D202, D203, D204, D205: Cost (none) -> 0.65; Distributor 1 (none) -> DigiKey; Distributor 1 PN (none) -> 160-1772-ND
- Q201, Q202, Q203, Q204, Q205: AssemblyType (none) -> SMT; Cost (none) -> 0.0475; Distributor 1 (none) -> JLCPCB; Distributor 1 PN (none) -> C94515
- R201, R202, R203, R204, R205, R206, R207, R208, R209, R210: AssemblyType (none) -> SMT; Cost (none) -> 0.0015
Changed lines of the file:
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@@
+      (effects (font (size 1.27 1.27)) hide)
+    )
+    (property "AssemblyType" "SMT" (id 9) (at 76.2 93.98 0)
+      (effects (font (size 1.27 1.27)) hide)
+    )
+    (property "Cost" "0.0015" (id 10) (at 76.2 93.98 0)
       (effects (font (size 1.27 1.27)) hide)
     )
@@
       (effects (font (size 1.27 1.27)) hide)
     )
+    (property "AssemblyType" "SMT" (id 9) (at 88.9 78.74 0)
+      (effects (font (size 1.27 1.27)) hide)
+    )
+    (property "Cost" "0.0015" (id 10) (at 88.9 78.74 0)
+      (effects (font (size 1.27 1.27)) hide)
+    )
     (pin "1")
     (pin "2")
@@
       (effects (font (size 1.27 1.27)) hide)
     )
+    (property "AssemblyType" "SMT" (id 9) (at 106.68 93.98 0)
+      (effects (font (size 1.27 1.27)) hide)
+    )
+    (property "Cost" "0.0015" (id 10) (at 106.68 93.98 0)
+      (effects (font (size 1.27 1.27)) hide)
+    )
     (pin "1")
     (pin "2")
@@
       (effects (font (size 1.27 1.27)) hide)
     )
+    (property "AssemblyType" "SMT" (id 9) (at 119.38 78.74 0)
+      (effects (font (size 1.27 1.27)) hide)
+    )
+    (property "Cost" "0.0015" (id 10) (at 119.38 78.74 0)
+      (effects (font (size 1.27 1.27)) hide)
+    )
     (pin "1")
     (pin "2")
@@
       (effects (font (size 1.27 1.27)) hide)
     )
+    (property "AssemblyType" "SMT" (id 9) (at 137.16 93.98 0)
+      (effects (font (size 1.27 1.27)) hide)
+    )
+    (property "Cost" "0.0015" (id 10) (at 137.16 93.98 0)
+      (effects (font (size 1.27 1.27)) hide)
+    )
     (pin "1")
     (pin "2")
@@
       (effects (font (size 1.27 1.27)) hide)
     )
+    (property "AssemblyType" "SMT" (id 9) (at 149.86 78.74 0)
+      (effects (font (size 1.27 1.27)) hide)
+    )
+    (property "Cost" "0.0015" (id 10) (at 149.86 78.74 0)
+      (effects (font (size 1.27 1.27)) hide)
+    )
     (pin "1")
     (pin "2")
@@
       (effects (font (size 1.27 1.27)) hide)
     )
+    (property "AssemblyType" "SMT" (id 9) (at 167.64 93.98 0)
+      (effects (font (size 1.27 1.27)) hide)
+    )
+    (property "Cost" "0.0015" (id 10) (at 167.64 93.98 0)
+      (effects (font (size 1.27 1.27)) hide)
+    )
     (pin "1")
     (pin "2")
@@
       (effects (font (size 1.27 1.27)) hide)
     )
+    (property "AssemblyType" "SMT" (id 9) (at 180.34 78.74 0)
+      (effects (font (size 1.27 1.27)) hide)
+    )
+    (property "Cost" "0.0015" (id 10) (at 180.34 78.74 0)
+      (effects (font (size 1.27 1.27)) hide)
+    )
     (pin "1")
     (pin "2")
@@
       (effects (font (size 1.27 1.27)) hide)
     )
+    (property "AssemblyType" "SMT" (id 9) (at 198.12 93.98 0)
+      (effects (font (size 1.27 1.27)) hide)
+    )
+    (property "Cost" "0.0015" (id 10) (at 198.12 93.98 0)
+      (effects (font (size 1.27 1.27)) hide)
+    )
     (pin "1")
     (pin "2")
@@
       (effects (font (size 1.27 1.27)) hide)
     )
+    (property "AssemblyType" "SMT" (id 9) (at 210.82 78.74 0)
+      (effects (font (size 1.27 1.27)) hide)
+    )
+    (property "Cost" "0.0015" (id 10) (at 210.82 78.74 0)
+      (effects (font (size 1.27 1.27)) hide)
+    )
     (pin "1")
     (pin "2")
@@
       (effects (font (size 1.27 1.27)) hide)
     )
+    (property "Cost" "0.65" (id 14) (at 119.38 90.17 0)
+      (effects (font (size 1.27 1.27)) hide)
+    )
+    (property "Distributor 1" "DigiKey" (id 15) (at 119.38 90.17 0)
+      (effects (font (size 1.27 1.27)) hide)
+    )
+    (property "Distributor 1 PN" "160-1772-ND" (id 16) (at 119.38 90.17 0)
+      (effects (font (size 1.27 1.27)) hide)
+    )
     (pin "1")
     (pin "2")
@@
       (effects (font (size 1.27 1.27)) hide)
     )
+    (property "Cost" "0.65" (id 14) (at 149.86 90.17 0)
+      (effects (font (size 1.27 1.27)) hide)
+    )
+    (property "Distributor 1" "DigiKey" (id 15) (at 149.86 90.17 0)
+      (effects (font (size 1.27 1.27)) hide)
+    )
+    (property "Distributor 1 PN" "160-1772-ND" (id 16) (at 149.86 90.17 0)
+      (effects (font (size 1.27 1.27)) hide)
+    )
     (pin "1")
     (pin "2")
@@
       (effects (font (size 1.27 1.27)) hide)
     )
+    (property "Cost" "0.65" (id 14) (at 180.34 90.17 0)
+      (effects (font (size 1.27 1.27)) hide)
+    )
+    (property "Distributor 1" "DigiKey" (id 15) (at 180.34 90.17 0)
+      (effects (font (size 1.27 1.27)) hide)
+    )
+    (property "Distributor 1 PN" "160-1772-ND" (id 16) (at 180.34 90.17 0)
+      (effects (font (size 1.27 1.27)) hide)
+    )
     (pin "1")
     (pin "2")
@@
       (effects (font (size 1.27 1.27)) hide)
     )
+    (property "Cost" "0.65" (id 14) (at 210.82 90.17 0)
+      (effects (font (size 1.27 1.27)) hide)
+    )
+    (property "Distributor 1" "DigiKey" (id 15) (at 210.82 90.17 0)
+      (effects (font (size 1.27 1.27)) hide)
+    )
+    (property "Distributor 1 PN" "160-1772-ND" (id 16) (at 210.82 90.17 0)
+      (effects (font (size 1.27 1.27)) hide)
+    )
     (pin "1")
     (pin "2")
@@
     )
     (property "AssemblyType" "HAND" (id 13) (at 88.9 90.17 0)
+      (effects (font (size 1.27 1.27)) hide)
+    )
+    (property "Cost" "0.65" (id 14) (at 88.9 90.17 0)
+      (effects (font (size 1.27 1.27)) hide)
+    )
+    (property "Distributor 1" "DigiKey" (id 15) (at 88.9 90.17 0)
+      (effects (font (size 1.27 1.27)) hide)
+    )
+    (property "Distributor 1 PN" "160-1772-ND" (id 16) (at 88.9 90.17 0)
       (effects (font (size 1.27 1.27)) hide)
     )
@@
       (effects (font (size 1.524 1.524)) (justify left) hide)
     )
+    (property "AssemblyType" "SMT" (id 13) (at 86.36 100.33 0)
+      (effects (font (size 1.27 1.27)) hide)
+    )
+    (property "Distributor 1" "JLCPCB" (id 14) (at 86.36 100.33 0)
+      (effects (font (size 1.27 1.27)) hide)
+    )
+    (property "Distributor 1 PN" "C94515" (id 15) (at 86.36 100.33 0)
+      (effects (font (size 1.27 1.27)) hide)
+    )
+    (property "Cost" "0.0475" (id 16) (at 86.36 100.33 0)
+      (effects (font (size 1.27 1.27)) hide)
+    )
     (pin "1")
     (pin "2")
@@
       (effects (font (size 1.524 1.524)) (justify left) hide)
     )
+    (property "AssemblyType" "SMT" (id 13) (at 208.28 100.33 0)
+      (effects (font (size 1.27 1.27)) hide)
+    )
+    (property "Distributor 1" "JLCPCB" (id 14) (at 208.28 100.33 0)
+      (effects (font (size 1.27 1.27)) hide)
+    )
+    (property "Distributor 1 PN" "C94515" (id 15) (at 208.28 100.33 0)
+      (effects (font (size 1.27 1.27)) hide)
+    )
+    (property "Cost" "0.0475" (id 16) (at 208.28 100.33 0)
+      (effects (font (size 1.27 1.27)) hide)
+    )
     (pin "1")
     (pin "2")
@@
       (effects (font (size 1.524 1.524)) (justify left) hide)
     )
+    (property "AssemblyType" "SMT" (id 13) (at 177.8 100.33 0)
+      (effects (font (size 1.27 1.27)) hide)
+    )
+    (property "Distributor 1" "JLCPCB" (id 14) (at 177.8 100.33 0)
+      (effects (font (size 1.27 1.27)) hide)
+    )
+    (property "Distributor 1 PN" "C94515" (id 15) (at 177.8 100.33 0)
+      (effects (font (size 1.27 1.27)) hide)
+    )
+    (property "Cost" "0.0475" (id 16) (at 177.8 100.33 0)
+      (effects (font (size 1.27 1.27)) hide)
+    )
     (pin "1")
     (pin "2")
@@
       (effects (font (size 1.524 1.524)) (justify left) hide)
     )
+    (property "AssemblyType" "SMT" (id 13) (at 147.32 100.33 0)
+      (effects (font (size 1.27 1.27)) hide)
+    )
+    (property "Distributor 1" "JLCPCB" (id 14) (at 147.32 100.33 0)
+      (effects (font (size 1.27 1.27)) hide)
+    )
+    (property "Distributor 1 PN" "C94515" (id 15) (at 147.32 100.33 0)
+      (effects (font (size 1.27 1.27)) hide)
+    )
+    (property "Cost" "0.0475" (id 16) (at 147.32 100.33 0)
+      (effects (font (size 1.27 1.27)) hide)
+    )
     (pin "1")
     (pin "2")
@@
       (effects (font (size 1.524 1.524)) (justify left) hide)
     )
-    (pin "1")
+    (property "AssemblyType" "SMT" (id 13) (at 116.84 100.33 0)
+      (effects (font (size 1.27 1.27)) hide)
+    )
+    (property "Distributor 1" "JLCPCB" (id 14) (at 116.84 100.33 0)
+      (effects (font (size 1.27 1.27)) hide)
+    )
+    (property "Distributor 1 PN" "C94515" (id 15) (at 116.84 100.33 0)
+      (effects (font (size 1.27 1.27)) hide)
+    )
+    (property "Cost" "0.0475" (id 16) (at 116.84 100.33 0)
+      (effects (font (size 1.27 1.27)) hide)
+    )
+    (pin "1")
