File: Hardware/GeneralPurposeAlarmDevicePCB/GeneralPurposeAlarmDevicePCB/SPI Peripherial.kicad_sch (KiCad schematic)
At the start: 6 parts

Commit message: Updated footprints and schematic Signed-off-by: lokimetasmith <lokimail@gmail.com>
Parts:
- F401: renamed from F?; value (none) -> Polyfuse_Small; footprint (none) -> Fuse:Fuse_0603_1608Metric
- J401: value (none) -> RJ12_6P6C_HORZ; footprint (none) -> GeneralPurposeAlarmDevicePCB:RJ12_Amphenol_54601
- R401, R402, R403, R404: renamed from R?; value (none) -> 330; footprint (none) -> Resistor_SMD:R_0603_1608Metric
Changed lines of the file:
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@@
   (symbol (lib_id "Device:R") (at 132.08 100.33 270) (unit 1)
     (in_bom yes) (on_board yes)
-    (property "Reference" "R?" (id 0) (at 130.81 95.25 90))
-    (property "Value" "" (id 1) (at 132.08 97.79 90))
-    (property "Footprint" "" (id 2) (at 132.08 98.552 90)
+    (property "Reference" "R401" (id 0) (at 130.81 95.25 90))
+    (property "Value" "330" (id 1) (at 132.08 97.79 90))
+    (property "Footprint" "Resistor_SMD:R_0603_1608Metric" (id 2) (at 132.08 98.552 90)
       (effects (font (size 1.27 1.27)) hide)
     )
@@
   (symbol (lib_id "Device:R") (at 142.24 106.68 270) (unit 1)
     (in_bom yes) (on_board yes)
-    (property "Reference" "R?" (id 0) (at 140.97 101.6 90))
-    (property "Value" "" (id 1) (at 142.24 104.14 90))
-    (property "Footprint" "" (id 2) (at 142.24 104.902 90)
+    (property "Reference" "R402" (id 0) (at 140.97 101.6 90))
+    (property "Value" "330" (id 1) (at 142.24 104.14 90))
+    (property "Footprint" "Resistor_SMD:R_0603_1608Metric" (id 2) (at 142.24 104.902 90)
       (effects (font (size 1.27 1.27)) hide)
     )
@@
   (symbol (lib_id "Device:R") (at 153.67 113.03 270) (unit 1)
     (in_bom yes) (on_board yes)
-    (property "Reference" "R?" (id 0) (at 152.4 107.95 90))
-    (property "Value" "" (id 1) (at 153.67 110.49 90))
-    (property "Footprint" "" (id 2) (at 153.67 111.252 90)
+    (property "Reference" "R403" (id 0) (at 152.4 107.95 90))
+    (property "Value" "330" (id 1) (at 153.67 110.49 90))
+    (property "Footprint" "Resistor_SMD:R_0603_1608Metric" (id 2) (at 153.67 111.252 90)
       (effects (font (size 1.27 1.27)) hide)
     )
@@
   (symbol (lib_id "Device:R") (at 185.42 123.19 270) (unit 1)
     (in_bom yes) (on_board yes)
-    (property "Reference" "R?" (id 0) (at 184.15 118.11 90))
-    (property "Value" "" (id 1) (at 185.42 120.65 90))
-    (property "Footprint" "" (id 2) (at 185.42 121.412 90)
+    (property "Reference" "R404" (id 0) (at 184.15 118.11 90))
+    (property "Value" "330" (id 1) (at 185.42 120.65 90))
+    (property "Footprint" "Resistor_SMD:R_0603_1608Metric" (id 2) (at 185.42 121.412 90)
       (effects (font (size 1.27 1.27)) hide)
     )
@@
   (symbol (lib_id "power:GND") (at 123.19 107.95 0) (unit 1)
     (in_bom yes) (on_board yes)
-    (property "Reference" "#PWR?" (id 0) (at 123.19 114.3 0)
+    (property "Reference" "#PWR0401" (id 0) (at 123.19 114.3 0)
       (effects (font (size 1.27 1.27)) hide)
     )
-    (property "Value" "" (id 1) (at 125.73 107.95 0))
+    (property "Value" "GND" (id 1) (at 125.73 107.95 0))
     (property "Footprint" "" (id 2) (at 123.19 107.95 0)
       (effects (font (size 1.27 1.27)) hide)
@@
     (in_bom yes) (on_board yes)
     (property "Reference" "J401" (id 0) (at 105.5878 91.2622 0))
-    (property "Value" "" (id 1) (at 105.5878 93.5736 0))
-    (property "Footprint" "" (id 2) (at 104.14 107.315 90)
+    (property "Value" "RJ12_6P6C_HORZ" (id 1) (at 105.5878 93.5736 0))
+    (property "Footprint" "GeneralPurposeAlarmDevicePCB:RJ12_Amphenol_54601" (id 2) (at 104.14 107.315 90)
       (effects (font (size 1.27 1.27)) hide)
     )
@@
   (symbol (lib_id "Device:Polyfuse_Small") (at 186.69 102.87 270) (unit 1)
     (in_bom yes) (on_board yes)
-    (property "Reference" "F?" (id 0) (at 186.69 97.663 90))
-    (property "Value" "" (id 1) (at 187.96 105.41 90))
-    (property "Footprint" "" (id 2) (at 181.61 104.14 0)
+    (property "Reference" "F401" (id 0) (at 186.69 97.663 90))
+    (property "Value" "Polyfuse_Small" (id 1) (at 187.96 105.41 90))
+    (property "Footprint" "Fuse:Fuse_0603_1608Metric" (id 2) (at 181.61 104.14 0)
       (effects (font (size 1.27 1.27)) (justify left) hide)
     )

Commit message: Update buzzer foot print. Fully connect all parts. Fix numerous silkscreen conflicts. Mix of metric and imperial grid.
Parts:
- J401: AssemblyType (none) -> HAND
Changed lines of the file:
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@@
       (effects (font (size 1.27 1.27)) hide)
     )
+    (property "AssemblyType" "HAND" (id 12) (at 104.14 107.95 0))
     (pin "1")
     (pin "2")
@@
       (effects (font (size 1.27 1.27)) (justify left) hide)
     )
-    (property "Datasheet" "https://datasheet.lcsc.com/lcsc/1806131741_Littelfuse-0603L075SLYR_C207016.pdf" (id 3) (at 186.69 102.87 0)
+    (property "Datasheet" "~" (id 3) (at 186.69 102.87 0)
       (effects (font (size 1.27 1.27)) hide)
     )

Commit message: Mature the BOM parts. Remove misspelled fields. Add some costs.
Parts:
- J401: Assembly Type HAND -> (none)
- R401, R402, R403, R404: footprint Resistor_SMD:R_0603_1608Metric -> Resistor_SMD:R_0603_1608Metric_Pad0.98x0.95mm_HandSolder
Changed lines of the file:
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@@
     (property "Reference" "R401" (id 0) (at 130.81 95.25 90))
     (property "Value" "330" (id 1) (at 132.08 97.79 90))
-    (property "Footprint" "Resistor_SMD:R_0603_1608Metric" (id 2) (at 132.08 98.552 90)
+    (property "Footprint" "Resistor_SMD:R_0603_1608Metric_Pad0.98x0.95mm_HandSolder" (id 2) (at 132.08 98.552 90)
       (effects (font (size 1.27 1.27)) hide)
     )
@@
     (property "Reference" "R402" (id 0) (at 140.97 101.6 90))
     (property "Value" "330" (id 1) (at 142.24 104.14 90))
-    (property "Footprint" "Resistor_SMD:R_0603_1608Metric" (id 2) (at 142.24 104.902 90)
+    (property "Footprint" "Resistor_SMD:R_0603_1608Metric_Pad0.98x0.95mm_HandSolder" (id 2) (at 142.24 104.902 90)
       (effects (font (size 1.27 1.27)) hide)
     )
@@
     (property "Reference" "R403" (id 0) (at 152.4 107.95 90))
     (property "Value" "330" (id 1) (at 153.67 110.49 90))
-    (property "Footprint" "Resistor_SMD:R_0603_1608Metric" (id 2) (at 153.67 111.252 90)
+    (property "Footprint" "Resistor_SMD:R_0603_1608Metric_Pad0.98x0.95mm_HandSolder" (id 2) (at 153.67 111.252 90)
       (effects (font (size 1.27 1.27)) hide)
     )
@@
     (property "Reference" "R404" (id 0) (at 184.15 118.11 90))
     (property "Value" "330" (id 1) (at 185.42 120.65 90))
-    (property "Footprint" "Resistor_SMD:R_0603_1608Metric" (id 2) (at 185.42 121.412 90)
+    (property "Footprint" "Resistor_SMD:R_0603_1608Metric_Pad0.98x0.95mm_HandSolder" (id 2) (at 185.42 121.412 90)
       (effects (font (size 1.27 1.27)) hide)
     )
@@
       (effects (font (size 1.27 1.27)) hide)
     )
-    (property "Assembly Type" "HAND" (id 10) (at 105.5878 95.885 0))
+    (property "Assembly Type" "" (id 10) (at 105.5878 95.885 0))
     (property "MPN" "5555165-1" (id 11) (at 104.14 107.95 0)
       (effects (font (size 1.27 1.27)) hide)

Commit message: Update a lot of cost and PNs from JLCPCB and some Digikey.
Parts:
- F401: AssemblyType (none) -> SMT; Cost (none) -> 0.2448; Distributor 1 (none) -> JLCPCB; Distributor 1 PN (none) -> C207017
- J401: Cost (none) -> 0.8901
- R401, R402, R403, R404: AssemblyType (none) -> SMT; Cost (none) -> 0.0015
Changed lines of the file:
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@@
+      (effects (font (size 1.27 1.27)) hide)
+    )
+    (property "AssemblyType" "SMT" (id 9) (at 132.08 100.33 0)
+      (effects (font (size 1.27 1.27)) hide)
+    )
+    (property "Cost" "0.0015" (id 10) (at 132.08 100.33 0)
       (effects (font (size 1.27 1.27)) hide)
     )
@@
       (effects (font (size 1.27 1.27)) hide)
     )
+    (property "AssemblyType" "SMT" (id 9) (at 142.24 106.68 0)
+      (effects (font (size 1.27 1.27)) hide)
+    )
+    (property "Cost" "0.0015" (id 10) (at 142.24 106.68 0)
+      (effects (font (size 1.27 1.27)) hide)
+    )
     (pin "1")
     (pin "2")
@@
       (effects (font (size 1.27 1.27)) hide)
     )
+    (property "AssemblyType" "SMT" (id 9) (at 153.67 113.03 0)
+      (effects (font (size 1.27 1.27)) hide)
+    )
+    (property "Cost" "0.0015" (id 10) (at 153.67 113.03 0)
+      (effects (font (size 1.27 1.27)) hide)
+    )
     (pin "1")
     (pin "2")
@@
       (effects (font (size 1.27 1.27)) hide)
     )
+    (property "AssemblyType" "SMT" (id 9) (at 185.42 123.19 0)
+      (effects (font (size 1.27 1.27)) hide)
+    )
+    (property "Cost" "0.0015" (id 10) (at 185.42 123.19 0)
+      (effects (font (size 1.27 1.27)) hide)
+    )
     (pin "1")
     (pin "2")
@@
     )
     (property "AssemblyType" "HAND" (id 12) (at 104.14 107.95 0))
+    (property "Cost" "0.8901" (id 13) (at 104.14 107.95 0)
+      (effects (font (size 1.27 1.27)) hide)
+    )
     (pin "1")
     (pin "2")
@@
       (effects (font (size 1.27 1.27)) hide)
     )
+    (property "AssemblyType" "SMT" (id 6) (at 186.69 102.87 0)
+      (effects (font (size 1.27 1.27)) hide)
+    )
+    (property "Cost" "0.2448" (id 7) (at 186.69 102.87 0)
+      (effects (font (size 1.27 1.27)) hide)
+    )
+    (property "Description" "6V 1A 50A -40℃~+85℃ 1.8A 40mΩ 300ms 120mΩ 0603 Resettable Fuses ROHS" (id 8) (at 186.69 102.87 0)
+      (effects (font (size 1.27 1.27)) hide)
+    )
+    (property "Distributor 1" "JLCPCB" (id 9) (at 186.69 102.87 0)
+      (effects (font (size 1.27 1.27)) hide)
+    )
+    (property "Distributor 1 PN" "C207017" (id 10) (at 186.69 102.87 0)
+      (effects (font (size 1.27 1.27)) hide)
+    )
