File: Hardware/GeneralPurposeAlarmDevicePCB/GeneralPurposeAlarmDevicePCB/USB_UART.kicad_sch (KiCad schematic)
At the start: 10 parts

Commit message: Updated footprints and schematic Signed-off-by: lokimetasmith <lokimail@gmail.com>
Parts:
- C501, C503: renamed from C?; value (none) -> 100nF; footprint (none) -> Capacitor_SMD:C_0603_1608Metric_Pad1.08x0.95mm_HandSolder
- C502: renamed from C?; value (none) -> 47uF 16V; footprint (none) -> Capacitor_SMD:CP_Elec_5x5.4; symbol GeneralPurposeAlarmDevicePCB-rescue:CP-Device -> Device:C_Polarized
- D501: renamed from D?; value (none) -> RED 0603; footprint (none) -> LED_SMD:LED_0603_1608Metric; symbol GeneralPurposeAlarmDevicePCB-rescue:LTST-C171KRKT-dk_LED-Indication-Discrete -> Device:LED
- J501: value (none) -> USB_B_Micro; footprint (none) -> Connector_USB:USB_Micro-B_Wuerth_629105150521
- R501, R502, R503: renamed from R?; value (none) -> 330R; footprint (none) -> Resistor_SMD:R_0603_1608Metric
- R504: renamed from R?; value (none) -> 4K7; footprint (none) -> Resistor_SMD:R_0603_1608Metric
- U501: renamed from U?; value (none) -> CH340E; footprint (none) -> Package_SO:MSOP-10_3x3mm_P0.5mm
Connections:
- net GND: now also C502.2, D501.2 (A)
- net VBUS: now also C502.1
- net at R501.2: now also D501.1 (K)

Commit message: Update buzzer foot print. Fully connect all parts. Fix numerous silkscreen conflicts. Mix of metric and imperial grid.
Parts:
- J501: footprint Connector_USB:USB_Micro-B_Wuerth_629105150521 -> GeneralPurposeAlarmDevicePCB:USB_Micro-B_Amphenol_10118194_Horizontal; Distributor 1 PN ??? C132563 -> C132563; MPN  (none) -> 10118194-0001LF; Manufacturer  (none) -> Amphenol ICC
Connections:
- net VBUS renamed VBus
Changed lines of the file:
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@@
     (effects (font (size 1.27 1.27)) (justify left bottom))
   )
-  (hierarchical_label "VBUS" (shape passive) (at 212.09 76.2 0)
+  (hierarchical_label "VBus" (shape passive) (at 212.09 76.2 0)
     (effects (font (size 1.27 1.27)) (justify left))
   )
@@
     (property "Reference" "J501" (id 0) (at 94.1578 83.3882 0))
     (property "Value" "USB_B_Micro" (id 1) (at 94.1578 85.6996 0))
-    (property "Footprint" "Connector_USB:USB_Micro-B_Wuerth_629105150521" (id 2) (at 96.52 96.52 0)
+    (property "Footprint" "GeneralPurposeAlarmDevicePCB:USB_Micro-B_Amphenol_10118194_Horizontal" (id 2) (at 96.52 96.52 0)
       (effects (font (size 1.27 1.27)) hide)
     )
@@
       (effects (font (size 1.27 1.27)) hide)
     )
-    (property "Distributor 1 PN" "???   C132563" (id 5) (at 92.71 95.25 0)
+    (property "Distributor 1 PN" "C132563" (id 5) (at 92.71 95.25 0)
       (effects (font (size 1.27 1.27)) hide)
     )
@@
       (effects (font (size 1.27 1.27)) hide)
     )
+    (property "Manufacturer " "Amphenol ICC" (id 8) (at 92.71 95.25 0)
+      (effects (font (size 1.27 1.27)) hide)
+    )
+    (property "MPN " "10118194-0001LF" (id 9) (at 92.71 95.25 0)
+      (effects (font (size 1.27 1.27)) hide)
+    )

Commit message: Add USB footprint 3D model for 10118194.
Parts:
- J501: MPN Wuerth_629105150521 ??? 10118194-0001LF -> 10118194-0001LF ???Wuerth_629105150521 ??? Molex 1050170001; Manufacturer Wuerth_629105150521 ??? Amphenol ICC -> Amphenol ICC ??? Wuerth ???Molex
Changed lines of the file:
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@@
       (effects (font (size 1.27 1.27)) hide)
     )
-    (property "Manufacturer" "Wuerth_629105150521  ???  Amphenol ICC" (id 6) (at 92.71 95.25 0)
+    (property "Manufacturer" "Amphenol ICC ???  Wuerth  ???Molex" (id 6) (at 92.71 95.25 0)
       (effects (font (size 1.27 1.27)) hide)
     )
-    (property "MPN" "Wuerth_629105150521  ??? 10118194-0001LF" (id 7) (at 92.71 95.25 0)
+    (property "MPN" "10118194-0001LF ???Wuerth_629105150521  ??? Molex 1050170001" (id 7) (at 92.71 95.25 0)
       (effects (font (size 1.27 1.27)) hide)
     )

Commit message: Add 7805 alternative for linear regulator, Add test points on power supply nets, add MechanicalPartsPlacement.pdf.
Parts:
- added TP201: TP_VBus, TestPoint:TestPoint_Loop_D2.54mm_Drill1.5mm_Beaded, symbol Connector:TestPoint
- added TP202: TP_V3, TestPoint:TestPoint_Loop_D2.54mm_Drill1.5mm_Beaded, symbol Connector:TestPoint
- added TP_nCTS201: TestPoint_nCTS, TestPoint:TestPoint_Loop_D2.54mm_Drill1.5mm_Beaded, symbol Connector:TestPoint
Connections:
- net GND: now also D501.1 (K); no longer D501.2 (A)
- net VBus: now also TP201.1
- net at C503.1, U501.10 (V3): now also TP202.1
- net at R504.2, U501.5 (~{CTS}): now also TP_nCTS201.1
- net at R501.2: now also D501.2 (A); no longer D501.1 (K)
Other:
- moved on the sheet: D501, R504
Changed lines of the file:
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@@
   (junction (at 154.94 76.2) (diameter 0) (color 0 0 0 0)
   )
+  (junction (at 175.26 105.41) (diameter 0) (color 0 0 0 0)
+  )
   (junction (at 120.65 76.2) (diameter 0) (color 0 0 0 0)
   )
   (junction (at 106.68 76.2) (diameter 0) (color 0 0 0 0)
+  )
+  (junction (at 137.16 78.74) (diameter 0) (color 0 0 0 0)
+  )
+  (junction (at 114.3 76.2) (diameter 0) (color 0 0 0 0)
   )
   (junction (at 154.94 116.84) (diameter 0) (color 0 0 0 0)
@@
   (no_connect (at 100.33 100.33))
   (no_connect (at 165.1 107.95))
+  (wire (pts (xy 114.3 76.2) (xy 106.68 76.2))
+    (stroke (width 0) (type default) (color 0 0 0 0))
+  )
   (wire (pts (xy 154.94 116.84) (xy 175.26 116.84))
     (stroke (width 0) (type default) (color 0 0 0 0))
@@
     (stroke (width 0) (type default) (color 0 0 0 0))
   )
+  (wire (pts (xy 175.26 105.41) (xy 193.04 105.41))
+    (stroke (width 0) (type default) (color 0 0 0 0))
+  )
   (wire (pts (xy 140.97 107.95) (xy 137.16 107.95))
     (stroke (width 0) (type default) (color 0 0 0 0))
@@
     (stroke (width 0) (type default) (color 0 0 0 0))
   )
-  (wire (pts (xy 175.26 116.84) (xy 175.26 110.49))
+  (wire (pts (xy 175.26 116.84) (xy 175.26 114.3))
     (stroke (width 0) (type default) (color 0 0 0 0))
   )
@@
     (stroke (width 0) (type default) (color 0 0 0 0))
   )
+  (wire (pts (xy 137.16 71.12) (xy 137.16 78.74))
+    (stroke (width 0) (type default) (color 0 0 0 0))
+  )
   (wire (pts (xy 129.54 107.95) (xy 125.73 107.95))
     (stroke (width 0) (type default) (color 0 0 0 0))
@@
     (stroke (width 0) (type default) (color 0 0 0 0))
   )
-  (wire (pts (xy 166.37 102.87) (xy 166.37 95.25))
+  (wire (pts (xy 175.26 105.41) (xy 175.26 106.68))
+    (stroke (width 0) (type default) (color 0 0 0 0))
+  )
+  (wire (pts (xy 166.37 101.6) (xy 166.37 95.25))
+    (stroke (width 0) (type default) (color 0 0 0 0))
+  )
+  (wire (pts (xy 166.37 101.6) (xy 175.26 101.6))
+    (stroke (width 0) (type default) (color 0 0 0 0))
+  )
+  (wire (pts (xy 114.3 72.39) (xy 114.3 76.2))
     (stroke (width 0) (type default) (color 0 0 0 0))
   )
@@
     (stroke (width 0) (type default) (color 0 0 0 0))
   )
-  (wire (pts (xy 120.65 76.2) (xy 106.68 76.2))
-    (stroke (width 0) (type default) (color 0 0 0 0))
-  )
-  (wire (pts (xy 175.26 102.87) (xy 166.37 102.87))
+  (wire (pts (xy 120.65 76.2) (xy 114.3 76.2))
+    (stroke (width 0) (type default) (color 0 0 0 0))
+  )
+  (wire (pts (xy 175.26 101.6) (xy 175.26 105.41))
     (stroke (width 0) (type default) (color 0 0 0 0))
   )
@@
   )
   (text "TX is Output\nRX is Input\n/CTS is Input\n/RTS is Output"
-    (at 185.42 107.95 0)
+    (at 234.95 95.25 0)
     (effects (font (size 1.27 1.27)) (justify left bottom))
   )
@@
     (pin "2")
   )
-  (symbol (lib_id "Device:LED") (at 121.92 107.95 180) (unit 1)
-    (in_bom yes) (on_board yes)
-    (property "Reference" "D501" (id 0) (at 121.92 104.14 0)
+  (symbol (lib_id "Device:LED") (at 121.92 107.95 0) (mirror x) (unit 1)
+    (in_bom yes) (on_board yes)
+    (property "Reference" "D501" (id 0) (at 123.19 105.41 0)
       (effects (font (size 1.524 1.524)))
     )
-    (property "Value" "RED 0603" (id 1) (at 125.73 113.03 0)
+    (property "Value" "RED 0603" (id 1) (at 124.46 110.49 0)
       (effects (font (size 1.524 1.524)))
     )
@@
       (effects (font (size 1.27 1.27)) hide)
     )
-    (property "Distributor 1 PN" "C2286" (id 5) (at 116.84 118.11 0)
+    (property "Distributor 1 PN" "C2286" (id 5) (at 127 118.11 0)
       (effects (font (size 1.524 1.524)) (justify left) hide)
     )
-    (property "MPN" "KT-0603R" (id 6) (at 116.84 120.65 0)
+    (property "MPN" "KT-0603R" (id 6) (at 127 120.65 0)
       (effects (font (size 1.524 1.524)) (justify left) hide)
     )
-    (property "Category" "Optoelectronics" (id 7) (at 116.84 123.19 0)
+    (property "Category" "Optoelectronics" (id 7) (at 127 123.19 0)
       (effects (font (size 1.524 1.524)) (justify left) hide)
     )
-    (property "Family" "LED Indication - Discrete" (id 8) (at 116.84 125.73 0)
+    (property "Family" "LED Indication - Discrete" (id 8) (at 127 125.73 0)
       (effects (font (size 1.524 1.524)) (justify left) hide)
     )
-    (property "Description" "LED RED CLEAR SMD" (id 9) (at 116.84 133.35 0)
+    (property "Description" "LED RED CLEAR SMD" (id 9) (at 127 133.35 0)
       (effects (font (size 1.524 1.524)) (justify left) hide)
     )
-    (property "Manufacturer" "Hubei KENTO Elec" (id 10) (at 116.84 135.89 0)
+    (property "Manufacturer" "Hubei KENTO Elec" (id 10) (at 127 135.89 0)
       (effects (font (size 1.524 1.524)) (justify left) hide)
     )
-    (property "Status" "Active" (id 11) (at 116.84 138.43 0)
+    (property "Status" "Active" (id 11) (at 127 138.43 0)
       (effects (font (size 1.524 1.524)) (justify left) hide)
     )
@@
     (pin "1")
   )
-  (symbol (lib_id "Device:R") (at 175.26 106.68 180) (unit 1)
-    (in_bom yes) (on_board yes)
-    (property "Reference" "R504" (id 0) (at 179.07 105.41 0))
-    (property "Value" "4K7" (id 1) (at 179.07 107.95 0))
-    (property "Footprint" "Resistor_SMD:R_0603_1608Metric" (id 2) (at 177.038 106.68 90)
-      (effects (font (size 1.27 1.27)) hide)
-    )
-    (property "Datasheet" "~" (id 3) (at 175.26 106.68 0)
-      (effects (font (size 1.27 1.27)) hide)
-    )
-    (property "Distributor 1" "JLCPCB" (id 4) (at 175.26 106.68 90)
-      (effects (font (size 1.27 1.27)) hide)
-    )
-    (property "Distributor 1 PN" "C269713" (id 5) (at 175.26 106.68 90)
-      (effects (font (size 1.27 1.27)) hide)
-    )
-    (property "Manufacturer" "TyoHM" (id 6) (at 175.26 106.68 90)
-      (effects (font (size 1.27 1.27)) hide)
-    )
-    (property "MPN" "RMC 0603 4K7 F N" (id 7) (at 175.26 106.68 90)
-      (effects (font (size 1.27 1.27)) hide)
-    )
-    (property "Description" "1W ±1% 4.7kΩ 0603 Chip Resistor - Surface Mount ROHS" (id 8) (at 175.26 106.68 0)
+  (symbol (lib_id "Device:R") (at 175.26 110.49 180) (unit 1)
+    (in_bom yes) (on_board yes)
+    (property "Reference" "R504" (id 0) (at 179.07 109.22 0))
+    (property "Value" "4K7" (id 1) (at 179.07 111.76 0))
+    (property "Footprint" "Resistor_SMD:R_0603_1608Metric" (id 2) (at 177.038 110.49 90)
+      (effects (font (size 1.27 1.27)) hide)
+    )
+    (property "Datasheet" "~" (id 3) (at 175.26 110.49 0)
+      (effects (font (size 1.27 1.27)) hide)
+    )
+    (property "Distributor 1" "JLCPCB" (id 4) (at 175.26 110.49 90)
+      (effects (font (size 1.27 1.27)) hide)
+    )
+    (property "Distributor 1 PN" "C269713" (id 5) (at 175.26 110.49 90)
+      (effects (font (size 1.27 1.27)) hide)
+    )
+    (property "Manufacturer" "TyoHM" (id 6) (at 175.26 110.49 90)
+      (effects (font (size 1.27 1.27)) hide)
+    )
+    (property "MPN" "RMC 0603 4K7 F N" (id 7) (at 175.26 110.49 90)
+      (effects (font (size 1.27 1.27)) hide)
+    )
+    (property "Description" "1W ±1% 4.7kΩ 0603 Chip Resistor - Surface Mount ROHS" (id 8) (at 175.26 110.49 0)
       (effects (font (size 1.27 1.27)) hide)
     )
@@
       (effects (font (size 1.27 1.27)) hide)
     )
+    (pin "1")
+  )
+  (symbol (lib_id "Connector:TestPoint") (at 114.3 72.39 0) (unit 1)
+    (in_bom yes) (on_board yes)
+    (property "Reference" "TP201" (id 0) (at 115.57 68.58 0)
+      (effects (font (size 1.27 1.27)) (justify left))
+    )
+    (property "Value" "TP_VBus" (id 1) (at 115.57 71.12 0)
+      (effects (font (size 1.27 1.27)) (justify left))
+    )
+    (property "Footprint" "TestPoint:TestPoint_Loop_D2.54mm_Drill1.5mm_Beaded" (id 2) (at 119.38 72.39 0)
+      (effects (font (size 1.27 1.27)) hide)
+    )
+    (property "Datasheet" "~" (id 3) (at 119.38 72.39 0)
+      (effects (font (size 1.27 1.27)) hide)
+    )
+    (pin "1")
+  )
+  (symbol (lib_id "Connector:TestPoint") (at 137.16 71.12 0) (unit 1)
+    (in_bom yes) (on_board yes)
+    (property "Reference" "TP202" (id 0) (at 138.43 67.31 0)
+      (effects (font (size 1.27 1.27)) (justify left))
+    )
+    (property "Value" "TP_V3" (id 1) (at 138.43 69.85 0)
+      (effects (font (size 1.27 1.27)) (justify left))
+    )
+    (property "Footprint" "TestPoint:TestPoint_Loop_D2.54mm_Drill1.5mm_Beaded" (id 2) (at 142.24 71.12 0)
+      (effects (font (size 1.27 1.27)) hide)
+    )
+    (property "Datasheet" "~" (id 3) (at 142.24 71.12 0)
+      (effects (font (size 1.27 1.27)) hide)
+    )
+    (pin "1")
+  )
+  (symbol (lib_id "Connector:TestPoint") (at 193.04 105.41 0) (unit 1)
+    (in_bom yes) (on_board yes)
+    (property "Reference" "TP_nCTS201" (id 0) (at 194.31 101.6 0)
+      (effects (font (size 1.27 1.27)) (justify left))
+    )
+    (property "Value" "TestPoint_nCTS" (id 1) (at 194.31 104.14 0)
+      (effects (font (size 1.27 1.27)) (justify left))
+    )
+    (property "Footprint" "TestPoint:TestPoint_Loop_D2.54mm_Drill1.5mm_Beaded" (id 2) (at 198.12 105.41 0)
+      (effects (font (size 1.27 1.27)) hide)
+    )
+    (property "Datasheet" "~" (id 3) (at 198.12 105.41 0)
+      (effects (font (size 1.27 1.27)) hide)
+    )

Commit message: Change TP to show value on F silk screen. Make REF DES smaller.
Parts:
- TP201: value TP_VBus -> VBus
- TP202: value TP_V3 -> V3
- TP203: renamed from TP_nCTS201; value TestPoint_nCTS -> nCTS
Changed lines of the file:
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@@
       (effects (font (size 1.27 1.27)) (justify left))
     )
-    (property "Value" "TP_VBus" (id 1) (at 115.57 71.12 0)
+    (property "Value" "VBus" (id 1) (at 115.57 71.12 0)
       (effects (font (size 1.27 1.27)) (justify left))
     )
@@
       (effects (font (size 1.27 1.27)) (justify left))
     )
-    (property "Value" "TP_V3" (id 1) (at 138.43 69.85 0)
+    (property "Value" "V3" (id 1) (at 138.43 69.85 0)
       (effects (font (size 1.27 1.27)) (justify left))
     )
@@
   (symbol (lib_id "Connector:TestPoint") (at 193.04 105.41 0) (unit 1)
     (in_bom yes) (on_board yes)
-    (property "Reference" "TP_nCTS201" (id 0) (at 194.31 101.6 0)
+    (property "Reference" "TP203" (id 0) (at 194.31 101.6 0)
       (effects (font (size 1.27 1.27)) (justify left))
     )
-    (property "Value" "TestPoint_nCTS" (id 1) (at 194.31 104.14 0)
+    (property "Value" "nCTS" (id 1) (at 194.31 104.14 0)
       (effects (font (size 1.27 1.27)) (justify left))
     )

Commit message: Mature the BOM parts. Remove misspelled fields. Add some costs.
Parts:
- removed J501: USB_B_Micro, GeneralPurposeAlarmDevicePCB:USB_Micro-B_Amphenol_10118194_Horizontal, symbol GPAD_SCH_LIB:USB_B_Micro
- added J501: USB_B_Micro_Local, GeneralPurposeAlarmDevicePCB:USB_Micro-B_Amphenol_10118194_Horizontal, symbol GPAD_SCH_LIB:USB_B_Micro_Local
- R501, R502, R503, R504: footprint Resistor_SMD:R_0603_1608Metric -> Resistor_SMD:R_0603_1608Metric_Pad0.98x0.95mm_HandSolder
- TP201, TP202, TP203: AssemblyType (none) -> HAND
Connections:
- net GND: now also J501.5 (GND), J501.6 (Shield)
- net VBus: now also J501.1 (VBUS)
- net at U501.1 (UD+): now also J501.3 (D+)
- net at U501.2 (UD-): now also J501.2 (D-)
Changed lines of the file:
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@@
     (property "Reference" "R502" (id 0) (at 171.45 82.55 90))
     (property "Value" "330R" (id 1) (at 172.72 85.09 90))
-    (property "Footprint" "Resistor_SMD:R_0603_1608Metric" (id 2) (at 172.72 85.852 90)
+    (property "Footprint" "Resistor_SMD:R_0603_1608Metric_Pad0.98x0.95mm_HandSolder" (id 2) (at 172.72 85.852 90)
       (effects (font (size 1.27 1.27)) hide)
     )
@@
     (property "Reference" "R503" (id 0) (at 171.45 91.44 90))
     (property "Value" "330R" (id 1) (at 172.72 93.98 90))
-    (property "Footprint" "Resistor_SMD:R_0603_1608Metric" (id 2) (at 172.72 94.742 90)
+    (property "Footprint" "Resistor_SMD:R_0603_1608Metric_Pad0.98x0.95mm_HandSolder" (id 2) (at 172.72 94.742 90)
       (effects (font (size 1.27 1.27)) hide)
     )
@@
     (property "Reference" "R501" (id 0) (at 132.08 102.87 90))
     (property "Value" "330R" (id 1) (at 133.35 105.41 90))
-    (property "Footprint" "Resistor_SMD:R_0603_1608Metric" (id 2) (at 133.35 106.172 90)
+    (property "Footprint" "Resistor_SMD:R_0603_1608Metric_Pad0.98x0.95mm_HandSolder" (id 2) (at 133.35 106.172 90)
       (effects (font (size 1.27 1.27)) hide)
     )
@@
     (property "Reference" "R504" (id 0) (at 179.07 109.22 0))
     (property "Value" "4K7" (id 1) (at 179.07 111.76 0))
-    (property "Footprint" "Resistor_SMD:R_0603_1608Metric" (id 2) (at 177.038 110.49 90)
+    (property "Footprint" "Resistor_SMD:R_0603_1608Metric_Pad0.98x0.95mm_HandSolder" (id 2) (at 177.038 110.49 90)
       (effects (font (size 1.27 1.27)) hide)
     )
@@
     (pin "2")
   )
-  (symbol (lib_id "GPAD_SCH_LIB:USB_B_Micro") (at 92.71 95.25 0) (unit 1)
-    (in_bom yes) (on_board yes)
-    (property "Reference" "J501" (id 0) (at 94.1578 83.3882 0))
-    (property "Value" "USB_B_Micro" (id 1) (at 94.1578 85.6996 0))
+  (symbol (lib_id "power:GND") (at 90.17 113.03 0) (unit 1)
+    (in_bom yes) (on_board yes)
+    (property "Reference" "#PWR0501" (id 0) (at 90.17 119.38 0)
+      (effects (font (size 1.27 1.27)) hide)
+    )
+    (property "Value" "GND" (id 1) (at 90.297 117.4242 0))
+    (property "Footprint" "" (id 2) (at 90.17 113.03 0)
+      (effects (font (size 1.27 1.27)) hide)
+    )
+    (property "Datasheet" "" (id 3) (at 90.17 113.03 0)
+      (effects (font (size 1.27 1.27)) hide)
+    )
+    (pin "1")
+  )
+  (symbol (lib_id "power:GND") (at 93.98 113.03 0) (unit 1)
+    (in_bom yes) (on_board yes)
+    (property "Reference" "#PWR0502" (id 0) (at 93.98 119.38 0)
+      (effects (font (size 1.27 1.27)) hide)
+    )
+    (property "Value" "GND" (id 1) (at 94.107 117.4242 0))
+    (property "Footprint" "" (id 2) (at 93.98 113.03 0)
+      (effects (font (size 1.27 1.27)) hide)
+    )
+    (property "Datasheet" "" (id 3) (at 93.98 113.03 0)
+      (effects (font (size 1.27 1.27)) hide)
+    )
+    (pin "1")
+  )
+  (symbol (lib_id "GPAD_SCH_LIB:USB_B_Micro_Local") (at 92.71 95.25 0) (unit 1)
+    (in_bom yes) (on_board yes) (fields_autoplaced)
+    (property "Reference" "J501" (id 0) (at 92.71 82.55 0))
+    (property "Value" "USB_B_Micro_Local" (id 1) (at 92.71 85.09 0))
     (property "Footprint" "GeneralPurposeAlarmDevicePCB:USB_Micro-B_Amphenol_10118194_Horizontal" (id 2) (at 96.52 96.52 0)
       (effects (font (size 1.27 1.27)) hide)
@@
       (effects (font (size 1.27 1.27)) hide)
     )
-    (property "Manufacturer " "Amphenol ICC" (id 8) (at 92.71 95.25 0)
-      (effects (font (size 1.27 1.27)) hide)
-    )
-    (property "MPN " "10118194-0001LF" (id 9) (at 92.71 95.25 0)
+    (property "AssemblyType" "HAND" (id 8) (at 92.71 95.25 0)
       (effects (font (size 1.27 1.27)) hide)
     )
@@
     (pin "6")
   )
-  (symbol (lib_id "power:GND") (at 90.17 113.03 0) (unit 1)
-    (in_bom yes) (on_board yes)
-    (property "Reference" "#PWR0501" (id 0) (at 90.17 119.38 0)
-      (effects (font (size 1.27 1.27)) hide)
-    )
-    (property "Value" "GND" (id 1) (at 90.297 117.4242 0))
-    (property "Footprint" "" (id 2) (at 90.17 113.03 0)
-      (effects (font (size 1.27 1.27)) hide)
-    )
-    (property "Datasheet" "" (id 3) (at 90.17 113.03 0)
-      (effects (font (size 1.27 1.27)) hide)
-    )
-    (pin "1")
-  )
-  (symbol (lib_id "power:GND") (at 93.98 113.03 0) (unit 1)
-    (in_bom yes) (on_board yes)
-    (property "Reference" "#PWR0502" (id 0) (at 93.98 119.38 0)
-      (effects (font (size 1.27 1.27)) hide)
-    )
-    (property "Value" "GND" (id 1) (at 94.107 117.4242 0))
-    (property "Footprint" "" (id 2) (at 93.98 113.03 0)
-      (effects (font (size 1.27 1.27)) hide)
-    )
-    (property "Datasheet" "" (id 3) (at 93.98 113.03 0)
-      (effects (font (size 1.27 1.27)) hide)
-    )
-    (pin "1")
-  )
   (symbol (lib_id "Connector:TestPoint") (at 114.3 72.39 0) (unit 1)
     (in_bom yes) (on_board yes)
@@
       (effects (font (size 1.27 1.27)) hide)
     )
+    (property "AssemblyType" "HAND" (id 4) (at 114.3 72.39 0)
+      (effects (font (size 1.27 1.27)) hide)
+    )
     (pin "1")
   )
@@
       (effects (font (size 1.27 1.27)) hide)
     )
+    (property "AssemblyType" "HAND" (id 4) (at 137.16 71.12 0)
+      (effects (font (size 1.27 1.27)) hide)
+    )
     (pin "1")
   )
@@
       (effects (font (size 1.27 1.27)) hide)
     )
+    (property "AssemblyType" "HAND" (id 4) (at 193.04 105.41 0)
+      (effects (font (size 1.27 1.27)) hide)
+    )
