File: Hardware/GeneralPurposeAlarmDevicePCB/GeneralPurposeAlarmDevicePCB/USB_UART.kicad_sch (KiCad schematic)
At the start: 13 parts, among them J501 USB_B_Micro_Local, U501 CH340E

Commit message: Update a lot of cost and PNs from JLCPCB and some Digikey.
Parts:
- C501, C503: AssemblyType (none) -> SMT; Cost (none) -> 0.0021
- C502: AssemblyType (none) -> SMT; Cost (none) -> 0.038
- D501: AssemblyType (none) -> SMT; Cost (none) -> 0.0054
- J501: Cost (none) -> 0.2042
- R501, R502, R503, R504: AssemblyType (none) -> SMT; Cost (none) -> 0.0015
- U501: AssemblyType (none) -> SMT; Cost (none) -> 0.3845
Changed lines of the file:
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@@
+      (effects (font (size 1.27 1.27)) hide)
+    )
+    (property "AssemblyType" "SMT" (id 10) (at 154.94 97.79 0)
+      (effects (font (size 1.27 1.27)) hide)
+    )
+    (property "Cost" "0.3845" (id 11) (at 154.94 97.79 0)
       (effects (font (size 1.27 1.27)) hide)
     )
@@
       (effects (font (size 1.27 1.27)) hide)
     )
+    (property "AssemblyType" "SMT" (id 9) (at 172.72 87.63 0)
+      (effects (font (size 1.27 1.27)) hide)
+    )
+    (property "Cost" "0.0015" (id 10) (at 172.72 87.63 0)
+      (effects (font (size 1.27 1.27)) hide)
+    )
     (pin "1")
     (pin "2")
@@
       (effects (font (size 1.27 1.27)) hide)
     )
+    (property "AssemblyType" "SMT" (id 9) (at 172.72 96.52 0)
+      (effects (font (size 1.27 1.27)) hide)
+    )
+    (property "Cost" "0.0015" (id 10) (at 172.72 96.52 0)
+      (effects (font (size 1.27 1.27)) hide)
+    )
     (pin "1")
     (pin "2")
@@
       (effects (font (size 1.27 1.27)) hide)
     )
+    (property "AssemblyType" "SMT" (id 9) (at 137.16 82.55 0)
+      (effects (font (size 1.27 1.27)) hide)
+    )
+    (property "Cost" "0.0021" (id 10) (at 137.16 82.55 0)
+      (effects (font (size 1.27 1.27)) hide)
+    )
     (pin "1")
     (pin "2")
@@
       (effects (font (size 1.27 1.27)) hide)
     )
+    (property "AssemblyType" "SMT" (id 8) (at 120.65 82.55 0)
+      (effects (font (size 1.27 1.27)) hide)
+    )
+    (property "Cost" "0.038" (id 9) (at 120.65 82.55 0)
+      (effects (font (size 1.27 1.27)) hide)
+    )
     (pin "1")
     (pin "2")
@@
     )
     (property "Description" "50V 100nF X7R ±10% 0603 Multilayer Ceramic Capacitors MLCC - SMD/SMT ROHS" (id 8) (at 106.68 82.55 0)
+      (effects (font (size 1.27 1.27)) hide)
+    )
+    (property "AssemblyType" "SMT" (id 9) (at 106.68 82.55 0)
+      (effects (font (size 1.27 1.27)) hide)
+    )
+    (property "Cost" "0.0021" (id 10) (at 106.68 82.55 0)
       (effects (font (size 1.27 1.27)) hide)
     )
@@
       (effects (font (size 1.27 1.27)) hide)
     )
+    (property "AssemblyType" "SMT" (id 9) (at 133.35 107.95 0)
+      (effects (font (size 1.27 1.27)) hide)
+    )
+    (property "Cost" "0.0015" (id 10) (at 133.35 107.95 0)
+      (effects (font (size 1.27 1.27)) hide)
+    )
     (pin "1")
     (pin "2")
@@
     (property "Status" "Active" (id 11) (at 127 138.43 0)
       (effects (font (size 1.524 1.524)) (justify left) hide)
+    )
+    (property "AssemblyType" "SMT" (id 12) (at 121.92 107.95 0)
+      (effects (font (size 1.27 1.27)) hide)
+    )
+    (property "Cost" "0.0054" (id 13) (at 121.92 107.95 0)
+      (effects (font (size 1.27 1.27)) hide)
     )
     (pin "1")
@@
     )
     (property "Description" "1W ±1% 4.7kΩ 0603 Chip Resistor - Surface Mount ROHS" (id 8) (at 175.26 110.49 0)
+      (effects (font (size 1.27 1.27)) hide)
+    )
+    (property "AssemblyType" "SMT" (id 9) (at 175.26 110.49 0)
+      (effects (font (size 1.27 1.27)) hide)
+    )
+    (property "Cost" "0.0015" (id 10) (at 175.26 110.49 0)
       (effects (font (size 1.27 1.27)) hide)
     )
@@
       (effects (font (size 1.27 1.27)) hide)
     )
+    (property "Cost" "0.2042" (id 9) (at 92.71 95.25 0)
+      (effects (font (size 1.27 1.27)) hide)
+    )
+    (property "Description" "USB 2.0 1 5 Female Micro-B SMD USB Connectors ROHS" (id 10) (at 92.71 95.25 0)
+      (effects (font (size 1.27 1.27)) hide)
+    )

Commit message: Route some power. Move transistors and resistors near LEDs for signall access.
Other:
- note added: "Place R503 near uControler TX pin."
Changed lines of the file:
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@@
+    (effects (font (size 1.27 1.27)) (justify left bottom))
+  )
+  (text "Place R503 near uControler TX pin." (at 177.8 93.98 0)
     (effects (font (size 1.27 1.27)) (justify left bottom))
   )
