File: Hardware/PolyVent_SPI_Controller/PolyVent_SPI_Controller.kicad_pcb (KiCad board)
At the start: 2 copper layers, 100 x 80 mm, 65 parts, among them J1 09231486921, J102 RJ12_6P6C_HORZ, J103 0.100_2Pin, J201 S04B-XASK-1(LF)(SN), Q101 BSS138, Q102 BSS138, Q103 BSS138, Q104 BSS138, Q201 BSS138, Q202 BSS138

Commit message: Update with Poly Fuse, Chip Select DIPs. Power LEDs.
Parts:
- removed R120: DNI, Resistor_SMD:R_0603_1608Metric_Pad0.98x0.95mm_HandSolder
- removed R121, R122, R123: 1R, Resistor_SMD:R_0603_1608Metric_Pad0.98x0.95mm_HandSolder
- added D101: RED 0603, LED_SMD:LED_0603_1608Metric_Pad1.05x0.95mm_HandSolder, F.Cu at (181.6, 78.1)
- added D102: RED 0603, LED_SMD:LED_0603_1608Metric_Pad1.05x0.95mm_HandSolder, F.Cu at (181.6, 74.9)
- added D103: RED 0603, LED_SMD:LED_0603_1608Metric_Pad1.05x0.95mm_HandSolder, F.Cu at (181.6, 71.8)
- added F101: Polyfuse_Small, Fuse:Fuse_0603_1608Metric, F.Cu at (114.3, 106.2)
- added F102: Polyfuse_Small, Fuse:Fuse_0603_1608Metric, F.Cu at (113.0, 108.6)
- added F103: Polyfuse_Small, Fuse:Fuse_0603_1608Metric, F.Cu at (113.8, 114.3)
- added J202: 0.100_2Pin, Connector_PinHeader_2.54mm:PinHeader_1x02_P2.54mm_Vertical, F.Cu at (181.0, 104.8)
- added R207: DNI, Resistor_SMD:R_0603_1608Metric_Pad0.98x0.95mm_HandSolder, F.Cu at (174.0, 104.1)
- added R208: DNI, Resistor_SMD:R_0603_1608Metric_Pad0.98x0.95mm_HandSolder, F.Cu at (174.0, 101.0)
- added SW101: SW_DIP_x08, PubInv_PCB:SMDIP-16_L11.39_W6.7mm, F.Cu at (127.8, 89.9)
- added SW102: SW_DIP_x08, PubInv_PCB:SMDIP-16_L11.39_W6.7mm, F.Cu at (127.8, 75.9)
- added TP203: SDA_5V, TestPoint:TestPoint_Loop_D2.54mm_Drill1.5mm_Beaded, F.Cu at (194.9, 123.2)
- R111: value 2K -> 1K
- R114: value 10K -> 1K
- R116: value 1R -> 10K
- R117, R118, R119: value DNI -> 1K
- TP108: value +12V -> TP_GND
- TP109: value TP_GND -> +12V
- TP202: value SDA_5V -> I2C_VCC
- moved TP108 82.6 mm to (194.3, 80.6)
- moved TP109 82.2 mm to (122.6, 122.6)
- moved R118 66.3 mm to (177.4, 74.9)
- moved R117 66.3 mm to (177.2, 78.1)
- moved R119 66.1 mm to (177.2, 71.8)
- moved Graphic1 51.7 mm to (170.4, 71.9)
- moved R116 35.4 mm to (142.9, 109.2), turned to 0 degrees
- moved TP202 20.9 mm to (188.0, 103.5)
- moved R115 9.61 mm to (141.6, 95.2)
- moved R114 7.65 mm to (144.1, 86.4), turned to 0 degrees
- moved TP101 3.49 mm to (180.0, 84.8)
- moved C105 2.02 mm to (119.9, 105.7)
- moved R205 1.02 mm to (182.6, 111.8)
- turned R111 to 0 degrees
Connections:
- J201 pad 1: +5V -> /I2C_Level_Shifter/I2C_VCC
- R111 pad 1: /MISO -> Net-(R111-Pad1)
- R111 pad 2: GND -> /MISO
- R114 pad 1: +3.3V -> GND
- R114 pad 2: /SCK -> Net-(R111-Pad1)
- R115 pad 2: /MOSI -> /SCK
- R116 pad 1: Net-(Q101-Pad2) -> +3.3V
- R116 pad 2: /CS_15 -> /MOSI
- R117 pad 1: Net-(Q101-Pad2) -> Net-(D101-Pad2)
- R117 pad 2: /CS_11 -> +12V
- R118 pad 1: Net-(Q101-Pad2) -> Net-(D102-Pad2)
- R118 pad 2: /CS_12 -> +5V
- R119 pad 1: Net-(Q101-Pad2) -> Net-(D103-Pad2)
- R119 pad 2: /CS_13 -> +3.3V
- TP108 pad 1: +12V -> GND
- TP109 pad 1: GND -> +12V
- TP202 pad 1: /I2C_Level_Shifter/SDA_5V -> /I2C_Level_Shifter/I2C_VCC
Routing:
- net +12V: track 25.5 -> 181.6 mm
- net +3.3V: track 166.5 -> 211.6 mm
- net /CS_9: track 0.00 -> 36.9 mm, vias 0 -> 1
- net /CS_10: track 0.00 -> 36.7 mm, vias 0 -> 1
- net /CS_1: track 0.00 -> 32.9 mm, vias 0 -> 3
- net /CS_8: track 0.00 -> 32.2 mm, vias 0 -> 3
- net /CS_2: track 0.00 -> 28.8 mm, vias 0 -> 3
- net /CS_3: track 0.00 -> 27.9 mm, vias 0 -> 3
- net /CS_12: track 8.30 -> 35.2 mm
- net /CS_13: track 7.37 -> 34.1 mm
- net /CS_15: track 8.64 -> 34.6 mm, vias 1 -> 3
- net /CS_11: track 9.61 -> 35.4 mm
- net /CS_6: track 0.00 -> 25.7 mm, vias 0 -> 3
- net /CS_5: track 0.00 -> 25.4 mm, vias 0 -> 3
- net /I2C_Level_Shifter/I2C_VCC: track 0.00 -> 25.1 mm
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Other:
- board text added: "+12V"
- board text added: "+3.3V"
- board text added: "+5V"
- board text added: "CS_1"
- board text added: "CS_10"
- board text added: "CS_11"
- board text added: "CS_12"
- board text added: "CS_13"
- board text added: "CS_14"
- board text added: "CS_15"
- board text added: "CS_2"
- board text added: "CS_3"
- board text added: "CS_4"
- board text added: "CS_5"
- board text added: "CS_6"
- board text added: "CS_7"
- board text added: "CS_8"
- board text added: "CS_9"

Commit message: Update PCB for fewer appatures on ground.
Parts:
- moved Graphic1 1.55 mm to (170.2, 70.4)
Routing:
- net Net-(Q101-Pad2): track 92.3 -> 93.4 mm
- net /SDA: track 96.2 -> 95.2 mm
- net /SCK: track 46.1 -> 46.7 mm
- net GND: vias 60 -> 62
Other:
- board text added: "20221124"

Commit message: Add buck regulator for ControllerVCC.
Parts:
- added R120: 1R0, Resistor_SMD:R_0603_1608Metric_Pad0.98x0.95mm_HandSolder, F.Cu at (187.5, 126.7)
- added U101: DC_DC_small, DC_DC_LM2596_small:DC_DC_LM2596_small, F.Cu at (158.2, 132.8)
- moved Q101 4.35 mm to (147.7, 117.6)
- moved R107 4.35 mm to (147.8, 121.4)
- moved R112 4.35 mm to (144.0, 117.6)
- moved R106 4.35 mm to (152.9, 121.4)
- moved TP105 4.35 mm to (152.9, 117.0)
Routing:
- net /SDA: track 95.2 -> 85.5 mm
- net +12V: track 181.6 -> 191.1 mm
- net +3.3V: track 211.6 -> 204.4 mm
- net Net-(R120-Pad2): track 0.00 -> 6.56 mm, vias 0 -> 1
- net +5V: track 183.9 -> 179.0 mm
- net /nCS: track 70.7 -> 66.2 mm
- net Net-(Q101-Pad2): track 93.4 -> 91.9 mm
- net /ControllerVcc: track 143.7 -> 144.6 mm
- net GND: vias 62 -> 66
