File: Hardware/PolyVent_SPI_Controller/PolyVent_SPI_Controller.kicad_pcb (KiCad board)
At the start: 2 copper layers, 100 x 80 mm, 75 parts, among them J1 09231486921, J102 RJ12_6P6C_HORZ, J103 0.100_2Pin, J201 S04B-XASK-1(LF)(SN), J202 0.100_2Pin, Q101 BSS138, Q102 BSS138, Q103 BSS138, Q104 BSS138, Q201 BSS138, Q202 BSS138, SW101 SW_DIP_x08, SW102 SW_DIP_x08, U101 DC_DC_small

Commit message: Change Buck Regulator for 1700x830 footprint. Update PDFs.
Parts:
- U101: footprint DC_DC_LM2596_small:DC_DC_LM2596_small -> PubInv_PCB:DC_DC_LM2596_small1700x830
- moved U101 14.1 mm to (144.5, 129.8)
- moved TP109 9.55 mm to (113.0, 123.2)
- moved R106 3.54 mm to (151.6, 118.1)
- moved R107 3.31 mm to (147.7, 118.1)
- moved Q101 2.54 mm to (147.7, 115.1)
- moved R112 2.54 mm to (144.0, 115.1)
- moved TP105 1.78 mm to (152.9, 115.2)
Routing:
- net Net-(R120-Pad2): track 6.56 -> 26.8 mm, vias 1 -> 3
- net +12V: track 191.1 -> 181.4 mm
- net +3.3V: track 204.4 -> 206.6 mm
- net +5V: track 179.0 -> 177.5 mm
- net /ControllerVcc: track 144.6 -> 143.2 mm
- net /nCS: track 66.2 -> 65.6 mm
- net Net-(Q101-Pad2): track 91.9 -> 92.4 mm
- net GND: vias 66 -> 76
