File: Hardware/PolyVent_SPI_Controller/PolyVent_SPI_Controller.kicad_pcb (KiCad board)
At the start: 2 copper layers, 100 x 80 mm, 75 parts, among them J1 09231486921, J102 RJ12_6P6C_HORZ, J103 0.100_2Pin, J201 S04B-XASK-1(LF)(SN), J202 0.100_2Pin, Q101 BSS138, Q102 BSS138, Q103 BSS138, Q104 BSS138, Q201 BSS138, Q202 BSS138, SW101 SW_DIP_x08, SW102 SW_DIP_x08, U101 DC_DC_small

Commit message: Increase size on power traces and vias. Move and edit model number text.
Connections:
- J1 pad 43: /SDA -> Net-(R120-Pad2)
- Q202 pad 2: /SDA -> Net-(R120-Pad2)
- R202 pad 2: /SDA -> Net-(R120-Pad2)
Routing:
- net Net-(R120-Pad2): track 26.8 -> 112.7 mm, vias 3 -> 8
- net /SDA: track 85.9 -> 0.00 mm, vias 5 -> 0
- net /ControllerVcc: track 143.2 -> 146.1 mm
- net +12V: track 181.4 -> 182.3 mm
- net /nCS: track 65.6 -> 64.9 mm
Other:
- board text added: "By: Public Invention"
- board text added: "Model: PolyVent_SPI_Controller"
- board text added: "Revision: 0.1 20221124"
- board text removed: "20221124"
- board text removed: "PolyVent_SPI_Controller"
- board text removed: "Public Invention"
- board text removed: "Revision 0.1"

Commit message: Update the Schematic and BOM for FET level shift. Make some parts DNI.
Parts:
- J1: value 09231486921 -> Plug 48 Way
- R103, R104, R105, R107, R111, R114: value 1K -> DNI
- R106, R109, R110, R113: value 10K -> 1K
Connections:
- J1 pad 43: Net-(R120-Pad2) -> /SDA
- Q202 pad 2: Net-(R120-Pad2) -> /SDA
- R202 pad 2: Net-(R120-Pad2) -> /SDA
Routing:
- net /SDA: track 0.00 -> 85.9 mm, vias 0 -> 5
- net Net-(R120-Pad2): track 112.7 -> 27.0 mm, vias 8 -> 3
