File: Hardware/PolyVent_SPI_Controller/I2C_Level_Shifter.kicad_sch (KiCad schematic)
At the start: 13 parts, among them J201 S04B-XASK-1(LF)(SN), Q201 BSS138, Q202 BSS138

Commit message: Update to KiCad files for PolyVent BOM update.
Parts:
- C201, C202, Q201, Q202, R201, R202, R203, R204, R205, R206: LongLead (none) -> NO
- TP201, TP202: Cost (none) -> NA; LongLead (none) -> NO
Changed lines of the file:
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@@
+      (effects (font (size 1.27 1.27)) hide)
+    )
+    (property "LongLead" "NO" (id 11) (at 190.5 86.36 0)
       (effects (font (size 1.27 1.27)) hide)
     )
@@
     )
     (property "Cost" "0.0015" (id 7) (at 147.32 106.68 0)
+      (effects (font (size 1.27 1.27)) hide)
+    )
+    (property "LongLead" "NO" (id 8) (at 147.32 106.68 0)
       (effects (font (size 1.27 1.27)) hide)
     )
@@
       (effects (font (size 1.27 1.27)) hide)
     )
+    (property "LongLead" "NO" (id 11) (at 190.5 91.44 0)
+      (effects (font (size 1.27 1.27)) hide)
+    )
     (pin "1")
     (pin "2")
@@
       (effects (font (size 1.27 1.27)) hide)
     )
+    (property "Cost" "NA" (id 7) (at 204.47 97.79 0)
+      (effects (font (size 1.27 1.27)) hide)
+    )
+    (property "LongLead" "NO" (id 8) (at 204.47 97.79 0)
+      (effects (font (size 1.27 1.27)) hide)
+    )
     (pin "1")
   )
@@
       (effects (font (size 1.27 1.27)) hide)
     )
+    (property "LongLead" "NO" (id 8) (at 135.89 64.77 0)
+      (effects (font (size 1.27 1.27)) hide)
+    )
     (pin "1")
     (pin "2")
@@
       (effects (font (size 1.27 1.27)) hide)
     )
+    (property "LongLead" "NO" (id 8) (at 124.46 71.12 0)
+      (effects (font (size 1.27 1.27)) hide)
+    )
     (pin "1")
     (pin "2")
@@
     )
     (property "Cost" "0.0015" (id 7) (at 147.32 53.34 0)
+      (effects (font (size 1.27 1.27)) hide)
+    )
+    (property "LongLead" "NO" (id 8) (at 147.32 53.34 0)
       (effects (font (size 1.27 1.27)) hide)
     )
@@
       (effects (font (size 1.27 1.27)) hide)
     )
+    (property "LongLead" "NO" (id 10) (at 234.95 99.06 0)
+      (effects (font (size 1.27 1.27)) hide)
+    )
     (pin "1")
     (pin "2")
@@
       (effects (font (size 1.27 1.27)) hide)
     )
+    (property "LongLead" "NO" (id 10) (at 223.52 99.06 0)
+      (effects (font (size 1.27 1.27)) hide)
+    )
     (pin "1")
     (pin "2")
@@
     )
     (property "Distributor 1 PN" "NA" (id 6) (at 204.47 82.55 0)
+      (effects (font (size 1.27 1.27)) hide)
+    )
+    (property "Cost" "NA" (id 7) (at 204.47 82.55 0)
+      (effects (font (size 1.27 1.27)) hide)
+    )
+    (property "LongLead" "NO" (id 8) (at 204.47 82.55 0)
       (effects (font (size 1.27 1.27)) hide)
     )
@@
       (effects (font (size 1.27 1.27)) hide)
     )
+    (property "LongLead" "NO" (id 8) (at 135.89 118.11 0)
+      (effects (font (size 1.27 1.27)) hide)
+    )
     (pin "1")
     (pin "2")
@@
       (effects (font (size 1.27 1.27)) hide)
     )
+    (property "LongLead" "NO" (id 8) (at 124.46 124.46 0)
+      (effects (font (size 1.27 1.27)) hide)
+    )

Commit message: Update with Poly Fuse, Chip Select DIPs. Power LEDs.
Parts:
- added J202: 0.100_2Pin, Connector_PinHeader_2.54mm:PinHeader_1x02_P2.54mm_Vertical, symbol GPAD_SCH_LIB:22-23-2021
- added R207, R208: DNI, Resistor_SMD:R_0603_1608Metric_Pad0.98x0.95mm_HandSolder, symbol Device:R
- added TP202: I2C_VCC, TestPoint:TestPoint_Loop_D2.54mm_Drill1.5mm_Beaded, symbol Connector:TestPoint
- renumbered TP202 to TP203
Connections:
- net +5V: now also R207.2; no longer J201.1
- new net +12V: J202.2, R208.2
- new net I2C_VCC: J201.1, J202.1, R207.1, R208.1, TP202.1
Other:
- note added: "Power to I2C interface, 5V or 12V."

Commit message: Update the Schematic and BOM for FET level shift. Make some parts DNI.
Parts:
- J201: Manufacturer JST -> JST Sales America
- Q201, Q202: MPN (none) -> BSS138; Manufacturer (none) -> Yangzhou Yangjie Elec Tech
- R201, R202, R203, R204: MPN (none) -> RMC 0603 10K F N; Manufacturer (none) -> TyoHM
- TP201, TP202, TP203: AssemblyType HAND -> DNI
Changed lines of the file:
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@@
+      (effects (font (size 1.27 1.27)) hide)
+    )
+    (property "Description" "100mW ±1% 10kΩ 0603 Chip Resistor - Surface Mount ROHS" (id 9) (at 147.32 106.68 0)
+      (effects (font (size 1.27 1.27)) hide)
+    )
+    (property "MPN" "RMC 0603 10K F N" (id 10) (at 147.32 106.68 0)
+      (effects (font (size 1.27 1.27)) hide)
+    )
+    (property "Manufacturer" "TyoHM" (id 11) (at 147.32 106.68 0)
       (effects (font (size 1.27 1.27)) hide)
     )
@@
       (effects (font (size 1.27 1.27)) hide)
     )
-    (property "AssemblyType" "HAND" (id 4) (at 204.47 97.79 0)
+    (property "AssemblyType" "DNI" (id 4) (at 204.47 97.79 0)
       (effects (font (size 1.27 1.27)) hide)
     )
@@
       (effects (font (size 1.27 1.27)) hide)
     )
+    (property "Description" "50V 220mA 3.5Ω@10V,220mA 360mW 1.5V@1mA N Channel SOT-23 MOSFETs ROHS" (id 9) (at 135.89 64.77 0)
+      (effects (font (size 1.27 1.27)) hide)
+    )
+    (property "MPN" "BSS138" (id 10) (at 135.89 64.77 0)
+      (effects (font (size 1.27 1.27)) hide)
+    )
+    (property "Manufacturer" "Yangzhou Yangjie Elec Tech" (id 11) (at 135.89 64.77 0)
+      (effects (font (size 1.27 1.27)) hide)
+    )
     (pin "1")
     (pin "2")
@@
       (effects (font (size 1.27 1.27)) hide)
     )
+    (property "Description" "100mW ±1% 10kΩ 0603 Chip Resistor - Surface Mount ROHS" (id 9) (at 124.46 71.12 0)
+      (effects (font (size 1.27 1.27)) hide)
+    )
+    (property "MPN" "RMC 0603 10K F N" (id 10) (at 124.46 71.12 0)
+      (effects (font (size 1.27 1.27)) hide)
+    )
+    (property "Manufacturer" "TyoHM" (id 11) (at 124.46 71.12 0)
+      (effects (font (size 1.27 1.27)) hide)
+    )
     (pin "1")
     (pin "2")
@@
     )
     (property "LongLead" "NO" (id 8) (at 147.32 53.34 0)
+      (effects (font (size 1.27 1.27)) hide)
+    )
+    (property "Description" "100mW ±1% 10kΩ 0603 Chip Resistor - Surface Mount ROHS" (id 9) (at 147.32 53.34 0)
+      (effects (font (size 1.27 1.27)) hide)
+    )
+    (property "MPN" "RMC 0603 10K F N" (id 10) (at 147.32 53.34 0)
+      (effects (font (size 1.27 1.27)) hide)
+    )
+    (property "Manufacturer" "TyoHM" (id 11) (at 147.32 53.34 0)
       (effects (font (size 1.27 1.27)) hide)
     )
@@
       (effects (font (size 1.27 1.27)) hide)
     )
-    (property "Datasheet" "~" (id 3) (at 234.95 99.06 0)
+    (property "Datasheet" "https://datasheet.lcsc.com/lcsc/1811082118_YAGEO-CC0603JRNPO9BN390_C107049.pdf" (id 3) (at 234.95 99.06 0)
       (effects (font (size 1.27 1.27)) hide)
     )
@@
       (effects (font (size 1.27 1.27)) hide)
     )
+    (property "Description" "50V 39pF NP0 ±5% 0603 Multilayer Ceramic Ca" (id 11) (at 234.95 99.06 0)
+      (effects (font (size 1.27 1.27)) hide)
+    )
     (pin "1")
     (pin "2")
@@
       (effects (font (size 1.27 1.27)) hide)
     )
-    (property "Datasheet" "~" (id 3) (at 223.52 99.06 0)
+    (property "Datasheet" "https://datasheet.lcsc.com/lcsc/1811082118_YAGEO-CC0603JRNPO9BN390_C107049.pdf" (id 3) (at 223.52 99.06 0)
       (effects (font (size 1.27 1.27)) hide)
     )
@@
       (effects (font (size 1.27 1.27)) hide)
     )
+    (property "Description" "50V 39pF NP0 ±5% 0603 Multilayer Ceramic Ca" (id 11) (at 223.52 99.06 0)
+      (effects (font (size 1.27 1.27)) hide)
+    )
     (pin "1")
     (pin "2")
@@
       (effects (font (size 1.27 1.27)) hide)
     )
-    (property "AssemblyType" "HAND" (id 4) (at 191.77 25.4 0)
+    (property "AssemblyType" "DNI" (id 4) (at 191.77 25.4 0)
       (effects (font (size 1.27 1.27)) hide)
     )
@@
       (effects (font (size 1.27 1.27)) hide)
     )
-    (property "AssemblyType" "HAND" (id 4) (at 204.47 82.55 0)
+    (property "AssemblyType" "DNI" (id 4) (at 204.47 82.55 0)
       (effects (font (size 1.27 1.27)) hide)
     )
@@
       (effects (font (size 1.27 1.27)) hide)
     )
+    (property "Description" "50V 220mA 3.5Ω@10V,220mA 360mW 1.5V@1mA N Channel SOT-23 MOSFETs ROHS" (id 9) (at 135.89 118.11 0)
+      (effects (font (size 1.27 1.27)) hide)
+    )
+    (property "MPN" "BSS138" (id 10) (at 135.89 118.11 0)
+      (effects (font (size 1.27 1.27)) hide)
+    )
+    (property "Manufacturer" "Yangzhou Yangjie Elec Tech" (id 11) (at 135.89 118.11 0)
+      (effects (font (size 1.27 1.27)) hide)
+    )
     (pin "1")
     (pin "2")
@@
       (effects (font (size 1.524 1.524)) (justify left) hide)
     )
-    (property "Manufacturer" "JST" (id 9) (at 215.9 88.9 0)
+    (property "Manufacturer" "JST Sales America" (id 9) (at 215.9 88.9 0)
       (effects (font (size 1.524 1.524)) (justify left) hide)
     )
@@
       (effects (font (size 1.27 1.27)) hide)
     )
+    (property "Description" "Do Not Insert" (id 9) (at 212.09 33.02 0)
+      (effects (font (size 1.27 1.27)) hide)
+    )
     (pin "1")
     (pin "2")
@@
       (effects (font (size 1.27 1.27)) hide)
     )
+    (property "Description" "Do Not Insert" (id 9) (at 212.09 25.4 0)
+      (effects (font (size 1.27 1.27)) hide)
+    )
     (pin "1")
     (pin "2")
@@
       (effects (font (size 1.27 1.27)) hide)
     )
+    (property "Description" "100mW ±1% 10kΩ 0603 Chip Resistor - Surface Mount ROHS" (id 9) (at 124.46 124.46 0)
+      (effects (font (size 1.27 1.27)) hide)
+    )
+    (property "MPN" "RMC 0603 10K F N" (id 10) (at 124.46 124.46 0)
+      (effects (font (size 1.27 1.27)) hide)
+    )
+    (property "Manufacturer" "TyoHM" (id 11) (at 124.46 124.46 0)
+      (effects (font (size 1.27 1.27)) hide)
+    )
