File: Hardware/PolyVent_SPI_Controller/PolyVent_SPI_Controller.kicad_sch (KiCad schematic)
At the start: 47 parts, among them J1 09231486921, J102 RJ12_6P6C_HORZ, J103 0.100_2Pin, Q101 BSS138, Q102 BSS138, Q103 BSS138, Q104 BSS138

Commit message: Update to KiCad files for PolyVent BOM update.
Parts:
- C101, C102, C103, C104, C105, C106, C107, Q101, Q102, Q103, Q104, R101, R102, R103, R104, R105, R106, R107, R108, R109, R110, R111, R112, R113, R114, R115, R116, R117, R118, R119, R120, R121, R122, R123: LongLead (none) -> NO
- TP101, TP102, TP103, TP104, TP105, TP106, TP107, TP108, TP109: Cost (none) -> NA; LongLead (none) -> NO

Commit message: Update with Poly Fuse, Chip Select DIPs. Power LEDs.
Parts:
- removed R116, R121, R122, R123: 1R, Resistor_SMD:R_0603_1608Metric_Pad0.98x0.95mm_HandSolder, symbol Device:R
- removed R120: DNI, Resistor_SMD:R_0603_1608Metric_Pad0.98x0.95mm_HandSolder, symbol Device:R
- added D101, D102, D103: RED 0603, LED_SMD:LED_0603_1608Metric_Pad1.05x0.95mm_HandSolder, symbol Device:LED
- added F101, F102, F103: Polyfuse_Small, Fuse:Fuse_0603_1608Metric, symbol Device:Polyfuse_Small
- added R114: 1K, Resistor_SMD:R_0603_1608Metric_Pad0.98x0.95mm_HandSolder, symbol Device:R
- added SW101, SW102: SW_DIP_x08, PubInv_PCB:SMDIP-16_L11.39_W6.7mm, symbol Switch:SW_DIP_x08
- R111: value 2K -> 1K; Distributor 1 PN C269690 -> C269704
- R117, R118, R119: value DNI -> 1K; Distributor 1 NA -> JLCPCB; Distributor 1 PN NA -> C269704
- renumbered MF1 to MF101, R114 to R115, R115 to R116, TP109 to TP108, TP108 to TP109
Connections:
- net +12V: now also R117.2, F103.2
- net +3.3V: now also R119.2, F101.2
- net +5V: now also R118.2, F102.2
- net 24V/12V: now also F103.1
- net 3.3V: now also F101.1
- net 5V: now also F102.1
- net CS_1: now also SW101.15
- net CS_10: now also SW102.15
- net CS_11: now also SW102.14; no longer R117.2
- net CS_12: now also SW102.13; no longer R118.2
- net CS_13: now also SW102.12; no longer R119.2
- net CS_14: now also SW102.11
- net CS_15: now also SW102.10
- net CS_2: now also SW101.14
- net CS_3: now also SW101.13
- net CS_4: now also SW101.12
- net CS_5: now also SW101.11
- net CS_6: now also SW101.10
- net CS_7: now also SW101.9
- net CS_8: now also SW101.16
- net CS_9: now also SW102.16
- net GND: now also D101.1 (K), D102.1 (K), D103.1 (K), R114.1; no longer R111.2
- net MISO: now also R111.2; no longer R111.1
- net at Q101.2 (S), R107.2, R112.2: now also SW101.1, SW101.2, SW101.3, SW101.4, SW101.5, SW101.6, SW101.7, SW101.8, SW102.1, SW102.2, SW102.3, SW102.4, SW102.5, SW102.6, SW102.7, SW102.8; no longer R117.1, R118.1, R119.1
- new net: R111.1, R114.2
- new net: D101.2 (A), R117.1
- new net: D102.2 (A), R118.1
- new net: D103.2 (A), R119.1
- no-connect marks 0 -> 1
Other:
- moved on the sheet: C105, C106, TP106, TP107

Commit message: Add buck regulator for ControllerVCC.
Parts:
- added R120: 1R0, Resistor_SMD:R_0603_1608Metric_Pad0.98x0.95mm_HandSolder, symbol Device:R
- added U101: DC_DC_small, DC_DC_LM2596_small:DC_DC_LM2596_small, symbol Custom_dc_dc_small:DC_DC_small
Connections:
- net +12V: now also U101.1 (+IN)
- net ControllerVcc: now also R120.1
- net GND: now also U101.2 (-IN), U101.4 (-OUT)
- new net: R120.2, U101.3 (+OUT)
Other:
- note added: "Adjust U101 for about 9 to 12V at ControllerVcc"
- moved on the sheet: J103, R102

Commit message: Change Buck Regulator for 1700x830 footprint. Update PDFs.
Parts:
- D101, D102, D103: DK_Datasheet_Link http://optoelectronics.liteon.com/upload/download/DS22-2000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 -> (none)
- U101: footprint DC_DC_LM2596_small:DC_DC_LM2596_small -> PubInv_PCB:DC_DC_LM2596_small1700x830; AssemblyType (none) -> HAND; Cost (none) -> 1.495; Distributor 1 (none) -> Amazon; Distributor 1 PN (none) -> https://www.amazon.com/LM2596-Converter-Module-Supply-1-23V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; LongLead (none) -> YES; MPN (none) -> LM2596 DC-DC Buck Converter Step Down Module
Changed lines of the file:
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@@
       (effects (font (size 1.27 1.27)) hide)
     )
-    (property "Datasheet" "~" (id 3) (at 246.38 119.38 0)
+    (property "Datasheet" "http://optoelectronics.liteon.com/upload/download/DS22-2000-109/LTST-C171KRKT.pdf" (id 3) (at 246.38 119.38 0)
       (effects (font (size 1.27 1.27)) hide)
     )
@@
     (property "Status" "Active" (id 11) (at 215.9 114.3 0)
       (effects (font (size 1.524 1.524)) (justify left) hide)
-    )
-    (property "DK_Datasheet_Link" "http://optoelectronics.liteon.com/upload/download/DS22-2000-109/LTST-C171KRKT.pdf" (id 12) (at 361.95 254 0)
-      (effects (font (size 1.27 1.27)) hide)
     )
     (property "DK_Detail_Page" "/product-detail/en/lite-on-inc/LTST-C171KRKT/160-1427-1-ND/386800" (id 13) (at 361.95 254 0)
@@
       (effects (font (size 1.27 1.27)) hide)
     )
-    (property "Datasheet" "~" (id 3) (at 246.38 154.94 0)
+    (property "Datasheet" "http://optoelectronics.liteon.com/upload/download/DS22-2000-109/LTST-C171KRKT.pdf" (id 3) (at 246.38 154.94 0)
       (effects (font (size 1.27 1.27)) hide)
     )
@@
     (property "Status" "Active" (id 11) (at 215.9 149.86 0)
       (effects (font (size 1.524 1.524)) (justify left) hide)
-    )
-    (property "DK_Datasheet_Link" "http://optoelectronics.liteon.com/upload/download/DS22-2000-109/LTST-C171KRKT.pdf" (id 12) (at 361.95 289.56 0)
-      (effects (font (size 1.27 1.27)) hide)
     )
     (property "DK_Detail_Page" "/product-detail/en/lite-on-inc/LTST-C171KRKT/160-1427-1-ND/386800" (id 13) (at 361.95 289.56 0)
@@
       (effects (font (size 1.27 1.27)) hide)
     )
-    (property "Datasheet" "~" (id 3) (at 246.38 86.36 0)
+    (property "Datasheet" "http://optoelectronics.liteon.com/upload/download/DS22-2000-109/LTST-C171KRKT.pdf" (id 3) (at 246.38 86.36 0)
       (effects (font (size 1.27 1.27)) hide)
     )
@@
     (property "Status" "Active" (id 11) (at 215.9 81.28 0)
       (effects (font (size 1.524 1.524)) (justify left) hide)
-    )
-    (property "DK_Datasheet_Link" "http://optoelectronics.liteon.com/upload/download/DS22-2000-109/LTST-C171KRKT.pdf" (id 12) (at 361.95 220.98 0)
-      (effects (font (size 1.27 1.27)) hide)
     )
     (property "DK_Detail_Page" "/product-detail/en/lite-on-inc/LTST-C171KRKT/160-1427-1-ND/386800" (id 13) (at 361.95 220.98 0)
@@
       (effects (font (size 0.9906 0.9906)))
     )
-    (property "Footprint" "DC_DC_LM2596_small:DC_DC_LM2596_small" (id 2) (at 46.99 73.66 0)
+    (property "Footprint" "PubInv_PCB:DC_DC_LM2596_small1700x830" (id 2) (at 46.99 73.66 0)
       (effects (font (size 1.524 1.524)) hide)
     )
-    (property "Datasheet" "" (id 3) (at 46.99 59.69 0)
+    (property "Datasheet" "https://www.amazon.com/LM2596-Converter-Module-Supply-1-23V-30V/dp/B008BHBEE0" (id 3) (at 46.99 59.69 0)
       (effects (font (size 1.524 1.524)) hide)
+    )
+    (property "AssemblyType" "HAND" (id 4) (at 46.99 67.31 0)
+      (effects (font (size 1.27 1.27)) hide)
+    )
+    (property "Cost" "1.495" (id 5) (at 46.99 67.31 0)
+      (effects (font (size 1.27 1.27)) hide)
+    )
+    (property "Distributor 1" "Amazon" (id 6) (at 46.99 67.31 0)
+      (effects (font (size 1.27 1.27)) hide)
+    )
+    (property "Distributor 1 PN" "https://www.amazon.com/LM2596-Converter-Module-Supply-1-23V-30V/dp/B008BHBEE0" (id 7) (at 46.99 67.31 0)
+      (effects (font (size 1.27 1.27)) hide)
+    )
+    (property "LongLead" "YES" (id 8) (at 46.99 67.31 0)
+      (effects (font (size 1.27 1.27)) hide)
+    )
+    (property "MPN" "LM2596 DC-DC Buck Converter Step Down Module" (id 9) (at 46.99 67.31 0)
+      (effects (font (size 1.27 1.27)) hide)
     )
     (pin "1")
@@
     )
     (path "/f9c50344-e85e-43bb-87e6-abc050a44195"
-      (reference "U101") (unit 1) (value "DC_DC_small") (footprint "DC_DC_LM2596_small:DC_DC_LM2596_small")
-    )
-  )
+      (reference "U101") (unit 1) (value "DC_DC_small") (footprint "PubInv_PCB:DC_DC_LM2596_small1700x830")
+    )
+  )

Commit message: Increase size on power traces and vias. Move and edit model number text.
Changed lines of the file:
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@@
   (junction (at 152.4 50.8) (diameter 0) (color 0 0 0 0)
   )
+  (junction (at 64.77 59.69) (diameter 0) (color 0 0 0 0)
+  )
   (junction (at 207.01 30.48) (diameter 0) (color 0 0 0 0)
   )
@@
   (junction (at 38.1 43.18) (diameter 0) (color 0 0 0 0)
   )
+  (junction (at 38.1 49.53) (diameter 0) (color 0 0 0 0)
+  )
   (junction (at 46.99 105.41) (diameter 0) (color 0 0 0 0)
   )
@@
   (junction (at 162.56 22.86) (diameter 0) (color 0 0 0 0)
   )
+  (junction (at 57.15 63.5) (diameter 0) (color 0 0 0 0)
+  )
   (junction (at 64.77 53.34) (diameter 0) (color 0 0 0 0)
   )
@@
     (stroke (width 0) (type default) (color 0 0 0 0))
   )
+  (wire (pts (xy 64.77 59.69) (xy 64.77 53.34))
+    (stroke (width 0) (type default) (color 0 0 0 0))
+  )
   (wire (pts (xy 176.53 22.86) (xy 179.07 22.86))
     (stroke (width 0) (type default) (color 0 0 0 0))
   )
+  (wire (pts (xy 57.15 63.5) (xy 57.15 59.69))
+    (stroke (width 0) (type default) (color 0 0 0 0))
+  )
   (wire (pts (xy 184.15 142.24) (xy 209.55 142.24))
     (stroke (width 0) (type default) (color 0 0 0 0))
   )
+  (wire (pts (xy 57.15 59.69) (xy 52.07 59.69))
+    (stroke (width 0) (type default) (color 0 0 0 0))
+  )
   (wire (pts (xy 191.77 68.58) (xy 209.55 68.58))
     (stroke (width 0) (type default) (color 0 0 0 0))
@@
     (stroke (width 0) (type default) (color 0 0 0 0))
   )
-  (wire (pts (xy 64.77 63.5) (xy 64.77 53.34))
+  (wire (pts (xy 64.77 63.5) (xy 64.77 59.69))
     (stroke (width 0) (type default) (color 0 0 0 0))
   )
@@
     (stroke (width 0) (type default) (color 0 0 0 0))
   )
+  (wire (pts (xy 26.67 49.53) (xy 38.1 49.53))
+    (stroke (width 0) (type default) (color 0 0 0 0))
+  )
   (wire (pts (xy 177.8 137.16) (xy 209.55 137.16))
     (stroke (width 0) (type default) (color 0 0 0 0))
@@
     (stroke (width 0) (type default) (color 0 0 0 0))
   )
+  (wire (pts (xy 64.77 59.69) (xy 67.31 59.69))
+    (stroke (width 0) (type default) (color 0 0 0 0))
+  )
   (wire (pts (xy 97.79 55.88) (xy 100.33 55.88))
     (stroke (width 0) (type default) (color 0 0 0 0))
@@
     (stroke (width 0) (type default) (color 0 0 0 0))
   )
-  (wire (pts (xy 38.1 43.18) (xy 38.1 53.34))
+  (wire (pts (xy 38.1 43.18) (xy 38.1 49.53))
     (stroke (width 0) (type default) (color 0 0 0 0))
   )
@@
     (stroke (width 0) (type default) (color 0 0 0 0))
   )
+  (wire (pts (xy 38.1 49.53) (xy 38.1 53.34))
+    (stroke (width 0) (type default) (color 0 0 0 0))
+  )
   (wire (pts (xy 74.93 121.92) (xy 74.93 165.1))
     (stroke (width 0) (type default) (color 0 0 0 0))
@@
     (pin "2")
   )
+  (symbol (lib_id "power:PWR_FLAG") (at 67.31 59.69 0) (unit 1)
+    (in_bom yes) (on_board yes)
+    (property "Reference" "#FLG0108" (id 0) (at 67.31 57.785 0)
+      (effects (font (size 1.27 1.27)) hide)
+    )
+    (property "Value" "PWR_FLAG" (id 1) (at 71.12 54.61 0))
+    (property "Footprint" "" (id 2) (at 67.31 59.69 0)
+      (effects (font (size 1.27 1.27)) hide)
+    )
+    (property "Datasheet" "~" (id 3) (at 67.31 59.69 0)
+      (effects (font (size 1.27 1.27)) hide)
+    )
+    (pin "1")
+  )
   (symbol (lib_id "power:+3.3V") (at 137.16 132.08 0) (unit 1)
     (in_bom yes) (on_board yes) (fields_autoplaced)
@@
     (pin "2")
   )
+  (symbol (lib_id "power:PWR_FLAG") (at 52.07 59.69 0) (unit 1)
+    (in_bom yes) (on_board yes)
+    (property "Reference" "#FLG0106" (id 0) (at 52.07 57.785 0)
+      (effects (font (size 1.27 1.27)) hide)
+    )
+    (property "Value" "PWR_FLAG" (id 1) (at 55.88 54.61 0))
+    (property "Footprint" "" (id 2) (at 52.07 59.69 0)
+      (effects (font (size 1.27 1.27)) hide)
+    )
+    (property "Datasheet" "~" (id 3) (at 52.07 59.69 0)
+      (effects (font (size 1.27 1.27)) hide)
+    )
+    (pin "1")
+  )
   (symbol (lib_id "blank_card-eagle-import:GND") (at 63.5 134.62 0) (unit 1)
     (in_bom yes) (on_board yes)
@@
     (pin "4")
   )
+  (symbol (lib_id "power:PWR_FLAG") (at 26.67 49.53 0) (unit 1)
+    (in_bom yes) (on_board yes)
+    (property "Reference" "#FLG0107" (id 0) (at 26.67 47.625 0)
+      (effects (font (size 1.27 1.27)) hide)
+    )
+    (property "Value" "PWR_FLAG" (id 1) (at 30.48 44.45 0))
+    (property "Footprint" "" (id 2) (at 26.67 49.53 0)
+      (effects (font (size 1.27 1.27)) hide)
+    )
+    (property "Datasheet" "~" (id 3) (at 26.67 49.53 0)
+      (effects (font (size 1.27 1.27)) hide)
+    )
+    (pin "1")
+  )
   (symbol (lib_id "Connector:TestPoint") (at 215.9 163.83 0) (unit 1)
     (in_bom yes) (on_board yes)
@@
       (reference "#FLG0105") (unit 1) (value "PWR_FLAG") (footprint "")
     )
+    (path "/e08327f5-43de-4362-947c-c48e59fd1ce5"
+      (reference "#FLG0106") (unit 1) (value "PWR_FLAG") (footprint "")
+    )
+    (path "/f9e2cd98-8360-413b-9d11-952db75617e2"
+      (reference "#FLG0107") (unit 1) (value "PWR_FLAG") (footprint "")
+    )
+    (path "/3f9849a3-2e3b-424d-9f67-343c1c42b98d"
+      (reference "#FLG0108") (unit 1) (value "PWR_FLAG") (footprint "")
+    )
     (path "/85301209-d4e7-4865-8c28-2c9332fe340e"

Commit message: Update the Schematic and BOM for FET level shift. Make some parts DNI.
Parts:
- D101, D102, D103, F101, F102, F103, R120: LongLead (none) -> NO
- J1: value 09231486921 -> Plug 48 Way
- Q101, Q102, Q103, Q104: MPN (none) -> BSS138; Manufacturer (none) -> Yangzhou Yangjie Elec Tech
- R103, R104, R105, R107, R111, R114: value 1K -> DNI; MPN (none) -> RMC06031K1%N; Manufacturer (none) -> TyoHM
- R106, R109, R110, R113: value 10K -> 1K; Distributor 1 PN C269701 -> C269704; MPN (none) -> RMC06031K1%N; Manufacturer (none) -> TyoHM
- R108, R112, R115, R116: MPN (none) -> RMC 0603 10K F N; Manufacturer (none) -> TyoHM
- R117, R118, R119: MPN (none) -> RMC06031K1%N; Manufacturer (none) -> TyoHM
- TP101, TP102, TP103, TP104, TP105, TP106, TP107, TP108, TP109: AssemblyType HAND -> DNI
- U101: Cost 1.495 -> 1.798; Distributor 1 PN https://www.amazon.com/LM2596-Converter-Module-Supply-1-23V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 -> https://www.amazon.com/Zixtec-LM2596-Converter-Module-1-25V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
Other:
- note added: "J1 connector (Plug) to back plane bus. Signals are 3.3 Volt logic level."
- note removed: "J101 connector to bus is 3.3 Volt logic level."
