File: Hardware/GeneralPurposeAlarmDevicePCB/GeneralPurposeAlarmDevicePCB.kicad_pcb (KiCad board)
At the start: 2 copper layers, 137.2 x 83.8 mm, 128 parts, among them J101 Barrel_Jack_Switch_SMT, J102 0.100_2Pin, J103 0.100_2Pin, J105 S04B-XASK-1(LF)(SN), J401 RJ12_6P6C_HORZ, J501 USB_B_Micro_Local, J601 22-23-2021, J602 22-23-2021, Q201 MMBT2222A-7-F, Q202 MMBT2222A-7-F, Q203 MMBT2222A-7-F, Q204 MMBT2222A-7-F, Q205 MMBT2222A-7-F, Q301 BSS138, Q601 MMBT2222A-7-F, Q602 MMBT2907ALT1G, U101 LM7805_TO220, U102 PI_ATMEGA328P-AU-InOrder, U301 PCF8574AT, U302 LCD_20x4_Character-GPAD_SCH_L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, U501 CH340E

Commit message: Add JLCPCB place holder text to GPAD and PV_SPI_Conteroller. Create spead sheet for managing JLCPCB pick and place requirements.
Parts:
- added T1: JLC_ToolingHole_0576mm, PubInv_PCB:JLC_ToolingHole_0576mm, F.Cu at (61.0, 29.2)
- added T2: JLC_ToolingHole_0576mm, PubInv_PCB:JLC_ToolingHole_0576mm, F.Cu at (187.9, 29.2)
- added T3: JLC_ToolingHole_0576mm, PubInv_PCB:JLC_ToolingHole_0576mm, F.Cu at (61.0, 90.2)
Other:
- board text added: "JLCJLCJLCJLC"
Changed lines of the file:
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@@
     )
   )
+  (footprint "PubInv_PCB:JLC_ToolingHole_0576mm" (layer "F.Cu")
+    (at 187.941687 29.19542)
+    (fp_text reference "T2" (at 0.127 -1.524 unlocked) (layer "F.SilkS")
+      (effects (font (size 1 1) (thickness 0.15)))
+    )
+    (fp_text value "JLC_ToolingHole_0576mm" (at 0 1 unlocked) (layer "F.Fab")
+      (effects (font (size 1 1) (thickness 0.15)))
+    )
+    (fp_text user "${REFERENCE}" (at 0 2.5 unlocked) (layer "F.Fab")
+      (effects (font (size 1 1) (thickness 0.15)))
+    )
+    (fp_circle (center 0 0) (end 0.576 0) (layer "Edge.Cuts") (width 0.12) (fill none))
+  )
   (footprint "Resistor_SMD:R_0603_1608Metric_Pad0.98x0.95mm_HandSolder" (layer "F.Cu")
     (at 127 45.72 180)
@@
     )
   )
+  (footprint "PubInv_PCB:JLC_ToolingHole_0576mm" (layer "F.Cu")
+    (at 60.96 90.17)
+    (fp_text reference "T3" (at -3.302 2.286 unlocked) (layer "F.SilkS")
+      (effects (font (size 1 1) (thickness 0.15)))
+    )
+    (fp_text value "JLC_ToolingHole_0576mm" (at 0 1 unlocked) (layer "F.Fab")
+      (effects (font (size 1 1) (thickness 0.15)))
+    )
+    (fp_text user "${REFERENCE}" (at 0 2.5 unlocked) (layer "F.Fab")
+      (effects (font (size 1 1) (thickness 0.15)))
+    )
+    (fp_circle (center 0 0) (end 0.576 0) (layer "Edge.Cuts") (width 0.12) (fill none))
+  )
   (footprint "Package_TO_SOT_THT:TO-220-3_Horizontal_TabDown" (layer "F.Cu")
     (at 180.34 80.985)
@@
     )
   )
+  (footprint "PubInv_PCB:JLC_ToolingHole_0576mm" (layer "F.Cu")
+    (at 60.96 29.21)
+    (fp_text reference "T1" (at 0.127 -1.524 unlocked) (layer "F.SilkS")
+      (effects (font (size 1 1) (thickness 0.15)))
+    )
+    (fp_text value "JLC_ToolingHole_0576mm" (at 0 1 unlocked) (layer "F.Fab")
+      (effects (font (size 1 1) (thickness 0.15)))
+    )
+    (fp_text user "${REFERENCE}" (at 0 2.5 unlocked) (layer "F.Fab")
+      (effects (font (size 1 1) (thickness 0.15)))
+    )
+    (fp_circle (center 0 0) (end 0.576 0) (layer "Edge.Cuts") (width 0.12) (fill none))
+  )
   (footprint "TestPoint:TestPoint_Loop_D2.54mm_Drill1.5mm_Beaded" (layer "F.Cu")
     (at 102.235 82.55)
@@
     (effects (font (size 1.016 1.016) (thickness 0.254)))
   )
+  (gr_text "JLCJLCJLCJLC" (at 186.436 69.723 90) (layer "F.SilkS")
+    (effects (font (size 1 1) (thickness 0.15)))
+  )
   (gr_text "Power by\nController_Vcc" (at 167.005 83.82) (layer "F.SilkS")
     (effects (font (size 1.016 1.016) (thickness 0.254)))
@@
   (via (at 84.455 61.595) (size 0.8) (drill 0.4) (layers "F.Cu" "B.Cu") (free) (net 2))
   (via (at 113.9825 92.3925) (size 0.8) (drill 0.4) (layers "F.Cu" "B.Cu") (net 2))
-  (via (at 60.96 90.17) (size 0.8) (drill 0.4) (layers "F.Cu" "B.Cu") (free) (net 2))
+  (via (at 60.96 91.567) (size 0.8) (drill 0.4) (layers "F.Cu" "B.Cu") (free) (net 2))
   (via (at 110.73 51.86) (size 0.8) (drill 0.4) (layers "F.Cu" "B.Cu") (net 2))
   (via (at 134.62 27.94) (size 0.8) (drill 0.4) (layers "F.Cu" "B.Cu") (free) (net 2))

Commit message: Updateing for Version 2, 1K on BuiltinLED
Parts:
- R103: value 330R -> 1K
Changed lines of the file:
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@@
   (net 89 "Net-(A101-Pad3)")
   (net 90 "Net-(R311-Pad1)")
-  (net 91 "Net-(R110-Pad1)")
+  (net 91 "Net-(D105-Pad1)")
   (net 92 "Net-(D106-Pad2)")
   (footprint "Capacitor_SMD:CP_Elec_5x5.4" (layer "F.Cu")
@@
     (property "AssemblyType" "SMT")
     (property "Cost" "0.0015")
-    (property "Description" "0.1W ±1% 330Ω 0603 Chip Resistor - Surface Mount ROHS")
+    (property "Description" "0.1W ±1% 1kΩ 0603 Chip Resistor - Surface Mount ROHS")
     (property "Distributor 1" "JLCPCB")
-    (property "Distributor 1 PN" "C269711")
+    (property "Distributor 1 PN" "C269704")
     (property "MPN" "RMC06033301%N")
     (property "Manufacturer" "TyoHM")
@@
       (effects (font (size 1 1) (thickness 0.15)))
     )
-    (fp_text value "330R" (at 0 1.43) (layer "F.Fab")
+    (fp_text value "1K" (at 0 1.43) (layer "F.Fab")
       (effects (font (size 1 1) (thickness 0.15)))
     )
@@
     (fp_line (start -0.8 0.4125) (end -0.8 -0.4125) (layer "F.Fab") (width 0.1))
     (pad "1" smd roundrect (at -0.9125 0 180) (size 0.975 0.95) (layers "F.Cu" "F.Paste" "F.Mask") (roundrect_rratio 0.25)
-      (net 91 "Net-(R110-Pad1)") (pintype "passive"))
+      (net 91 "Net-(D105-Pad1)") (pintype "passive"))
     (pad "2" smd roundrect (at 0.9125 0 180) (size 0.975 0.95) (layers "F.Cu" "F.Paste" "F.Mask") (roundrect_rratio 0.25)
       (net 5 "+5V") (pintype "passive"))
@@
     (fp_arc (start 1.23 1.58) (mid -4.227431 0) (end 1.23 -1.58) (layer "B.Fab") (width 0.1))
     (pad "1" thru_hole rect locked (at -2.54 0) (size 2 2) (drill 1) (layers *.Cu *.Mask)
-      (net 91 "Net-(R110-Pad1)") (pintype "passive"))
+      (net 91 "Net-(D105-Pad1)") (pintype "passive"))
     (pad "2" thru_hole circle locked (at 0 0) (size 2 2) (drill 1) (layers *.Cu *.Mask)
       (net 2 "GND") (pintype "passive"))

Commit message: Add text to the UNO footprint front and back silk screen.
Parts:
- A101: footprint Module:Arduino_UNO_R3 -> GeneralPurposeAlarmDevicePCB:Arduino_UNO_R3_NoMountingHoles3D

Commit message: Enlarge_ground_around_U302_Pin_19.
Parts:
- moved C602 0.13 mm to (81.4, 83.8), turned to 180 degrees
Routing:
- net Light0: track 116.2 -> 114.6 mm
- net Switch_Mute: track 141.4 -> 142.4 mm, vias 4 -> 3
- net GND: vias 94 -> 101
Other:
- board text added: "CLK"
- board text added: "COPI"
- board text added: "SCL"
- board text added: "SDA"
- board text added: "nCS"
