File: Hardware/GeneralPurposeAlarmDevicePCB/GeneralPurposeAlarmDevicePCB.kicad_pcb (KiCad board)
At the start: 2 copper layers, 137.2 x 83.8 mm, 131 parts, among them J101 Barrel_Jack_Switch_SMT, J102 0.100_2Pin, J103 0.100_2Pin, J105 S04B-XASK-1(LF)(SN), J401 RJ12_6P6C_HORZ, J501 USB_B_Micro_Local, J601 22-23-2021, J602 22-23-2021, Q201 MMBT2222A-7-F, Q202 MMBT2222A-7-F, Q203 MMBT2222A-7-F, Q204 MMBT2222A-7-F, Q205 MMBT2222A-7-F, Q301 BSS138, Q601 MMBT2222A-7-F, Q602 MMBT2907ALT1G, T1 JLC_ToolingHole_0576mm, T2 JLC_ToolingHole_0576mm, T3 JLC_ToolingHole_0576mm, U101 LM7805_TO220, U102 PI_ATMEGA328P-AU-InOrder, U301 PCF8574AT, U302 LCD_20x4_Character-GPAD_SCH_L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, U501 CH340E

Commit message: MoveR104R105NearJ105
Parts:
- moved R104 39.4 mm to (139.1, 80.6), turned to 90 degrees
- moved R105 37.3 mm to (133.1, 83.1), turned to 90 degrees
- moved R310 17.7 mm to (178.7, 47.2)
Routing:
- net Net-(C114-Pad1): track 59.2 -> 8.81 mm, vias 5 -> 1
- net Net-(C113-Pad1): track 60.1 -> 11.5 mm, vias 5 -> 1
- net /LCD And I2C Interface/Vcc_LCD: track 124.5 -> 120.3 mm
- net Net-(R306-Pad1): track 43.9 -> 40.6 mm, vias 2 -> 0
- net +5V: track 456.4 -> 454.2 mm
- net ControllerRX: track 89.9 -> 91.4 mm
- net SDA: track 157.3 -> 155.8 mm, vias 2 -> 5
- net SCL: track 169.5 -> 170.4 mm, vias 2 -> 6
- net nRESET: track 54.9 -> 55.5 mm
- net COPI: track 87.8 -> 87.3 mm
- net GND: vias 101 -> 112

Commit message: Delete stray track.
Routing:
- net /LCD And I2C Interface/Vcc_LCD: track 120.3 -> 119.4 mm
Changed lines of the file:
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@@
   (segment (start 158.75 30.48) (end 163.195 30.48) (width 1.27) (layer "F.Cu") (net 67))
   (segment (start 162.900004 33.02) (end 161.925 33.995004) (width 1.27) (layer "F.Cu") (net 67))
-  (segment (start 177.5275 42.9075) (end 178.425 42.9075) (width 0.35) (layer "F.Cu") (net 67))
   (segment (start 135.89 34.925) (end 138.0725 37.1075) (width 0.35) (layer "F.Cu") (net 67))
   (segment (start 164.2375 27.94) (end 164.2375 27.220002) (width 0.35) (layer "F.Cu") (net 67))

Commit message: Make new schematic symbol and PCB symbol to correct pin numbers on JST connector. Generate new gerbers and drills.
Parts:
- J105: value S04B-XASK-1(LF)(SN) -> S04B-XASK-1(LF)(SN)Rev2; footprint GeneralPurposeAlarmDevicePCB:S04B-XASK-1(LF)(SN) -> GeneralPurposeAlarmDevicePCB:S04B-XASK-1(LF)(SN)Rev2
- moved J105 2.54 mm to (137.2, 104.1)
Connections:
- J105 pad 1: +5V -> Net-(C114-Pad1)
- J105 pad 2: Net-(C113-Pad1) -> GND
- J105 pad 3: GND -> Net-(C113-Pad1)
- J105 pad 4: Net-(C114-Pad1) -> +5V
Routing:
- net +5V: track 454.2 -> 456.8 mm
- net Net-(C114-Pad1): track 8.81 -> 11.4 mm
- net Net-(C113-Pad1): track 11.5 -> 14.0 mm
Other:
- outline, holes or cut-outs redrawn
- board text added: "General Purpouse Alarm Device, Public Invention, Rev 2.0 20230221"
- board text removed: "General Purpouse Alarm Device, Public Invention, Rev 2.0 20221113"
Changed lines of the file:
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@@
     )
   )
-  (footprint "GeneralPurposeAlarmDevicePCB:S04B-XASK-1(LF)(SN)" locked (layer "F.Cu")
-    (at 137.16 101.6 180)
-    (property "Assembly Type" "")
-    (property "AssemblyType" "HAND")
-    (property "Category" "Connectors, Interconnects")
-    (property "Cost" "0.1517")
-    (property "Description" "CONN HEADER R/A 4POS 2.5MM")
-    (property "Digi-Key_PN" "455-4090-ND")
-    (property "Distributor 1" "JLCPCB")
-    (property "Distributor 1 PN" "C265097")
-    (property "Distributor 2" "DigiKey  ")
-    (property "Distributor 2 PN" "455-4090-ND")
-    (property "Family" "Rectangular Connectors - Headers, Male Pins, Side Entery")
-    (property "MPN" "S04B-XASK-1(LF)(SN)")
-    (property "Manufacturer" "JST")
-    (property "Sheetfile" "GeneralPurposeAlarmDevicePCB.kicad_sch")
-    (property "Sheetname" "")
-    (property "Status" "Active")
-    (attr through_hole)
-    (fp_text reference "J105" (at -5.08 13.97 unlocked) (layer "F.SilkS")
-      (effects (font (size 1 1) (thickness 0.15)))
-    )
-    (fp_text value "S04B-XASK-1(LF)(SN)" (at 0.5 7.5 180 unlocked) (layer "F.Fab")
-      (effects (font (size 1 1) (thickness 0.15)))
-    )
-    (fp_text user "${REFERENCE}" (at 0.5 6 180 unlocked) (layer "F.Fab")
-      (effects (font (size 1 1) (thickness 0.15)))
-    )
-    (fp_line (start -2 3.5) (end -3 3.5) (layer "F.SilkS") (width 0.12))
-    (fp_line (start 2 3.5) (end 3 3.5) (layer "F.SilkS") (width 0.12))
-    (fp_line (start 0 5) (end 0 6) (layer "F.SilkS") (width 0.12))
-    (fp_line (start 0 2) (end 0 1) (layer "F.SilkS") (width 0.12))
-    (fp_rect (start -6.25 0) (end 6.25 12.6) (layer "F.SilkS") (width 0.12) (fill none))
-    (fp_circle (center -6.5 9.5) (end -5 9.5) (layer "F.SilkS") (width 0.12) (fill solid))
-    (pad "" thru_hole circle locked (at 0 3.5 180) (size 0 0) (drill oval 2.8 2) (layers *.Mask "Dwgs.User"))
-    (pad "1" thru_hole rect locked (at -3.75 9.2 180) (size 1.524 1.524) (drill 0.9) (layers *.Cu *.Mask)
-      (net 5 "+5V") (pintype "passive"))
-    (pad "2" thru_hole circle locked (at -1.25 9.2 180) (size 1.524 1.524) (drill 0.9) (layers *.Cu *.Mask)
-      (net 70 "Net-(C113-Pad1)") (pintype "passive"))
-    (pad "3" thru_hole circle locked (at 1.25 9.2 180) (size 1.524 1.524) (drill 0.9) (layers *.Cu *.Mask)
-      (net 2 "GND") (pintype "passive"))
-    (pad "4" thru_hole circle locked (at 3.75 9.2 180) (size 1.524 1.524) (drill 0.9) (layers *.Cu *.Mask)
-      (net 71 "Net-(C114-Pad1)") (pintype "passive"))
-    (model "${KIPRJMOD}/Parts/S04B-XASK-1/Cube.wrl"
-      (offset (xyz 6.35 0 0))
-      (scale (xyz 1 1 1))
-      (rotate (xyz 0 0 180))
-    )
-  )
   (footprint "Resistor_SMD:R_0603_1608Metric_Pad0.98x0.95mm_HandSolder" (layer "F.Cu")
     (at 139.065 80.645 90)
@@
     )
   )
+  (footprint "GeneralPurposeAlarmDevicePCB:S04B-XASK-1(LF)(SN)Rev2" locked (layer "F.Cu")
+    (at 137.16 104.14 180)
+    (property "Assembly Type" "HAND")
+    (property "Category" "Connectors, Interconnects")
+    (property "Description" "CONN HEADER R/A 4POS 2.5MM")
+    (property "Digi-Key_PN" "455-4090-ND")
+    (property "Distributor 1" "JLCPCB")
+    (property "Distributor 1 PN" "C265097")
+    (property "Distributor 2" "DigiKey  ")
+    (property "Distributor 2 PN" "455-4090-ND")
+    (property "Family" "Rectangular Connectors - Headers, Male Pins, Side Entery")
+    (property "MPN" "S04B-XASK-1(LF)(SN)")
+    (property "Manufacturer" "JST")
+    (property "Sheetfile" "GeneralPurposeAlarmDevicePCB.kicad_sch")
+    (property "Sheetname" "")
+    (property "Status" "Active")
+    (attr through_hole)
+    (fp_text reference "J105" (at -5.08 13.97 unlocked) (layer "F.SilkS")
+      (effects (font (size 1 1) (thickness 0.15)))
+    )
+    (fp_text value "S04B-XASK-1(LF)(SN)Rev2" (at 0.5 7.5 180 unlocked) (layer "F.Fab")
+      (effects (font (size 1 1) (thickness 0.15)))
+    )
+    (fp_text user "${REFERENCE}" (at 0.5 6 180 unlocked) (layer "F.Fab")
+      (effects (font (size 1 1) (thickness 0.15)))
+    )
+    (fp_line (start -2 3.5) (end -3 3.5) (layer "F.SilkS") (width 0.12))
+    (fp_line (start 0 5) (end 0 6) (layer "F.SilkS") (width 0.12))
+    (fp_line (start 0 2) (end 0 1) (layer "F.SilkS") (width 0.12))
+    (fp_line (start 2 3.5) (end 3 3.5) (layer "F.SilkS") (width 0.12))
+    (fp_rect (start -6.25 0) (end 6.25 12.6) (layer "F.SilkS") (width 0.12) (fill none))
+    (fp_circle (center 6.35 9.525) (end 7.85 9.525) (layer "F.SilkS") (width 0.12) (fill solid))
+    (pad "" thru_hole circle locked (at 0 3.5 180) (size 0 0) (drill oval 2.8 2) (layers *.Mask "Dwgs.User"))
+    (pad "1" thru_hole rect locked (at 3.75 9.2 180) (size 1.524 1.524) (drill 0.9) (layers *.Cu *.Mask)
+      (net 71 "Net-(C114-Pad1)") (pintype "passive"))
+    (pad "2" thru_hole circle locked (at 1.25 9.2 180) (size 1.524 1.524) (drill 0.9) (layers *.Cu *.Mask)
+      (net 2 "GND") (pintype "passive"))
+    (pad "3" thru_hole circle locked (at -1.25 9.2 180) (size 1.524 1.524) (drill 0.9) (layers *.Cu *.Mask)
+      (net 70 "Net-(C113-Pad1)") (pintype "passive"))
+    (pad "4" thru_hole circle locked (at -3.75 9.2 180) (size 1.524 1.524) (drill 0.9) (layers *.Cu *.Mask)
+      (net 5 "+5V") (pintype "passive"))
+    (model "${KIPRJMOD}/Parts/S04B-XASK-1/Cube.wrl"
+      (offset (xyz 6.35 0 0))
+      (scale (xyz 1 1 1))
+      (rotate (xyz 0 0 180))
+    )
+  )
   (footprint "TestPoint:TestPoint_Loop_D2.54mm_Drill1.5mm_Beaded" (layer "F.Cu")
     (at 104.14 98.425)
@@
   )
   (gr_line (start 193.04 17.78) (end 55.88 17.78) (layer "Edge.Cuts") (width 0.05))
-  (gr_line (start 55.88 101.6) (end 193.04 101.6) (layer "Edge.Cuts") (width 0.05))
   (gr_line (start 55.88 17.78) (end 55.88 101.6) (layer "Edge.Cuts") (width 0.05))
+  (gr_line (start 138.557 101.6) (end 193.04 101.6) (layer "Edge.Cuts") (width 0.05))
+  (gr_line (start 135.763 101.6) (end 55.88 101.6) (layer "Edge.Cuts") (width 0.05))
+  (gr_arc (start 137.541 99.568) (mid 138.25942 99.86558) (end 138.557 100.584) (layer "Edge.Cuts") (width 0.05))
+  (gr_arc (start 135.763 100.584) (mid 136.06058 99.86558) (end 136.779 99.568) (layer "Edge.Cuts") (width 0.05))
   (gr_line (start 193.04 101.6) (end 193.04 17.78) (layer "Edge.Cuts") (width 0.05))
+  (gr_line (start 137.541 99.568) (end 136.779 99.568) (layer "Edge.Cuts") (width 0.05))
+  (gr_line (start 135.763 101.6) (end 135.763 100.584) (layer "Edge.Cuts") (width 0.05))
+  (gr_line (start 138.557 101.6) (end 138.557 100.584) (layer "Edge.Cuts") (width 0.05))
   (gr_text "Contrast" (at 184.785 34.925) (layer "B.SilkS")
     (effects (font (size 1.016 1.016) (thickness 0.254)) (justify mirror))
@@
     (effects (font (size 0.762 0.762) (thickness 0.1524)))
   )
-  (gr_text "General Purpouse Alarm Device, Public Invention, Rev 2.0 20221113" (at 116.205 19.05) (layer "F.SilkS")
+  (gr_text "General Purpouse Alarm Device, Public Invention, Rev 2.0 20230221" (at 116.205 19.05) (layer "F.SilkS")
     (effects (font (size 1.27 1.27) (thickness 0.254)))
   )
@@
   (segment (start 140.91 87.69) (end 140.97 87.63) (width 0.2) (layer "B.Cu") (net 5))
   (segment (start 142.621 72.136) (end 142.621 77.597) (width 1.27) (layer "B.Cu") (net 5))
-  (segment (start 140.910005 92.399993) (end 140.910005 87.689995) (width 0.762) (layer "B.Cu") (net 5))
   (segment (start 140.97 87.63) (end 141.605 86.995) (width 0.762) (layer "B.Cu") (net 5))
   (segment (start 142.621 77.597) (end 142.494 77.724) (width 1.27) (layer "B.Cu") (net 5))
+  (segment (start 140.91 94.92001) (end 140.92999 94.94) (width 0.35) (layer "B.Cu") (net 5))
+  (segment (start 140.910005 94.939993) (end 140.910005 87.689995) (width 0.889) (layer "B.Cu") (net 5))
   (segment (start 141.605 86.995) (end 141.605 86.36) (width 0.762) (layer "B.Cu") (net 5))
+  (segment (start 140.91 94.94) (end 140.910005 94.939995) (width 0.762) (layer "B.Cu") (net 5))
   (segment (start 106.68 89.3075) (end 107.0875 88.9) (width 0.254) (layer "F.Cu") (net 6))
   (segment (start 106.2725 89.3075) (end 106.68 89.3075) (width 0.2) (layer "F.Cu") (net 6))
@@
   (segment (start 139.065 85.3175) (end 138.6575 85.725) (width 0.25) (layer "F.Cu") (net 70))
   (via (at 139.065 87.63) (size 0.8) (drill 0.4) (layers "F.Cu" "B.Cu") (net 70))
-  (segment (start 138.41001 92.399993) (end 138.41001 88.28499) (width 0.635) (layer "B.Cu") (net 70))
+  (segment (start 138.43 88.30498) (end 138.43 94.939993) (width 0.889) (layer "B.Cu") (net 70))
   (segment (start 138.41 88.285) (end 139.065 87.63) (width 0.2) (layer "B.Cu") (net 70))
+  (segment (start 138.41001 88.28499) (end 138.42999 88.30497) (width 0.635) (layer "B.Cu") (net 70))
   (segment (start 133.1225 85.725) (end 133.1225 84.0475) (width 0.2) (layer "F.Cu") (net 71))
   (segment (start 132.715 86.1325) (end 133.1225 85.725) (width 0.2) (layer "F.Cu") (net 71))
   (segment (start 132.715 87.63) (end 132.715 86.1325) (width 0.2) (layer "F.Cu") (net 71))
   (via (at 132.715 87.63) (size 0.8) (drill 0.4) (layers "F.Cu" "B.Cu") (net 71))
-  (segment (start 133.41 88.325) (end 132.715 87.63) (width 0.2) (layer "B.Cu") (net 71))
-  (segment (start 133.409995 92.399993) (end 133.409995 88.324995) (width 0.635) (layer "B.Cu") (net 71))
+  (segment (start 132.715 87.63) (end 133.42999 88.34499) (width 0.381) (layer "B.Cu") (net 71))
+  (segment (start 133.429985 88.344985) (end 133.429985 94.939993) (width 0.889) (layer "B.Cu") (net 71))
   (segment (start 134.62 65.786) (end 139.446 65.786) (width 0.508) (layer "F.Cu") (net 72))
   (segment (start 139.446 65.786) (end 139.7 66.04) (width 0.25) (layer "F.Cu") (net 72))
