File: Hardware/GeneralPurposeAlarmDevicePCB/GeneralPurposeAlarmDevicePCB.kicad_pcb (KiCad board)
At the start: 2 copper layers, 137.2 x 83.8 mm, 131 parts, among them J101 Barrel_Jack_Switch_SMT, J102 0.100_2Pin, J103 0.100_2Pin, J105 S04B-XASK-1(LF)(SN)Rev2, J401 RJ12_6P6C_HORZ, J501 USB_B_Micro_Local, J601 22-23-2021, J602 22-23-2021, Q201 MMBT2222A-7-F, Q202 MMBT2222A-7-F, Q203 MMBT2222A-7-F, Q204 MMBT2222A-7-F, Q205 MMBT2222A-7-F, Q301 BSS138, Q601 MMBT2222A-7-F, Q602 MMBT2907ALT1G, T1 JLC_ToolingHole_0576mm, T2 JLC_ToolingHole_0576mm, T3 JLC_ToolingHole_0576mm, U101 LM7805_TO220, U102 PI_ATMEGA328P-AU-InOrder, U301 PCF8574AT, U302 LCD_20x4_Character-GPAD_SCH_L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, U501 CH340E

Commit message: Add Adafruit buzzer to PCB. DRC no errors. Trivial warnings.
Parts:
- added R506: DNI, Resistor_SMD:R_0603_1608Metric_Pad0.98x0.95mm_HandSolder, F.Cu at (59.2, 73.4)
- added R507: 1R, Resistor_SMD:R_0603_1608Metric_Pad0.98x0.95mm_HandSolder, F.Cu at (66.3, 89.5)
- added R508: 1R, Resistor_SMD:R_0603_1608Metric_Pad0.98x0.95mm_HandSolder, F.Cu at (58.9, 89.4)
- BZ601: value Buzzer_12.2mm_H6.5mm -> Buzzer_Adafruit_P1536A; footprint Buzzer_Beeper:Buzzer_TDK_PS1240P02BT_D12.2mm_H6.5mm -> GeneralPurposeAlarmDevicePCB:Buzzer_12.2mm_9.7mm_7.62mm
- Q601: value MMBT2222A-7-F -> BSS138
- Q602: value MMBT2907ALT1G -> DNI
- R604: value 1R -> DNI
- moved R505 31.9 mm to (59.8, 57.7)
- moved R112 2.17 mm to (126.7, 47.9)
- moved D106 1.93 mm to (129.0, 45.2)
- moved BZ601 1.44 mm to (74.9, 86.4)
- turned C601 to 180 degrees
Connections:
- BZ601 pad 1: Net-(BZ601-Pad1) -> /AlarmAudio/VccBuzzer
- BZ601 pad 2: GND -> Net-(BZ601-Pad2)
- J601 pad 1: Net-(BZ601-Pad1) -> /AlarmAudio/VccBuzzer
- J601 pad 2: GND -> Net-(BZ601-Pad2)
- Q601 pad 3: /AlarmAudio/VccBuzzer -> Net-(Q601-Pad3)
- R604 pad 1: Net-(BZ601-Pad1) -> Net-(BZ601-Pad2)
Routing:
- net Net-(Q601-Pad3): track 0.00 -> 24.1 mm
- net /AlarmAudio/VccBuzzer: track 19.4 -> 43.5 mm, vias 0 -> 1
- net Net-(BZ601-Pad1): track 19.8 -> 0.00 mm, vias 1 -> 0
- net Net-(BZ601-Pad2): track 0.00 -> 16.1 mm, vias 0 -> 1
- net GND: track 136.0 -> 131.9 mm, vias 112 -> 114
- net Net-(Q601-Pad2): track 6.76 -> 9.04 mm
- net +5V: track 456.8 -> 457.9 mm
- net Light0: track 114.6 -> 113.9 mm
- net Net-(Q601-Pad1): track 79.0 -> 78.3 mm
Other:
- board text added: "General Purpouse Alarm Device, Public Invention, Rev 2.0 20230228"
- board text removed: "External Speaker"
- board text removed: "General Purpouse Alarm Device, Public Invention, Rev 2.0 20230221"

Commit message: Update U301 for JLCPCB in stock, Break and then fix SCH library because of illigal character in sch symbol name.
Parts:
- R401, R402, R403, R404, R605: value 330 -> 330R
- U301: value PCF8574AT -> PCF8574AT_3_518
Changed lines of the file:
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@@
     (property "Description" "TRANS PNP 60V 0.6A SOT23")
     (property "Digi-Key_PN" "MMBT2907ALT1GOSCT-ND")
-    (property "Distributor 1" "JCLPCB")
-    (property "Distributor 1 PN" "C40752")
+    (property "Distributor 1" "DNI")
+    (property "Distributor 1 PN" "DNI")
+    (property "Distributor 2" "JCLPCB")
+    (property "Distributor 2 PN" "C40752")
     (property "Family" "Transistors - Bipolar (BJT) - Single")
     (property "MPN" "MMBT2907ALT1G")
@@
       (effects (font (size 1 1) (thickness 0.15)))
     )
-    (fp_text value "330" (at 0 1.43 90) (layer "F.Fab")
+    (fp_text value "330R" (at 0 1.43 90) (layer "F.Fab")
       (effects (font (size 1 1) (thickness 0.15)))
     )
@@
     (tags "SOIC SO")
     (property "AssemblyType" "SMT")
-    (property "Cost" "0.6414")
-    (property "Description" "Remote 8-bit I/O expander for I2C-bus with interrupt")
+    (property "Cost" "1.87")
     (property "Distributor 1" "JLCPCB")
-    (property "Distributor 1 PN" "C83193")
-    (property "MPN" "PCF8574AT/3,512")
-    (property "Manufacturer" "NXP Semicon")
+    (property "Distributor 1 PN" "C86832")
+    (property "MPN" "PCF8574AT_3_518")
     (property "Sheetfile" "LCD And I2C Interface.kicad_sch")
     (property "Sheetname" "LCD And I2C Interface")
@@
       (effects (font (size 1 1) (thickness 0.15)))
     )
-    (fp_text value "PCF8574AT" (at 0 6.1 180) (layer "F.Fab")
+    (fp_text value "PCF8574AT_3_518" (at 0 6.1 180) (layer "F.Fab")
       (effects (font (size 1 1) (thickness 0.15)))
     )
@@
     (property "Distributor 1" "JLCPCB")
     (property "Distributor 1 PN" "C269704")
-    (property "MPN" "RMC06033301%N")
+    (property "MPN" "RMC06031K1%N")
     (property "Manufacturer" "TyoHM")
     (property "Sheetfile" "GeneralPurposeAlarmDevicePCB.kicad_sch")
@@
     (property "AssemblyType" "SMT")
     (property "Cost" "0.0015")
-    (property "Description" "0.1W ±5% 1Ω 0603 Chip Resistor - Surface Mount ROHS")
-    (property "Distributor 1" "JLCPCB")
-    (property "Distributor 1 PN" "C269434")
+    (property "Description" "DNI")
+    (property "Distributor 1" "DNI")
+    (property "Distributor 1 PN" "DNI")
     (property "MPN" "RMC060315%N")
     (property "Manufacturer" "TyoHM")
@@
     (property "Cost" "0.0015")
     (property "Description" "DNI")
-    (property "Distributor 1" "JLCPCB")
+    (property "Distributor 1" "DNI")
     (property "Distributor 1 PN" "DNI")
     (property "MPN" "DNI")
@@
     (property "Cost" "0.0015")
     (property "Description" "DNI")
-    (property "Distributor 1" "JLCPCB")
+    (property "Distributor 1" "DNI")
     (property "Distributor 1 PN" "DNI")
     (property "MPN" "DNI")
@@
     (property "Cost" "0.0015")
     (property "Description" "DNI")
-    (property "Distributor 1" "JLCPCB")
+    (property "Distributor 1" "DNI")
     (property "Distributor 1 PN" "DNI")
     (property "MPN" "DNI")
@@
     (property "Cost" "0.0015")
     (property "Description" "DNI")
-    (property "Distributor 1" "JLCPCB")
+    (property "Distributor 1" "DNI")
     (property "Distributor 1 PN" "DNI")
     (property "MPN" "DNI")
@@
       (effects (font (size 1 1) (thickness 0.15)))
     )
-    (fp_text value "330" (at 0 1.43 -90) (layer "F.Fab")
+    (fp_text value "330R" (at 0 1.43 -90) (layer "F.Fab")
       (effects (font (size 1 1) (thickness 0.15)))
     )
@@
       (effects (font (size 1 1) (thickness 0.15)))
     )
-    (fp_text value "330" (at 0 1.43 -90) (layer "F.Fab")
+    (fp_text value "330R" (at 0 1.43 -90) (layer "F.Fab")
       (effects (font (size 1 1) (thickness 0.15)))
     )
@@
       (effects (font (size 1 1) (thickness 0.15)))
     )
-    (fp_text value "330" (at 0 1.43 -90) (layer "F.Fab")
+    (fp_text value "330R" (at 0 1.43 -90) (layer "F.Fab")
       (effects (font (size 1 1) (thickness 0.15)))
     )
@@
       (effects (font (size 1 1) (thickness 0.15)))
     )
-    (fp_text value "330" (at 0 1.43 -90) (layer "F.Fab")
+    (fp_text value "330R" (at 0 1.43 -90) (layer "F.Fab")
       (effects (font (size 1 1) (thickness 0.15)))
     )
@@
     (property "AssemblyType" "SMT")
     (property "Cost" "0.0015")
-    (property "Description" "0.1W ±5% 1Ω 0603 Chip Resistor - Surface Mount ROHS")
-    (property "Distributor 1" "JLCPCB")
-    (property "Distributor 1 PN" "C269434")
+    (property "Description" "DNI")
+    (property "Distributor 1" "DNI")
+    (property "Distributor 1 PN" "DNI")
     (property "MPN" "RMC060315%N")
     (property "Manufacturer" "TyoHM")
@@
     (fp_line (start -1.27 -2.92) (end -1.27 2.88) (layer "F.Fab") (width 0.1))
     (fp_line (start -0.562893 0) (end -1.27 0.5) (layer "F.Fab") (width 0.1))
-    (pad "1" thru_hole roundrect (at 0 0 180) (size 1.74 2.19) (drill 1.19) (layers *.Cu *.Mask) (roundrect_rratio 0.143678)
+    (pad "1" thru_hole roundrect (at 0 0 180) (size 1.74 2.19) (drill 1.19) (layers *.Cu *.Mask) (roundrect_rratio 0.1436781609)
       (net 67 "Switch_Mute") (pintype "passive"))
     (pad "2" thru_hole oval (at 2.54 0 180) (size 1.74 2.19) (drill 1.19) (layers *.Cu *.Mask)
@@
     (property "Assembly Type" "HAND")
     (property "Category" "Connectors, Interconnects")
+    (property "Cost" "0.15")
     (property "Description" "CONN HEADER R/A 4POS 2.5MM")
     (property "Digi-Key_PN" "455-4090-ND")
@@
     (property "Cost" "4.99")
     (property "Description" "")
-    (property "Distributor 1" "Aliexpress")
-    (property "Distributor 1 PN" "https://www.aliexpress.com/item/3256803213374992.html")
-    (property "Distributor 2" "Amazon")
-    (property "Distributor 2 PN" "https://www.amazon.com/GeeekPi-Interface-Adapter-Backlight-Raspberry/dp/B07QLRD3TM/ref=sr_1_2")
+    (property "Distributor 1" "eBay   Aliexpress")
+    (property "Distributor 1 PN" "403534100457 ")
+    (property "Distributor 2" "Amazon  / Aliexpress")
+    (property "Distributor 2 PN" "https://www.amazon.com/GeeekPi-Interface-Adapter-Backlight-Raspberry/dp/B07QLRD3TM/ref=sr_1_2 /  https://www.aliexpress.com/item/3256803213374992.html")
     (property "MPN" "")
     (property "MPN " "")

Commit message: Update LED standoff in PCB library and PCB.
Parts:
- added MF103: U_Box_V104_General_Alarm_Device_LED_Standoff, GeneralPurposeAlarmDevicePCB:U_Box_V104_General_Alarm_Device_LED_Standoff, B.Cu at (186.7, 54.6)
- added MF601: U_Box_V104_General_Alarm_Device_LED_Standoff, GeneralPurposeAlarmDevicePCB:U_Box_V104_General_Alarm_Device_LED_Standoff, B.Cu at (71.1, 72.4)
- added MF602: U_Box_V104_General_Alarm_Device_LED_Standoff, GeneralPurposeAlarmDevicePCB:U_Box_V104_General_Alarm_Device_LED_Standoff, B.Cu at (71.1, 59.8)
- added MF603: U_Box_V104_General_Alarm_Device_LED_Standoff, GeneralPurposeAlarmDevicePCB:U_Box_V104_General_Alarm_Device_LED_Standoff, B.Cu at (71.1, 47.0)
- added MF604: U_Box_V104_General_Alarm_Device_LED_Standoff, GeneralPurposeAlarmDevicePCB:U_Box_V104_General_Alarm_Device_LED_Standoff, B.Cu at (71.1, 34.2)
- added MF605: U_Box_V104_General_Alarm_Device_LED_Standoff, GeneralPurposeAlarmDevicePCB:U_Box_V104_General_Alarm_Device_LED_Standoff, B.Cu at (71.1, 21.6)

Commit message: Add PCB Layout for Battery Circuitry
Also created several Capstone Specific BOMs/PDFs
Parts:
- added C702: 10uF, Capacitor_SMD:C_0603_1608Metric_Pad1.08x0.95mm_HandSolder, F.Cu at (167.6, 68.5)
- added D701: ORANGE 0603, LED_SMD:LED_0603_1608Metric, F.Cu at (149.9, 63.5)
- added D702: GREEN 0603, LED_SMD:LED_0603_1608Metric, F.Cu at (152.4, 59.2)
- added D703: RED 0603, LED_SMD:LED_0603_1608Metric_Pad1.05x0.95mm_HandSolder, F.Cu at (157.5, 58.4)
- added D704: PMEG3020EP, Diode_SMD:D_SOD-128, F.Cu at (152.4, 71.1)
- added J701: BATT_JST, Connector_JST:JST_PH_S2B-PH-K_1x02_P2.00mm_Horizontal, F.Cu at (162.6, 68.6)
- added Q302: AOSS21311C, Package_TO_SOT_SMD:SOT-23, F.Cu at (128.0, 52.4)
- added R701: 330R, Resistor_SMD:R_0603_1608Metric_Pad0.98x0.95mm_HandSolder, F.Cu at (152.4, 66.0)
- added R702: 330R, Resistor_SMD:R_0603_1608Metric_Pad0.98x0.95mm_HandSolder, F.Cu at (154.9, 55.9)
- added R703: 330R, Resistor_SMD:R_0603_1608Metric_Pad0.98x0.95mm_HandSolder, F.Cu at (167.6, 55.9)
- added R704: 2K, Resistor_SMD:R_0603_1608Metric_Pad0.98x0.95mm_HandSolder, F.Cu at (162.6, 55.9)
- added R705: 1K, Resistor_SMD:R_0603_1608Metric_Pad0.98x0.95mm_HandSolder, F.Cu at (170.2, 50.8)
- added R706: 150K, Resistor_SMD:R_0603_1608Metric_Pad0.98x0.95mm_HandSolder, F.Cu at (167.6, 50.8)
- added TH701: 10k Therm, Resistor_SMD:R_0603_1608Metric_Pad0.98x0.95mm_HandSolder, F.Cu at (165.1, 50.8)
- added U701: MCP73833, Package_DFN_QFN:DFN-10-1EP_3x3mm_P0.5mm_EP1.7x2.5mm, F.Cu at (159.6, 52.7)
- moved R109 3.98 mm to (137.2, 54.3)
- moved R102 0.28 mm to (122.8, 66.0)
Connections:
- U102 pad 22: unconnected-(U102-Pad22) -> LCD power
Routing:
- net +5V: track 457.9 -> 521.9 mm
- net /LCD And I2C Interface/Vcc_LCD: track 119.4 -> 180.9 mm
- net Net-(D704-A): track 0.00 -> 47.9 mm
- net Vin: track 88.2 -> 121.6 mm
- net LCD power: track 0.00 -> 25.1 mm
- net Net-(U701-STAT1): track 0.00 -> 20.1 mm
- net Net-(D703-K): track 0.00 -> 12.5 mm
- net Net-(U701-THERM): track 0.00 -> 9.95 mm
- net Net-(U701-PG): track 0.00 -> 6.77 mm
- net VccController: track 151.8 -> 157.6 mm
- net Net-(U701-STAT2): track 0.00 -> 5.21 mm
- net Net-(R705-Pad2): track 0.00 -> 5.02 mm
- net PC0: track 31.0 -> 35.7 mm
- net Net-(D702-K): track 0.00 -> 4.50 mm
- net Net-(D701-K): track 0.00 -> 3.91 mm
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