File: Hardware/GeneralPurposeAlarmDevicePCB/GeneralPurposeAlarmDevicePCB.kicad_sch (KiCad schematic)
At the start: 52 parts, among them J101 Barrel_Jack_Switch_SMT, J102 0.100_2Pin, J103 0.100_2Pin, J105 S04B-XASK-1(LF)(SN), U101 LM7805_TO220, U102 PI_ATMEGA328P-AU-InOrder

Commit message: Update schematic for rework of Version 1 PCB for D7 and D10 and Reset to nRTS.
Connections:
- net GND: no longer C110.2
- net Light4: now also U102.11 (PD7); no longer U102.14 (PB2)
- net nCS: now also U102.14 (PB2); no longer U102.11 (PD7)
- new net nRTS: C110.2
Other:
- sheet USB_UART ports: added nRTS; removed none
- note added: "Note: Schematic Rev 1.2 reflects rework to PCB 20220726. D7 and D10 interchanged. C110 connects reset to U501 pin 4 nRTS."
- note added: "Note: Using 0603HandSolder for Rs and Cs."
- note removed: "Note: Check pad sized for 0603 and 0603HandSolder"
Changed lines of the file:
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@@
   (title_block
     (title "GeneralPurposeAlarmDevicePCB")
-    (date "2022-06-20")
-    (rev "0.0")
+    (date "2022-11-13")
+    (rev "1.2")
     (company "PublicInvention")
     (comment 1 "GNU Affero General Public License v3.0")
@@
     (stroke (width 0) (type default) (color 0 0 0 0))
   )
+  (wire (pts (xy 46.99 171.45) (xy 52.07 171.45))
+    (stroke (width 0) (type default) (color 0 0 0 0))
+  )
   (wire (pts (xy 186.69 24.13) (xy 186.69 27.94))
     (stroke (width 0) (type default) (color 0 0 0 0))
@@
     (stroke (width 0) (type default) (color 0 0 0 0))
   )
+  (wire (pts (xy 124.46 74.93) (xy 124.46 78.74))
+    (stroke (width 0) (type default) (color 0 0 0 0))
+  )
   (wire (pts (xy 182.88 104.14) (xy 189.23 104.14))
     (stroke (width 0) (type default) (color 0 0 0 0))
@@
     (stroke (width 0) (type default) (color 0 0 0 0))
   )
+  (wire (pts (xy 130.81 78.74) (xy 124.46 78.74))
+    (stroke (width 0) (type default) (color 0 0 0 0))
+  )
   (wire (pts (xy 74.93 95.25) (xy 76.2 95.25))
     (stroke (width 0) (type default) (color 0 0 0 0))
@@
     (effects (font (size 1.27 1.27)) (justify left bottom))
   )
+  (text "Note: Schematic Rev 1.2 reflects rework to PCB 20220726.\nD7 and D10 interchanged.\nC110 connects reset to U501 pin 4 nRTS."
+    (at 161.29 177.8 0)
+    (effects (font (size 1.27 1.27)) (justify left bottom))
+  )
   (text "Power Indicator" (at 138.43 48.26 0)
     (effects (font (size 1.27 1.27)) (justify left bottom))
@@
     (effects (font (size 1.27 1.27)) (justify left bottom))
   )
-  (text "Note: Check pad sized for 0603 and 0603HandSolder" (at 39.37 135.89 0)
+  (text "Note: Using 0603HandSolder for Rs and Cs." (at 161.29 170.18 0)
     (effects (font (size 1.27 1.27)) (justify left bottom))
   )
@@
     )
   )
-  (global_label "Light4" (shape output) (at 96.52 157.48 180) (fields_autoplaced)
+  (global_label "Light4" (shape output) (at 91.44 138.43 270) (fields_autoplaced)
     (effects (font (size 1.27 1.27)) (justify right))
-    (property "Intersheet References" "${INTERSHEET_REFS}" (id 0) (at 0 0 0)
+    (property "Intersheet References" "${INTERSHEET_REFS}" (id 0) (at -66.04 234.95 0)
       (effects (font (size 1.27 1.27)) hide)
     )
@@
     )
   )
+  (global_label "nRTS" (shape input) (at 52.07 171.45 0) (fields_autoplaced)
+    (effects (font (size 1.27 1.27)) (justify left))
+    (property "Intersheet References" "${INTERSHEET_REFS}" (id 0) (at 58.9904 171.3706 0)
+      (effects (font (size 1.27 1.27)) (justify left) hide)
+    )
+  )
   (global_label "Light1" (shape output) (at 236.22 143.51 180) (fields_autoplaced)
     (effects (font (size 1.27 1.27)) (justify right))
@@
     )
   )
+  (global_label "nRTS" (shape input) (at 130.81 78.74 0) (fields_autoplaced)
+    (effects (font (size 1.27 1.27)) (justify left))
+    (property "Intersheet References" "${INTERSHEET_REFS}" (id 0) (at 137.7304 78.6606 0)
+      (effects (font (size 1.27 1.27)) (justify left) hide)
+    )
+  )
   (global_label "Tone" (shape output) (at 173.99 138.43 180) (fields_autoplaced)
     (effects (font (size 1.27 1.27)) (justify right))
@@
     )
   )
-  (global_label "nCS" (shape output) (at 91.44 138.43 270) (fields_autoplaced)
+  (global_label "nCS" (shape output) (at 96.52 157.48 180) (fields_autoplaced)
     (effects (font (size 1.27 1.27)) (justify right))
-    (property "Intersheet References" "${INTERSHEET_REFS}" (id 0) (at 0 0 0)
+    (property "Intersheet References" "${INTERSHEET_REFS}" (id 0) (at 234.95 66.04 0)
       (effects (font (size 1.27 1.27)) hide)
     )
@@
     (pin "2")
   )
-  (symbol (lib_id "power:GND") (at 124.46 74.93 0) (unit 1)
-    (in_bom yes) (on_board yes)
-    (property "Reference" "#PWR0118" (id 0) (at 124.46 81.28 0)
-      (effects (font (size 1.27 1.27)) hide)
-    )
-    (property "Value" "GND" (id 1) (at 124.587 79.3242 0))
-    (property "Footprint" "" (id 2) (at 124.46 74.93 0)
-      (effects (font (size 1.27 1.27)) hide)
-    )
-    (property "Datasheet" "" (id 3) (at 124.46 74.93 0)
-      (effects (font (size 1.27 1.27)) hide)
-    )
-    (pin "1")
-  )
   (symbol (lib_id "Device:D_Schottky") (at 85.09 54.61 0) (mirror x) (unit 1)
     (in_bom yes) (on_board yes)
@@
       (effects (font (size 1.27 1.27)) (justify right))
     )
+    (pin "nRTS" input (at 46.99 171.45 0)
+      (effects (font (size 1.27 1.27)) (justify right))
+    )
   )
   (sheet (at 243.84 93.98) (size 20.32 31.75) (fields_autoplaced)
@@
       (reference "#PWR0117") (unit 1) (value "GND") (footprint "")
     )
-    (path "/00000000-0000-0000-0000-000062f990fb"
-      (reference "#PWR0118") (unit 1) (value "GND") (footprint "")
-    )
     (path "/00000000-0000-0000-0000-000062cbe01c"

Commit message: Update PCB for version 2. Update enclosure drawing to reflect the V1 enclosure assembly.
Parts:
- removed D105: LTL2R3KEK, GeneralPurposeAlarmDevicePCB:LED_5mm_Radial, symbol Device:LED
- added D105: LED_T1.75_CLEAR_RED, GeneralPurposeAlarmDevicePCB:LED_5mm_Radial, symbol GPAD_SCH_LIB:LED_T1.75_CLEAR_WHITE
Connections:
- net GND: now also D105.2
- net Light4: now also A101.22 (D7); no longer A101.25 (D10)
- net PC3: now also R103.2
- net SPI_SCK: no longer R103.2
- net nCS: now also A101.25 (D10); no longer A101.22 (D7)
- net at R110.1: now also D105.1
Other:
- note removed: "Note: Schematic Rev 1.2 reflects rework to PCB 20220726. D7 and D10 interchanged. C110 connects reset to U501 pin 4 nRTS."
- moved on the sheet: D102, MF101, R103

Commit message: Put BUILTIN LED and resistor back on D13. Add new LED and resistor for Wink on A3.
Parts:
- added D102: RED 0603, LED_SMD:LED_0603_1608Metric_Pad1.05x0.95mm_HandSolder, symbol Device:LED
- added R103: 330R, Resistor_SMD:R_0603_1608Metric_Pad0.98x0.95mm_HandSolder, symbol Device:R
- D106: renamed from D102; footprint digikey-footprints:0805 -> LED_SMD:LED_0603_1608Metric_Pad1.05x0.95mm_HandSolder
- MF101: value PCB_GPAD_VER1 -> PCB_GPAD_VER2
- XTAL101: Cost 0.0853 -> 0.08; DK_Datasheet_Link http://www.ndk.com/images/products/catalog/c_NX3225GD-STD-C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 -> https://datasheet.lcsc.com/lcsc/1811061718_TAE-Zhejiang-Abe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; DK_Detail_Page /product-detail/en/ndk-america-inc/NX3225GD-8MHZ-STD-CRA-3/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 -> (none); Digi-Key_PN 644-1178-1-ND -> (none); Distributor 1 PN TAXM16M2GLFBET2T -> C111377; MPN NX3225GD-8MHZ-STD-CRA-3 -> TAXM16M2GLFBET2T; Manufacturer NDK America, Inc. -> TAE(Zhejiang Abel Elec)
- renumbered R103 to R112
Connections:
- net GND: now also D102.1 (K)
- net SPI_SCK: now also R103.2
- new net: D102.2 (A), R103.1
Other:
- note added: "Wink LED"

Commit message: Updateing for Version 2, 1K on BuiltinLED
Parts:
- R103: value 330R -> 1K; Distributor 1 PN C269711 -> C269704
Changed lines of the file:
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@@
     (in_bom yes) (on_board yes)
     (property "Reference" "R103" (id 0) (at 125.73 129.54 90))
-    (property "Value" "330R" (id 1) (at 123.19 130.81 90))
+    (property "Value" "1K" (id 1) (at 123.19 130.81 90))
     (property "Footprint" "Resistor_SMD:R_0603_1608Metric_Pad0.98x0.95mm_HandSolder" (id 2) (at 122.428 130.81 90)
       (effects (font (size 1.27 1.27)) hide)
@@
       (effects (font (size 1.27 1.27)) hide)
     )
-    (property "Distributor 1 PN" "C269711" (id 5) (at 120.65 130.81 90)
+    (property "Distributor 1 PN" "C269704" (id 5) (at 120.65 130.81 90)
       (effects (font (size 1.27 1.27)) hide)
     )
@@
       (effects (font (size 1.27 1.27)) hide)
     )
-    (property "Description" "0.1W ±1% 330Ω 0603 Chip Resistor - Surface Mount ROHS" (id 8) (at 120.65 130.81 0)
+    (property "Description" "0.1W ±1% 1kΩ 0603 Chip Resistor - Surface Mount ROHS" (id 8) (at 120.65 130.81 0)
       (effects (font (size 1.27 1.27)) hide)
     )
@@
     )
     (path "/9db81953-12a5-4526-8251-7f652374b37b"
-      (reference "R103") (unit 1) (value "330R") (footprint "Resistor_SMD:R_0603_1608Metric_Pad0.98x0.95mm_HandSolder")
+      (reference "R103") (unit 1) (value "1K") (footprint "Resistor_SMD:R_0603_1608Metric_Pad0.98x0.95mm_HandSolder")
     )
     (path "/00000000-0000-0000-0000-000062d57aa0"

Commit message: Add text to the UNO footprint front and back silk screen.
Parts:
- A101: footprint Module:Arduino_UNO_R3 -> GeneralPurposeAlarmDevicePCB:Arduino_UNO_R3_NoMountingHoles3D
Changed lines of the file:
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@@
     (property "Reference" "A101" (id 0) (at 165.1 104.14 0))
     (property "Value" "Arduino_UNO_R3_Shield" (id 1) (at 173.99 107.95 0))
-    (property "Footprint" "Module:Arduino_UNO_R3" (id 2) (at 191.77 133.35 0)
+    (property "Footprint" "GeneralPurposeAlarmDevicePCB:Arduino_UNO_R3_NoMountingHoles3D" (id 2) (at 191.77 133.35 0)
       (effects (font (size 1.27 1.27) italic) hide)
     )
@@
     )
     (path "/00000000-0000-0000-0000-0000634841c0"
-      (reference "A101") (unit 1) (value "Arduino_UNO_R3_Shield") (footprint "Module:Arduino_UNO_R3")
+      (reference "A101") (unit 1) (value "Arduino_UNO_R3_Shield") (footprint "GeneralPurposeAlarmDevicePCB:Arduino_UNO_R3_NoMountingHoles3D")
     )
     (path "/00000000-0000-0000-0000-000062dd8e5f/5897491e-9402-49c5-a894-b7415b30b227"

Commit message: Enlarge_ground_around_U302_Pin_19.
Changed lines of the file:
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@@
-    (stroke (width 0) (type default) (color 0 0 0 0))
-  )
-  (wire (pts (xy 229.87 31.75) (xy 209.55 31.75))
     (stroke (width 0) (type default) (color 0 0 0 0))
   )
@@
     (stroke (width 0) (type default) (color 0 0 0 0))
   )
+  (wire (pts (xy 207.01 39.37) (xy 229.87 39.37))
+    (stroke (width 0) (type default) (color 0 0 0 0))
+  )
   (wire (pts (xy 55.88 68.58) (xy 91.44 68.58))
     (stroke (width 0) (type default) (color 0 0 0 0))
@@
     (stroke (width 0) (type default) (color 0 0 0 0))
   )
+  (wire (pts (xy 209.55 31.75) (xy 229.87 31.75))
+    (stroke (width 0) (type default) (color 0 0 0 0))
+  )
   (wire (pts (xy 142.24 31.75) (xy 142.24 24.13))
     (stroke (width 0) (type default) (color 0 0 0 0))
@@
     (stroke (width 0) (type default) (color 0 0 0 0))
   )
-  (wire (pts (xy 229.87 39.37) (xy 207.01 39.37))
-    (stroke (width 0) (type default) (color 0 0 0 0))
-  )

Commit message: Make new schematic symbol and PCB symbol to correct pin numbers on JST connector. Generate new gerbers and drills.
Parts:
- removed J105: S04B-XASK-1(LF)(SN), GeneralPurposeAlarmDevicePCB:S04B-XASK-1(LF)(SN), symbol GPAD_SCH_LIB:S04B-XASK-1(LF)(SN)
- added J105: S04B-XASK-1(LF)(SN)Rev2, GeneralPurposeAlarmDevicePCB:S04B-XASK-1(LF)(SN)Rev2, symbol GPAD_SCH_LIB:S04B-XASK-1(LF)(SN)Rev2
Connections:
- net +5V: now also J105.4
- net GND: now also J105.2
- net at C113.1, R104.1: now also J105.3
- net at C114.1, R105.1: now also J105.1
Changed lines of the file:
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@@
     (stroke (width 0) (type default) (color 0 0 0 0))
   )
-  (wire (pts (xy 240.03 67.31) (xy 246.38 67.31))
-    (stroke (width 0) (type default) (color 0 0 0 0))
-  )
   (wire (pts (xy 85.09 146.05) (xy 88.9 146.05))
     (stroke (width 0) (type default) (color 0 0 0 0))
@@
     (stroke (width 0) (type default) (color 0 0 0 0))
   )
-  (wire (pts (xy 228.6 62.23) (xy 246.38 62.23))
-    (stroke (width 0) (type default) (color 0 0 0 0))
-  )
   (wire (pts (xy 72.39 102.87) (xy 66.04 102.87))
     (stroke (width 0) (type default) (color 0 0 0 0))
   )
-  (wire (pts (xy 222.25 64.77) (xy 246.38 64.77))
-    (stroke (width 0) (type default) (color 0 0 0 0))
-  )
   (wire (pts (xy 218.44 62.23) (xy 228.6 62.23))
     (stroke (width 0) (type default) (color 0 0 0 0))
@@
     (stroke (width 0) (type default) (color 0 0 0 0))
   )
+  (wire (pts (xy 228.6 62.23) (xy 245.11 62.23))
+    (stroke (width 0) (type default) (color 0 0 0 0))
+  )
   (wire (pts (xy 110.49 24.13) (xy 113.03 24.13))
     (stroke (width 0) (type default) (color 0 0 0 0))
@@
     (stroke (width 0) (type default) (color 0 0 0 0))
   )
+  (wire (pts (xy 240.03 67.31) (xy 245.11 67.31))
+    (stroke (width 0) (type default) (color 0 0 0 0))
+  )
   (wire (pts (xy 116.84 68.58) (xy 119.38 68.58))
     (stroke (width 0) (type default) (color 0 0 0 0))
@@
     (stroke (width 0) (type default) (color 0 0 0 0))
   )
+  (wire (pts (xy 222.25 59.69) (xy 245.11 59.69))
+    (stroke (width 0) (type default) (color 0 0 0 0))
+  )
   (wire (pts (xy 152.4 58.42) (xy 152.4 107.95))
     (stroke (width 0) (type default) (color 0 0 0 0))
@@
     (stroke (width 0) (type default) (color 0 0 0 0))
   )
+  (wire (pts (xy 222.25 64.77) (xy 245.11 64.77))
+    (stroke (width 0) (type default) (color 0 0 0 0))
+  )
   (wire (pts (xy 25.4 33.02) (xy 25.4 40.64))
     (stroke (width 0) (type default) (color 0 0 0 0))
@@
     (stroke (width 0) (type default) (color 0 0 0 0))
   )
-  (wire (pts (xy 222.25 59.69) (xy 246.38 59.69))
-    (stroke (width 0) (type default) (color 0 0 0 0))
-  )
   (wire (pts (xy 77.47 54.61) (xy 77.47 58.42))
     (stroke (width 0) (type default) (color 0 0 0 0))
@@
     (pin "2")
   )
-  (symbol (lib_id "GPAD_SCH_LIB:S04B-XASK-1(LF)(SN)") (at 248.92 59.69 90) (mirror x) (unit 1)
-    (in_bom yes) (on_board yes)
-    (property "Reference" "J105" (id 0) (at 252.73 59.69 90)
-      (effects (font (size 1.27 1.27)) (justify right))
-    )
-    (property "Value" "S04B-XASK-1(LF)(SN)" (id 1) (at 243.84 69.85 90)
-      (effects (font (size 1.27 1.27)) (justify right))
-    )
-    (property "Footprint" "GeneralPurposeAlarmDevicePCB:S04B-XASK-1(LF)(SN)" (id 2) (at 243.84 64.77 0)
-      (effects (font (size 1.524 1.524)) (justify left) hide)
-    )
-    (property "Datasheet" "https://www.jst-mfg.com/product/pdf/eng/eXA1.pdf" (id 3) (at 241.3 64.77 0)
-      (effects (font (size 1.524 1.524)) (justify left) hide)
-    )
-    (property "Digi-Key_PN" "455-4090-ND" (id 4) (at 238.76 64.77 0)
-      (effects (font (size 1.524 1.524)) (justify left) hide)
-    )
-    (property "MPN" "S04B-XASK-1(LF)(SN)" (id 5) (at 236.22 64.77 0)
-      (effects (font (size 1.524 1.524)) (justify left) hide)
-    )
-    (property "Category" "Connectors, Interconnects" (id 6) (at 233.68 64.77 0)
-      (effects (font (size 1.524 1.524)) (justify left) hide)
-    )
-    (property "Family" "Rectangular Connectors - Headers, Male Pins, Side Entery" (id 7) (at 231.14 64.77 0)
-      (effects (font (size 1.524 1.524)) (justify left) hide)
-    )
-    (property "Description" "CONN HEADER R/A 4POS 2.5MM" (id 8) (at 223.52 64.77 0)
-      (effects (font (size 1.524 1.524)) (justify left) hide)
-    )
-    (property "Manufacturer" "JST" (id 9) (at 220.98 64.77 0)
-      (effects (font (size 1.524 1.524)) (justify left) hide)
-    )
-    (property "Status" "Active" (id 10) (at 218.44 64.77 0)
-      (effects (font (size 1.524 1.524)) (justify left) hide)
-    )
-    (property "Distributor 1" "JLCPCB" (id 11) (at 248.92 59.69 0)
-      (effects (font (size 1.27 1.27)) hide)
-    )
-    (property "Distributor 1 PN" "C265097" (id 12) (at 248.92 59.69 0)
-      (effects (font (size 1.27 1.27)) hide)
-    )
-    (property "Distributor 2" "DigiKey  " (id 13) (at 248.92 59.69 0)
-      (effects (font (size 1.27 1.27)) hide)
-    )
-    (property "Distributor 2 PN" "455-4090-ND" (id 14) (at 252.1712 65.6844 90)
-      (effects (font (size 1.27 1.27)) (justify right) hide)
-    )
-    (property "Assembly Type" "" (id 15) (at 308.61 -189.23 0)
-      (effects (font (size 1.27 1.27)) hide)
-    )
-    (property "AssemblyType" "HAND" (id 16) (at 248.92 59.69 0)
-      (effects (font (size 1.27 1.27)) hide)
-    )
-    (property "Cost" "0.1517" (id 17) (at 248.92 59.69 0)
-      (effects (font (size 1.27 1.27)) hide)
-    )
-    (pin "1")
-    (pin "2")
-    (pin "3")
-    (pin "4")
-  )
   (symbol (lib_id "power:GND") (at 222.25 69.85 0) (unit 1)
     (in_bom yes) (on_board yes)
@@
     (pin "2")
   )
+  (symbol (lib_id "GPAD_SCH_LIB:S04B-XASK-1(LF)(SN)Rev2") (at 247.65 59.69 90) (mirror x) (unit 1)
+    (in_bom yes) (on_board yes) (fields_autoplaced)
+    (property "Reference" "J105" (id 0) (at 251.46 62.2299 90)
+      (effects (font (size 1.27 1.27)) (justify right))
+    )
+    (property "Value" "S04B-XASK-1(LF)(SN)Rev2" (id 1) (at 251.46 64.7699 90)
+      (effects (font (size 1.27 1.27)) (justify right))
+    )
+    (property "Footprint" "GeneralPurposeAlarmDevicePCB:S04B-XASK-1(LF)(SN)Rev2" (id 2) (at 242.57 64.77 0)
+      (effects (font (size 1.524 1.524)) (justify left) hide)
+    )
+    (property "Datasheet" "https://www.jst-mfg.com/product/pdf/eng/eXA1.pdf" (id 3) (at 240.03 64.77 0)
+      (effects (font (size 1.524 1.524)) (justify left) hide)
+    )
+    (property "Digi-Key_PN" "455-4090-ND" (id 4) (at 237.49 64.77 0)
+      (effects (font (size 1.524 1.524)) (justify left) hide)
+    )
+    (property "MPN" "S04B-XASK-1(LF)(SN)" (id 5) (at 234.95 64.77 0)
+      (effects (font (size 1.524 1.524)) (justify left) hide)
+    )
+    (property "Category" "Connectors, Interconnects" (id 6) (at 232.41 64.77 0)
+      (effects (font (size 1.524 1.524)) (justify left) hide)
+    )
+    (property "Family" "Rectangular Connectors - Headers, Male Pins, Side Entery" (id 7) (at 229.87 64.77 0)
+      (effects (font (size 1.524 1.524)) (justify left) hide)
+    )
+    (property "Description" "CONN HEADER R/A 4POS 2.5MM" (id 8) (at 222.25 64.77 0)
+      (effects (font (size 1.524 1.524)) (justify left) hide)
+    )
+    (property "Manufacturer" "JST" (id 9) (at 219.71 64.77 0)
+      (effects (font (size 1.524 1.524)) (justify left) hide)
+    )
+    (property "Status" "Active" (id 10) (at 217.17 64.77 0)
+      (effects (font (size 1.524 1.524)) (justify left) hide)
+    )
+    (property "Distributor 1" "JLCPCB" (id 11) (at 247.65 59.69 0)
+      (effects (font (size 1.27 1.27)) hide)
+    )
+    (property "Distributor 1 PN" "C265097" (id 12) (at 247.65 59.69 0)
+      (effects (font (size 1.27 1.27)) hide)
+    )
+    (property "Distributor 2" "DigiKey  " (id 13) (at 247.65 59.69 0)
+      (effects (font (size 1.27 1.27)) hide)
+    )
+    (property "Distributor 2 PN" "455-4090-ND" (id 14) (at 247.65 59.69 0)
+      (effects (font (size 1.27 1.27)) hide)
+    )
+    (property "Assembly Type" "HAND" (id 15) (at 247.65 59.69 0)
+      (effects (font (size 1.27 1.27)) hide)
+    )
+    (pin "1")
+    (pin "2")
+    (pin "3")
+    (pin "4")
+  )
   (symbol (lib_id "Device:R") (at 213.36 118.11 270) (unit 1)
     (in_bom yes) (on_board yes)
@@
       (reference "J103") (unit 1) (value "0.100_2Pin") (footprint "Connector_PinHeader_2.54mm:PinHeader_1x02_P2.54mm_Vertical")
     )
-    (path "/00000000-0000-0000-0000-000062d4a7fc"
-      (reference "J105") (unit 1) (value "S04B-XASK-1(LF)(SN)") (footprint "GeneralPurposeAlarmDevicePCB:S04B-XASK-1(LF)(SN)")
+    (path "/4872c0e0-8d3c-46ac-8236-411065e3473b"
+      (reference "J105") (unit 1) (value "S04B-XASK-1(LF)(SN)Rev2") (footprint "GeneralPurposeAlarmDevicePCB:S04B-XASK-1(LF)(SN)Rev2")
     )
     (path "/00000000-0000-0000-0000-000062b93801/00000000-0000-0000-0000-000062d0d90d"
