File: Hardware/GeneralPurposeAlarmDevicePCB/GeneralPurposeAlarmDevicePCB.kicad_sch (KiCad schematic)
At the start: 55 parts, among them J101 Barrel_Jack_Switch_SMT, J102 0.100_2Pin, J103 0.100_2Pin, J105 S04B-XASK-1(LF)(SN)Rev2, U101 LM7805_TO220, U102 PI_ATMEGA328P-AU-InOrder

Commit message: Add Battery Control Circuitry
Added Battery Control Circuitry schematic as well as a MOSFET to turn on and off the LCD
Parts:
- D105: MPN (none) -> LTL2R3KEK
Other:
- added sheet Battery Control (Battery_Control.kicad_sch)
- sheet LCD And I2C Interface ports: added LCDPower; removed none

Commit message: Add PCB Layout for Battery Circuitry
Also created several Capstone Specific BOMs/PDFs
Connections:
- net LCD power: now reaches U102.22 (ADC7)
- no-connect marks 2 -> 1
Changed lines of the file:
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@@
   (junction (at 154.94 24.13) (diameter 0) (color 0 0 0 0)
   )
+  (junction (at 229.87 45.72) (diameter 0) (color 0 0 0 0)
+  )
   (junction (at 209.55 31.75) (diameter 0) (color 0 0 0 0)
   )
@@
   )
   (no_connect (at 113.03 107.95))
-  (no_connect (at 113.03 100.33))
   (wire (pts (xy 104.14 170.18) (xy 99.06 170.18))
     (stroke (width 0) (type default))
@@
     (stroke (width 0) (type default))
   )
+  (wire (pts (xy 113.03 100.33) (xy 118.11 100.33))
+    (stroke (width 0) (type default))
+  )
   (wire (pts (xy 144.78 31.75) (xy 142.24 31.75))
     (stroke (width 0) (type default))
@@
     (stroke (width 0) (type default))
   )
+  (wire (pts (xy 222.25 45.72) (xy 229.87 45.72))
+    (stroke (width 0) (type default))
+  )
   (wire (pts (xy 149.86 24.13) (xy 149.86 22.86))
     (stroke (width 0) (type default))
@@
   )
   (wire (pts (xy 146.05 71.12) (xy 147.32 71.12))
+    (stroke (width 0) (type default))
+  )
+  (wire (pts (xy 229.87 45.72) (xy 231.14 45.72))
     (stroke (width 0) (type default))
   )
@@
     )
   )
+  (global_label "LCD power" (shape input) (at 118.11 100.33 0) (fields_autoplaced)
+    (effects (font (size 1.27 1.27)) (justify left))
+    (property "Intersheetrefs" "${INTERSHEET_REFS}" (at 130.195 100.33 0)
+      (effects (font (size 1.27 1.27)) (justify left) hide)
+    )
+  )
   (global_label "nCS" (shape output) (at 96.52 157.48 180) (fields_autoplaced)
     (effects (font (size 1.27 1.27)) (justify right))
@@
       (effects (font (size 1.27 1.27)) (justify right) hide)
     )
+  )
+  (global_label "LCD power" (shape input) (at 222.25 45.72 180) (fields_autoplaced)
+    (effects (font (size 1.27 1.27)) (justify right))
+    (property "Intersheetrefs" "${INTERSHEET_REFS}" (at 210.165 45.72 0)
+      (effects (font (size 1.27 1.27)) (justify right) hide)
+    )
