File: Hardware/GeneralPurposeAlarmDevicePCB/GeneralPurposeAlarmDevicePCB.kicad_sch (KiCad schematic)
At the start: 54 parts, among them J101 Barrel_Jack_Switch_SMT, J102 0.100_2Pin, J103 0.100_2Pin, J105 S04B-XASK-1(LF)(SN)Rev2, U101 LM7805_TO220, U102 PI_ATMEGA328P-AU-InOrder

Commit message: Update U301 for JLCPCB in stock, Break and then fix SCH library because of illigal character in sch symbol name.
Parts:
- J105: Cost (none) -> 0.15
- R103: MPN RMC06033301%N -> RMC06031K1%N
- R106, R107: Distributor 1 JLCPCB -> DNI
Changed lines of the file:
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@@
       (effects (font (size 1.27 1.27)) hide)
     )
-    (property "Distributor 1" "JLCPCB" (id 4) (at 148.59 31.75 90)
+    (property "Distributor 1" "DNI" (id 4) (at 148.59 31.75 90)
       (effects (font (size 1.27 1.27)) hide)
     )
@@
       (effects (font (size 1.27 1.27)) hide)
     )
-    (property "Distributor 1" "JLCPCB" (id 4) (at 185.42 34.29 90)
+    (property "Distributor 1" "DNI" (id 4) (at 185.42 34.29 90)
       (effects (font (size 1.27 1.27)) hide)
     )
@@
       (effects (font (size 1.27 1.27)) hide)
     )
+    (property "Cost" "0.15" (id 16) (at 247.65 59.69 0)
+      (effects (font (size 1.27 1.27)) hide)
+    )
     (pin "1")
     (pin "2")
@@
       (effects (font (size 1.27 1.27)) hide)
     )
-    (property "MPN" "RMC06033301%N" (id 7) (at 120.65 130.81 90)
+    (property "MPN" "RMC06031K1%N" (id 7) (at 120.65 130.81 90)
       (effects (font (size 1.27 1.27)) hide)
     )
@@
     )
     (path "/00000000-0000-0000-0000-000062b93801/00000000-0000-0000-0000-000062b96d5b"
-      (reference "R401") (unit 1) (value "330") (footprint "Resistor_SMD:R_0603_1608Metric_Pad0.98x0.95mm_HandSolder")
+      (reference "R401") (unit 1) (value "330R") (footprint "Resistor_SMD:R_0603_1608Metric_Pad0.98x0.95mm_HandSolder")
     )
     (path "/00000000-0000-0000-0000-000062b93801/00000000-0000-0000-0000-000062b96d66"
-      (reference "R402") (unit 1) (value "330") (footprint "Resistor_SMD:R_0603_1608Metric_Pad0.98x0.95mm_HandSolder")
+      (reference "R402") (unit 1) (value "330R") (footprint "Resistor_SMD:R_0603_1608Metric_Pad0.98x0.95mm_HandSolder")
     )
     (path "/00000000-0000-0000-0000-000062b93801/00000000-0000-0000-0000-000062b96d71"
-      (reference "R403") (unit 1) (value "330") (footprint "Resistor_SMD:R_0603_1608Metric_Pad0.98x0.95mm_HandSolder")
+      (reference "R403") (unit 1) (value "330R") (footprint "Resistor_SMD:R_0603_1608Metric_Pad0.98x0.95mm_HandSolder")
     )
     (path "/00000000-0000-0000-0000-000062b93801/00000000-0000-0000-0000-000062b96d7c"
-      (reference "R404") (unit 1) (value "330") (footprint "Resistor_SMD:R_0603_1608Metric_Pad0.98x0.95mm_HandSolder")
+      (reference "R404") (unit 1) (value "330R") (footprint "Resistor_SMD:R_0603_1608Metric_Pad0.98x0.95mm_HandSolder")
     )
     (path "/00000000-0000-0000-0000-000062bc4e7e/00000000-0000-0000-0000-000062be31ed"
@@
     )
     (path "/00000000-0000-0000-0000-000062dd8e5f/00000000-0000-0000-0000-000062de23f8"
-      (reference "R605") (unit 1) (value "330") (footprint "Resistor_SMD:R_0603_1608Metric_Pad0.98x0.95mm_HandSolder")
+      (reference "R605") (unit 1) (value "330R") (footprint "Resistor_SMD:R_0603_1608Metric_Pad0.98x0.95mm_HandSolder")
     )
     (path "/00000000-0000-0000-0000-000062b871ee/7008cf90-b212-49d7-8b1b-23ef20575b82"
@@
       (reference "U102") (unit 1) (value "PI_ATMEGA328P-AU-InOrder") (footprint "Package_QFP:TQFP-32_7x7mm_P0.8mm")
     )
-    (path "/00000000-0000-0000-0000-000062b871ee/00000000-0000-0000-0000-000062b90f36"
-      (reference "U301") (unit 1) (value "PCF8574AT") (footprint "Package_SO:SOIC-16W_7.5x10.3mm_P1.27mm")
+    (path "/00000000-0000-0000-0000-000062b871ee/e051ebe0-83f1-4aa8-b0c7-b7b5af8758eb"
+      (reference "U301") (unit 1) (value "PCF8574AT_3_518") (footprint "Package_SO:SOIC-16W_7.5x10.3mm_P1.27mm")
     )
     (path "/00000000-0000-0000-0000-000062b871ee/2ab4402c-7d6e-4745-b7e2-2505e19e98be"

Commit message: Add LED Standoffs to Schematic. Bump version to 2.1
Parts:
- added MF103: U_Box_V104_General_Alarm_Device_LED_Standoff, GeneralPurposeAlarmDevicePCB:U_Box_V104_General_Alarm_Device_LED_Standoff, symbol GPAD_SCH_LIB:U_Box_V104_General_Alarm_Device_LED_Standoff
Changed lines of the file:
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@@
   (title_block
     (title "GeneralPurposeAlarmDevicePCB")
-    (date "2022-11-13")
-    (rev "2.0")
+    (date "2023-03-02")
+    (rev "2.1")
     (company "PublicInvention")
     (comment 1 "GNU Affero General Public License v3.0")
@@
     (pin "2")
   )
+  (symbol (lib_id "GPAD_SCH_LIB:U_Box_V104_General_Alarm_Device_LED_Standoff") (at 115.57 50.8 0) (unit 1)
+    (in_bom yes) (on_board yes) (fields_autoplaced)
+    (property "Reference" "MF103" (id 0) (at 120.65 49.5299 0)
+      (effects (font (size 1.27 1.27)) (justify left))
+    )
+    (property "Value" "U_Box_V104_General_Alarm_Device_LED_Standoff" (id 1) (at 120.65 52.0699 0)
+      (effects (font (size 1.27 1.27)) (justify left))
+    )
+    (property "Footprint" "GeneralPurposeAlarmDevicePCB:U_Box_V104_General_Alarm_Device_LED_Standoff" (id 2) (at 115.57 50.8 0)
+      (effects (font (size 1.27 1.27)) hide)
+    )
+    (property "Datasheet" "" (id 3) (at 115.57 50.8 0)
+      (effects (font (size 1.27 1.27)) hide)
+    )
+  )
   (symbol (lib_id "Device:C") (at 228.6 74.93 0) (unit 1)
     (in_bom yes) (on_board yes)
@@
       (reference "MF102") (unit 1) (value "ENCLOSURE_GPAD_VER1") (footprint "")
     )
+    (path "/9df02aba-ac24-40d4-aded-7ee5c2a5a8e2"
+      (reference "MF103") (unit 1) (value "U_Box_V104_General_Alarm_Device_LED_Standoff") (footprint "GeneralPurposeAlarmDevicePCB:U_Box_V104_General_Alarm_Device_LED_Standoff")
+    )
     (path "/00000000-0000-0000-0000-000062b871ee/fbcd2f6c-e85f-48ea-bb94-218dde6e448f"
       (reference "MF401") (unit 1) (value "Screw_4-40_0.375_Phillips") (footprint "NA")
@@
       (reference "MF412") (unit 1) (value "Nut_4-40_Lock,_External-Tooth") (footprint "NA")
     )
+    (path "/00000000-0000-0000-0000-000062b3ac2f/ea964b5b-02f6-40ab-8892-c36a3db6b068"
+      (reference "MF601") (unit 1) (value "U_Box_V104_General_Alarm_Device_LED_Standoff") (footprint "GeneralPurposeAlarmDevicePCB:U_Box_V104_General_Alarm_Device_LED_Standoff")
+    )
+    (path "/00000000-0000-0000-0000-000062b3ac2f/da8e7b02-3ac8-446f-b0c5-b1d9f9707be2"
+      (reference "MF602") (unit 1) (value "U_Box_V104_General_Alarm_Device_LED_Standoff") (footprint "GeneralPurposeAlarmDevicePCB:U_Box_V104_General_Alarm_Device_LED_Standoff")
+    )
+    (path "/00000000-0000-0000-0000-000062b3ac2f/a2b6516e-9ff6-4381-a43b-e1824330249d"
+      (reference "MF603") (unit 1) (value "U_Box_V104_General_Alarm_Device_LED_Standoff") (footprint "GeneralPurposeAlarmDevicePCB:U_Box_V104_General_Alarm_Device_LED_Standoff")
+    )
+    (path "/00000000-0000-0000-0000-000062b3ac2f/7e8dabd8-9dd3-4f9c-89bb-fae59fdcc0f5"
+      (reference "MF604") (unit 1) (value "U_Box_V104_General_Alarm_Device_LED_Standoff") (footprint "GeneralPurposeAlarmDevicePCB:U_Box_V104_General_Alarm_Device_LED_Standoff")
+    )
+    (path "/00000000-0000-0000-0000-000062b3ac2f/420e9d6e-e67c-486c-8424-10e52e74b3ba"
+      (reference "MF605") (unit 1) (value "U_Box_V104_General_Alarm_Device_LED_Standoff") (footprint "GeneralPurposeAlarmDevicePCB:U_Box_V104_General_Alarm_Device_LED_Standoff")
+    )
     (path "/00000000-0000-0000-0000-000062b3ac2f/00000000-0000-0000-0000-000062d15bd1"

Commit message: Update Manufacturing test with results of testing SN16-SN21. Make R103 DNI to unload the SPI nCS line.
Parts:
- R103: value 1K -> DNI
Changed lines of the file:
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@@
   (title_block
     (title "GeneralPurposeAlarmDevicePCB")
-    (date "2023-03-02")
-    (rev "2.1")
+    (date "2023-04-25")
+    (rev "2.2")
     (company "PublicInvention")
     (comment 1 "GNU Affero General Public License v3.0")
@@
     (in_bom yes) (on_board yes)
     (property "Reference" "R103" (id 0) (at 125.73 129.54 90))
-    (property "Value" "1K" (id 1) (at 123.19 130.81 90))
+    (property "Value" "DNI" (id 1) (at 123.19 130.81 90))
     (property "Footprint" "Resistor_SMD:R_0603_1608Metric_Pad0.98x0.95mm_HandSolder" (id 2) (at 122.428 130.81 90)
       (effects (font (size 1.27 1.27)) hide)
@@
     )
     (path "/9db81953-12a5-4526-8251-7f652374b37b"
-      (reference "R103") (unit 1) (value "1K") (footprint "Resistor_SMD:R_0603_1608Metric_Pad0.98x0.95mm_HandSolder")
+      (reference "R103") (unit 1) (value "DNI") (footprint "Resistor_SMD:R_0603_1608Metric_Pad0.98x0.95mm_HandSolder")
     )
     (path "/00000000-0000-0000-0000-000062d57aa0"
