File: Hardware/GeneralPurposeAlarmDevicePCB/SPI Peripherial.kicad_sch (KiCad schematic)
At the start: 6 parts, among them J401 RJ12_6P6C_HORZ

Commit message: Update U301 for JLCPCB in stock, Break and then fix SCH library because of illigal character in sch symbol name.
Parts:
- R401, R402, R403, R404: value 330 -> 330R
Changed lines of the file:
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@@
     (in_bom yes) (on_board yes)
     (property "Reference" "R401" (id 0) (at 130.81 95.25 90))
-    (property "Value" "330" (id 1) (at 132.08 97.79 90))
+    (property "Value" "330R" (id 1) (at 132.08 97.79 90))
     (property "Footprint" "Resistor_SMD:R_0603_1608Metric_Pad0.98x0.95mm_HandSolder" (id 2) (at 132.08 98.552 90)
       (effects (font (size 1.27 1.27)) hide)
@@
     (in_bom yes) (on_board yes)
     (property "Reference" "R402" (id 0) (at 140.97 101.6 90))
-    (property "Value" "330" (id 1) (at 142.24 104.14 90))
+    (property "Value" "330R" (id 1) (at 142.24 104.14 90))
     (property "Footprint" "Resistor_SMD:R_0603_1608Metric_Pad0.98x0.95mm_HandSolder" (id 2) (at 142.24 104.902 90)
       (effects (font (size 1.27 1.27)) hide)
@@
     (in_bom yes) (on_board yes)
     (property "Reference" "R403" (id 0) (at 152.4 107.95 90))
-    (property "Value" "330" (id 1) (at 153.67 110.49 90))
+    (property "Value" "330R" (id 1) (at 153.67 110.49 90))
     (property "Footprint" "Resistor_SMD:R_0603_1608Metric_Pad0.98x0.95mm_HandSolder" (id 2) (at 153.67 111.252 90)
       (effects (font (size 1.27 1.27)) hide)
@@
     (in_bom yes) (on_board yes)
     (property "Reference" "R404" (id 0) (at 184.15 118.11 90))
-    (property "Value" "330" (id 1) (at 185.42 120.65 90))
+    (property "Value" "330R" (id 1) (at 185.42 120.65 90))
     (property "Footprint" "Resistor_SMD:R_0603_1608Metric_Pad0.98x0.95mm_HandSolder" (id 2) (at 185.42 121.412 90)
       (effects (font (size 1.27 1.27)) hide)
