File: Hardware/GeneralPurposeAlarmDevicePCB/ESP32.kicad_sch (KiCad schematic)
At the start: 4 parts

Commit message: updated PCB1
Connections:
- net SCL: now also U?.36 (IO22); no longer U?.22 (SDI/SD1)
- net SDA: now also U?.33 (IO21); no longer U?.21 (SDO/SD0)
- net Tone: now also U?.26 (IO4); no longer U?.33 (IO21)
Changed lines of the file:
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@@
+    (stroke (width 0) (type default) (color 0 0 0 0))
+  )
+  (wire (pts (xy 147.32 57.15) (xy 153.67 57.15))
     (stroke (width 0) (type default) (color 0 0 0 0))
   )
@@
     (stroke (width 0) (type default) (color 0 0 0 0))
   )
-  (wire (pts (xy 114.3 77.47) (xy 116.84 77.47))
+  (wire (pts (xy 147.32 85.09) (xy 153.67 85.09))
     (stroke (width 0) (type default) (color 0 0 0 0))
   )
@@
     (stroke (width 0) (type default) (color 0 0 0 0))
   )
-  (wire (pts (xy 114.3 80.01) (xy 116.84 80.01))
-    (stroke (width 0) (type default) (color 0 0 0 0))
-  )
   (wire (pts (xy 101.6 41.91) (xy 101.6 46.99))
     (stroke (width 0) (type default) (color 0 0 0 0))
@@
     )
   )
-  (global_label "SCL" (shape input) (at 114.3 80.01 180) (fields_autoplaced)
-    (effects (font (size 1.27 1.27)) (justify right))
-    (property "Intersheet References" "${INTERSHEET_REFS}" (id 0) (at 326.39 -66.04 0)
-      (effects (font (size 1.27 1.27)) (justify left) hide)
+  (global_label "SDA" (shape input) (at 153.67 82.55 0) (fields_autoplaced)
+    (effects (font (size 1.27 1.27)) (justify left))
+    (property "Intersheet References" "${INTERSHEET_REFS}" (id 0) (at -58.42 -60.96 0)
+      (effects (font (size 1.27 1.27)) (justify right) hide)
+    )
+  )
+  (global_label "SCL" (shape input) (at 153.67 85.09 0) (fields_autoplaced)
+    (effects (font (size 1.27 1.27)) (justify left))
+    (property "Intersheet References" "${INTERSHEET_REFS}" (id 0) (at -58.42 -60.96 0)
+      (effects (font (size 1.27 1.27)) (justify right) hide)
     )
   )
@@
     )
   )
-  (global_label "Tone" (shape output) (at 153.67 82.55 0) (fields_autoplaced)
+  (global_label "Light4" (shape output) (at 153.67 69.85 0) (fields_autoplaced)
     (effects (font (size 1.27 1.27)) (justify left))
-    (property "Intersheet References" "${INTERSHEET_REFS}" (id 0) (at 327.66 -55.88 0)
+    (property "Intersheet References" "${INTERSHEET_REFS}" (id 0) (at 327.66 -73.66 0)
       (effects (font (size 1.27 1.27)) (justify left) hide)
     )
   )
-  (global_label "Light4" (shape output) (at 153.67 69.85 0) (fields_autoplaced)
+  (global_label "Tone" (shape output) (at 153.67 57.15 0) (fields_autoplaced)
     (effects (font (size 1.27 1.27)) (justify left))
-    (property "Intersheet References" "${INTERSHEET_REFS}" (id 0) (at 327.66 -73.66 0)
+    (property "Intersheet References" "${INTERSHEET_REFS}" (id 0) (at 327.66 -81.28 0)
       (effects (font (size 1.27 1.27)) (justify left) hide)
     )
@@
     )
   )
-  (global_label "SDA" (shape input) (at 114.3 77.47 180) (fields_autoplaced)
-    (effects (font (size 1.27 1.27)) (justify right))
-    (property "Intersheet References" "${INTERSHEET_REFS}" (id 0) (at 326.39 -66.04 0)
-      (effects (font (size 1.27 1.27)) (justify left) hide)
-    )
-  )

Commit message: updated PCB
Parts:
- removed D?: RED 0603, LED_SMD:LED_0603_1608Metric_Pad1.05x0.95mm_HandSolder, symbol Device:LED
- removed R? (x2): 330R, Resistor_SMD:R_0603_1608Metric_Pad0.98x0.95mm_HandSolder, symbol Device:R
- removed U?: ESP32-WROOM-32, RF_Module:ESP32-WROOM-32, symbol RF_Module:ESP32-WROOM-32
- added D?: RED 0603, LED_SMD:LED_0603_1608Metric_Pad1.05x0.95mm_HandSolder, symbol Device:LED
- added R? (x2): 330R, Resistor_SMD:R_0603_1608Metric_Pad0.98x0.95mm_HandSolder, symbol Device:R
- added U?: ESP32-WROOM-32, RF_Module:ESP32-WROOM-32, symbol RF_Module:ESP32-WROOM-32
Connections:
- net Attenuate: now also U?.16 (IO13)
- net CIPO: now also U?.31 (IO19)
- net COPI: now also U?.37 (IO23)
- net ControllerRX: now also U?.34 (RXD0/IO3)
- net ControllerTX: now also U?.35 (TXD0/IO1)
- net GND: now also D?.1 (K), U?.1 (GND), U?.15 (GND), U?.38 (GND), U?.39 (GND)
- net GPIO16: now also U?.27 (IO16)
- net GPIO17: now also U?.28 (IO17)
- net Light0: now also U?.10 (IO25)
- net Light1: now also U?.11 (IO26)
- net Light2: now also U?.12 (IO27)
- net Light3: now also U?.13 (IO14)
- net Light4: now also U?.23 (IO15)
- net PC0: now also U?.6 (IO34)
- net PC1: now also U?.7 (IO35)
- net PC2: now also U?.8 (IO32)
- net PC3: now also R?.2, U?.9 (IO33)
- net SCL: now also U?.36 (IO22)
- net SDA: now also U?.33 (IO21)
- net SPI_SCK: now also U?.30 (IO18)
- net Switch_Mute: now also U?.14 (IO12)
- net Tone: now also U?.26 (IO4)
- net Vin: now also U?.2 (VDD)
- net nCS: now also U?.29 (IO5)
- net nRESET: now also R?.1
- new net: D?.2 (A), R?.1
- new net: R?.2, U?.3 (EN)
- no-connect marks 0 -> 8
