File: Hardware/GeneralPurposeAlarmDevicePCB/Battery_Control.kicad_sch (KiCad schematic)
At the start: 16 parts, among them J703 BATT_JST, J703 BATT_Solder, U701 MCP73833

Commit message: Add PCB Layout for Battery Circuitry
Also created several Capstone Specific BOMs/PDFs
Parts:
- removed J703: BATT_Solder, Connector_PinSocket_2.54mm:PinSocket_1x02_P2.54mm_Vertical, symbol Connector_Generic:Conn_01x02
- renumbered R110 to R1, R110 to R2
Other:
- company: (none) -> PublicInvention
- title: (none) -> GeneralPurposeAlarmDevicePCB
- moved on the sheet: BT701, C702, D106, D701, D702, D704, J703, R1, R109, R110, R2, R704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
