File: Hardware/GeneralPurposeAlarmDevicePCB/LCD And I2C Interface.kicad_sch (KiCad schematic)
At the start: 31 parts, among them Q301 BSS138, U301 PCF8574AT, U302 LCD_20x4_Character-GPAD_SCH_L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

Commit message: Update PCB for version 2. Update enclosure drawing to reflect the V1 enclosure assembly.
Parts:
- added R312: 4K7, Resistor_SMD:R_0603_1608Metric_Pad0.98x0.95mm_HandSolder, symbol Device:R
- U301: footprint Package_SO:SOIC-16W_5.3x10.2mm_P1.27mm -> Package_SO:SOIC-16W_7.5x10.3mm_P1.27mm
Connections:
- net at R311.1, U301.7 (P3): now also R312.2; no longer Q301.1 (G)
- new net: Q301.1 (G), R312.1
Changed lines of the file:
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@@
     (title "GeneralPurposeAlarmDevicePCB")
     (date "2022-11-13")
-    (rev "1.2")
+    (rev "2.0")
     (company "PublicInvention")
     (comment 1 "GNU Affero General Public License v3.0")
@@
   (junction (at 195.58 40.64) (diameter 0) (color 0 0 0 0)
   )
+  (junction (at 203.2 106.68) (diameter 0) (color 0 0 0 0)
+  )
   (junction (at 133.35 82.55) (diameter 0) (color 0 0 0 0)
   )
@@
   (junction (at 195.58 52.07) (diameter 0) (color 0 0 0 0)
   )
-  (junction (at 203.2 104.14) (diameter 0) (color 0 0 0 0)
-  )
   (junction (at 198.12 59.69) (diameter 0) (color 0 0 0 0)
   )
@@
     (stroke (width 0) (type default) (color 0 0 0 0))
   )
+  (wire (pts (xy 203.2 106.68) (xy 204.47 106.68))
+    (stroke (width 0) (type default) (color 0 0 0 0))
+  )
   (wire (pts (xy 125.73 99.06) (xy 125.73 101.6))
     (stroke (width 0) (type default) (color 0 0 0 0))
@@
     (stroke (width 0) (type default) (color 0 0 0 0))
   )
+  (wire (pts (xy 212.09 106.68) (xy 213.36 106.68))
+    (stroke (width 0) (type default) (color 0 0 0 0))
+  )
   (wire (pts (xy 116.84 52.07) (xy 156.21 52.07))
     (stroke (width 0) (type default) (color 0 0 0 0))
@@
     (stroke (width 0) (type default) (color 0 0 0 0))
   )
+  (wire (pts (xy 213.36 104.14) (xy 213.36 106.68))
+    (stroke (width 0) (type default) (color 0 0 0 0))
+  )
   (wire (pts (xy 175.26 62.23) (xy 170.18 62.23))
     (stroke (width 0) (type default) (color 0 0 0 0))
@@
   )
   (wire (pts (xy 88.9 59.69) (xy 88.9 52.07))
-    (stroke (width 0) (type default) (color 0 0 0 0))
-  )
-  (wire (pts (xy 213.36 104.14) (xy 203.2 104.14))
     (stroke (width 0) (type default) (color 0 0 0 0))
   )
@@
     (property "Reference" "U301" (id 0) (at 147.32 60.96 0))
     (property "Value" "PCF8574AT" (id 1) (at 149.86 64.77 0))
-    (property "Footprint" "Package_SO:SOIC-16W_5.3x10.2mm_P1.27mm" (id 2) (at 156.21 85.09 0)
+    (property "Footprint" "Package_SO:SOIC-16W_7.5x10.3mm_P1.27mm" (id 2) (at 156.21 85.09 0)
       (effects (font (size 1.27 1.27)) hide)
     )
@@
     (pin "9")
   )
+  (symbol (lib_id "Device:R") (at 208.28 106.68 270) (unit 1)
+    (in_bom yes) (on_board yes)
+    (property "Reference" "R312" (id 0) (at 207.01 104.14 90))
+    (property "Value" "4K7" (id 1) (at 208.28 110.49 90))
+    (property "Footprint" "Resistor_SMD:R_0603_1608Metric_Pad0.98x0.95mm_HandSolder" (id 2) (at 208.28 104.902 90)
+      (effects (font (size 1.27 1.27)) hide)
+    )
+    (property "Datasheet" "~" (id 3) (at 208.28 106.68 0)
+      (effects (font (size 1.27 1.27)) hide)
+    )
+    (property "Distributor 1" "JLCPCB" (id 4) (at 208.28 106.68 90)
+      (effects (font (size 1.27 1.27)) hide)
+    )
+    (property "Distributor 1 PN" "C269713" (id 5) (at 208.28 106.68 90)
+      (effects (font (size 1.27 1.27)) hide)
+    )
+    (property "Manufacturer" "TyoHM" (id 6) (at 208.28 106.68 90)
+      (effects (font (size 1.27 1.27)) hide)
+    )
+    (property "MPN" "RMC 0603 4K7 F N" (id 7) (at 208.28 106.68 90)
+      (effects (font (size 1.27 1.27)) hide)
+    )
+    (property "Description" "1W ±1% 4.7kΩ 0603 Chip Resistor - Surface Mount ROHS" (id 8) (at 208.28 106.68 0)
+      (effects (font (size 1.27 1.27)) hide)
+    )
+    (property "AssemblyType" "SMT" (id 9) (at 208.28 106.68 0)
+      (effects (font (size 1.27 1.27)) hide)
+    )
+    (property "Cost" "0.0015" (id 10) (at 208.28 106.68 0)
+      (effects (font (size 1.27 1.27)) hide)
+    )
+    (pin "1")
+    (pin "2")
+  )
   (symbol (lib_id "GPAD_SCH_LIB:Nut_4-40_Lock,_External-Tooth") (at 55.88 156.21 0) (unit 1)

Commit message: Update LCD footprint for larger holes. Ground LCD holes.
Connections:
- net GND: now also U302.17 (MH1), U302.18 (MH2), U302.19 (MH3), U302.20 (MH4)
Other:
- note removed: "Backlight transistor gate(base) to PCF8547 pin 7 P3. If add base resistor can use MMBT2222 for transistor."
Changed lines of the file:
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@@
   (junction (at 185.42 52.07) (diameter 0) (color 0 0 0 0)
   )
+  (junction (at 196.85 73.66) (diameter 0) (color 0 0 0 0)
+  )
   (junction (at 185.42 97.79) (diameter 0) (color 0 0 0 0)
   )
@@
   (junction (at 107.95 52.07) (diameter 0) (color 0 0 0 0)
   )
+  (junction (at 196.85 68.58) (diameter 0) (color 0 0 0 0)
+  )
   (junction (at 195.58 52.07) (diameter 0) (color 0 0 0 0)
   )
@@
   (junction (at 203.2 40.64) (diameter 0) (color 0 0 0 0)
   )
+  (junction (at 196.85 71.12) (diameter 0) (color 0 0 0 0)
+  )
   (junction (at 167.64 52.07) (diameter 0) (color 0 0 0 0)
   )
@@
     (stroke (width 0) (type default) (color 0 0 0 0))
   )
+  (wire (pts (xy 196.85 73.66) (xy 199.39 73.66))
+    (stroke (width 0) (type default) (color 0 0 0 0))
+  )
+  (wire (pts (xy 195.58 66.04) (xy 196.85 66.04))
+    (stroke (width 0) (type default) (color 0 0 0 0))
+  )
   (wire (pts (xy 97.79 59.69) (xy 97.79 52.07))
     (stroke (width 0) (type default) (color 0 0 0 0))
@@
     (stroke (width 0) (type default) (color 0 0 0 0))
   )
+  (wire (pts (xy 196.85 71.12) (xy 196.85 73.66))
+    (stroke (width 0) (type default) (color 0 0 0 0))
+  )
   (wire (pts (xy 171.45 82.55) (xy 171.45 106.68))
     (stroke (width 0) (type default) (color 0 0 0 0))
@@
     (stroke (width 0) (type default) (color 0 0 0 0))
   )
+  (wire (pts (xy 199.39 73.66) (xy 199.39 76.2))
+    (stroke (width 0) (type default) (color 0 0 0 0))
+  )
   (wire (pts (xy 171.45 77.47) (xy 171.45 64.77))
     (stroke (width 0) (type default) (color 0 0 0 0))
@@
     (stroke (width 0) (type default) (color 0 0 0 0))
   )
+  (wire (pts (xy 196.85 66.04) (xy 196.85 68.58))
+    (stroke (width 0) (type default) (color 0 0 0 0))
+  )
   (wire (pts (xy 175.26 82.55) (xy 173.99 82.55))
     (stroke (width 0) (type default) (color 0 0 0 0))
@@
     (stroke (width 0) (type default) (color 0 0 0 0))
   )
+  (wire (pts (xy 196.85 68.58) (xy 196.85 71.12))
+    (stroke (width 0) (type default) (color 0 0 0 0))
+  )
   (wire (pts (xy 226.06 55.88) (xy 226.06 50.8))
     (stroke (width 0) (type default) (color 0 0 0 0))
@@
     (stroke (width 0) (type default) (color 0 0 0 0))
   )
+  (wire (pts (xy 195.58 68.58) (xy 196.85 68.58))
+    (stroke (width 0) (type default) (color 0 0 0 0))
+  )
   (wire (pts (xy 133.35 82.55) (xy 107.95 82.55))
     (stroke (width 0) (type default) (color 0 0 0 0))
@@
     (stroke (width 0) (type default) (color 0 0 0 0))
   )
+  (wire (pts (xy 195.58 71.12) (xy 196.85 71.12))
+    (stroke (width 0) (type default) (color 0 0 0 0))
+  )
   (wire (pts (xy 138.43 80.01) (xy 116.84 80.01))
     (stroke (width 0) (type default) (color 0 0 0 0))
@@
   )
   (wire (pts (xy 156.21 67.31) (xy 156.21 52.07))
+    (stroke (width 0) (type default) (color 0 0 0 0))
+  )
+  (wire (pts (xy 195.58 73.66) (xy 196.85 73.66))
     (stroke (width 0) (type default) (color 0 0 0 0))
   )
@@
     (effects (font (size 1.27 1.27)) (justify left bottom))
   )
-  (text "Backlight transistor gate(base) to PCF8547 pin 7 P3.\nIf add base resistor can use MMBT2222 for transistor."
-    (at 154.94 139.7 0)
-    (effects (font (size 1.27 1.27)) (justify left bottom))
-  )
   (label "Vcc_LCD" (at 232.41 40.64 0)
     (effects (font (size 1.27 1.27)) (justify left bottom))
@@
     (pin "15")
     (pin "16")
+    (pin "17")
+    (pin "18")
+    (pin "19")
     (pin "2")
+    (pin "20")
     (pin "3")
     (pin "4")
@@
     )
   )
+  (symbol (lib_id "power:GND") (at 199.39 76.2 0) (unit 1)
+    (in_bom yes) (on_board yes)
+    (property "Reference" "#PWR0126" (id 0) (at 199.39 82.55 0)
+      (effects (font (size 1.27 1.27)) hide)
+    )
+    (property "Value" "GND" (id 1) (at 199.517 80.5942 0))
+    (property "Footprint" "" (id 2) (at 199.39 76.2 0)
+      (effects (font (size 1.27 1.27)) hide)
+    )
+    (property "Datasheet" "" (id 3) (at 199.39 76.2 0)
+      (effects (font (size 1.27 1.27)) hide)
+    )
+    (pin "1")
+  )
   (symbol (lib_id "GPAD_SCH_LIB:Nut_4-40_Lock,_External-Tooth") (at 127 156.21 0) (unit 1)

Commit message: Update U301 for JLCPCB in stock, Break and then fix SCH library because of illigal character in sch symbol name.
Parts:
- removed U301: PCF8574AT, Package_SO:SOIC-16W_7.5x10.3mm_P1.27mm, symbol Interface_Expansion:PCF8574A
- added U301: PCF8574AT_3_518, Package_SO:SOIC-16W_7.5x10.3mm_P1.27mm, symbol GPAD_SCH_LIB:PCF8574AT_3_518
- R306, R308: Distributor 1 JLCPCB -> DNI
- U302: Distributor 1 Aliexpress -> eBay Aliexpress; Distributor 1 PN https://www.aliexpress.com/item/3256803213374992.html -> 403534100457; Distributor 2 Amazon -> Amazon / Aliexpress; Distributor 2 PN https://www.amazon.com/GeeekPi-Interface-Adapter-Backlight-Raspberry/dp/B07QLRD3TM/ref=sr_1_2 -> https://www.amazon.com/GeeekPi-Interface-Adapter-Backlight-Raspberry/dp/B07QLRD3TM/ref=sr_1_2 / https://www.aliexpress.com/item/3256803213374992.html
Connections:
- net GND: now also U301.8 (VSS)
- net SCL: now also U301.14 (SCL)
- net SDA: now also U301.15 (SDA)
- net Vcc_LCD: now also U301.16 (VDD)
- net at R303.1, R309.1: now also U301.1 (A0)
- net at U302.12 (DB5): now also U301.10 (P5)
- net at U302.13 (DB6): now also U301.11 (P6)
- net at U302.14 (DB7): now also U301.12 (P7)
- net at R304.1, TP402.1: now also U301.13 (~{INT})
- net at R302.1, R307.1: now also U301.2 (A1)
- net at R301.1, R305.1: now also U301.3 (A2)
- net at U302.4 (RS): now also U301.4 (P0)
- net at U302.5 (R/W): now also U301.5 (P1)
- net at U302.6 (E): now also U301.6 (P2)
- net at R311.1, R312.2: now also U301.7 (P3)
- net at U302.11 (DB4): now also U301.9 (P4)
Changed lines of the file:
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@@
     (pin "1")
-  )
-  (symbol (lib_id "Interface_Expansion:PCF8574A") (at 156.21 85.09 0) (unit 1)
-    (in_bom yes) (on_board yes)
-    (property "Reference" "U301" (id 0) (at 147.32 60.96 0))
-    (property "Value" "PCF8574AT" (id 1) (at 149.86 64.77 0))
-    (property "Footprint" "Package_SO:SOIC-16W_7.5x10.3mm_P1.27mm" (id 2) (at 156.21 85.09 0)
-      (effects (font (size 1.27 1.27)) hide)
-    )
-    (property "Datasheet" "http://www.nxp.com/documents/data_sheet/PCF8574_PCF8574A.pdf" (id 3) (at 156.21 85.09 0)
-      (effects (font (size 1.27 1.27)) hide)
-    )
-    (property "Distributor 1" "JLCPCB" (id 4) (at 156.21 85.09 0)
-      (effects (font (size 1.27 1.27)) hide)
-    )
-    (property "Distributor 1 PN" "C83193" (id 5) (at 156.21 85.09 0)
-      (effects (font (size 1.27 1.27)) hide)
-    )
-    (property "Manufacturer" "NXP Semicon" (id 6) (at 156.21 85.09 0)
-      (effects (font (size 1.27 1.27)) hide)
-    )
-    (property "Description" "Remote 8-bit I/O expander for I2C-bus with interrupt" (id 7) (at 156.21 85.09 0)
-      (effects (font (size 1.27 1.27)) hide)
-    )
-    (property "MPN" "PCF8574AT/3,512" (id 8) (at 156.21 85.09 0)
-      (effects (font (size 1.27 1.27)) hide)
-    )
-    (property "AssemblyType" "SMT" (id 9) (at 156.21 85.09 0)
-      (effects (font (size 1.27 1.27)) hide)
-    )
-    (property "Cost" "0.6414" (id 10) (at 156.21 85.09 0)
-      (effects (font (size 1.27 1.27)) hide)
-    )
-    (pin "1")
-    (pin "10")
-    (pin "11")
-    (pin "12")
-    (pin "13")
-    (pin "14")
-    (pin "15")
-    (pin "16")
-    (pin "2")
-    (pin "3")
-    (pin "4")
-    (pin "5")
-    (pin "6")
-    (pin "7")
-    (pin "8")
-    (pin "9")
   )
   (symbol (lib_id "Device:R") (at 107.95 63.5 180) (unit 1)
@@
       (effects (font (size 1.27 1.27)) hide)
     )
-    (property "Distributor 1" "JLCPCB" (id 4) (at 226.06 59.69 90)
+    (property "Distributor 1" "DNI" (id 4) (at 226.06 59.69 90)
       (effects (font (size 1.27 1.27)) hide)
     )
@@
       (effects (font (size 1.27 1.27)) hide)
     )
-    (property "Distributor 1" "JLCPCB" (id 4) (at 226.06 72.39 90)
+    (property "Distributor 1" "DNI" (id 4) (at 226.06 72.39 90)
       (effects (font (size 1.27 1.27)) hide)
     )
@@
       (effects (font (size 1.27 1.27)) hide)
     )
-    (property "Distributor 1" "Aliexpress" (id 4) (at 157.988 94.996 0)
-      (effects (font (size 1.27 1.27)) hide)
-    )
-    (property "Distributor 1 PN" "https://www.aliexpress.com/item/3256803213374992.html" (id 5) (at 182.88 97.536 0)
-      (effects (font (size 1.27 1.27)) hide)
-    )
-    (property "Distributor 2" "Amazon" (id 6) (at 156.972 100.584 0)
-      (effects (font (size 1.27 1.27)) hide)
-    )
-    (property "Distributor 2 PN" "https://www.amazon.com/GeeekPi-Interface-Adapter-Backlight-Raspberry/dp/B07QLRD3TM/ref=sr_1_2" (id 7) (at 205.486 102.87 0)
+    (property "Distributor 1" "eBay   Aliexpress" (id 4) (at 157.988 94.996 0)
+      (effects (font (size 1.27 1.27)) hide)
+    )
+    (property "Distributor 1 PN" "403534100457 " (id 5) (at 182.88 97.536 0)
+      (effects (font (size 1.27 1.27)) hide)
+    )
+    (property "Distributor 2" "Amazon  / Aliexpress" (id 6) (at 156.972 100.584 0)
+      (effects (font (size 1.27 1.27)) hide)
+    )
+    (property "Distributor 2 PN" "https://www.amazon.com/GeeekPi-Interface-Adapter-Backlight-Raspberry/dp/B07QLRD3TM/ref=sr_1_2 /  https://www.aliexpress.com/item/3256803213374992.html" (id 7) (at 205.486 102.87 0)
       (effects (font (size 1.27 1.27)) hide)
     )
@@
     (pin "1")
   )
+  (symbol (lib_id "GPAD_SCH_LIB:PCF8574AT_3_518") (at 156.21 85.09 0) (unit 1)
+    (in_bom yes) (on_board yes)
+    (property "Reference" "U301" (id 0) (at 149.86 63.5 0)
+      (effects (font (size 1.27 1.27)) (justify left))
+    )
+    (property "Value" "PCF8574AT_3_518" (id 1) (at 137.16 66.04 0)
+      (effects (font (size 1.27 1.27)) (justify left))
+    )
+    (property "Footprint" "Package_SO:SOIC-16W_7.5x10.3mm_P1.27mm" (id 2) (at 156.21 85.09 0)
+      (effects (font (size 1.27 1.27)) hide)
+    )
+    (property "Datasheet" "https://datasheet.lcsc.com/lcsc/1811151526_NXP-Semicon-PCF8574AT-3-518_C86832.pdf" (id 3) (at 156.21 85.09 0)
+      (effects (font (size 1.27 1.27)) hide)
+    )
+    (property "AssemblyType" "SMT" (id 4) (at 156.21 85.09 0)
+      (effects (font (size 1.27 1.27)) hide)
+    )
+    (property "Cost" "1.87" (id 5) (at 156.21 85.09 0)
+      (effects (font (size 1.27 1.27)) hide)
+    )
+    (property "Distributor 1" "JLCPCB" (id 6) (at 156.21 85.09 0)
+      (effects (font (size 1.27 1.27)) hide)
+    )
+    (property "Distributor 1 PN" "C86832" (id 7) (at 156.21 85.09 0)
+      (effects (font (size 1.27 1.27)) hide)
+    )
+    (property "MPN" "PCF8574AT_3_518" (id 8) (at 156.21 85.09 0)
+      (effects (font (size 1.27 1.27)) hide)
+    )
+    (pin "1")
+    (pin "10")
+    (pin "11")
+    (pin "12")
+    (pin "13")
+    (pin "14")
+    (pin "15")
+    (pin "16")
+    (pin "2")
+    (pin "3")
+    (pin "4")
+    (pin "5")
+    (pin "6")
+    (pin "7")
+    (pin "8")
+    (pin "9")
+  )
   (symbol (lib_id "GPAD_SCH_LIB:Spacer_0.0182x0.125 inch") (at 125.73 138.43 0) (unit 1)
