File: Hardware/GeneralPurposeAlarmDevicePCB/LCD And I2C Interface.kicad_sch (KiCad schematic)
At the start: 32 parts, among them Q301 BSS138, U301 PCF8574AT_3_518, U302 LCD_20x4_Character-GPAD_SCH_L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

Commit message: Fix schematic broken by the "/" in the hex nut.
Parts:
- removed MF403, MF406, MF409, MF412: Nut_4-40_3/16, symbol GPAD_SCH_LIB:Nut_4-40_3/16
- added MF403, MF406, MF409, MF412: Nut_4-40_0.1875, symbol GPAD_SCH_LIB:Nut_4-40_0.1875
