File: Hardware/GeneralPurposeAlarmDevicePCB/AlarmAudio.kicad_sch (KiCad schematic)
At the start: 14 parts, among them J601 22-23-2021, Q601 MMBT2222A-7-F, Q602 MMBT2907ALT1G

Commit message: Update PCB for version 2. Update enclosure drawing to reflect the V1 enclosure assembly.
Parts:
- added J602: 22-23-2021, Connector_Molex:Molex_KK-254_AE-6410-02A_1x02_P2.54mm_Vertical, symbol GPAD_SCH_LIB:22-23-2021
Connections:
- net GND: now also J602.2
- net Switch_Mute: now also J602.1
Changed lines of the file:
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@@
     (title "GeneralPurposeAlarmDevicePCB")
     (date "2022-11-13")
-    (rev "1.2")
+    (rev "2.0")
     (company "PublicInvention")
     (comment 1 "GNU Affero General Public License v3.0")
@@
   (junction (at 101.6 48.26) (diameter 0) (color 0 0 0 0)
   )
+  (junction (at 74.93 118.11) (diameter 0) (color 0 0 0 0)
+  )
   (junction (at 123.19 71.12) (diameter 0) (color 0 0 0 0)
   )
@@
     (stroke (width 0) (type default) (color 0 0 0 0))
   )
+  (wire (pts (xy 74.93 139.7) (xy 77.47 139.7))
+    (stroke (width 0) (type default) (color 0 0 0 0))
+  )
   (wire (pts (xy 102.87 90.17) (xy 110.49 90.17))
     (stroke (width 0) (type default) (color 0 0 0 0))
@@
     (stroke (width 0) (type default) (color 0 0 0 0))
   )
+  (wire (pts (xy 74.93 118.11) (xy 81.28 118.11))
+    (stroke (width 0) (type default) (color 0 0 0 0))
+  )
   (wire (pts (xy 93.98 118.11) (xy 95.25 118.11))
     (stroke (width 0) (type default) (color 0 0 0 0))
@@
     (stroke (width 0) (type default) (color 0 0 0 0))
   )
-  (wire (pts (xy 64.77 118.11) (xy 81.28 118.11))
+  (wire (pts (xy 77.47 137.16) (xy 74.93 137.16))
+    (stroke (width 0) (type default) (color 0 0 0 0))
+  )
+  (wire (pts (xy 64.77 118.11) (xy 74.93 118.11))
     (stroke (width 0) (type default) (color 0 0 0 0))
   )
@@
     (stroke (width 0) (type default) (color 0 0 0 0))
   )
+  (wire (pts (xy 74.93 139.7) (xy 74.93 142.24))
+    (stroke (width 0) (type default) (color 0 0 0 0))
+  )
   (wire (pts (xy 62.23 134.62) (xy 62.23 137.16))
     (stroke (width 0) (type default) (color 0 0 0 0))
@@
   )
   (wire (pts (xy 102.87 71.12) (xy 110.49 71.12))
+    (stroke (width 0) (type default) (color 0 0 0 0))
+  )
+  (wire (pts (xy 74.93 118.11) (xy 74.93 137.16))
     (stroke (width 0) (type default) (color 0 0 0 0))
   )
@@
     (pin "2")
   )
+  (symbol (lib_id "power:GND") (at 74.93 142.24 0) (unit 1)
+    (in_bom yes) (on_board yes)
+    (property "Reference" "#PWR0118" (id 0) (at 74.93 148.59 0)
+      (effects (font (size 1.27 1.27)) hide)
+    )
+    (property "Value" "GND" (id 1) (at 75.057 146.6342 0))
+    (property "Footprint" "" (id 2) (at 74.93 142.24 0)
+      (effects (font (size 1.27 1.27)) hide)
+    )
+    (property "Datasheet" "" (id 3) (at 74.93 142.24 0)
+      (effects (font (size 1.27 1.27)) hide)
+    )
+    (pin "1")
+  )
   (symbol (lib_id "Device:Buzzer") (at 190.5 90.17 0) (unit 1)
     (in_bom yes) (on_board yes) (fields_autoplaced)
@@
     (pin "4")
   )
+  (symbol (lib_id "GPAD_SCH_LIB:22-23-2021") (at 80.01 137.16 90) (mirror x) (unit 1)
+    (in_bom yes) (on_board yes)
+    (property "Reference" "J602" (id 0) (at 83.82 134.62 90)
+      (effects (font (size 1.27 1.27)) (justify right))
+    )
+    (property "Value" "22-23-2021" (id 1) (at 76.2 143.51 90)
+      (effects (font (size 1.27 1.27)) (justify right))
+    )
+    (property "Footprint" "Connector_Molex:Molex_KK-254_AE-6410-02A_1x02_P2.54mm_Vertical" (id 2) (at 74.93 142.24 0)
+      (effects (font (size 1.524 1.524)) (justify left) hide)
+    )
+    (property "Datasheet" "https://media.digikey.com/pdf/Data%20Sheets/Molex%20PDFs/A-6373-N_Series_Dwg_2010-12-03.pdf" (id 3) (at 72.39 142.24 0)
+      (effects (font (size 1.524 1.524)) (justify left) hide)
+    )
+    (property "Digi-Key_PN" "WM4200-ND" (id 4) (at 69.85 142.24 0)
+      (effects (font (size 1.524 1.524)) (justify left) hide)
+    )
+    (property "MPN" "22-23-2021" (id 5) (at 67.31 142.24 0)
+      (effects (font (size 1.524 1.524)) (justify left) hide)
+    )
+    (property "Category" "Connectors, Interconnects" (id 6) (at 64.77 142.24 0)
+      (effects (font (size 1.524 1.524)) (justify left) hide)
+    )
+    (property "Family" "Rectangular Connectors - Headers, Male Pins" (id 7) (at 62.23 142.24 0)
+      (effects (font (size 1.524 1.524)) (justify left) hide)
+    )
+    (property "DK_Datasheet_Link" "https://media.digikey.com/pdf/Data%20Sheets/Molex%20PDFs/A-6373-N_Series_Dwg_2010-12-03.pdf" (id 8) (at 59.69 142.24 0)
+      (effects (font (size 1.524 1.524)) (justify left) hide)
+    )
+    (property "DK_Detail_Page" "/product-detail/en/molex/22-23-2021/WM4200-ND/26667" (id 9) (at 57.15 142.24 0)
+      (effects (font (size 1.524 1.524)) (justify left) hide)
+    )
+    (property "Description" "CONN HEADER VERT 2POS 2.54MM" (id 10) (at 54.61 142.24 0)
+      (effects (font (size 1.524 1.524)) (justify left) hide)
+    )
+    (property "Manufacturer" "Molex" (id 11) (at 52.07 142.24 0)
+      (effects (font (size 1.524 1.524)) (justify left) hide)
+    )
+    (property "Status" "Active" (id 12) (at 49.53 142.24 0)
+      (effects (font (size 1.524 1.524)) (justify left) hide)
+    )
+    (property "Assembly Type" "" (id 13) (at 191.77 -57.15 0)
+      (effects (font (size 1.27 1.27)) hide)
+    )
+    (property "AssemblyType" "HAND" (id 14) (at 80.01 137.16 0)
+      (effects (font (size 1.27 1.27)) hide)
+    )
+    (property "Cost" "0.22000" (id 15) (at 80.01 137.16 0)
+      (effects (font (size 1.27 1.27)) hide)
+    )
+    (property "Distributor 1" "DigiKey" (id 16) (at 80.01 137.16 0)
+      (effects (font (size 1.27 1.27)) hide)
+    )
+    (property "Distributor 1 PN" "900-0022232021-ND" (id 17) (at 80.01 137.16 0)
+      (effects (font (size 1.27 1.27)) hide)
+    )
+    (pin "1")
+    (pin "2")
+  )
   (symbol (lib_id "power:GND") (at 132.08 99.06 0) (unit 1)

Commit message: Schematic symbol and library part Adafruit buzzer. Change schematic buzzer circuit to switch Adafruit buzzer.
Parts:
- removed BZ601: Buzzer_12.2mm_H6.5mm, Buzzer_Beeper:Buzzer_TDK_PS1240P02BT_D12.2mm_H6.5mm, symbol Device:Buzzer
- added BZ601: Buzzer_Adafruit_P1536A, GeneralPurposeAlarmDevicePCB:Buzzer_12.2mm_9.7mm_7.62mm, symbol GPAD_SCH_LIB:Buzzer_Adafruit_P1536A
- added R506: DNI, Resistor_SMD:R_0603_1608Metric_Pad0.98x0.95mm_HandSolder, symbol Device:R
- added R507, R508: 1R, Resistor_SMD:R_0603_1608Metric_Pad0.98x0.95mm_HandSolder, symbol Device:R
- R604: value 1R -> DNI
Connections:
- net GND: now also R508.1; no longer J601.2
- net VccBuzzer: now also J601.1, BZ601.1 (-), R506.2; no longer Q601.3 (C)
- net at R604.1: now also J601.2, BZ601.2 (+), R507.1; no longer J601.1
- net at Q601.2 (E), Q602.2 (E), R604.2: now also R508.2
- new net: Q601.3 (C), R506.1, R507.2
Other:
- moved on the sheet: J601

Commit message: Add Adafruit buzzer to PCB. DRC no errors. Trivial warnings.
Parts:
- removed Q601: MMBT2222A-7-F, Package_TO_SOT_SMD:SOT-23, symbol GPAD_SCH_LIB:MMBT2222A-7-F
- added Q601: BSS138, Package_TO_SOT_SMD:SOT-23, symbol Transistor_FET:BSS138
- Q602: value MMBT2907ALT1G -> DNI
Connections:
- net at Q602.2 (E), R508.2, R604.2: now also Q601.2 (S)
- net at Q602.1 (B), R505.2, R602.1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: now also Q601.1 (G)
- net at R506.1, R507.2: now also Q601.3 (D)
Changed lines of the file:
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@@
     (pin "2")
-  )
-  (symbol (lib_id "GPAD_SCH_LIB:MMBT2222A-7-F") (at 134.62 60.96 0) (unit 1)
-    (in_bom yes) (on_board yes)
-    (property "Reference" "Q601" (id 0) (at 139.3952 59.6138 0)
-      (effects (font (size 1.524 1.524)) (justify left))
-    )
-    (property "Value" "MMBT2222A-7-F" (id 1) (at 139.3952 62.3062 0)
-      (effects (font (size 1.524 1.524)) (justify left))
-    )
-    (property "Footprint" "Package_TO_SOT_SMD:SOT-23" (id 2) (at 139.7 55.88 0)
-      (effects (font (size 1.524 1.524)) (justify left) hide)
-    )
-    (property "Datasheet" "https://www.diodes.com/assets/Datasheets/ds30041.pdf" (id 3) (at 139.7 53.34 0)
-      (effects (font (size 1.524 1.524)) (justify left) hide)
-    )
-    (property "Digi-Key_PN" "MMBT2222A-FDICT-ND" (id 4) (at 139.7 50.8 0)
-      (effects (font (size 1.524 1.524)) (justify left) hide)
-    )
-    (property "MPN" "MMBT2222A-7-F" (id 5) (at 139.7 48.26 0)
-      (effects (font (size 1.524 1.524)) (justify left) hide)
-    )
-    (property "Category" "Discrete Semiconductor Products" (id 6) (at 139.7 45.72 0)
-      (effects (font (size 1.524 1.524)) (justify left) hide)
-    )
-    (property "Family" "Transistors - Bipolar (BJT) - Single" (id 7) (at 139.7 43.18 0)
-      (effects (font (size 1.524 1.524)) (justify left) hide)
-    )
-    (property "DK_Datasheet_Link" "https://www.diodes.com/assets/Datasheets/ds30041.pdf" (id 8) (at 139.7 40.64 0)
-      (effects (font (size 1.524 1.524)) (justify left) hide)
-    )
-    (property "DK_Detail_Page" "/product-detail/en/diodes-incorporated/MMBT2222A-7-F/MMBT2222A-FDICT-ND/815723" (id 9) (at 139.7 38.1 0)
-      (effects (font (size 1.524 1.524)) (justify left) hide)
-    )
-    (property "Description" "TRANS NPN 40V 0.6A SMD SOT23-3" (id 10) (at 139.7 35.56 0)
-      (effects (font (size 1.524 1.524)) (justify left) hide)
-    )
-    (property "Manufacturer" "Diodes Incorporated" (id 11) (at 139.7 33.02 0)
-      (effects (font (size 1.524 1.524)) (justify left) hide)
-    )
-    (property "Status" "Active" (id 12) (at 139.7 30.48 0)
-      (effects (font (size 1.524 1.524)) (justify left) hide)
-    )
-    (property "AssemblyType" "SMT" (id 13) (at 134.62 60.96 0)
-      (effects (font (size 1.27 1.27)) hide)
-    )
-    (property "Distributor 1" "JLCPCB" (id 14) (at 134.62 60.96 0)
-      (effects (font (size 1.27 1.27)) hide)
-    )
-    (property "Distributor 1 PN" "C94515" (id 15) (at 134.62 60.96 0)
-      (effects (font (size 1.27 1.27)) hide)
-    )
-    (property "Cost" "0.0475" (id 16) (at 134.62 60.96 0)
-      (effects (font (size 1.27 1.27)) hide)
-    )
-    (pin "1")
-    (pin "2")
-    (pin "3")
   )
   (symbol (lib_id "Device:R") (at 99.06 90.17 90) (unit 1)
@@
       (effects (font (size 1.524 1.524)) (justify left))
     )
-    (property "Value" "MMBT2907ALT1G" (id 1) (at 139.3952 76.1238 0)
+    (property "Value" "DNI" (id 1) (at 139.3952 76.1238 0)
       (effects (font (size 1.524 1.524)) (justify left))
     )
@@
     (pin "2")
   )
+  (symbol (lib_id "Transistor_FET:BSS138") (at 134.62 60.96 0) (unit 1)
+    (in_bom yes) (on_board yes)
+    (property "Reference" "Q601" (id 0) (at 139.8016 59.7916 0)
+      (effects (font (size 1.27 1.27)) (justify left))
+    )
+    (property "Value" "BSS138" (id 1) (at 139.8016 62.103 0)
+      (effects (font (size 1.27 1.27)) (justify left))
+    )
+    (property "Footprint" "Package_TO_SOT_SMD:SOT-23" (id 2) (at 139.7 62.865 0)
+      (effects (font (size 1.27 1.27) italic) (justify left) hide)
+    )
+    (property "Datasheet" "https://www.onsemi.com/pub/Collateral/BSS138-D.PDF" (id 3) (at 134.62 60.96 0)
+      (effects (font (size 1.27 1.27)) (justify left) hide)
+    )
+    (property "Description" "N-Channel Enhancement Mode Field Effect Transistor" (id 4) (at 134.62 60.96 0)
+      (effects (font (size 1.27 1.27)) hide)
+    )
+    (property "Distributor 1" "JLCPCB" (id 5) (at 134.62 60.96 0)
+      (effects (font (size 1.27 1.27)) hide)
+    )
+    (property "Distributor 1 PN" "C400505" (id 6) (at 134.62 60.96 0)
+      (effects (font (size 1.27 1.27)) hide)
+    )
+    (property "Manufacturer" "Yangzhou Yangjie Electronic Technology Co., Ltd" (id 8) (at 134.62 60.96 0)
+      (effects (font (size 1.27 1.27)) hide)
+    )
+    (property "MPN" "BSS138" (id 9) (at 134.62 60.96 0)
+      (effects (font (size 1.27 1.27)) hide)
+    )
+    (property "AssemblyType" "SMT" (id 10) (at 134.62 60.96 0)
+      (effects (font (size 1.27 1.27)) hide)
+    )
+    (property "Cost" "0.0196" (id 11) (at 134.62 60.96 0)
+      (effects (font (size 1.27 1.27)) hide)
+    )
+    (pin "1")
+    (pin "2")
+    (pin "3")
+  )
   (symbol (lib_id "Connector:TestPoint") (at 101.6 43.18 0) (unit 1)

Commit message: Update U301 for JLCPCB in stock, Break and then fix SCH library because of illigal character in sch symbol name.
Parts:
- Q602: Distributor 1 JCLPCB -> DNI; Distributor 1 PN C40752 -> DNI; Distributor 2 (none) -> JCLPCB; Distributor 2 PN (none) -> C40752
- R506, R604: Distributor 1 JLCPCB -> DNI; Distributor 1 PN C269434 -> DNI
- R605: value 330 -> 330R
Changed lines of the file:
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@@
       (effects (font (size 1.27 1.27)) hide)
     )
-    (property "Distributor 1" "JLCPCB" (id 4) (at 165.1 68.58 90)
-      (effects (font (size 1.27 1.27)) hide)
-    )
-    (property "Distributor 1 PN" "C269434" (id 5) (at 165.1 68.58 90)
+    (property "Distributor 1" "DNI" (id 4) (at 165.1 68.58 90)
+      (effects (font (size 1.27 1.27)) hide)
+    )
+    (property "Distributor 1 PN" "DNI" (id 5) (at 165.1 68.58 90)
       (effects (font (size 1.27 1.27)) hide)
     )
@@
       (effects (font (size 1.27 1.27)) hide)
     )
-    (property "Description" "0.1W ±5% 1Ω 0603 Chip Resistor - Surface Mount ROHS" (id 8) (at 165.1 68.58 0)
+    (property "Description" "DNI" (id 8) (at 165.1 68.58 0)
       (effects (font (size 1.27 1.27)) hide)
     )
@@
     (in_bom yes) (on_board yes)
     (property "Reference" "R605" (id 0) (at 97.79 87.63 90))
-    (property "Value" "330" (id 1) (at 99.06 93.98 90))
+    (property "Value" "330R" (id 1) (at 99.06 93.98 90))
     (property "Footprint" "Resistor_SMD:R_0603_1608Metric_Pad0.98x0.95mm_HandSolder" (id 2) (at 99.06 91.948 90)
       (effects (font (size 1.27 1.27)) hide)
@@
       (effects (font (size 1.27 1.27)) hide)
     )
-    (property "Distributor 1" "JCLPCB" (id 14) (at 134.62 77.47 0)
-      (effects (font (size 1.27 1.27)) hide)
-    )
-    (property "Distributor 1 PN" "C40752" (id 15) (at 134.62 77.47 0)
+    (property "Distributor 1" "DNI" (id 14) (at 134.62 77.47 0)
+      (effects (font (size 1.27 1.27)) hide)
+    )
+    (property "Distributor 1 PN" "DNI" (id 15) (at 134.62 77.47 0)
       (effects (font (size 1.27 1.27)) hide)
     )
     (property "Cost" "0.0374" (id 16) (at 134.62 77.47 0)
+      (effects (font (size 1.27 1.27)) hide)
+    )
+    (property "Distributor 2" "JCLPCB" (id 17) (at 134.62 77.47 0)
+      (effects (font (size 1.27 1.27)) hide)
+    )
+    (property "Distributor 2 PN" "C40752" (id 18) (at 134.62 77.47 0)
       (effects (font (size 1.27 1.27)) hide)
     )
@@
       (effects (font (size 1.27 1.27)) hide)
     )
-    (property "Distributor 1" "JLCPCB" (id 4) (at 125.73 48.26 90)
-      (effects (font (size 1.27 1.27)) hide)
-    )
-    (property "Distributor 1 PN" "C269434" (id 5) (at 125.73 48.26 90)
+    (property "Distributor 1" "DNI" (id 4) (at 125.73 48.26 90)
+      (effects (font (size 1.27 1.27)) hide)
+    )
+    (property "Distributor 1 PN" "DNI" (id 5) (at 125.73 48.26 90)
       (effects (font (size 1.27 1.27)) hide)
     )
@@
       (effects (font (size 1.27 1.27)) hide)
     )
-    (property "Description" "0.1W ±5% 1Ω 0603 Chip Resistor - Surface Mount ROHS" (id 8) (at 125.73 48.26 0)
-      (effects (font (size 1.27 1.27)) hide)
-    )
+    (property "Description" "DNI" (id 8) (at 125.73 48.26 0)
+      (effects (font (size 1.27 1.27)) hide)
+    )

Commit message: Update schematic with note on additional vendor information on buzzer.
Other:
- note added: "Notes on Buzzer vendors Units assembled with these two parts are similar in performance but not identical. Assemble SN 22, 23, 24 and 25 with Digikey number 433-WST-1210T-ND. Assemble SN 26, 27, 28 , 29 and 30 with Digikey number 102-CMI-1295-0585T-ND. And Assemble SN ?16, 17, 18 , and 19? with Adafruit part."
Changed lines of the file:
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@@
     (stroke (width 0) (type default) (color 0 0 0 0))
   )
-  (image (at 260.35 175.26) (scale 0.75)
+  (image (at 255.27 179.07) (scale 0.75)
     (data
       iVBORw0KGgoAAAANSUhEUgAAASAAAAEgCAYAAAAUg66AAAAABHNCSVQICAgIfAhkiAAAAAlwSFlz
@@
     )
   )
+  (text "Notes on Buzzer vendors\nUnits assembled with these two parts are similar in performance but not identical.  \nAssemble SN 22, 23, 24 and 25 with Digikey number 433-WST-1210T-ND.\nAssemble SN 26, 27, 28 , 29 and 30 with Digikey number 102-CMI-1295-0585T-ND.\n\nAnd Assemble SN ?16, 17, 18 , and 19? with Adafruit part.\n"
+    (at 168.91 30.48 0)
+    (effects (font (size 1.27 1.27)) (justify left bottom))
+  )
   (text "For external \"speaker\"." (at 195.58 59.69 0)
