File: Hardware/GeneralPurposeAlarmDevicePCB/AlarmLights5.kicad_sch (KiCad schematic)
At the start: 20 parts, among them Q201 MMBT2222A-7-F, Q202 MMBT2222A-7-F, Q203 MMBT2222A-7-F, Q204 MMBT2222A-7-F, Q205 MMBT2222A-7-F

Commit message: Update PCB for version 2. Update enclosure drawing to reflect the V1 enclosure assembly.
Changed lines of the file:
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@@
     (title "GeneralPurposeAlarmDevicePCB")
     (date "2022-11-13")
-    (rev "1.2")
+    (rev "2.0")
     (company "PublicInvention")
     (comment 1 "GNU Affero General Public License v3.0")
@@
   (symbol (lib_id "Device:R") (at 76.2 93.98 180) (unit 1)
     (in_bom yes) (on_board yes)
-    (property "Reference" "R201" (id 0) (at 78.74 90.17 0))
+    (property "Reference" "R201" (id 0) (at 81.28 92.71 0))
     (property "Value" "4K7" (id 1) (at 80.01 95.25 0))
     (property "Footprint" "Resistor_SMD:R_0603_1608Metric_Pad0.98x0.95mm_HandSolder" (id 2) (at 77.978 93.98 90)
@@
   (symbol (lib_id "Device:R") (at 106.68 93.98 180) (unit 1)
     (in_bom yes) (on_board yes)
-    (property "Reference" "R203" (id 0) (at 109.22 92.71 0))
+    (property "Reference" "R203" (id 0) (at 111.76 92.71 0))
     (property "Value" "4K7" (id 1) (at 110.49 95.25 0))
     (property "Footprint" "Resistor_SMD:R_0603_1608Metric_Pad0.98x0.95mm_HandSolder" (id 2) (at 108.458 93.98 90)
@@
   (symbol (lib_id "Device:R") (at 137.16 93.98 180) (unit 1)
     (in_bom yes) (on_board yes)
-    (property "Reference" "R205" (id 0) (at 139.7 92.71 0))
+    (property "Reference" "R205" (id 0) (at 142.24 92.71 0))
     (property "Value" "4K7" (id 1) (at 140.97 95.25 0))
     (property "Footprint" "Resistor_SMD:R_0603_1608Metric_Pad0.98x0.95mm_HandSolder" (id 2) (at 138.938 93.98 90)
@@
   (symbol (lib_id "Device:R") (at 167.64 93.98 180) (unit 1)
     (in_bom yes) (on_board yes)
-    (property "Reference" "R207" (id 0) (at 170.18 92.71 0))
+    (property "Reference" "R207" (id 0) (at 172.72 92.71 0))
     (property "Value" "4K7" (id 1) (at 171.45 95.25 0))
     (property "Footprint" "Resistor_SMD:R_0603_1608Metric_Pad0.98x0.95mm_HandSolder" (id 2) (at 169.418 93.98 90)
@@
   (symbol (lib_id "Device:R") (at 198.12 93.98 180) (unit 1)
     (in_bom yes) (on_board yes)
-    (property "Reference" "R209" (id 0) (at 200.66 92.71 0))
+    (property "Reference" "R209" (id 0) (at 204.47 92.71 0))
     (property "Value" "4K7" (id 1) (at 201.93 95.25 0))
     (property "Footprint" "Resistor_SMD:R_0603_1608Metric_Pad0.98x0.95mm_HandSolder" (id 2) (at 199.898 93.98 90)

Commit message: Add LED Standoffs to Schematic. Bump version to 2.1
Parts:
- added MF601, MF602, MF603, MF604, MF605: U_Box_V104_General_Alarm_Device_LED_Standoff, GeneralPurposeAlarmDevicePCB:U_Box_V104_General_Alarm_Device_LED_Standoff, symbol GPAD_SCH_LIB:U_Box_V104_General_Alarm_Device_LED_Standoff
Changed lines of the file:
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@@
   (title_block
     (title "GeneralPurposeAlarmDevicePCB")
-    (date "2022-11-13")
-    (rev "2.0")
+    (date "2023-03-02")
+    (rev "2.1")
     (company "PublicInvention")
     (comment 1 "GNU Affero General Public License v3.0")
@@
     (pin "3")
   )
+  (symbol (lib_id "GPAD_SCH_LIB:U_Box_V104_General_Alarm_Device_LED_Standoff") (at 210.82 124.46 0) (unit 1)
+    (in_bom yes) (on_board yes) (fields_autoplaced)
+    (property "Reference" "MF605" (id 0) (at 215.9 123.1899 0)
+      (effects (font (size 1.27 1.27)) (justify left))
+    )
+    (property "Value" "U_Box_V104_General_Alarm_Device_LED_Standoff" (id 1) (at 215.9 125.7299 0)
+      (effects (font (size 1.27 1.27)) (justify left))
+    )
+    (property "Footprint" "GeneralPurposeAlarmDevicePCB:U_Box_V104_General_Alarm_Device_LED_Standoff" (id 2) (at 210.82 124.46 0)
+      (effects (font (size 1.27 1.27)) hide)
+    )
+    (property "Datasheet" "" (id 3) (at 210.82 124.46 0)
+      (effects (font (size 1.27 1.27)) hide)
+    )
+  )
+  (symbol (lib_id "GPAD_SCH_LIB:U_Box_V104_General_Alarm_Device_LED_Standoff") (at 180.34 130.81 0) (unit 1)
+    (in_bom yes) (on_board yes) (fields_autoplaced)
+    (property "Reference" "MF604" (id 0) (at 185.42 129.5399 0)
+      (effects (font (size 1.27 1.27)) (justify left))
+    )
+    (property "Value" "U_Box_V104_General_Alarm_Device_LED_Standoff" (id 1) (at 185.42 132.0799 0)
+      (effects (font (size 1.27 1.27)) (justify left))
+    )
+    (property "Footprint" "GeneralPurposeAlarmDevicePCB:U_Box_V104_General_Alarm_Device_LED_Standoff" (id 2) (at 180.34 130.81 0)
+      (effects (font (size 1.27 1.27)) hide)
+    )
+    (property "Datasheet" "" (id 3) (at 180.34 130.81 0)
+      (effects (font (size 1.27 1.27)) hide)
+    )
+  )
+  (symbol (lib_id "GPAD_SCH_LIB:U_Box_V104_General_Alarm_Device_LED_Standoff") (at 151.13 123.19 0) (unit 1)
+    (in_bom yes) (on_board yes) (fields_autoplaced)
+    (property "Reference" "MF603" (id 0) (at 156.21 121.9199 0)
+      (effects (font (size 1.27 1.27)) (justify left))
+    )
+    (property "Value" "U_Box_V104_General_Alarm_Device_LED_Standoff" (id 1) (at 156.21 124.4599 0)
+      (effects (font (size 1.27 1.27)) (justify left))
+    )
+    (property "Footprint" "GeneralPurposeAlarmDevicePCB:U_Box_V104_General_Alarm_Device_LED_Standoff" (id 2) (at 151.13 123.19 0)
+      (effects (font (size 1.27 1.27)) hide)
+    )
+    (property "Datasheet" "" (id 3) (at 151.13 123.19 0)
+      (effects (font (size 1.27 1.27)) hide)
+    )
+  )
+  (symbol (lib_id "GPAD_SCH_LIB:U_Box_V104_General_Alarm_Device_LED_Standoff") (at 119.38 129.54 0) (unit 1)
+    (in_bom yes) (on_board yes) (fields_autoplaced)
+    (property "Reference" "MF602" (id 0) (at 124.46 128.2699 0)
+      (effects (font (size 1.27 1.27)) (justify left))
+    )
+    (property "Value" "U_Box_V104_General_Alarm_Device_LED_Standoff" (id 1) (at 124.46 130.8099 0)
+      (effects (font (size 1.27 1.27)) (justify left))
+    )
+    (property "Footprint" "GeneralPurposeAlarmDevicePCB:U_Box_V104_General_Alarm_Device_LED_Standoff" (id 2) (at 119.38 129.54 0)
+      (effects (font (size 1.27 1.27)) hide)
+    )
+    (property "Datasheet" "" (id 3) (at 119.38 129.54 0)
+      (effects (font (size 1.27 1.27)) hide)
+    )
+  )
+  (symbol (lib_id "GPAD_SCH_LIB:U_Box_V104_General_Alarm_Device_LED_Standoff") (at 88.9 120.65 0) (unit 1)
+    (in_bom yes) (on_board yes) (fields_autoplaced)
+    (property "Reference" "MF601" (id 0) (at 93.98 119.3799 0)
+      (effects (font (size 1.27 1.27)) (justify left))
+    )
+    (property "Value" "U_Box_V104_General_Alarm_Device_LED_Standoff" (id 1) (at 93.98 121.9199 0)
+      (effects (font (size 1.27 1.27)) (justify left))
+    )
+    (property "Footprint" "GeneralPurposeAlarmDevicePCB:U_Box_V104_General_Alarm_Device_LED_Standoff" (id 2) (at 88.9 120.65 0)
+      (effects (font (size 1.27 1.27)) hide)
+    )
+    (property "Datasheet" "" (id 3) (at 88.9 120.65 0)
+      (effects (font (size 1.27 1.27)) hide)
+    )
+  )
 )
