File: Hardware/GeneralPurposeAlarmDevicePCB/USB_UART.kicad_sch (KiCad schematic)
At the start: 13 parts, among them J501 USB_B_Micro_Local, U501 CH340E

Commit message: Update schematic for rework of Version 1 PCB for D7 and D10 and Reset to nRTS.
Connections:
- net nRTS: now reaches U501.4 (~{RTS})
Changed lines of the file:
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@@
   (title_block
     (title "GeneralPurposeAlarmDevicePCB")
-    (date "2022-06-20")
-    (rev "0.0")
+    (date "2022-11-13")
+    (rev "1.2")
     (company "PublicInvention")
     (comment 1 "GNU Affero General Public License v3.0")
@@
     (stroke (width 0) (type default) (color 0 0 0 0))
   )
+  (wire (pts (xy 165.1 107.95) (xy 167.64 107.95))
+    (stroke (width 0) (type default) (color 0 0 0 0))
+  )
   (wire (pts (xy 100.33 97.79) (xy 144.78 97.79))
     (stroke (width 0) (type default) (color 0 0 0 0))
@@
     (stroke (width 0) (type default) (color 0 0 0 0))
   )
+  (wire (pts (xy 167.64 115.57) (xy 167.64 107.95))
+    (stroke (width 0) (type default) (color 0 0 0 0))
+  )
   (wire (pts (xy 90.17 113.03) (xy 90.17 105.41))
     (stroke (width 0) (type default) (color 0 0 0 0))
   )
   (wire (pts (xy 120.65 76.2) (xy 114.3 76.2))
+    (stroke (width 0) (type default) (color 0 0 0 0))
+  )
+  (wire (pts (xy 213.36 115.57) (xy 167.64 115.57))
     (stroke (width 0) (type default) (color 0 0 0 0))
   )
@@
     (effects (font (size 1.27 1.27)) (justify left))
   )
+  (hierarchical_label "nRTS" (shape input) (at 213.36 115.57 0)
+    (effects (font (size 1.27 1.27)) (justify left))
+  )

Commit message: Update PCB for version 2. Update enclosure drawing to reflect the V1 enclosure assembly.
Connections:
- no-connect marks 2 -> 1
Changed lines of the file:
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@@
     (title "GeneralPurposeAlarmDevicePCB")
     (date "2022-11-13")
-    (rev "1.2")
+    (rev "2.0")
     (company "PublicInvention")
     (comment 1 "GNU Affero General Public License v3.0")
@@
   )
   (no_connect (at 100.33 100.33))
-  (no_connect (at 165.1 107.95))
   (wire (pts (xy 114.3 76.2) (xy 106.68 76.2))
     (stroke (width 0) (type default) (color 0 0 0 0))
@@
     (stroke (width 0) (type default) (color 0 0 0 0))
   )
+  (wire (pts (xy 165.1 107.95) (xy 167.64 107.95))
+    (stroke (width 0) (type default) (color 0 0 0 0))
+  )
   (wire (pts (xy 144.78 100.33) (xy 140.97 100.33))
     (stroke (width 0) (type default) (color 0 0 0 0))
   )
-  (wire (pts (xy 165.1 107.95) (xy 167.64 107.95))
-    (stroke (width 0) (type default) (color 0 0 0 0))
-  )
