File: Hardware/GPAD2/GeneralPurposeAlarmDevicePCB_DFPlayer/GeneralPurposeAlarmDevicePCB_DFPlayer.kicad_sch (KiCad schematic)
At the start: 56 parts, among them J101 Barrel_Jack_Switch_SMT, J102 0.100_2Pin, J103 0.100_2Pin, J105 S04B-XASK-1(LF)(SN)Rev2, U101 LM7805_TO220, U102 PI_ATMEGA328P-AU-InOrder

Commit message: updated kicad
Parts:
- added D?: RED 0603, LED_SMD:LED_0603_1608Metric_Pad1.05x0.95mm_HandSolder, symbol Device:LED
- added R? (x2): 330R, Resistor_SMD:R_0603_1608Metric_Pad0.98x0.95mm_HandSolder, symbol Device:R
- added U?: ESP32-DEVKITC, MODULE_ESP32-DEVKITC, symbol ESP32-DEVKITC:ESP32-DEVKITC
Connections:
- net Attenuate: now also U?.15 (IO13)
- net CIPO: now also U?.31 (IO19)
- net COPI: now also U?.37 (IO23)
- net ControllerRX: now also U?.34 (RXD0)
- net ControllerTX: now also U?.35 (TXD0)
- net GND: now also D?.1 (K), U?.14 (GND1), U?.32 (GND2), U?.38 (GND3)
- net GPIO16: now also U?.27 (IO16)
- net GPIO17: now also U?.28 (IO17)
- net Light0: now also U?.24 (IO2)
- net Light1: now also U?.10 (IO26)
- net Light2: now also U?.9 (IO25)
- net Light3: now also U?.12 (IO14)
- net Light4: now also U?.23 (IO15)
- net PC0: now also U?.5 (IO34)
- net PC1: now also U?.6 (IO35)
- net PC2: now also U?.7 (IO32)
- net PC3: now also R?.2, U?.8 (IO33)
- net SCL: now also U?.36 (IO22)
- net SDA: now also U?.33 (IO21)
- net SPI_SCK: now also U?.30 (IO18)
- net Switch_Mute: now also U?.13 (IO12)
- net Tone: now also U?.26 (IO4)
- net VccController: now also U?.19 (EXT_5V)
- net nCS: now also U?.29 (IO5)
- net nRESET: now also R?.1
- new net: D?.2 (A), R?.1
- new net: R?.2, U?.2 (EN)
- new net 3.3V: U?.1 (3V3)
- no-connect marks 2 -> 12
Other:
- removed sheet Esp32
- note added: "Hook to the ground or leave unconnect"
- moved on the sheet: C103, C104, C106, C107, C110, C111, C112, D102, D103, H101, H102, H103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

Commit message: Updated all needed files for hardware
Parts:
- removed A101: Arduino_UNO_R3_Shield, GeneralPurposeAlarmDevicePCB:Arduino_UNO_R3_NoMountingHoles3D, symbol GPAD_SCH_LIB:Arduino_UNO_R3_Shield
- removed D106: RED 0603, LED_SMD:LED_0603_1608Metric_Pad1.05x0.95mm_HandSolder, symbol Device:LED
- removed R111, R112: 330R, Resistor_SMD:R_0603_1608Metric_Pad0.98x0.95mm_HandSolder, symbol Device:R
- removed TP105: 3.3V, TestPoint:TestPoint_Loop_D2.54mm_Drill1.5mm_Beaded, symbol Connector:TestPoint
- removed U?: PAM8403, PAM8403, symbol PAM8403:PAM8403
- removed U?: DFR0299, MODULE_DFR0299, symbol DFR0299:DFR0299
Connections:
- net Light3: no longer U102.13 (PB1)
Other:
- note added: "Notes: ESP32 Pin to ATmega328 IO34 PC0 IO35 PC1 IO32 PC2 IO33 PC3 IO21 PC4 (SDA) IO22 PC5 RXD0 PD0 TXD0 PD1 IO12 PD2 IO2 PD3 IO13 PD4 IO26 PD5 IO25 PD6 IO15 PD7 IO4 PB0 IO14 PB1 IO5 PB2 IO23 PB3 IO19 PB4 IO18 PB5"
- note removed: "Notes: Arduino Pin to ATmega328 A0 PC0 A1 PC1 A2 PC2 A3 PC3 A4 PC4 A5 PC5 D0 PD0 D1 PD1 D2 PD2 'D3 PD3 D4 PD4 `D5 PD5 `D6 PD6 D7 PD7 D8 PB0 `D9 PB1 `D10 PB2 `D11 PB3 D12 PB4 D13 PB5 Remark: PC4 as SDA PC5 as SCL is conventional UNO pinout. Same for Rx and Tx."
- note removed: "UNO Headers"
- note removed: "Wink LED"
- moved on the sheet: R?

Commit message: Updated Hardware
Other:
- note added: "GPAD2 version (modified by hardware team) Bryan's team: Nguyen Vu, Bryan Tran, Van Nguyen, Baraa Ahmad"
- note removed: "Note: Using 0603HandSolder for Rs and Cs."
Changed lines of the file:
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@@
     (effects (font (size 1.27 1.27)) (justify left bottom))
   )
-  (text "Note: Using 0603HandSolder for Rs and Cs." (at 161.29 170.18 0)
-    (effects (font (size 1.27 1.27)) (justify left bottom))
+  (text "GPAD2 version (modified by hardware team)\nBryan's team: Nguyen Vu, Bryan Tran, Van Nguyen, Baraa Ahmad"
+    (at 161.29 170.18 0)
+    (effects (font (size 1.5 1.5) (thickness 0.4) bold) (justify left bottom))
   )
   (label "+5V" (at 116.84 24.13 0)
