File: Hardware/GPAD2/GeneralPurposeAlarmDevicePCB_DFPlayer/SDcard.kicad_sch (KiCad schematic)
At the start: 2 parts

Commit message: Updated all needed files for hardware
Connections:
- no-connect marks 0 -> 9
Other:
- title: (none) -> GeneralPurposeAlarmDevicePCB
- moved on the sheet: R1, U?
Changed lines of the file:
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@@
 (kicad_sch (version 20211123) (generator eeschema)
   (paper "A4")
-  (junction (at 91.44 82.55) (diameter 0) (color 0 0 0 0)
+  (title_block
+    (title "GeneralPurposeAlarmDevicePCB")
+    (date "2023-04-27")
+    (comment 1 "GPAD2 version")
+    (comment 2 "Drawn by Nguyen Vu")
   )
-  (junction (at 81.28 100.33) (diameter 0) (color 0 0 0 0)
+  (junction (at 164.846 82.296) (diameter 0) (color 0 0 0 0)
   )
-  (wire (pts (xy 78.74 67.31) (xy 86.36 67.31))
+  (junction (at 154.686 100.076) (diameter 0) (color 0 0 0 0)
+  )
+  (no_connect (at 121.666 79.756))
+  (no_connect (at 152.146 87.376))
+  (no_connect (at 121.666 92.456))
+  (no_connect (at 121.666 87.376))
+  (no_connect (at 121.666 72.136))
+  (no_connect (at 121.666 77.216))
+  (no_connect (at 152.146 89.916))
+  (no_connect (at 121.666 94.996))
+  (no_connect (at 121.666 84.836))
+  (wire (pts (xy 152.146 67.056) (xy 159.766 67.056))
     (stroke (width 0) (type default) (color 0 0 0 0))
   )
-  (wire (pts (xy 78.74 72.39) (xy 83.82 72.39))
+  (wire (pts (xy 152.146 72.136) (xy 157.226 72.136))
     (stroke (width 0) (type default) (color 0 0 0 0))
   )
-  (wire (pts (xy 78.74 82.55) (xy 91.44 82.55))
+  (wire (pts (xy 152.146 82.296) (xy 164.846 82.296))
     (stroke (width 0) (type default) (color 0 0 0 0))
   )
-  (wire (pts (xy 78.74 100.33) (xy 81.28 100.33))
+  (wire (pts (xy 152.146 100.076) (xy 154.686 100.076))
     (stroke (width 0) (type default) (color 0 0 0 0))
   )
-  (wire (pts (xy 86.36 60.96) (xy 86.36 67.31))
+  (wire (pts (xy 159.766 60.706) (xy 159.766 67.056))
     (stroke (width 0) (type default) (color 0 0 0 0))
   )
-  (wire (pts (xy 78.74 74.93) (xy 83.82 74.93))
+  (wire (pts (xy 152.146 74.676) (xy 157.226 74.676))
     (stroke (width 0) (type default) (color 0 0 0 0))
   )
-  (wire (pts (xy 78.74 80.01) (xy 96.52 80.01))
+  (wire (pts (xy 152.146 79.756) (xy 169.926 79.756))
     (stroke (width 0) (type default) (color 0 0 0 0))
   )
-  (wire (pts (xy 91.44 82.55) (xy 105.41 82.55))
+  (wire (pts (xy 164.846 82.296) (xy 178.816 82.296))
     (stroke (width 0) (type default) (color 0 0 0 0))
   )
-  (wire (pts (xy 91.44 82.55) (xy 91.44 92.71))
+  (wire (pts (xy 164.846 82.296) (xy 164.846 92.456))
     (stroke (width 0) (type default) (color 0 0 0 0))
   )
-  (wire (pts (xy 81.28 100.33) (xy 81.28 104.14))
+  (wire (pts (xy 154.686 100.076) (xy 154.686 103.886))
     (stroke (width 0) (type default) (color 0 0 0 0))
   )
-  (wire (pts (xy 81.28 100.33) (xy 91.44 100.33))
+  (wire (pts (xy 154.686 100.076) (xy 164.846 100.076))
     (stroke (width 0) (type default) (color 0 0 0 0))
   )
-  (hierarchical_label "GPIO17" (shape input) (at 96.52 80.01 0)
+  (hierarchical_label "GPIO17" (shape input) (at 169.926 79.756 0)
     (effects (font (size 1.27 1.27)) (justify left))
   )
-  (hierarchical_label "DacLeft" (shape output) (at 83.82 74.93 0)
+  (hierarchical_label "DacLeft" (shape output) (at 157.226 74.676 0)
     (effects (font (size 1.27 1.27)) (justify left))
   )
-  (hierarchical_label "DacRight" (shape output) (at 83.82 72.39 0)
+  (hierarchical_label "DacRight" (shape output) (at 157.226 72.136 0)
     (effects (font (size 1.27 1.27)) (justify left))
   )
-  (hierarchical_label "GPIO16" (shape input) (at 105.41 82.55 0)
+  (hierarchical_label "GPIO16" (shape input) (at 178.816 82.296 0)
     (effects (font (size 1.27 1.27)) (justify left))
   )
-  (symbol (lib_id "power:+5V") (at 86.36 60.96 0) (unit 1)
+  (symbol (lib_id "power:+5V") (at 159.766 60.706 0) (unit 1)
     (in_bom yes) (on_board yes)
-    (property "Reference" "#PWR?" (id 0) (at 86.36 64.77 0)
+    (property "Reference" "#PWR?" (id 0) (at 159.766 64.516 0)
       (effects (font (size 1.27 1.27)) hide)
     )
-    (property "Value" "+5V" (id 1) (at 86.741 56.5658 0))
-    (property "Footprint" "" (id 2) (at 86.36 60.96 0)
+    (property "Value" "+5V" (id 1) (at 160.147 56.3118 0))
+    (property "Footprint" "" (id 2) (at 159.766 60.706 0)
       (effects (font (size 1.27 1.27)) hide)
     )
-    (property "Datasheet" "" (id 3) (at 86.36 60.96 0)
+    (property "Datasheet" "" (id 3) (at 159.766 60.706 0)
       (effects (font (size 1.27 1.27)) hide)
     )
     (pin "1")
   )
-  (symbol (lib_id "power:GND") (at 81.28 104.14 0) (unit 1)
+  (symbol (lib_id "power:GND") (at 154.686 103.886 0) (unit 1)
     (in_bom yes) (on_board yes)
-    (property "Reference" "#PWR?" (id 0) (at 81.28 110.49 0)
+    (property "Reference" "#PWR?" (id 0) (at 154.686 110.236 0)
       (effects (font (size 1.27 1.27)) hide)
     )
-    (property "Value" "GND" (id 1) (at 81.407 108.5342 0))
-    (property "Footprint" "" (id 2) (at 81.28 104.14 0)
+    (property "Value" "GND" (id 1) (at 154.813 108.2802 0))
+    (property "Footprint" "" (id 2) (at 154.686 103.886 0)
       (effects (font (size 1.27 1.27)) hide)
     )
-    (property "Datasheet" "" (id 3) (at 81.28 104.14 0)
+    (property "Datasheet" "" (id 3) (at 154.686 103.886 0)
       (effects (font (size 1.27 1.27)) hide)
     )
     (pin "1")
   )
-  (symbol (lib_id "DFR0299:DFR0299") (at 63.5 82.55 0) (unit 1)
+  (symbol (lib_id "DFR0299:DFR0299") (at 136.906 82.296 0) (unit 1)
     (in_bom yes) (on_board yes) (fields_autoplaced)
-    (property "Reference" "U?" (id 0) (at 63.5 59.69 0))
-    (property "Value" "DFR0299" (id 1) (at 63.5 62.23 0))
-    (property "Footprint" "MODULE_DFR0299" (id 2) (at 63.5 82.55 0)
+    (property "Reference" "U?" (id 0) (at 136.906 59.436 0))
+    (property "Value" "DFR0299" (id 1) (at 136.906 61.976 0))
+    (property "Footprint" "MODULE_DFR0299" (id 2) (at 136.906 82.296 0)
       (effects (font (size 1.27 1.27)) (justify bottom) hide)
     )
-    (property "Datasheet" "" (id 3) (at 63.5 82.55 0)
+    (property "Datasheet" "" (id 3) (at 136.906 82.296 0)
       (effects (font (size 1.27 1.27)) hide)
     )
-    (property "MP" "DFR0299" (id 4) (at 63.5 82.55 0)
+    (property "MP" "DFR0299" (id 4) (at 136.906 82.296 0)
       (effects (font (size 1.27 1.27)) (justify bottom) hide)
     )
-    (property "PRICE" "None" (id 5) (at 63.5 82.55 0)
+    (property "PRICE" "None" (id 5) (at 136.906 82.296 0)
       (effects (font (size 1.27 1.27)) (justify bottom) hide)
     )
-    (property "PACKAGE" "None" (id 6) (at 63.5 82.55 0)
+    (property "PACKAGE" "None" (id 6) (at 136.906 82.296 0)
       (effects (font (size 1.27 1.27)) (justify bottom) hide)
     )
-    (property "MF" "DFRobot" (id 7) (at 63.5 82.55 0)
+    (property "MF" "DFRobot" (id 7) (at 136.906 82.296 0)
       (effects (font (size 1.27 1.27)) (justify bottom) hide)
     )
-    (property "AVAILABILITY" "Unavailable" (id 8) (at 63.5 82.55 0)
+    (property "AVAILABILITY" "Unavailable" (id 8) (at 136.906 82.296 0)
       (effects (font (size 1.27 1.27)) (justify bottom) hide)
     )
-    (property "DESCRIPTION" "Dfplayer - a Mini Mp3 Player" (id 9) (at 63.5 82.55 0)
+    (property "DESCRIPTION" "Dfplayer - a Mini Mp3 Player" (id 9) (at 136.906 82.296 0)
       (effects (font (size 1.27 1.27)) (justify bottom) hide)
     )
@@
     (pin "9")
   )
-  (symbol (lib_id "Device:R") (at 91.44 96.52 0) (unit 1)
+  (symbol (lib_id "Device:R") (at 164.846 96.266 0) (unit 1)
     (in_bom yes) (on_board yes) (fields_autoplaced)
-    (property "Reference" "R1" (id 0) (at 93.98 95.2499 0)
+    (property "Reference" "R1" (id 0) (at 167.386 94.9959 0)
       (effects (font (size 1.27 1.27)) (justify left))
     )
-    (property "Value" "10k" (id 1) (at 93.98 97.7899 0)
+    (property "Value" "10k" (id 1) (at 167.386 97.5359 0)
       (effects (font (size 1.27 1.27)) (justify left))
     )
-    (property "Footprint" "" (id 2) (at 89.662 96.52 90)
+    (property "Footprint" "" (id 2) (at 163.068 96.266 90)
       (effects (font (size 1.27 1.27)) hide)
     )
-    (property "Datasheet" "~" (id 3) (at 91.44 96.52 0)
+    (property "Datasheet" "~" (id 3) (at 164.846 96.266 0)
       (effects (font (size 1.27 1.27)) hide)
     )

Commit message: Updated Hardware
Other:
- note added: "GPAD2 version (modified by hardware team) Bryan's team: Nguyen Vu, Bryan Tran, Van Nguyen, Baraa Ahmad"
Changed lines of the file:
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@@
     (stroke (width 0) (type default) (color 0 0 0 0))
+  )
+  (text "GPAD2 version (modified by hardware team)\nBryan's team: Nguyen Vu, Bryan Tran, Van Nguyen, Baraa Ahmad"
+    (at 177.038 159.766 0)
+    (effects (font (size 1.5 1.5) (thickness 0.4) bold) (justify left bottom))
   )
   (hierarchical_label "GPIO17" (shape input) (at 169.926 79.756 0)
